Commit message: 完善Readme.md,调整world中机器人位置

File: src/alfa_robot_description/urdf/alfa_robot.urdf.xacro (robot description, xacro)
@@ -16,5 +16,5 @@
   <!-- set prefix if multiple robots are used -->
   <xacro:alfa_robot prefix="$(arg prefix)" parent="world">
-    <origin xyz="0 0 0" rpy="0 0 0"/>          <!-- position robot in the world -->
+    <origin xyz="0 0 0.09" rpy="0 0 0"/>          <!-- position robot in the world -->
   </xacro:alfa_robot>
   <xacro:alfa_robot_ros2_control
