Commit message: 只修改discription

File: src/alfa_robot_description/install/alfa_robot_description/share/alfa_robot_description/urdf/alfa_robot/alfa_robot_macro.xacro (robot description, xacro)
@@ -8,12 +8,12 @@
     <link name="${prefix}base_link">
       <inertial>
-        <origin xyz="3.7315E-08 -7.4812E-06 0.017979" rpy="0 0 0"/>
-        <mass value="11.681"/>
-        <inertia ixx="0.33161" ixy="0" ixz="0" iyy="0.33161" iyz="0" izz="0.6611"/>
-      </inertial>
-      <visual>
-        <origin xyz="0 0 0" rpy="0 0 0"/>
-        <geometry>
-          <mesh filename="package://alfa_robot_description/meshes/alfa_robot/visual/base.STL"/>
+        <origin xyz="-0.44193110855616 0.000259961331933109 0.176428166472852" rpy="0 0 0"/>
+        <mass value="394.931465036981"/>
+        <inertia ixx="66.5681215725466" ixy="5.74775273893285E-10" ixz="9.85014992290203" iyy="65.6389024339403" iyz="2.76043934386688E-09" izz="112.938477587322"/>
+      </inertial>
+      <visual>
+        <origin xyz="0 0 0" rpy="0 0 0"/>
+        <geometry>
+          <mesh filename="package://alfa_robot_description/meshes/alfa_robot/visual/base_link.STL"/>
         </geometry>
         <material name="blue"/>
@@ -22,5 +22,5 @@
         <origin xyz="0 0 0" rpy="0 0 0"/>
         <geometry>
-          <mesh filename="package://alfa_robot_description/meshes/alfa_robot/collision/base.STL"/>
+          <mesh filename="package://alfa_robot_description/meshes/alfa_robot/collision/base_link.STL"/>
         </geometry>
       </collision>
@@ -29,7 +29,7 @@
     <link name="${prefix}turn_link">
       <inertial>
-        <origin xyz="-5.4556E-05 0.094864 0.74374" rpy="0 0 0"/>
-        <mass value="52.536"/>
-        <inertia ixx="10.303" ixy="0" ixz="0" iyy="10.345" iyz="0" izz="1.0442"/>
+        <origin xyz="8.3102236387753E-05 -5.6319532371063E-13 0.854091510931534" rpy="0 0 0"/>
+        <mass value="93.4308976427189"/>
+        <inertia ixx="39.2606066773154" ixy="6.93889405615743E-18" ixz="-5.06230387770105E-13" iyy="39.2606066773154" iyz="2.34703241842353E-11" izz="1.49032676193219"/>
       </inertial>
       <visual>
@@ -50,7 +50,7 @@
     <link name="${prefix}updown_link">
       <inertial>
-        <origin xyz="0.0201090104029969 0.0803972373261843 0.0984366062782738" rpy="0 0 0"/>
-        <mass value="22.9526820845594"/>
-        <inertia ixx="0.164263278076855" ixy="0" ixz="0" iyy="0.152416211091917" iyz="0" izz="0.278538027798598"/>
+        <origin xyz="-0.297917412220348 -3.47192615164638E-07 0.0811648445824145" rpy="0 0 0"/>
+        <mass value="49.32553657462"/>
+        <inertia ixx="0.931332356925864" ixy="9.94007584674414E-06" ixz="0.066855170904404" iyy="1.73410727221432" iyz="-8.33331169026236E-07" izz="2.04445451860146"/>
       </inertial>
       <visual>
@@ -68,10 +68,136 @@
       </collision>
     </link>
+    <!-- plate (new link) -->
+    <link name="${prefix}plate_link">
+      <inertial>
+        <origin xyz="0.0698918884158706 7.79931674799172E-15 -0.0265000000000004" rpy="0 0 0"/>
+        <mass value="5.63390000000005"/>
+        <inertia ixx="0.0596659645833342" ixy="-9.2486172257981E-16" ixz="-5.64097728970053E-17" iyy="0.0554411298589926" iyz="-2.02970605311345E-14" izz="0.112469490258993"/>
+      </inertial>
+      <visual>
+        <origin xyz="0 0 0" rpy="0 0 0"/>
+        <geometry>
+          <mesh filename="package://alfa_robot_description/meshes/alfa_robot/visual/plate.STL"/>
+        </geometry>
+        <material name="white"/>
+      </visual>
+      <collision>
+        <origin xyz="0 0 0" rpy="0 0 0"/>
+        <geometry>
+          <mesh filename="package://alfa_robot_description/meshes/alfa_robot/collision/plate.STL"/>
+        </geometry>
+      </collision>
+    </link>
     <!-- leftarmbase (link name differs from joint for GZ compatibility) -->
+    <link name="${prefix}rightarmbase_link">
+      <inertial>
+        <origin xyz="-0.0636796126431308 0.0122577193728348 0.0451053264420542" rpy="0 0 0"/>
+        <mass value="12.5747563662381"/>
+        <inertia ixx="0.101345095416832" ixy="-0.0130489080354425" ixz="0.0363217436443393" iyy="0.783542694113494" iyz="0.00243382729312609" izz="0.751203346059042"/>
+      </inertial>
+      <visual>
+        <origin xyz="0 0 0" rpy="0 0 0"/>
+        <geometry>
+          <mesh filename="package://alfa_robot_description/meshes/alfa_robot/visual/rightarmbase.STL"/>
+        </geometry>
+        <material name="white"/>
+      </visual>
+      <collision>
+        <origin xyz="0 0 0" rpy="0 0 0"/>
+        <geometry>
+          <mesh filename="package://alfa_robot_description/meshes/alfa_robot/collision/rightarmbase.STL"/>
+        </geometry>
+      </collision>
+    </link>
+    <!-- leftjoint1 (link name differs from joint for GZ compatibility) -->
+    <link name="${prefix}rightjoint1_link">
+      <inertial>
+        <origin xyz="0.573415246499549 -4.59374950527724E-05 0.0242655456595022" rpy="0 0 0"/>
+        <mass value="2.70490666316"/>
+        <inertia ixx="0.0126377757573578" ixy="0.00720527645040998" ixz="-0.00117248770906348" iyy="0.048686796094863" iyz="2.68796611524638E-05" izz="0.0514547540806274"/>
+      </inertial>
+      <visual>
+        <origin xyz="0 0 0" rpy="0 0 0"/>
+        <geometry>
+          <mesh filename="package://alfa_robot_description/meshes/alfa_robot/visual/rightjoint1.STL"/>
+        </geometry>
+        <material name="white"/>
+      </visual>
+      <collision>
+        <origin xyz="0 0 0" rpy="0 0 0"/>
+        <geometry>
+          <mesh filename="package://alfa_robot_description/meshes/alfa_robot/collision/rightjoint1.STL"/>
+        </geometry>
+      </collision>
+    </link>
+    <!-- leftjoint2 (link name differs from joint for GZ compatibility) -->
+    <link name="${prefix}rightjoint2_link">
+      <inertial>
+        <origin xyz="0.0974924803763488 0.00121089642420269 0.0312499999989556" rpy="0 0 0"/>
+        <mass value="3.87102034080653"/>
+        <inertia ixx="0.00877438403522921" ixy="-0.000323257298214455" ixz="-6.23575529358465E-18" iyy="0.0347966708621837" iyz="-1.25198249100768E-19" izz="0.0391798661983104"/>
+      </inertial>
+      <visual>
+        <origin xyz="0 0 0" rpy="0 0 0"/>
+        <geometry>
+          <mesh filename="package://alfa_robot_description/meshes/alfa_robot/visual/rightjoint2.STL"/>
+        </geometry>
+        <material name="white"/>
+      </visual>
+      <collision>
+        <origin xyz="0 0 0" rpy="0 0 0"/>
+        <geometry>
+          <mesh filename="package://alfa_robot_description/meshes/alfa_robot/collision/rightjoint2.STL"/>
+        </geometry>
+      </collision>
+    </link>
+    <!-- leftjoint3 (link name differs from joint for GZ compatibility) -->
+    <link name="${prefix}rightjoint3_link">
+      <inertial>
+        <origin xyz="-1.19792535313579E-06 -0.000259105444550378 0.0735910770497341" rpy="0 0 0"/>
+        <mass value="2.16307538045068"/>
+        <inertia ixx="0.00756201455703306" ixy="9.47660614357424E-06" ixz="4.55435043254249E-08" iyy="0.00986535032315377" iyz="1.11493916689321E-05" izz="0.00512470452023724"/>
+      </inertial>
+      <visual>
+        <origin xyz="0 0 0" rpy="0 0 0"/>
+        <geometry>
+          <mesh filename="package://alfa_robot_description/meshes/alfa_robot/visual/rightjoint3.STL"/>
+        </geometry>
+        <material name="white"/>
+      </visual>
+      <collision>
+        <origin xyz="0 0 0" rpy="0 0 0"/>
+        <geometry>
+          <mesh filename="package://alfa_robot_description/meshes/alfa_robot/collision/rightjoint3.STL"/>
+        </geometry>
+      </collision>
+    </link>
+    <!-- leftjoint4 (link name differs from joint for GZ compatibility) -->
+    <link name="${prefix}rightjoint4_link">
+      <inertial>
+        <origin xyz="0.175697729205423 -0.00674464490596161 -0.0110129395688763" rpy="0 0 0"/>
+        <mass value="9.92773566678187"/>
+        <inertia ixx="0.0636499915289178" ixy="0.00193403162826374" ixz="0.0237125239968199" iyy="0.138062467565159" iyz="-0.000500914594551876" izz="0.123364066774707"/>
+      </inertial>
+      <visual>
+        <origin xyz="0 0 0" rpy="0 0 0"/>
+        <geometry>
+          <mesh filename="package://alfa_robot_description/meshes/alfa_robot/visual/rightjoint4.STL"/>
+        </geometry>
+        <material name="white"/>
+      </visual>
+      <collision>
+        <origin xyz="0 0 0" rpy="0 0 0"/>
+        <geometry>
+          <mesh filename="package://alfa_robot_description/meshes/alfa_robot/collision/rightjoint4.STL"/>
+        </geometry>
+      </collision>
+    </link>
+    <!-- rightarmbase (link name differs from joint for GZ compatibility) -->
     <link name="${prefix}leftarmbase_link">
       <inertial>
-        <origin xyz="0.29757 -0.16382 0.17861" rpy="0 0 0"/>
-        <mass value="18.562"/>
-        <inertia ixx="0.79163" ixy="0" ixz="0" iyy="0.43754" iyz="0" izz="0.39477"/>
+        <origin xyz="-0.0497615746360321 -0.0246057688749117 0.0430343814698384" rpy="0 0 0"/>
+        <mass value="13.1823257277416"/>
+        <inertia ixx="0.104088812848048" ixy="0.013834486847352" ixz="0.0505635371163732" iyy="0.863382985023394" iyz="-0.00307573195386396" izz="0.828453194049388"/>
       </inertial>
       <visual>
@@ -89,10 +215,10 @@
       </collision>
     </link>
-    <!-- leftjoint1 (link name differs from joint for GZ compatibility) -->
+    <!-- rightjoint1 (link name differs from joint for GZ compatibility) -->
     <link name="${prefix}leftjoint1_link">
       <inertial>
-        <origin xyz="0.00502820177318375 0.0342161631641283 0.281401807518592" rpy="0 0 0"/>
-        <mass value="2.1850126782898"/>
-        <inertia ixx="0.0182045859844161" ixy="0" ixz="0" iyy="0.0178203341545887" iyz="0" izz="0.00307285467353774"/>
+        <origin xyz="0.57341524650029 4.58601160402972E-05 0.0242655456596959" rpy="0 0 0"/>
+        <mass value="2.70490666316309"/>
+        <inertia ixx="0.0126378005178209" ixy="-0.00720533280334168" ixz="-0.001172487709181" iyy="0.0486867960951763" iyz="-2.68816757577675E-05" izz="0.051454778841387"/>
       </inertial>
       <visual>
@@ -110,10 +236,10 @@
       </collision>
     </link>
-    <!-- leftjoint2 (link name differs from joint for GZ compatibility) -->
+    <!-- rightjoint2 (link name differs from joint for GZ compatibility) -->
     <link name="${prefix}leftjoint2_link">
       <inertial>
-        <origin xyz="-0.149017202271686 -0.000289955936075892 0.0195313938678338" rpy="0 0 0"/>
-        <mass value="1.30575454209857"/>
-        <inertia ixx="0.00160201811072687" ixy="0" ixz="0" iyy="0.0045017939044488" iyz="0" izz="0.00558222979330651"/>
+        <origin xyz="0.0982222389567129 2.77555756156289E-16 0.0280872172763753" rpy="0 0 0"/>
+        <mass value="3.80063815279185"/>
+        <inertia ixx="0.00855142309151201" ixy="-6.9931040125315E-18" ixz="0.000737698249610721" iyy="0.03409027056488" iyz="6.71273610699033E-19" izz="0.038449314153095"/>
       </inertial>
       <visual>
@@ -131,10 +257,10 @@
       </collision>
     </link>
-    <!-- leftjoint3 (link name differs from joint for GZ compatibility) -->
+    <!-- rightjoint3 (link name differs from joint for GZ compatibility) -->
     <link name="${prefix}leftjoint3_link">
       <inertial>
-        <origin xyz="4.32362620763627E-05 0.00090464696325504 0.0847683944898301" rpy="0 0 0"/>
-        <mass value="1.2829930846756"/>
-        <inertia ixx="0.00201630610415181" ixy="0" ixz="0" iyy="0.00302769103356114" iyz="0" izz="0.00227450005359758"/>
+        <origin xyz="0.00424368697534261 0.000259106738649706 0.0734709611355132" rpy="0 0 0"/>
+        <mass value="2.16310625460758"/>
+        <inertia ixx="0.00755389789683751" ixy="-6.42921999609667E-07" ixz="-0.000140310452236765" iyy="0.00986541284670613" iyz="-1.11309098584596E-05" izz="0.0051328070950562"/>
       </inertial>
       <visual>
@@ -152,10 +278,10 @@
       </collision>
     </link>
-    <!-- leftjoint4 (link name differs from joint for GZ compatibility) -->
+    <!-- rightjoint4 (link name differs from joint for GZ compatibility) -->
     <link name="${prefix}leftjoint4_link">
       <inertial>
-        <origin xyz="-0.192813505520282 -0.00671906082576801 -0.0056742418931493" rpy="0 0 0"/>
-        <mass value="1.70355283014671"/>
-        <inertia ixx="0.00487993158594216" ixy="0" ixz="0" iyy="0.00449383295362854" iyz="0" izz="0.00373716891794887"/>
+        <origin xyz="0.179805345971669 0.00027459738144453 0.0111248225390411" rpy="0 0 0"/>
+        <mass value="9.59771353822043"/>
+        <inertia ixx="0.0623468092864488" ixy="-0.000903417557492398" ixz="-0.0234301373942001" iyy="0.130723241701585" iyz="-0.000423930246625516" izz="0.115651820367604"/>
       </inertial>
       <visual>
@@ -170,214 +296,4 @@
         <geometry>
           <mesh filename="package://alfa_robot_description/meshes/alfa_robot/collision/leftjoint4.STL"/>
-        </geometry>
-      </collision>
-    </link>
-    <!-- rightarmbase (link name differs from joint for GZ compatibility) -->
-    <link name="${prefix}rightarmbase_link">
-      <inertial>
-        <origin xyz="0.0568652250818897 0.0787348857644462 0.00280311476846101" rpy="0 0 0"/>
-        <mass value="6.19361408901838"/>
-        <inertia ixx="0.0557032604337449" ixy="0" ixz="0" iyy="0.0270932354936772" iyz="0" izz="0.0553565785725355"/>
-      </inertial>
-      <visual>
-        <origin xyz="0 0 0" rpy="0 0 0"/>
-        <geometry>
-          <mesh filename="package://alfa_robot_description/meshes/alfa_robot/visual/rightarmbase.STL"/>
-        </geometry>
-        <material name="white"/>
-      </visual>
-      <collision>
-        <origin xyz="0 0 0" rpy="0 0 0"/>
-        <geometry>
-          <mesh filename="package://alfa_robot_description/meshes/alfa_robot/collision/rightarmbase.STL"/>
-        </geometry>
-      </collision>
-    </link>
-    <!-- rightjoint1 (link name differs from joint for GZ compatibility) -->
-    <link name="${prefix}rightjoint1_link">
-      <inertial>
-        <origin xyz="0.0125188483480216 -0.0276314408365126 0.290315233804106" rpy="0 0 0"/>
-        <mass value="1.84782059002931"/>
-        <inertia ixx="0.00887650044662994" ixy="0" ixz="0" iyy="0.00849110110359986" iyz="0" izz="0.00297285321308238"/>
-      </inertial>
-      <visual>
-        <origin xyz="0 0 0" rpy="0 0 0"/>
-        <geometry>
-          <mesh filename="package://alfa_robot_description/meshes/alfa_robot/visual/rightjoint1.STL"/>
-        </geometry>
-        <material name="white"/>
-      </visual>
-      <collision>
-        <origin xyz="0 0 0" rpy="0 0 0"/>
-        <geometry>
-          <mesh filename="package://alfa_robot_description/meshes/alfa_robot/collision/rightjoint1.STL"/>
-        </geometry>
-      </collision>
-    </link>
-    <!-- rightjoint2 (link name differs from joint for GZ compatibility) -->
-    <link name="${prefix}rightjoint2_link">
-      <inertial>
-        <origin xyz="-0.1474146108181 0.00338572158786365 0.0189953911214911" rpy="0 0 0"/>
-        <mass value="1.30873868902494"/>
-        <inertia ixx="0.00160436190994309" ixy="0" ixz="0" iyy="0.00450351560284405" iyz="0" izz="0.00558274700030671"/>
-      </inertial>
-      <visual>
-        <origin xyz="0 0 0" rpy="0 0 0"/>
-        <geometry>
-          <mesh filename="package://alfa_robot_description/meshes/alfa_robot/visual/rightjoint2.STL"/>
-        </geometry>
-        <material name="white"/>
-      </visual>
-      <collision>
-        <origin xyz="0 0 0" rpy="0 0 0"/>
-        <geometry>
-          <mesh filename="package://alfa_robot_description/meshes/alfa_robot/collision/rightjoint2.STL"/>
-        </geometry>
-      </collision>
-    </link>
-    <!-- rightjoint3 (link name differs from joint for GZ compatibility) -->
-    <link name="${prefix}rightjoint3_link">
-      <inertial>
-        <origin xyz="0.000636075551307513 -0.000732173079496579 0.0855214235064663" rpy="0 0 0"/>
-        <mass value="1.26746478497369"/>
-        <inertia ixx="0.00201192504269909" ixy="0" ixz="0" iyy="0.00302323826204887" iyz="0" izz="0.0022699433487247"/>
-      </inertial>
-      <visual>
-        <origin xyz="0 0 0" rpy="0 0 0"/>
-        <geometry>
-          <mesh filename="package://alfa_robot_description/meshes/alfa_robot/visual/rightjoint3.STL"/>
-        </geometry>
-        <material name="white"/>
-      </visual>
-      <collision>
-        <origin xyz="0 0 0" rpy="0 0 0"/>
-        <geometry>
-          <mesh filename="package://alfa_robot_description/meshes/alfa_robot/collision/rightjoint3.STL"/>
-        </geometry>
-      </collision>
-    </link>
-    <!-- rightjoint4 (link name differs from joint for GZ compatibility) -->
-    <link name="${prefix}rightjoint4_link">
-      <inertial>
-        <origin xyz="0.19373426132831 -0.00481885161982026 -0.0070966670102961" rpy="0 0 0"/>
-        <mass value="1.798511332725"/>
-        <inertia ixx="0.00490614728606829" ixy="0" ixz="0" iyy="0.00452071247048926" iyz="0" izz="0.00376343860760531"/>
-      </inertial>
-      <visual>
-        <origin xyz="0 0 0" rpy="0 0 0"/>
-        <geometry>
-          <mesh filename="package://alfa_robot_description/meshes/alfa_robot/visual/rightjoint4.STL"/>
-        </geometry>
-        <material name="white"/>
-      </visual>
-      <collision>
-        <origin xyz="0 0 0" rpy="0 0 0"/>
-        <geometry>
-          <mesh filename="package://alfa_robot_description/meshes/alfa_robot/collision/rightjoint4.STL"/>
-        </geometry>
-      </collision>
-    </link>
-    <!-- base_chassis_link -->
-    <link name="${prefix}base_chassis_link">
-      <inertial>
-        <origin xyz="0.055638 -0.051873 0.029822" rpy="0 0 0"/>
-        <mass value="270"/>
-        <inertia ixx="1.2255" ixy="-0.00010878" ixz="0.00012664" iyy="0.82719" iyz="0.0048512" izz="2.0056"/>
-      </inertial>
-      <visual>
-        <origin xyz="0 0 0" rpy="0 0 0"/>
-        <geometry>
-          <mesh filename="package://alfa_robot_description/meshes/alfa_robot/visual/base_chassis.STL"/>
-        </geometry>
-        <material name="white"/>
-      </visual>
-      <collision>
-        <origin xyz="0 0 0" rpy="0 0 0"/>
-        <geometry>
-          <mesh filename="package://alfa_robot_description/meshes/alfa_robot/visual/base_chassis.STL"/>
-        </geometry>
-      </collision>
-    </link>
-    <!-- left back (link name differs from joint for GZ compatibility) -->
-    <link name="${prefix}left back_link">
-      <inertial>
-        <origin xyz="0 0 0" rpy="0 0 0"/>
-        <mass value="20"/>
-        <inertia ixx="0.0034435" ixy="0" ixz="0" iyy="0.0034435" iyz="0" izz="0.0068283"/>
-      </inertial>
-      <visual>
-        <origin xyz="0 0 0" rpy="0 0 0"/>
-        <geometry>
-          <mesh filename="package://alfa_robot_description/meshes/alfa_robot/visual/leftback.STL"/>
-        </geometry>
-        <material name="white"/>
-      </visual>
-      <collision>
-        <origin xyz="0 0 0" rpy="0 0 0"/>
-        <geometry>
-          <mesh filename="package://alfa_robot_description/meshes/alfa_robot/collision/wheel.STL"/>
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