Commit message: 1

File: src/alfa_robot_description/urdf/alfa_robot/alfa_robot_macro.ros2_control.xacro (robot description, xacro)
@@ -41,10 +41,10 @@
           <param name="safe_position_leftjoint1">0.0</param>
           <param name="safe_position_leftjoint2">0.0</param>
-          <param name="safe_position_leftjoint3">-1.57</param>
+          <param name="safe_position_leftjoint3">0.0</param>
           <param name="safe_position_leftjoint4">0.0</param>
           <param name="safe_position_rightarmbase">0.0</param>
           <param name="safe_position_rightjoint1">0.0</param>
           <param name="safe_position_rightjoint2">0.0</param>
-          <param name="safe_position_rightjoint3">-1.57</param>
+          <param name="safe_position_rightjoint3">0.0</param>
           <param name="safe_position_rightjoint4">0.0</param>
         </xacro:unless>

File: src/alfa_robot_description/urdf/alfa_robot/alfa_robot_macro.xacro (robot description, xacro)
@@ -383,4 +383,8 @@
       </collision>
     </link>
+    <!-- right_ee_link (virtual end effector for MoveIt2 planning) -->
+    <link name="${prefix}right_ee_link"/>
+    <!-- left_ee_link (virtual end effector for MoveIt2 planning) -->
+    <link name="${prefix}left_ee_link"/>
     <!-- END LINKS -->
     <!-- JOINTS -->
@@ -404,5 +408,5 @@
       <child link="${prefix}updown_link"/>
       <axis xyz="0 0 1"/>
-      <limit lower="-0.15" upper="1" effort="0" velocity="0"/>
+      <limit lower="-0.15" upper="1" effort="1000" velocity="1000"/>
     </joint>
     <!-- leftarmbase -->
@@ -412,5 +416,5 @@
       <child link="${prefix}leftarmbase_link"/>
       <axis xyz="0 0 1"/>
-      <limit lower="-0.3" upper="0.3" effort="0" velocity="0"/>
+      <limit lower="-0.15" upper="0.15" effort="1000" velocity="1000"/>
     </joint>
     <!-- leftjoint1 -->
@@ -420,5 +424,5 @@
       <child link="${prefix}leftjoint1_link"/>
       <axis xyz="0 0 1"/>
-      <limit lower="-0.5" upper="0.5" effort="0" velocity="0"/>
+      <limit lower="0" upper="0.5" effort="1000" velocity="1000"/>
     </joint>
     <!-- leftjoint2 -->
@@ -437,9 +441,16 @@
     </joint>
     <!-- leftjoint4 -->
-    <joint name="${prefix}leftjoint4" type="continuous">
+    <joint name="${prefix}leftjoint4" type="revolute">
       <origin xyz="0.00058164 0.044646 0.115" rpy="-1.5708 0 -0.013027"/>
       <parent link="${prefix}leftjoint3_link"/>
       <child link="${prefix}leftjoint4_link"/>
       <axis xyz="0 0 -1"/>
+      <limit lower="-3.14" upper="0" effort="1000" velocity="1000"/>
+    </joint>
+    <!-- left_ee_joint (virtual fixed joint for MoveIt2 end effector) -->
+    <joint name="${prefix}left_ee_joint" type="fixed">
+      <origin xyz="-0.275 -0.0308 -0.02825" rpy="0 0 0"/>
+      <parent link="${prefix}leftjoint4_link"/>
+      <child link="${prefix}left_ee_link"/>
     </joint>
     <!-- rightarmbase -->
@@ -449,5 +460,5 @@
       <child link="${prefix}rightarmbase_link"/>
       <axis xyz="0 0 -1"/>
-      <limit lower="-0.3" upper="0.3" effort="0" velocity="0"/>
+      <limit lower="-0.15" upper="0.15" effort="1000" velocity="1000"/>
     </joint>
     <!-- rightjoint1 -->
@@ -457,5 +468,5 @@
       <child link="${prefix}rightjoint1_link"/>
       <axis xyz="0 0 1"/>
-      <limit lower="0" upper="0.5" effort="0" velocity="0"/>
+      <limit lower="0" upper="0.5" effort="1000" velocity="1000"/>
     </joint>
     <!-- rightjoint2 -->
@@ -474,9 +485,16 @@
     </joint>
     <!-- rightjoint4 -->
-    <joint name="${prefix}rightjoint4" type="continuous">
+    <joint name="${prefix}rightjoint4" type="revolute">
       <origin xyz="-0.0003624 -0.044649 0.115" rpy="-1.5708 0 3.1335"/>
       <parent link="${prefix}rightjoint3_link"/>
       <child link="${prefix}rightjoint4_link"/>
       <axis xyz="0 0 1"/>
+      <limit lower="-3.14" upper="0" effort="1000" velocity="1000"/>
+    </joint>
+    <!-- right_ee_joint (virtual fixed joint for MoveIt2 end effector) -->
+    <joint name="${prefix}right_ee_joint" type="fixed">
+      <origin xyz="0.275 -0.0308 -0.02825" rpy="0 0 0"/>
+      <parent link="${prefix}rightjoint4_link"/>
+      <child link="${prefix}right_ee_link"/>
     </joint>
     <!-- base_chassis_link_joint -->
@@ -492,5 +510,5 @@
       <child link="${prefix}left back_link"/>
       <axis xyz="0 0 -1"/>
-      <limit effort="0" velocity="10"/>
+      <limit effort="1000" velocity="10"/>
     </joint>
     <!-- left forward -->
@@ -500,5 +518,5 @@
       <child link="${prefix}left forward_link"/>
       <axis xyz="0 0 -1"/>
-      <limit effort="0" velocity="10"/>
+      <limit effort="1000" velocity="10"/>
     </joint>
     <!-- right back -->
@@ -508,5 +526,5 @@
       <child link="${prefix}right back_link"/>
       <axis xyz="0 0 -1"/>
-      <limit effort="0" velocity="10"/>
+      <limit effort="1000" velocity="10"/>
     </joint>
     <!-- right forward -->
@@ -516,5 +534,5 @@
       <child link="${prefix}right forward_link"/>
       <axis xyz="0 0 -1"/>
-      <limit effort="0" velocity="10"/>
+      <limit effort="1000" velocity="10"/>
     </joint>
     <!-- END JOINTS -->

Commit message: URDF中添加雷达相机

File: src/alfa_robot_description/urdf/alfa_robot/alfa_robot_macro.ros2_control.xacro (robot description, xacro)
@@ -86,9 +86,69 @@
         <state_interface name="acceleration"/>
       </joint>
+      <!-- rightarmbase (prismatic) -->
+      <joint name="${prefix}rightarmbase">
+        <command_interface name="position">
+          <param name="min">0</param>
+          <param name="max">0.16</param>
+        </command_interface>
+        <state_interface name="position">
+          <param name="initial_value">0.0</param>
+        </state_interface>
+        <state_interface name="velocity"/>
+        <state_interface name="acceleration"/>
+      </joint>
+      <!-- rightjoint1 (prismatic) -->
+      <joint name="${prefix}rightjoint1">
+        <command_interface name="position">
+          <param name="min">0</param>
+          <param name="max">0.5</param>
+        </command_interface>
+        <state_interface name="position">
+          <param name="initial_value">0.0</param>
+        </state_interface>
+        <state_interface name="velocity"/>
+        <state_interface name="acceleration"/>
+      </joint>
+      <!-- rightjoint2 (continuous) -->
+      <joint name="${prefix}rightjoint2">
+        <command_interface name="position">
+          <param name="min">-3.14159</param>
+          <param name="max">3.14159</param>
+        </command_interface>
+        <state_interface name="position">
+          <param name="initial_value">0.0</param>
+        </state_interface>
+        <state_interface name="velocity"/>
+        <state_interface name="acceleration"/>
+      </joint>
+      <!-- rightjoint3 (continuous) -->
+      <joint name="${prefix}rightjoint3">
+        <command_interface name="position">
+          <param name="min">-3.14159</param>
+          <param name="max">3.14159</param>
+        </command_interface>
+        <state_interface name="position">
+          <param name="initial_value">0.0</param>
+        </state_interface>
+        <state_interface name="velocity"/>
+        <state_interface name="acceleration"/>
+      </joint>
+      <!-- rightjoint4 (continuous) -->
+      <joint name="${prefix}rightjoint4">
+        <command_interface name="position">
+          <param name="min">-3.14159</param>
+          <param name="max">3.14159</param>
+        </command_interface>
+        <state_interface name="position">
+          <param name="initial_value">0.0</param>
+        </state_interface>
+        <state_interface name="velocity"/>
+        <state_interface name="acceleration"/>
+      </joint>
       <!-- leftarmbase (prismatic) -->
-      <joint name="${prefix}rightarmbase">
-        <command_interface name="position">
-          <param name="min">0</param>
-          <param name="max">0.16</param>
+      <joint name="${prefix}leftarmbase">
+        <command_interface name="position">
+          <param name="min">0</param>
+          <param name="max">0.2</param>
         </command_interface>
         <state_interface name="position">
@@ -99,5 +159,5 @@
       </joint>
       <!-- leftjoint1 (prismatic) -->
-      <joint name="${prefix}rightjoint1">
+      <joint name="${prefix}leftjoint1">
         <command_interface name="position">
           <param name="min">0</param>
@@ -111,5 +171,5 @@
       </joint>
       <!-- leftjoint2 (continuous) -->
-      <joint name="${prefix}rightjoint2">
+      <joint name="${prefix}leftjoint2">
         <command_interface name="position">
           <param name="min">-3.14159</param>
@@ -123,64 +183,4 @@
       </joint>
       <!-- leftjoint3 (continuous) -->
-      <joint name="${prefix}rightjoint3">
-        <command_interface name="position">
-          <param name="min">-3.14159</param>
-          <param name="max">3.14159</param>
-        </command_interface>
-        <state_interface name="position">
-          <param name="initial_value">0.0</param>
-        </state_interface>
-        <state_interface name="velocity"/>
-        <state_interface name="acceleration"/>
-      </joint>
-      <!-- leftjoint4 (continuous) -->
-      <joint name="${prefix}rightjoint4">
-        <command_interface name="position">
-          <param name="min">-3.14159</param>
-          <param name="max">3.14159</param>
-        </command_interface>
-        <state_interface name="position">
-          <param name="initial_value">0.0</param>
-        </state_interface>
-        <state_interface name="velocity"/>
-        <state_interface name="acceleration"/>
-      </joint>
-      <!-- rightarmbase (prismatic) -->
-      <joint name="${prefix}leftarmbase">
-        <command_interface name="position">
-          <param name="min">0</param>
-          <param name="max">0.2</param>
-        </command_interface>
-        <state_interface name="position">
-          <param name="initial_value">0.0</param>
-        </state_interface>
-        <state_interface name="velocity"/>
-        <state_interface name="acceleration"/>
-      </joint>
-      <!-- rightjoint1 (prismatic) -->
-      <joint name="${prefix}leftjoint1">
-        <command_interface name="position">
-          <param name="min">0</param>
-          <param name="max">0.5</param>
-        </command_interface>
-        <state_interface name="position">
-          <param name="initial_value">0.0</param>
-        </state_interface>
-        <state_interface name="velocity"/>
-        <state_interface name="acceleration"/>
-      </joint>
-      <!-- rightjoint2 (continuous) -->
-      <joint name="${prefix}leftjoint2">
-        <command_interface name="position">
-          <param name="min">-3.14159</param>
-          <param name="max">3.14159</param>
-        </command_interface>
-        <state_interface name="position">
-          <param name="initial_value">0.0</param>
-        </state_interface>
-        <state_interface name="velocity"/>
-        <state_interface name="acceleration"/>
-      </joint>
-      <!-- rightjoint3 (continuous) -->
       <joint name="${prefix}leftjoint3">
         <command_interface name="position">
@@ -194,5 +194,5 @@
         <state_interface name="acceleration"/>
       </joint>
-      <!-- rightjoint4 (continuous) -->
+      <!-- leftjoint4 (revolute) -->
       <joint name="${prefix}leftjoint4">
         <command_interface name="position">

File: src/alfa_robot_description/urdf/alfa_robot/alfa_robot_macro.xacro (robot description, xacro)
@@ -296,4 +296,48 @@
         <geometry>
           <mesh filename="package://alfa_robot_description/meshes/alfa_robot/collision/leftjoint4.STL"/>
+        </geometry>
+      </collision>
+    </link>
+    <!-- camera -->
+    <link name="${prefix}camera_link">
+      <inertial>
+        <origin xyz="-0.0128838261972163 0.00026531291498777 0.00027897095170859" rpy="0 0 0"/>
+        <mass value="0.0247923828845652"/>
+        <inertia ixx="3.5668701541101E-05" ixy="-1.36439346012497E-08" ixz="-2.61698308401705E-08"
+                 iyy="2.83830455101906E-06" iyz="2.73948631199571E-08" izz="3.34987859138971E-05"/>
+      </inertial>
+      <visual>
+        <origin xyz="0 0 0" rpy="0 0 0"/>
+        <geometry>
+          <mesh filename="package://alfa_robot_description/meshes/alfa_robot/visual/camera.STL"/>
+        </geometry>
+        <material name="white"/>
+      </visual>
+      <collision>
+        <origin xyz="0 0 0" rpy="0 0 0"/>
+        <geometry>
+          <mesh filename="package://alfa_robot_description/meshes/alfa_robot/collision/camera.STL"/>
+        </geometry>
+      </collision>
+    </link>
+    <!-- lidar -->
+    <link name="${prefix}lidar_link">
+      <inertial>
+        <origin xyz="-0.00468733327842979 -6.25961285910526E-06 -0.016722032751983" rpy="0 0 0"/>
+        <mass value="0.141886849294983"/>
+        <inertia ixx="4.37633098241424E-05" ixy="-5.36171297405178E-09" ixz="7.01471703806087E-06"
+                 iyy="4.50759714359166E-05" iyz="9.27886666435768E-10" izz="6.68414722762209E-05"/>
+      </inertial>
+      <visual>
+        <origin xyz="0 0 0" rpy="0 0 0"/>
+        <geometry>
+          <mesh filename="package://alfa_robot_description/meshes/alfa_robot/visual/lidar.STL"/>
+        </geometry>
+        <material name="arm_grey"/>
+      </visual>
+      <collision>
+        <origin xyz="0 0 0" rpy="0 0 0"/>
+        <geometry>
+          <mesh filename="package://alfa_robot_description/meshes/alfa_robot/collision/lidar.STL"/>
         </geometry>
       </collision>
@@ -426,4 +470,16 @@
       <child link="${prefix}left_ee_link"/>
     </joint>
+    <!-- camera -->
+    <joint name="${prefix}camera" type="fixed">
+      <origin xyz="0.51384 0 0.07785" rpy="0 0 0"/>
+      <parent link="${prefix}updown_link"/>
+      <child link="${prefix}camera_link"/>
+    </joint>
+    <!-- lidar -->
+    <joint name="${prefix}lidar" type="fixed">
+      <origin xyz="0.46082 0 0.13841" rpy="0 0 0"/>
+      <parent link="${prefix}updown_link"/>
+      <child link="${prefix}lidar_link"/>
+    </joint>
     <!-- END JOINTS -->
   </xacro:macro>
