Commit message: feat: 左臂升级为7自由度，新增leftjoint6关节
URDF/Xacro更改:
- 新增 leftjoint6 关节和 link，类型为 prismatic (直线，行程0-15cm)
- leftjoint4 从 prismatic 改为 continuous (旋转)
- 更新 leftarmbase/leftjoint1 运动范围
- 更新所有左臂关节的惯性参数和碰撞网格
- 更新末端执行器位置到 leftjoint6_link

控制器配置更新:
- all_position_controller、left_arm_controller 等新增 leftjoint6
- MoveIt SRDF 和 ros2_controllers 配置更新

.gitignore 更新:
- 允许 meshes 目录下的 STL 文件被跟踪

Co-Authored-By: Claude Opus 4.7 <noreply@anthropic.com>

File: src/alfa_robot_description/urdf/alfa_robot/alfa_robot_macro.ros2_control.xacro (robot description, xacro)
@@ -45,4 +45,5 @@
           <param name="safe_position_leftjoint4">0.0</param>
           <param name="safe_position_leftjoint5">0.0</param>
+          <param name="safe_position_leftjoint6">0.0</param>
           <param name="safe_position_rightarmbase">0.0</param>
           <param name="safe_position_rightjoint1">0.0</param>
@@ -152,6 +153,6 @@
       <joint name="${prefix}leftarmbase">
         <command_interface name="position">
-          <param name="min">-0.16</param>
-          <param name="max">0</param>
+          <param name="min">0</param>
+          <param name="max">0.14</param>
         </command_interface>
         <state_interface name="position">
@@ -165,5 +166,5 @@
         <command_interface name="position">
           <param name="min">0</param>
-          <param name="max">0.45</param>
+          <param name="max">0.42</param>
         </command_interface>
         <state_interface name="position">
@@ -197,9 +198,9 @@
         <state_interface name="acceleration"/>
       </joint>
-      <!-- leftjoint4 (prismatic) -->
+      <!-- leftjoint4 (continuous) -->
       <joint name="${prefix}leftjoint4">
         <command_interface name="position">
-          <param name="min">0</param>
-          <param name="max">0.22</param>
+          <param name="min">-3.14159</param>
+          <param name="max">3.14159</param>
         </command_interface>
         <state_interface name="position">
@@ -214,4 +215,16 @@
           <param name="min">-3.14159</param>
           <param name="max">3.14159</param>
+        </command_interface>
+        <state_interface name="position">
+          <param name="initial_value">0.0</param>
+        </state_interface>
+        <state_interface name="velocity"/>
+        <state_interface name="acceleration"/>
+      </joint>
+      <!-- leftjoint6 (prismatic, new end effector extension) -->
+      <joint name="${prefix}leftjoint6">
+        <command_interface name="position">
+          <param name="min">0</param>
+          <param name="max">0.15</param>
         </command_interface>
         <state_interface name="position">

File: src/alfa_robot_description/urdf/alfa_robot/alfa_robot_macro.xacro (robot description, xacro)
@@ -29,7 +29,7 @@
     <link name="${prefix}turn_link">
       <inertial>
-        <origin xyz="8.3102236387753E-05 -5.6319532371063E-13 0.854091510931534" rpy="0 0 0"/>
-        <mass value="93.4308976427189"/>
-        <inertia ixx="39.2606066773154" ixy="6.93889405615743E-18" ixz="-5.06230387770105E-13" iyy="39.2606066773154" iyz="2.34703241842353E-11" izz="1.49032676193219"/>
+        <origin xyz="-0.0697894032768815 -0.00012433244764639 0.982155423971065" rpy="0 0 0"/>
+        <mass value="42.0737844290435"/>
+        <inertia ixx="10.0720353784748" ixy="-1.75362629131178E-06" ixz="5.29823321336754E-05" iyy="10.0937833616587" iyz="1.43589075450652E-06" izz="0.327199381319826"/>
       </inertial>
       <visual>
@@ -50,7 +50,7 @@
     <link name="${prefix}updown_link">
       <inertial>
-        <origin xyz="-0.297917412220348 -3.47192615164638E-07 0.0811648445824145" rpy="0 0 0"/>
-        <mass value="49.32553657462"/>
-        <inertia ixx="0.931332356925864" ixy="9.94007584674414E-06" ixz="0.066855170904404" iyy="1.73410727221432" iyz="-8.33331169026236E-07" izz="2.04445451860146"/>
+        <origin xyz="-0.196828632659582 0.0148673483555221 0.0956849238503419" rpy="0 0 0"/>
+        <mass value="26.931167747836"/>
+        <inertia ixx="0.231217459750122" ixy="2.93337887014215E-05" ixz="0.000951254936009737" iyy="0.178754005132662" iyz="-1.44830456938328E-05" izz="0.348822965146485"/>
       </inertial>
       <visual>
@@ -92,7 +92,7 @@
     <link name="${prefix}rightarmbase_link">
       <inertial>
-        <origin xyz="-0.0636796126431308 0.0122577193728348 0.0451053264420542" rpy="0 0 0"/>
-        <mass value="12.5747563662381"/>
-        <inertia ixx="0.101345095416832" ixy="-0.0130489080354425" ixz="0.0363217436443393" iyy="0.783542694113494" iyz="0.00243382729312609" izz="0.751203346059042"/>
+        <origin xyz="0.0065184830076993 0.0166887762268038 0.0522668634862797" rpy="0 0 0"/>
+        <mass value="6.84202784607225"/>
+        <inertia ixx="0.0164013007938562" ixy="9.83820122469931E-06" ixz="0.000389797205690543" iyy="0.0925933973563738" iyz="-0.000135019154076589" izz="0.0913226513514585"/>
       </inertial>
       <visual>
@@ -113,7 +113,7 @@
     <link name="${prefix}rightjoint1_link">
       <inertial>
-        <origin xyz="0.573415246499549 -4.59374950527724E-05 0.0242655456595022" rpy="0 0 0"/>
-        <mass value="2.70490666316"/>
-        <inertia ixx="0.0126377757573578" ixy="0.00720527645040998" ixz="-0.00117248770906348" iyy="0.048686796094863" iyz="2.68796611524638E-05" izz="0.0514547540806274"/>
+        <origin xyz="0.363254870237073 -0.00430635985497407 0.00399546521565419" rpy="0 0 0"/>
+        <mass value="2.46184783942628"/>
+        <inertia ixx="0.00349086639926755" ixy="-2.69181048005308E-07" ixz="1.18635671701878E-06" iyy="0.0377537678958155" iyz="-8.95938402086781E-05" izz="0.0384323225293085"/>
       </inertial>
       <visual>
@@ -134,7 +134,7 @@
     <link name="${prefix}rightjoint2_link">
       <inertial>
-        <origin xyz="0.0974924803763488 0.00121089642420269 0.0312499999989556" rpy="0 0 0"/>
-        <mass value="3.87102034080653"/>
-        <inertia ixx="0.00877438403522921" ixy="-0.000323257298214455" ixz="-6.23575529358465E-18" iyy="0.0347966708621837" iyz="-1.25198249100768E-19" izz="0.0391798661983104"/>
+        <origin xyz="0.150409645725255 0.00448982924374308 0.0188845887503852" rpy="0 0 0"/>
+        <mass value="2.48976780370709"/>
+        <inertia ixx="0.00317772693030281" ixy="-6.94923571222452E-05" ixz="3.53574425014485E-07" iyy="0.00869746381533899" iyz="2.83263029765993E-08" izz="0.0108712453298436"/>
       </inertial>
       <visual>
@@ -155,7 +155,7 @@
     <link name="${prefix}rightjoint3_link">
       <inertial>
-        <origin xyz="-1.19792535313579E-06 -0.000259105444550378 0.0735910770497341" rpy="0 0 0"/>
-        <mass value="2.16307538045068"/>
-        <inertia ixx="0.00756201455703306" ixy="9.47660614357424E-06" ixz="4.55435043254249E-08" iyy="0.00986535032315377" iyz="1.11493916689321E-05" izz="0.00512470452023724"/>
+        <origin xyz="-2.6889792636986E-05 0.00177301957246101 0.0771138491168442" rpy="0 0 0"/>
+        <mass value="2.36049013572046"/>
+        <inertia ixx="0.00371444525711301" ixy="6.97171051907141E-06" ixz="6.54275051629753E-07" iyy="0.00546440283832201" iyz="-3.57400059517791E-07" izz="0.00425607026205507"/>
       </inertial>
       <visual>
@@ -176,7 +176,7 @@
     <link name="${prefix}rightjoint4_link">
       <inertial>
-        <origin xyz="0.175697729205423 -0.00674464490596161 -0.0110129395688763" rpy="0 0 0"/>
-        <mass value="9.92773566678187"/>
-        <inertia ixx="0.0636499915289178" ixy="0.00193403162826374" ixz="0.0237125239968199" iyy="0.138062467565159" iyz="-0.000500914594551876" izz="0.123364066774707"/>
+        <origin xyz="0.168114701096427 -0.011285572595106 -0.0157488023557206" rpy="0 0 0"/>
+        <mass value="1.71170101112419"/>
+        <inertia ixx="0.00484207681591099" ixy="-6.65777874958895E-05" ixz="-9.07857869658426E-06" iyy="0.00422266337154443" iyz="9.33417209316671E-07" izz="0.00348624434926117"/>
       </inertial>
       <visual>
@@ -197,7 +197,7 @@
     <link name="${prefix}leftarmbase_link">
       <inertial>
-        <origin xyz="0.00858986048627108 -0.0287669594343616 0.0499555606572781" rpy="0 0 0"/>
-        <mass value="7.06520786855791"/>
-        <inertia ixx="0.0164730270054741" ixy="9.84172584812845E-06" ixz="0.000387662666781538" iyy="0.0926777572077124" iyz="0.000120939157760669" izz="0.0913979516362821"/>
+        <origin xyz="0.00858986048699223 -0.0287669594345854 0.0499555606572479" rpy="0 0 0"/>
+        <mass value="7.06520786853071"/>
+        <inertia ixx="0.0164730270054181" ixy="9.84172582142273E-06" ixz="0.000387662666799276" iyy="0.0926777572076808" iyz="0.0001209391577568" izz="0.091397951636245"/>
       </inertial>
       <visual>
@@ -218,7 +218,7 @@
     <link name="${prefix}leftjoint1_link">
       <inertial>
-        <origin xyz="0.374415906775149 -0.00904923744463459 -0.0148960568987655" rpy="0 0 0"/>
-        <mass value="2.37583354079001"/>
-        <inertia ixx="0.00207304785493464" ixy="1.02796852110949E-06" ixz="1.72939416918191E-06" iyy="0.0375730763919683" iyz="9.61510248922564E-06" izz="0.0381102083862888"/>
+        <origin xyz="0.32398542150288 0.0675146775051429 -0.0136862113102643" rpy="0 0 0"/>
+        <mass value="2.48077826581444"/>
+        <inertia ixx="0.0026348787049079" ixy="-2.78509690352211E-07" ixz="2.27753599606112E-06" iyy="0.0378277422884527" iyz="3.74055166687532E-05" izz="0.0384178105950815"/>
       </inertial>
       <visual>
@@ -239,7 +239,7 @@
     <link name="${prefix}leftjoint2_link">
       <inertial>
-        <origin xyz="-3.31662261210397E-06 -0.0765366527672894 0.0979391100942644" rpy="0 0 0"/>
-        <mass value="0.86529067490259"/>
-        <inertia ixx="0.00132661283538382" ixy="-1.59054446085595E-07" ixz="3.24265168911163E-07" iyy="0.00116106049969607" iyz="-1.07921267015626E-06" izz="0.00137430337463552"/>
+        <origin xyz="0.00998125570987396 -0.0501508012211525 0.0836125943851177" rpy="0 0 0"/>
+        <mass value="0.924094586385747"/>
+        <inertia ixx="0.00138886172299487" ixy="-9.60798584640597E-07" ixz="-2.47998998359295E-07" iyy="0.00126018297864274" iyz="6.56045281312999E-07" izz="0.0014853923148985"/>
       </inertial>
       <visual>
@@ -260,7 +260,7 @@
     <link name="${prefix}leftjoint3_link">
       <inertial>
-        <origin xyz="0.211965218493119 0.0178758106324586 0.00251195422528849" rpy="0 0 0"/>
-        <mass value="0.80983551449458"/>
-        <inertia ixx="0.000895661134764477" ixy="-1.74285015573192E-07" ixz="1.55325395906594E-06" iyy="0.00203081725363" iyz="-7.18963040487278E-10" izz="0.00212477105992021"/>
+        <origin xyz="0.225299625739963 1.60107813145238E-05 -0.0720438220450934" rpy="0 0 0"/>
+        <mass value="1.34400405454488"/>
+        <inertia ixx="0.00147896138599604" ixy="1.09234424169219E-06" ixz="-3.74484328782169E-07" iyy="0.0027517586466101" iyz="-1.75900999614053E-08" izz="0.00279083369334524"/>
       </inertial>
       <visual>
@@ -281,7 +281,7 @@
     <link name="${prefix}leftjoint4_link">
       <inertial>
-        <origin xyz="0.0844096980098743 -0.0538627242829748 -2.30167658230584E-05" rpy="0 0 0"/>
-        <mass value="0.87429812902866"/>
-        <inertia ixx="0.00141845889439953" ixy="8.7764400516495E-05" ixz="2.05978166736258E-07" iyy="0.00123345158654823" iyz="-1.07921281417646E-06" izz="0.00149174666442669"/>
+        <origin xyz="0.0100204605383918 -0.00985679814963347 0.0840089075623952" rpy="0 0 0"/>
+        <mass value="0.983457322359293"/>
+        <inertia ixx="0.00146324457982104" ixy="-1.07921279553368E-06" ixz="2.05978166819893E-07" iyy="0.00136637778648993" iyz="-3.51454994521712E-07" izz="0.00151815899256312"/>
       </inertial>
       <visual>
@@ -302,7 +302,7 @@
     <link name="${prefix}leftjoint5_link">
       <inertial>
-        <origin xyz="0.0961218883209607 4.05763946975668E-06 -0.0115836008735541" rpy="0 0 0"/>
-        <mass value="0.798597769370932"/>
-        <inertia ixx="0.00254664839147289" ixy="-9.91166552698404E-09" ixz="1.01070951103748E-05" iyy="0.0012909021102841" iyz="3.11289977467224E-09" izz="0.00196072810117326"/>
+        <origin xyz="0.0101785346040691 9.30231893336853E-06 0.114866949892092" rpy="0 0 0"/>
+        <mass value="1.05113789872684"/>
+        <inertia ixx="0.00202470522047338" ixy="1.84484199834478E-08" ixz="-0.000306186752830273" iyy="0.00328579639703018" iyz="7.17708515637608E-10" izz="0.00340020564373822"/>
       </inertial>
       <visual>
@@ -317,4 +317,25 @@
         <geometry>
           <mesh filename="package://alfa_robot_description/meshes/alfa_robot/collision/leftjoint5.STL"/>
+        </geometry>
+      </collision>
+    </link>
+    <!-- leftjoint6 (new link for end effector extension) -->
+    <link name="${prefix}leftjoint6_link">
+      <inertial>
+        <origin xyz="0.0338349899428319 2.18158824338843E-14 1.47522838389591E-09" rpy="0 0 0"/>
+        <mass value="0.763196071605449"/>
+        <inertia ixx="0.00324062849151741" ixy="6.82020341217245E-19" ixz="-3.87057635370163E-16" iyy="0.0019198659327465" iyz="-1.80691312979497E-18" izz="0.00150433027221572"/>
+      </inertial>
+      <visual>
+        <origin xyz="0 0 0" rpy="0 0 0"/>
+        <geometry>
+          <mesh filename="package://alfa_robot_description/meshes/alfa_robot/visual/leftjoint6.STL"/>
+        </geometry>
+        <material name="blue"/>
+      </visual>
+      <collision>
+        <origin xyz="0 0 0" rpy="0 0 0"/>
+        <geometry>
+          <mesh filename="package://alfa_robot_description/meshes/alfa_robot/collision/leftjoint6.STL"/>
         </geometry>
       </collision>
@@ -323,8 +344,7 @@
     <link name="${prefix}camera_link">
       <inertial>
-        <origin xyz="-0.0128838261972163 0.00026531291498777 0.00027897095170859" rpy="0 0 0"/>
-        <mass value="0.0247923828845652"/>
-        <inertia ixx="3.5668701541101E-05" ixy="-1.36439346012497E-08" ixz="-2.61698308401705E-08"
-                 iyy="2.83830455101906E-06" iyz="2.73948631199571E-08" izz="3.34987859138971E-05"/>
+        <origin xyz="-0.0129500032830805 3.27763982552187E-08 8.59781135176263E-10" rpy="0 0 0"/>
+        <mass value="0.0884229444440941"/>
+        <inertia ixx="0.000108966100127413" ixy="4.24530017226163E-12" ixz="1.30809093461559E-12" iyy="1.08349581479197E-05" iyz="1.58450016026868E-10" izz="0.000108016955483713"/>
       </inertial>
       <visual>
@@ -345,8 +365,7 @@
     <link name="${prefix}lidar_link">
       <inertial>
-        <origin xyz="-0.00468733327842979 -6.25961285910526E-06 -0.016722032751983" rpy="0 0 0"/>
-        <mass value="0.141886849294983"/>
-        <inertia ixx="4.37633098241424E-05" ixy="-5.36171297405178E-09" ixz="7.01471703806087E-06"
-                 iyy="4.50759714359166E-05" iyz="9.27886666435768E-10" izz="6.68414722762209E-05"/>
+        <origin xyz="-0.000765897194240361 5.34294830600857E-16 -0.00285836724227106" rpy="0 0 0"/>
+        <mass value="0.296061195729235"/>
+        <inertia ixx="0.000229195879552691" ixy="-5.34979264059518E-18" ixz="-7.69967406090194E-06" iyy="0.000231259000999259" iyz="8.30310887470795E-18" izz="0.000202523426202246"/>
       </inertial>
       <visual>
@@ -385,9 +404,9 @@
     <!-- updown -->
     <joint name="${prefix}updown" type="prismatic">
-      <origin xyz="-0.23547 0 0.45934" rpy="0 0 0"/>
+      <origin xyz="-0.23547 0 0.57771" rpy="0 0 0"/>
       <parent link="${prefix}turn_link"/>
       <child link="${prefix}updown_link"/>
       <axis xyz="0 0 1"/>
-      <limit lower="0" upper="0.95" effort="1000" velocity="1"/>
+      <limit lower="0" upper="1" effort="1000" velocity="1"/>
     </joint>
     <!-- plate (new joint) -->
@@ -401,41 +420,41 @@
     <!-- leftarmbase -->
     <joint name="${prefix}rightarmbase" type="prismatic">
-      <origin xyz="-0.16145 -0.31517 0.146" rpy="0 0 0"/>
+      <origin xyz="-0.16145 -0.47517 0.146" rpy="0 0 0"/>
       <parent link="${prefix}updown_link"/>
       <child link="${prefix}rightarmbase_link"/>
-      <axis xyz="0 -1 0"/>
-      <limit lower="0" upper="0.12" effort="1000" velocity="1000"/>
+      <axis xyz="0 1 0"/>
+      <limit lower="0" upper="0.16" effort="1000" velocity="0.5"/>
     </joint>
     <!-- leftjoint1 -->
     <joint name="${prefix}rightjoint1" type="prismatic">
-      <origin xyz="0.11412 0.024997 0.07136" rpy="0 0 0"/>
+      <origin xyz="0.08729 0.024997 0.07136" rpy="0 0 0"/>
       <parent link="${prefix}rightarmbase_link"/>
       <child link="${prefix}rightjoint1_link"/>
       <axis xyz="1 0 0"/>
-      <limit lower="0" upper="0.4" effort="1000" velocity="1000"/>
+      <limit lower="0" upper="0.5" effort="1000" velocity="0.5"/>
     </joint>
     <!-- leftjoint2 -->
-    <joint name="${prefix}rightjoint2" type="revolute">
+    <joint name="${prefix}rightjoint2" type="continuous">
       <origin xyz="0.67445 -0.035997 0.04964" rpy="0 1.5708 0"/>
       <parent link="${prefix}rightjoint1_link"/>
       <child link="${prefix}rightjoint2_link"/>
       <axis xyz="0 0 1"/>
-      <limit lower="-2.35" upper="2.35" effort="1000" velocity="1000"/>
+      <limit lower="-3.14" upper="3.14" effort="0" velocity="0"/>
     </joint>
     <!-- leftjoint3 -->
-    <joint name="${prefix}rightjoint3" type="revolute">
+    <joint name="${prefix}rightjoint3" type="continuous">
       <origin xyz="0.19998 0.0021836 0.0834" rpy="0 0 0"/>
       <parent link="${prefix}rightjoint2_link"/>
       <child link="${prefix}rightjoint3_link"/>
       <axis xyz="0 0 1"/>
-      <limit lower="-2.35" upper="2.35" effort="1000" velocity="1000"/>
+      <limit lower="-3.14" upper="3.14" effort="0" velocity="0"/>
     </joint>
     <!-- leftjoint4 -->
-    <joint name="${prefix}rightjoint4" type="revolute">
+    <joint name="${prefix}rightjoint4" type="continuous">
       <origin xyz="-0.00022361 -0.054349 0.105" rpy="1.5708 -0.11346 -0.0041142"/>
       <parent link="${prefix}rightjoint3_link"/>
       <child link="${prefix}rightjoint4_link"/>
       <axis xyz="0 0 1"/>
-      <limit lower="0" upper="3.14" effort="1000" velocity="1000"/>
+      <limit lower="-3.14" upper="3.14" effort="0" velocity="0"/>
     </joint>
     <!-- left_ee_joint (virtual fixed joint for MoveIt2 end effector) -->
@@ -447,21 +466,21 @@
     <!-- rightarmbase -->
     <joint name="${prefix}leftarmbase" type="prismatic">
-      <origin xyz="-0.16145 0.4695 0.146" rpy="0 0 0"/>
+      <origin xyz="-0.16145 0.3282 0.146" rpy="0 0 0"/>
       <parent link="${prefix}updown_link"/>
       <child link="${prefix}leftarmbase_link"/>
       <axis xyz="0 1 0"/>
-      <limit lower="-0.16" upper="0" effort="1000" velocity="0.5"/>
+      <limit lower="0" upper="0.14" effort="1000" velocity="0.5"/>
     </joint>
     <!-- rightjoint1 -->
     <joint name="${prefix}leftjoint1" type="prismatic">
-      <origin xyz="0.094579 -0.021899 0.088" rpy="0 0 0"/>
+      <origin xyz="0.15658 -0.096099 0.086" rpy="0 0 0"/>
       <parent link="${prefix}leftarmbase_link"/>
       <child link="${prefix}leftjoint1_link"/>
       <axis xyz="1 0 0"/>
-      <limit lower="0" upper="0.45" effort="1000" velocity="0.5"/>
+      <limit lower="0" upper="0.42" effort="1000" velocity="0.5"/>
     </joint>
     <!-- rightjoint2 -->
     <joint name="${prefix}leftjoint2" type="continuous">
-      <origin xyz="0.74035 0.0209 0.033" rpy="0 1.5708 0"/>
+      <origin xyz="0.67335 0.10135 0.04" rpy="0 1.5708 0"/>
       <parent link="${prefix}leftjoint1_link"/>
       <child link="${prefix}leftjoint2_link"/>
@@ -471,5 +490,5 @@
     <!-- rightjoint3 -->
     <joint name="${prefix}leftjoint3" type="continuous">
-      <origin xyz="0 -0.035 0.11" rpy="1.5708 -1.5708 0"/>
+      <origin xyz="0.01 0.0058 0.098" rpy="1.5708 -1.5708 0"/>
       <parent link="${prefix}leftjoint2_link"/>
       <child link="${prefix}leftjoint3_link"/>
@@ -478,23 +497,31 @@
     </joint>
     <!-- rightjoint4 -->
-    <joint name="${prefix}leftjoint4" type="prismatic">
-      <origin xyz="0.376 0.026 0.0023" rpy="1.5708 0 0"/>
+    <joint name="${prefix}leftjoint4" type="continuous">
+      <origin xyz="0.3418 -0.01 -0.082" rpy="1.5708 0 1.5708"/>
       <parent link="${prefix}leftjoint3_link"/>
       <child link="${prefix}leftjoint4_link"/>
+      <axis xyz="0 0 1"/>
+      <limit lower="-3.14" upper="3.14" effort="0" velocity="0"/>
+    </joint>
+    <!-- leftjoint5 (new joint for 6DOF) -->
+    <joint name="${prefix}leftjoint5" type="continuous">
+      <origin xyz="0.01 -0.0022 0.098" rpy="1.5708 -1.5708 0"/>
+      <parent link="${prefix}leftjoint4_link"/>
+      <child link="${prefix}leftjoint5_link"/>
+      <axis xyz="0 0 1"/>
+      <limit lower="-3.14" upper="3.14" effort="0" velocity="0"/>
+    </joint>
+    <!-- leftjoint6 (new joint for end effector extension) -->
+    <joint name="${prefix}leftjoint6" type="prismatic">
+      <origin xyz="0.13 0 0.1435" rpy="1.5708 0 0"/>
+      <parent link="${prefix}leftjoint5_link"/>
+      <child link="${prefix}leftjoint6_link"/>
       <axis xyz="1 0 0"/>
       <limit lower="0" upper="0.15" effort="0" velocity="0"/>
     </joint>
-    <!-- leftjoint5 (new joint for 6DOF) -->
-    <joint name="${prefix}leftjoint5" type="continuous">
-      <origin xyz="0.092 0.0018 0" rpy="-1.5708 0 0"/>
-      <parent link="${prefix}leftjoint4_link"/>
-      <child link="${prefix}leftjoint5_link"/>
-      <axis xyz="0 0 1"/>
-      <limit lower="-3.14" upper="3.14" effort="0" velocity="0"/>
-    </joint>
-    <!-- right_ee_joint (virtual fixed joint for MoveIt2 end effector) -->
+    <!-- left_ee_joint (virtual fixed joint for MoveIt2 end effector) -->
     <joint name="${prefix}left_ee_joint" type="fixed">
       <origin xyz="0.05 0 0" rpy="0 0 0"/>
-      <parent link="${prefix}leftjoint5_link"/>
+      <parent link="${prefix}leftjoint6_link"/>
       <child link="${prefix}left_ee_link"/>
     </joint>
