Commit message: gazebo仿真实现，待调节控制器

File: src/alfa_robot_description/urdf/alfa_robot/alfa_robot_macro.xacro (robot description, xacro)
@@ -22,10 +22,10 @@
         <origin xyz="0 0 0" rpy="0 0 0"/>
         <geometry>
-          <mesh filename="package://alfa_robot_description/meshes/alfa_robot/visual/base.STL"/>
-        </geometry>
-      </collision>
-    </link>
-    <!-- turn -->
-    <link name="${prefix}turn">
+          <mesh filename="package://alfa_robot_description/meshes/alfa_robot/collision/base.STL"/>
+        </geometry>
+      </collision>
+    </link>
+    <!-- turn (link name differs from joint for GZ compatibility) -->
+    <link name="${prefix}turn_link">
       <inertial>
         <origin xyz="-5.4556E-05 0.094864 0.74374" rpy="0 0 0"/>
@@ -43,10 +43,10 @@
         <origin xyz="0 0 0" rpy="0 0 0"/>
         <geometry>
-          <mesh filename="package://alfa_robot_description/meshes/alfa_robot/visual/turn.STL"/>
-        </geometry>
-      </collision>
-    </link>
-    <!-- updown -->
-    <link name="${prefix}updown">
+          <mesh filename="package://alfa_robot_description/meshes/alfa_robot/collision/turn.STL"/>
+        </geometry>
+      </collision>
+    </link>
+    <!-- updown (link name differs from joint for GZ compatibility) -->
+    <link name="${prefix}updown_link">
       <inertial>
         <origin xyz="0.0201090104029969 0.0803972373261843 0.0984366062782738" rpy="0 0 0"/>
@@ -64,10 +64,10 @@
         <origin xyz="0 0 0" rpy="0 0 0"/>
         <geometry>
-          <mesh filename="package://alfa_robot_description/meshes/alfa_robot/visual/updown.STL"/>
-        </geometry>
-      </collision>
-    </link>
-    <!-- leftarmbase -->
-    <link name="${prefix}leftarmbase">
+          <mesh filename="package://alfa_robot_description/meshes/alfa_robot/collision/updown.STL"/>
+        </geometry>
+      </collision>
+    </link>
+    <!-- leftarmbase (link name differs from joint for GZ compatibility) -->
+    <link name="${prefix}leftarmbase_link">
       <inertial>
         <origin xyz="0.29757 -0.16382 0.17861" rpy="0 0 0"/>
@@ -85,10 +85,10 @@
         <origin xyz="0 0 0" rpy="0 0 0"/>
         <geometry>
-          <mesh filename="package://alfa_robot_description/meshes/alfa_robot/visual/leftarmbase.STL"/>
-        </geometry>
-      </collision>
-    </link>
-    <!-- leftjoint1 -->
-    <link name="${prefix}leftjoint1">
+          <mesh filename="package://alfa_robot_description/meshes/alfa_robot/collision/leftarmbase.STL"/>
+        </geometry>
+      </collision>
+    </link>
+    <!-- leftjoint1 (link name differs from joint for GZ compatibility) -->
+    <link name="${prefix}leftjoint1_link">
       <inertial>
         <origin xyz="0.00502820177318375 0.0342161631641283 0.281401807518592" rpy="0 0 0"/>
@@ -106,10 +106,10 @@
         <origin xyz="0 0 0" rpy="0 0 0"/>
         <geometry>
-          <mesh filename="package://alfa_robot_description/meshes/alfa_robot/visual/leftjoint1.STL"/>
-        </geometry>
-      </collision>
-    </link>
-    <!-- leftjoint2 -->
-    <link name="${prefix}leftjoint2">
+          <mesh filename="package://alfa_robot_description/meshes/alfa_robot/collision/leftjoint1.STL"/>
+        </geometry>
+      </collision>
+    </link>
+    <!-- leftjoint2 (link name differs from joint for GZ compatibility) -->
+    <link name="${prefix}leftjoint2_link">
       <inertial>
         <origin xyz="-0.149017202271686 -0.000289955936075892 0.0195313938678338" rpy="0 0 0"/>
@@ -127,10 +127,10 @@
         <origin xyz="0 0 0" rpy="0 0 0"/>
         <geometry>
-          <mesh filename="package://alfa_robot_description/meshes/alfa_robot/visual/leftjoint2.STL"/>
-        </geometry>
-      </collision>
-    </link>
-    <!-- leftjoint3 -->
-    <link name="${prefix}leftjoint3">
+          <mesh filename="package://alfa_robot_description/meshes/alfa_robot/collision/leftjoint2.STL"/>
+        </geometry>
+      </collision>
+    </link>
+    <!-- leftjoint3 (link name differs from joint for GZ compatibility) -->
+    <link name="${prefix}leftjoint3_link">
       <inertial>
         <origin xyz="4.32362620763627E-05 0.00090464696325504 0.0847683944898301" rpy="0 0 0"/>
@@ -148,10 +148,10 @@
         <origin xyz="0 0 0" rpy="0 0 0"/>
         <geometry>
-          <mesh filename="package://alfa_robot_description/meshes/alfa_robot/visual/leftjoint3.STL"/>
-        </geometry>
-      </collision>
-    </link>
-    <!-- leftjoint4 -->
-    <link name="${prefix}leftjoint4">
+          <mesh filename="package://alfa_robot_description/meshes/alfa_robot/collision/leftjoint3.STL"/>
+        </geometry>
+      </collision>
+    </link>
+    <!-- leftjoint4 (link name differs from joint for GZ compatibility) -->
+    <link name="${prefix}leftjoint4_link">
       <inertial>
         <origin xyz="-0.192813505520282 -0.00671906082576801 -0.0056742418931493" rpy="0 0 0"/>
@@ -169,10 +169,10 @@
         <origin xyz="0 0 0" rpy="0 0 0"/>
         <geometry>
-          <mesh filename="package://alfa_robot_description/meshes/alfa_robot/visual/leftjoint4.STL"/>
-        </geometry>
-      </collision>
-    </link>
-    <!-- rightarmbase -->
-    <link name="${prefix}rightarmbase">
+          <mesh filename="package://alfa_robot_description/meshes/alfa_robot/collision/leftjoint4.STL"/>
+        </geometry>
+      </collision>
+    </link>
+    <!-- rightarmbase (link name differs from joint for GZ compatibility) -->
+    <link name="${prefix}rightarmbase_link">
       <inertial>
         <origin xyz="0.0568652250818897 0.0787348857644462 0.00280311476846101" rpy="0 0 0"/>
@@ -190,10 +190,10 @@
         <origin xyz="0 0 0" rpy="0 0 0"/>
         <geometry>
-          <mesh filename="package://alfa_robot_description/meshes/alfa_robot/visual/rightarmbase.STL"/>
-        </geometry>
-      </collision>
-    </link>
-    <!-- rightjoint1 -->
-    <link name="${prefix}rightjoint1">
+          <mesh filename="package://alfa_robot_description/meshes/alfa_robot/collision/rightarmbase.STL"/>
+        </geometry>
+      </collision>
+    </link>
+    <!-- rightjoint1 (link name differs from joint for GZ compatibility) -->
+    <link name="${prefix}rightjoint1_link">
       <inertial>
         <origin xyz="0.0125188483480216 -0.0276314408365126 0.290315233804106" rpy="0 0 0"/>
@@ -211,10 +211,10 @@
         <origin xyz="0 0 0" rpy="0 0 0"/>
         <geometry>
-          <mesh filename="package://alfa_robot_description/meshes/alfa_robot/visual/rightjoint1.STL"/>
-        </geometry>
-      </collision>
-    </link>
-    <!-- rightjoint2 -->
-    <link name="${prefix}rightjoint2">
+          <mesh filename="package://alfa_robot_description/meshes/alfa_robot/collision/rightjoint1.STL"/>
+        </geometry>
+      </collision>
+    </link>
+    <!-- rightjoint2 (link name differs from joint for GZ compatibility) -->
+    <link name="${prefix}rightjoint2_link">
       <inertial>
         <origin xyz="-0.1474146108181 0.00338572158786365 0.0189953911214911" rpy="0 0 0"/>
@@ -232,10 +232,10 @@
         <origin xyz="0 0 0" rpy="0 0 0"/>
         <geometry>
-          <mesh filename="package://alfa_robot_description/meshes/alfa_robot/visual/rightjoint2.STL"/>
-        </geometry>
-      </collision>
-    </link>
-    <!-- rightjoint3 -->
-    <link name="${prefix}rightjoint3">
+          <mesh filename="package://alfa_robot_description/meshes/alfa_robot/collision/rightjoint2.STL"/>
+        </geometry>
+      </collision>
+    </link>
+    <!-- rightjoint3 (link name differs from joint for GZ compatibility) -->
+    <link name="${prefix}rightjoint3_link">
       <inertial>
         <origin xyz="0.000636075551307513 -0.000732173079496579 0.0855214235064663" rpy="0 0 0"/>
@@ -253,10 +253,10 @@
         <origin xyz="0 0 0" rpy="0 0 0"/>
         <geometry>
-          <mesh filename="package://alfa_robot_description/meshes/alfa_robot/visual/rightjoint3.STL"/>
-        </geometry>
-      </collision>
-    </link>
-    <!-- rightjoint4 -->
-    <link name="${prefix}rightjoint4">
+          <mesh filename="package://alfa_robot_description/meshes/alfa_robot/collision/rightjoint3.STL"/>
+        </geometry>
+      </collision>
+    </link>
+    <!-- rightjoint4 (link name differs from joint for GZ compatibility) -->
+    <link name="${prefix}rightjoint4_link">
       <inertial>
         <origin xyz="0.19373426132831 -0.00481885161982026 -0.0070966670102961" rpy="0 0 0"/>
@@ -274,5 +274,5 @@
         <origin xyz="0 0 0" rpy="0 0 0"/>
         <geometry>
-          <mesh filename="package://alfa_robot_description/meshes/alfa_robot/visual/rightjoint4.STL"/>
+          <mesh filename="package://alfa_robot_description/meshes/alfa_robot/collision/rightjoint4.STL"/>
         </geometry>
       </collision>
@@ -299,6 +299,6 @@
       </collision>
     </link>
-    <!-- left back -->
-    <link name="${prefix}left back">
+    <!-- left back (link name differs from joint for GZ compatibility) -->
+    <link name="${prefix}left back_link">
       <inertial>
         <origin xyz="0 0 0" rpy="0 0 0"/>
@@ -316,10 +316,10 @@
         <origin xyz="0 0 0" rpy="0 0 0"/>
         <geometry>
-          <mesh filename="package://alfa_robot_description/meshes/alfa_robot/visual/leftback.STL"/>
-        </geometry>
-      </collision>
-    </link>
-    <!-- left forward -->
-    <link name="${prefix}left forward">
+          <mesh filename="package://alfa_robot_description/meshes/alfa_robot/collision/wheel.STL"/>
+        </geometry>
+      </collision>
+    </link>
+    <!-- left forward (link name differs from joint for GZ compatibility) -->
+    <link name="${prefix}left forward_link">
       <inertial>
         <origin xyz="0 0 0" rpy="0 0 0"/>
@@ -337,10 +337,10 @@
         <origin xyz="0 0 0" rpy="0 0 0"/>
         <geometry>
-          <mesh filename="package://alfa_robot_description/meshes/alfa_robot/visual/leftforward.STL"/>
-        </geometry>
-      </collision>
-    </link>
-    <!-- right back -->
-    <link name="${prefix}right back">
+          <mesh filename="package://alfa_robot_description/meshes/alfa_robot/collision/wheel.STL"/>
+        </geometry>
+      </collision>
+    </link>
+    <!-- right back (link name differs from joint for GZ compatibility) -->
+    <link name="${prefix}right back_link">
       <inertial>
         <origin xyz="0 0 0" rpy="0 0 0"/>
@@ -358,10 +358,10 @@
         <origin xyz="0 0 0" rpy="0 0 0"/>
         <geometry>
-          <mesh filename="package://alfa_robot_description/meshes/alfa_robot/visual/rightback.STL"/>
-        </geometry>
-      </collision>
-    </link>
-    <!-- right forward -->
-    <link name="${prefix}right forward">
+          <mesh filename="package://alfa_robot_description/meshes/alfa_robot/collision/wheel.STL"/>
+        </geometry>
+      </collision>
+    </link>
+    <!-- right forward (link name differs from joint for GZ compatibility) -->
+    <link name="${prefix}right forward_link">
       <inertial>
         <origin xyz="0 0 0" rpy="0 0 0"/>
@@ -379,5 +379,5 @@
         <origin xyz="0 0 0" rpy="0 0 0"/>
         <geometry>
-          <mesh filename="package://alfa_robot_description/meshes/alfa_robot/visual/rightforward.STL"/>
+          <mesh filename="package://alfa_robot_description/meshes/alfa_robot/collision/wheel.STL"/>
         </geometry>
       </collision>
@@ -395,5 +395,5 @@
       <origin xyz="0 -0.020495 0.089" rpy="0 0 0"/>
       <parent link="${prefix}base_link"/>
-      <child link="${prefix}turn"/>
+      <child link="${prefix}turn_link"/>
       <axis xyz="0 0 -1"/>
     </joint>
@@ -401,6 +401,6 @@
     <joint name="${prefix}updown" type="prismatic">
       <origin xyz="0.00014192 0.30273 0.47937" rpy="0 0 0"/>
-      <parent link="${prefix}turn"/>
-      <child link="${prefix}updown"/>
+      <parent link="${prefix}turn_link"/>
+      <child link="${prefix}updown_link"/>
       <axis xyz="0 0 1"/>
       <limit lower="-0.15" upper="1" effort="0" velocity="0"/>
@@ -409,6 +409,6 @@
     <joint name="${prefix}leftarmbase" type="prismatic">
       <origin xyz="-0.34911 0.11493 0.16" rpy="0.00046884 1.5708 0"/>
-      <parent link="${prefix}updown"/>
-      <child link="${prefix}leftarmbase"/>
+      <parent link="${prefix}updown_link"/>
+      <child link="${prefix}leftarmbase_link"/>
       <axis xyz="0 0 -1"/>
       <limit lower="-0.3" upper="0.3" effort="0" velocity="0"/>
@@ -417,6 +417,6 @@
     <joint name="${prefix}leftjoint1" type="prismatic">
       <origin xyz="-0.072146 -0.11751 0.044163" rpy="-1.5708 0 3.1416"/>
-      <parent link="${prefix}leftarmbase"/>
-      <child link="${prefix}leftjoint1"/>
+      <parent link="${prefix}leftarmbase_link"/>
+      <child link="${prefix}leftjoint1_link"/>
       <axis xyz="0 0 1"/>
       <limit lower="0" upper="0.5" effort="0" velocity="0"/>
@@ -425,6 +425,6 @@
     <joint name="${prefix}leftjoint2" type="continuous">
       <origin xyz="0.048854 0.065162 0.51445" rpy="0 0 0"/>
-      <parent link="${prefix}leftjoint1"/>
-      <child link="${prefix}leftjoint2"/>
+      <parent link="${prefix}leftjoint1_link"/>
+      <child link="${prefix}leftjoint2_link"/>
       <axis xyz="0 0 -1"/>
     </joint>
@@ -432,6 +432,6 @@
     <joint name="${prefix}leftjoint3" type="continuous">
       <origin xyz="-0.2 -0.00036724 0.0734" rpy="0 0 0"/>
-      <parent link="${prefix}leftjoint2"/>
-      <child link="${prefix}leftjoint3"/>
+      <parent link="${prefix}leftjoint2_link"/>
+      <child link="${prefix}leftjoint3_link"/>
       <axis xyz="0 0 -1"/>
     </joint>
@@ -439,6 +439,6 @@
     <joint name="${prefix}leftjoint4" type="continuous">
       <origin xyz="0.00058164 0.044646 0.115" rpy="-1.5708 0 -0.013027"/>
-      <parent link="${prefix}leftjoint3"/>
-      <child link="${prefix}leftjoint4"/>
+      <parent link="${prefix}leftjoint3_link"/>
+      <child link="${prefix}leftjoint4_link"/>
       <axis xyz="0 0 -1"/>
     </joint>
@@ -446,6 +446,6 @@
     <joint name="${prefix}rightarmbase" type="prismatic">
       <origin xyz="0.34777 0.1146 0.16" rpy="-0.00046884 -1.5708 0"/>
-      <parent link="${prefix}updown"/>
-      <child link="${prefix}rightarmbase"/>
+      <parent link="${prefix}updown_link"/>
+      <child link="${prefix}rightarmbase_link"/>
       <axis xyz="0 0 -1"/>
       <limit lower="-0.3" upper="0.3" effort="0" velocity="0"/>
@@ -454,6 +454,6 @@
     <joint name="${prefix}rightjoint1" type="prismatic">
       <origin xyz="0.072146 -0.11412 0.044162" rpy="1.5708 0 0"/>
-      <parent link="${prefix}rightarmbase"/>
-      <child link="${prefix}rightjoint1"/>
+      <parent link="${prefix}rightarmbase_link"/>
+      <child link="${prefix}rightjoint1_link"/>
       <axis xyz="0 0 1"/>
       <limit lower="0" upper="0.5" effort="0" velocity="0"/>
@@ -462,6 +462,6 @@
     <joint name="${prefix}rightjoint2" type="continuous">
       <origin xyz="0.048854 -0.065162 0.51445" rpy="0 0 0"/>
-      <parent link="${prefix}rightjoint1"/>
-      <child link="${prefix}rightjoint2"/>
+      <parent link="${prefix}rightjoint1_link"/>
+      <child link="${prefix}rightjoint2_link"/>
       <axis xyz="0 0 -1"/>
     </joint>
@@ -469,6 +469,6 @@
     <joint name="${prefix}rightjoint3" type="continuous">
       <origin xyz="-0.19996 0.0038023 0.0734" rpy="0 0 0"/>
-      <parent link="${prefix}rightjoint2"/>
-      <child link="${prefix}rightjoint3"/>
+      <parent link="${prefix}rightjoint2_link"/>
+      <child link="${prefix}rightjoint3_link"/>
       <axis xyz="0 0 1"/>
     </joint>
@@ -476,6 +476,6 @@
     <joint name="${prefix}rightjoint4" type="continuous">
       <origin xyz="-0.0003624 -0.044649 0.115" rpy="-1.5708 0 3.1335"/>
-      <parent link="${prefix}rightjoint3"/>
-      <child link="${prefix}rightjoint4"/>
+      <parent link="${prefix}rightjoint3_link"/>
+      <child link="${prefix}rightjoint4_link"/>
       <axis xyz="0 0 1"/>
     </joint>
@@ -490,5 +490,5 @@
       <origin xyz="0.463 -0.439 0.086" rpy="-1.5708 0 -1.5708"/>
       <parent link="${prefix}base_chassis_link"/>
-      <child link="${prefix}left back"/>
+      <child link="${prefix}left back_link"/>
       <axis xyz="0 0 -1"/>
       <limit effort="0" velocity="10"/>
@@ -498,5 +498,5 @@
       <origin xyz="0.463 0.439 0.086" rpy="-1.5708 0 -1.5708"/>
       <parent link="${prefix}base_chassis_link"/>
-      <child link="${prefix}left forward"/>
+      <child link="${prefix}left forward_link"/>
       <axis xyz="0 0 -1"/>
       <limit effort="0" velocity="10"/>
@@ -506,5 +506,5 @@
       <origin xyz="-0.463 -0.439 0.086" rpy="1.5708 0 -1.5708"/>
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
Commit message: 修复PDO、分了两个缓存区、修复心跳包存在延迟读取导致关闭后重启

File: src/alfa_robot_description/urdf/alfa_robot/alfa_robot_macro.xacro (robot description, xacro)
@@ -411,5 +411,5 @@
       <parent link="${prefix}updown_link"/>
       <child link="${prefix}leftarmbase_link"/>
-      <axis xyz="0 0 -1"/>
+      <axis xyz="0 0 1"/>
       <limit lower="-0.3" upper="0.3" effort="0" velocity="0"/>
     </joint>
@@ -420,5 +420,5 @@
       <child link="${prefix}leftjoint1_link"/>
       <axis xyz="0 0 1"/>
-      <limit lower="0" upper="0.5" effort="0" velocity="0"/>
+      <limit lower="-0.5" upper="0.5" effort="0" velocity="0"/>
     </joint>
     <!-- leftjoint2 -->

Commit message: 这个是试用的联调提交，因为urdf与实机不符因此只能以此妥协的xacro方案，机械结构与实机一致，但目前的urdf在组装上并不是合法的

File: src/alfa_robot_description/urdf/alfa_robot/alfa_robot_macro.xacro (robot description, xacro)
@@ -471,8 +471,8 @@
     <!-- rightjoint3 -->
     <joint name="${prefix}leftjoint3" type="continuous">
-      <origin xyz="0 -0.035 0.11" rpy="1.5708 -1.5708 0"/>
+      <origin xyz="0 -0.035 0.11" rpy="0 -1.5708 0"/>
       <parent link="${prefix}leftjoint2_link"/>
       <child link="${prefix}leftjoint3_link"/>
-      <axis xyz="0 0 1"/>
+      <axis xyz="0 1 0"/>
       <limit lower="-3.14" upper="3.14" effort="0" velocity="0"/>
     </joint>

Commit message: 将初始角度与实机同步

File: src/alfa_robot_description/urdf/alfa_robot/alfa_robot_macro.xacro (robot description, xacro)
@@ -471,5 +471,5 @@
     <!-- rightjoint3 -->
     <joint name="${prefix}leftjoint3" type="continuous">
-      <origin xyz="0 -0.035 0.11" rpy="0 -1.5708 0"/>
+      <origin xyz="0 -0.035 0.11" rpy="0 0 0"/>
       <parent link="${prefix}leftjoint2_link"/>
       <child link="${prefix}leftjoint3_link"/>
