Commit message: feat: 左臂升级为6自由度，新增leftjoint5关节
URDF/Xacro更改:
- 新增 leftjoint5 关节和 link，类型为 continuous (旋转)
- leftjoint4 从旋转关节改为直线关节 (prismatic)
- 更新左臂各关节的 DH 参数、惯性参数和碰撞网格
- 更新 leftarmbase/leftjoint1-4 的运动范围限制
- 末端执行器从 leftjoint4_link 移至 leftjoint5_link

MoveIt配置更改:
- left_arm 组新增 leftjoint5 关节
- 更新控制器配置包含 leftjoint5
- 更新碰撞检测配置

硬件接口更改:
- 新增 PlaceholderJoint 类用于临时占用未知协议的关节槽位
- 新增 safe_position_leftjoint5 参数

Co-Authored-By: Claude Opus 4.7 <noreply@anthropic.com>

File: src/alfa_robot_description/urdf/alfa_robot/alfa_robot_macro.xacro (robot description, xacro)
@@ -197,7 +197,7 @@
     <link name="${prefix}leftarmbase_link">
       <inertial>
-        <origin xyz="-0.0497615746360321 -0.0246057688749117 0.0430343814698384" rpy="0 0 0"/>
-        <mass value="13.1823257277416"/>
-        <inertia ixx="0.104088812848048" ixy="0.013834486847352" ixz="0.0505635371163732" iyy="0.863382985023394" iyz="-0.00307573195386396" izz="0.828453194049388"/>
+        <origin xyz="0.00858986048627108 -0.0287669594343616 0.0499555606572781" rpy="0 0 0"/>
+        <mass value="7.06520786855791"/>
+        <inertia ixx="0.0164730270054741" ixy="9.84172584812845E-06" ixz="0.000387662666781538" iyy="0.0926777572077124" iyz="0.000120939157760669" izz="0.0913979516362821"/>
       </inertial>
       <visual>
@@ -218,7 +218,7 @@
     <link name="${prefix}leftjoint1_link">
       <inertial>
-        <origin xyz="0.57341524650029 4.58601160402972E-05 0.0242655456596959" rpy="0 0 0"/>
-        <mass value="2.70490666316309"/>
-        <inertia ixx="0.0126378005178209" ixy="-0.00720533280334168" ixz="-0.001172487709181" iyy="0.0486867960951763" iyz="-2.68816757577675E-05" izz="0.051454778841387"/>
+        <origin xyz="0.374415906775149 -0.00904923744463459 -0.0148960568987655" rpy="0 0 0"/>
+        <mass value="2.37583354079001"/>
+        <inertia ixx="0.00207304785493464" ixy="1.02796852110949E-06" ixz="1.72939416918191E-06" iyy="0.0375730763919683" iyz="9.61510248922564E-06" izz="0.0381102083862888"/>
       </inertial>
       <visual>
@@ -239,7 +239,7 @@
     <link name="${prefix}leftjoint2_link">
       <inertial>
-        <origin xyz="0.0982222389567129 2.77555756156289E-16 0.0280872172763753" rpy="0 0 0"/>
-        <mass value="3.80063815279185"/>
-        <inertia ixx="0.00855142309151201" ixy="-6.9931040125315E-18" ixz="0.000737698249610721" iyy="0.03409027056488" iyz="6.71273610699033E-19" izz="0.038449314153095"/>
+        <origin xyz="-3.31662261210397E-06 -0.0765366527672894 0.0979391100942644" rpy="0 0 0"/>
+        <mass value="0.86529067490259"/>
+        <inertia ixx="0.00132661283538382" ixy="-1.59054446085595E-07" ixz="3.24265168911163E-07" iyy="0.00116106049969607" iyz="-1.07921267015626E-06" izz="0.00137430337463552"/>
       </inertial>
       <visual>
@@ -260,7 +260,7 @@
     <link name="${prefix}leftjoint3_link">
       <inertial>
-        <origin xyz="0.00424368697534261 0.000259106738649706 0.0734709611355132" rpy="0 0 0"/>
-        <mass value="2.16310625460758"/>
-        <inertia ixx="0.00755389789683751" ixy="-6.42921999609667E-07" ixz="-0.000140310452236765" iyy="0.00986541284670613" iyz="-1.11309098584596E-05" izz="0.0051328070950562"/>
+        <origin xyz="0.211965218493119 0.0178758106324586 0.00251195422528849" rpy="0 0 0"/>
+        <mass value="0.80983551449458"/>
+        <inertia ixx="0.000895661134764477" ixy="-1.74285015573192E-07" ixz="1.55325395906594E-06" iyy="0.00203081725363" iyz="-7.18963040487278E-10" izz="0.00212477105992021"/>
       </inertial>
       <visual>
@@ -281,7 +281,7 @@
     <link name="${prefix}leftjoint4_link">
       <inertial>
-        <origin xyz="0.179805345971669 0.00027459738144453 0.0111248225390411" rpy="0 0 0"/>
-        <mass value="9.59771353822043"/>
-        <inertia ixx="0.0623468092864488" ixy="-0.000903417557492398" ixz="-0.0234301373942001" iyy="0.130723241701585" iyz="-0.000423930246625516" izz="0.115651820367604"/>
+        <origin xyz="0.0844096980098743 -0.0538627242829748 -2.30167658230584E-05" rpy="0 0 0"/>
+        <mass value="0.87429812902866"/>
+        <inertia ixx="0.00141845889439953" ixy="8.7764400516495E-05" ixz="2.05978166736258E-07" iyy="0.00123345158654823" iyz="-1.07921281417646E-06" izz="0.00149174666442669"/>
       </inertial>
       <visual>
@@ -296,4 +296,25 @@
         <geometry>
           <mesh filename="package://alfa_robot_description/meshes/alfa_robot/collision/leftjoint4.STL"/>
+        </geometry>
+      </collision>
+    </link>
+    <!-- leftjoint5 (new link for 6DOF) -->
+    <link name="${prefix}leftjoint5_link">
+      <inertial>
+        <origin xyz="0.0961218883209607 4.05763946975668E-06 -0.0115836008735541" rpy="0 0 0"/>
+        <mass value="0.798597769370932"/>
+        <inertia ixx="0.00254664839147289" ixy="-9.91166552698404E-09" ixz="1.01070951103748E-05" iyy="0.0012909021102841" iyz="3.11289977467224E-09" izz="0.00196072810117326"/>
+      </inertial>
+      <visual>
+        <origin xyz="0 0 0" rpy="0 0 0"/>
+        <geometry>
+          <mesh filename="package://alfa_robot_description/meshes/alfa_robot/visual/leftjoint5.STL"/>
+        </geometry>
+        <material name="white"/>
+      </visual>
+      <collision>
+        <origin xyz="0 0 0" rpy="0 0 0"/>
+        <geometry>
+          <mesh filename="package://alfa_robot_description/meshes/alfa_robot/collision/leftjoint5.STL"/>
         </geometry>
       </collision>
@@ -426,46 +447,54 @@
     <!-- rightarmbase -->
     <joint name="${prefix}leftarmbase" type="prismatic">
-      <origin xyz="-0.16145 0.32 0.146" rpy="0 0 0"/>
+      <origin xyz="-0.16145 0.4695 0.146" rpy="0 0 0"/>
       <parent link="${prefix}updown_link"/>
       <child link="${prefix}leftarmbase_link"/>
       <axis xyz="0 1 0"/>
-      <limit lower="0" upper="0.12" effort="1000" velocity="1000"/>
+      <limit lower="-0.16" upper="0" effort="1000" velocity="0.5"/>
     </joint>
     <!-- rightjoint1 -->
     <joint name="${prefix}leftjoint1" type="prismatic">
-      <origin xyz="0.11412 -0.036996 0.07136" rpy="0 0 0"/>
+      <origin xyz="0.094579 -0.021899 0.088" rpy="0 0 0"/>
       <parent link="${prefix}leftarmbase_link"/>
       <child link="${prefix}leftjoint1_link"/>
       <axis xyz="1 0 0"/>
-      <limit lower="0" upper="0.4" effort="1000" velocity="1000"/>
+      <limit lower="0" upper="0.45" effort="1000" velocity="0.5"/>
     </joint>
     <!-- rightjoint2 -->
     <joint name="${prefix}leftjoint2" type="continuous">
-      <origin xyz="0.67445 0.035997 0.04964" rpy="-0.65703 1.5397 -0.65679"/>
+      <origin xyz="0.74035 0.0209 0.033" rpy="0 1.5708 0"/>
       <parent link="${prefix}leftjoint1_link"/>
       <child link="${prefix}leftjoint2_link"/>
       <axis xyz="0 0 1"/>
-      <limit lower="-2.35" upper="2.35" effort="1000" velocity="1000"/>
+      <limit lower="-3.14" upper="3.14" effort="0" velocity="0"/>
     </joint>
     <!-- rightjoint3 -->
     <joint name="${prefix}leftjoint3" type="continuous">
-      <origin xyz="0.20199 0.00030029 0.078444" rpy="0.00026875 -0.033043 0.010884"/>
+      <origin xyz="0 -0.035 0.11" rpy="1.5708 -1.5708 0"/>
       <parent link="${prefix}leftjoint2_link"/>
       <child link="${prefix}leftjoint3_link"/>
       <axis xyz="0 0 1"/>
-      <limit lower="-2.35" upper="2.35" effort="1000" velocity="1000"/>
+      <limit lower="-3.14" upper="3.14" effort="0" velocity="0"/>
     </joint>
     <!-- rightjoint4 -->
-    <joint name="${prefix}leftjoint4" type="revolute">
-      <origin xyz="0.0060547 0.05435 0.10483" rpy="1.5708 0 0"/>
+    <joint name="${prefix}leftjoint4" type="prismatic">
+      <origin xyz="0.376 0.026 0.0023" rpy="1.5708 0 0"/>
       <parent link="${prefix}leftjoint3_link"/>
       <child link="${prefix}leftjoint4_link"/>
-      <axis xyz="0 0 1"/>
-      <limit lower="0" upper="3.14" effort="1000" velocity="1000"/>
+      <axis xyz="1 0 0"/>
+      <limit lower="0" upper="0.22" effort="0" velocity="0"/>
+    </joint>
+    <!-- leftjoint5 (new joint for 6DOF) -->
+    <joint name="${prefix}leftjoint5" type="continuous">
+      <origin xyz="0.092 0.0018 0" rpy="-1.5708 0 0"/>
+      <parent link="${prefix}leftjoint4_link"/>
+      <child link="${prefix}leftjoint5_link"/>
+      <axis xyz="0 0 1"/>
+      <limit lower="-3.14" upper="3.14" effort="0" velocity="0"/>
     </joint>
     <!-- right_ee_joint (virtual fixed joint for MoveIt2 end effector) -->
     <joint name="${prefix}left_ee_joint" type="fixed">
-      <origin xyz="0.275 -0.0308 -0.02825" rpy="0 0 0"/>
-      <parent link="${prefix}leftjoint4_link"/>
+      <origin xyz="0.05 0 0" rpy="0 0 0"/>
+      <parent link="${prefix}leftjoint5_link"/>
       <child link="${prefix}left_ee_link"/>
     </joint>

Commit message: fix: 修正电缸参数配置
- URDF: leftjoint4 电缸行程限制从 0.22m 改为 0.15m
- CylinderDriver: 编码器分辨率从 200000 改为 2000000 脉冲/米 (10000脉冲/5mm)
- 硬件配置: 更新 zero_offset 为 -24995000

Co-Authored-By: Claude Opus 4.7 <noreply@anthropic.com>

File: src/alfa_robot_description/urdf/alfa_robot/alfa_robot_macro.xacro (robot description, xacro)
@@ -483,5 +483,5 @@
       <child link="${prefix}leftjoint4_link"/>
       <axis xyz="1 0 0"/>
-      <limit lower="0" upper="0.22" effort="0" velocity="0"/>
+      <limit lower="0" upper="0.15" effort="0" velocity="0"/>
     </joint>
     <!-- leftjoint5 (new joint for 6DOF) -->

Commit message: fix: 修正 leftjoint3/leftjoint5 关节坐标系方向
- leftjoint3: rpy 从 1.5708 改为 -1.5708
- leftjoint5: rpy 从 1.5708 改为 -1.5708

Co-Authored-By: Claude Opus 4.7 <noreply@anthropic.com>

File: src/alfa_robot_description/urdf/alfa_robot/alfa_robot_macro.xacro (robot description, xacro)
@@ -490,5 +490,5 @@
     <!-- rightjoint3 -->
     <joint name="${prefix}leftjoint3" type="continuous">
-      <origin xyz="0.01 0.0058 0.098" rpy="1.5708 -1.5708 0"/>
+      <origin xyz="0.01 0.0058 0.098" rpy="-1.5708 -1.5708 0"/>
       <parent link="${prefix}leftjoint2_link"/>
       <child link="${prefix}leftjoint3_link"/>
@@ -506,5 +506,5 @@
     <!-- leftjoint5 (new joint for 6DOF) -->
     <joint name="${prefix}leftjoint5" type="continuous">
-      <origin xyz="0.01 -0.0022 0.098" rpy="1.5708 -1.5708 0"/>
+      <origin xyz="0.01 -0.0022 0.098" rpy="-1.5708 -1.5708 0"/>
       <parent link="${prefix}leftjoint4_link"/>
       <child link="${prefix}leftjoint5_link"/>

Commit message: feat: v2.0 左臂关节方向修正 + MoveIt 控制启动文件
- 修正 leftjoint2/3/5 的关节方向（反转旋转方向）
- 调整 leftjoint3 限位范围：-0.3 ~ π rad
- 为 left_arm_controller 添加 leftjoint5 关节
- 新增 rviz_moveit_control.launch.py 启动文件
  - 组合硬件控制 + MoveIt 规划 + RViz 可视化
  - 支持通过 RViz MotionPlanning 插件控制实机
- 添加 use_rviz 启动参数，允许禁用 RViz

Co-Authored-By: Claude Opus 4.7 <noreply@anthropic.com>

File: src/alfa_robot_description/urdf/alfa_robot/alfa_robot_macro.xacro (robot description, xacro)
@@ -453,5 +453,5 @@
       <limit lower="-0.16" upper="0" effort="1000" velocity="0.5"/>
     </joint>
-    <!-- rightjoint1 -->
+<!-- rightjoint1 -->
     <joint name="${prefix}leftjoint1" type="prismatic">
       <origin xyz="0.094579 -0.021899 0.088" rpy="0 0 0"/>
@@ -462,20 +462,23 @@
     </joint>
     <!-- rightjoint2 -->
-    <joint name="${prefix}leftjoint2" type="continuous">
-      <origin xyz="0.74035 0.0209 0.033" rpy="0 1.5708 0"/>
+    <joint name="${prefix}leftjoint2" type="revolute">
+      <!-- 修改了 rpy，追加了绕 Z 轴 180 度的旋转 -->
+      <origin xyz="0.74035 0.0209 0.033" rpy="3.14159 -1.5708 0"/>
       <parent link="${prefix}leftjoint1_link"/>
       <child link="${prefix}leftjoint2_link"/>
       <axis xyz="0 0 1"/>
-      <limit lower="-3.14" upper="3.14" effort="0" velocity="0"/>
+      <limit lower="-3.14" upper="3.14" effort="100" velocity="1.0"/>
     </joint>
     <!-- rightjoint3 -->
-    <joint name="${prefix}leftjoint3" type="continuous">
-      <origin xyz="0 -0.035 0.11" rpy="0 0 0"/>
+    <joint name="${prefix}leftjoint3" type="revolute">
+      <!-- 修改了 rpy，追加了绕 Y 轴 180 度的旋转 -->
+      <origin xyz="0 -0.035 0.11" rpy="0 3.14159 0"/>
       <parent link="${prefix}leftjoint2_link"/>
       <child link="${prefix}leftjoint3_link"/>
       <axis xyz="0 1 0"/>
-      <limit lower="-3.14" upper="3.14" effort="0" velocity="0"/>
+      <limit lower="-0.3" upper="3.14" effort="100" velocity="1.0"/>
     </joint>
     <!-- rightjoint4 -->
+    <!-- 后续的关节 origin 完全不需要修改！因为它们的父坐标系已经旋转到位了 -->
     <joint name="${prefix}leftjoint4" type="prismatic">
       <origin xyz="0.376 0.026 0.0023" rpy="1.5708 0 0"/>
@@ -483,13 +486,13 @@
       <child link="${prefix}leftjoint4_link"/>
       <axis xyz="1 0 0"/>
-      <limit lower="0" upper="0.15" effort="0" velocity="0"/>
+      <limit lower="0" upper="0.15" effort="100" velocity="0.1"/>
     </joint>
     <!-- leftjoint5 (new joint for 6DOF) -->
-    <joint name="${prefix}leftjoint5" type="continuous">
+    <joint name="${prefix}leftjoint5" type="revolute">
       <origin xyz="0.092 0.0018 0" rpy="-1.5708 0 0"/>
       <parent link="${prefix}leftjoint4_link"/>
       <child link="${prefix}leftjoint5_link"/>
       <axis xyz="0 0 1"/>
-      <limit lower="-3.14" upper="3.14" effort="0" velocity="0"/>
+      <limit lower="-1.57" upper="1.57" effort="100" velocity="1.0"/>
     </joint>
     <!-- right_ee_joint (virtual fixed joint for MoveIt2 end effector) -->

Commit message: fix: 关节类型修正为 revolute + IK benchmark 关节限位修复
URDF:
- 右臂/左臂 joint2-5 从 continuous 改为 revolute，补充 effort/velocity
- 关节限位与 joint_limits.yaml 保持一致

joint_limits.yaml:
- left/right joint2-5 添加 has_position_limits + min/max_position

ik_benchmark:
- setToRandomPositions 后强制 clamp 到 URDF 限位范围
- 修复 continuous 关节未正确限位导致 FK 生成越界目标的问题

replay_ik_benchmark:
- 修正关节名称（移除 "turn"），匹配 dual_arm_with_base 组
- 新增 --count/--seed 参数支持随机抽样回放

Co-Authored-By: Claude Opus 4.7 <noreply@anthropic.com>

File: src/alfa_robot_description/urdf/alfa_robot/alfa_robot_macro.xacro (robot description, xacro)
@@ -477,34 +477,34 @@
     </joint>
     <!-- rightjoint2 -->
-    <joint name="${prefix}rightjoint2" type="continuous">
+    <joint name="${prefix}rightjoint2" type="revolute">
       <origin xyz="0.67335 -0.10135 0.04" rpy="0 1.5708 0"/>
       <parent link="${prefix}rightjoint1_link"/>
       <child link="${prefix}rightjoint2_link"/>
       <axis xyz="0 0 1"/>
-      <limit lower="-3.14" upper="3.14" effort="0" velocity="0"/>
+      <limit lower="-3.14159265" upper="3.14159265" effort="1000" velocity="0.5"/>
     </joint>
     <!-- rightjoint3 -->
-    <joint name="${prefix}rightjoint3" type="continuous">
+    <joint name="${prefix}rightjoint3" type="revolute">
       <origin xyz="0.01 -0.0058 0.098" rpy="1.5708 -1.5708 0"/>
       <parent link="${prefix}rightjoint2_link"/>
       <child link="${prefix}rightjoint3_link"/>
       <axis xyz="0 0 1"/>
-      <limit lower="-3.14" upper="3.14" effort="0" velocity="0"/>
+      <limit lower="-1.57079632" upper="1.57079632" effort="1000" velocity="0.5"/>
     </joint>
     <!-- rightjoint4 -->
-    <joint name="${prefix}rightjoint4" type="continuous">
+    <joint name="${prefix}rightjoint4" type="revolute">
       <origin xyz="0.3418 0.01 -0.082" rpy="-1.5708 0 -1.5708"/>
       <parent link="${prefix}rightjoint3_link"/>
       <child link="${prefix}rightjoint4_link"/>
       <axis xyz="0 0 1"/>
-      <limit lower="-3.14" upper="3.14" effort="0" velocity="0"/>
+      <limit lower="-3.14159265" upper="3.14159265" effort="1000" velocity="0.5"/>
     </joint>
     <!-- rightjoint5 (new joint for 6DOF, Y-axis mirror of leftjoint5) -->
-    <joint name="${prefix}rightjoint5" type="continuous">
+    <joint name="${prefix}rightjoint5" type="revolute">
       <origin xyz="0.01 0.0022 0.098" rpy="1.5708 -1.5708 0"/>
       <parent link="${prefix}rightjoint4_link"/>
       <child link="${prefix}rightjoint5_link"/>
       <axis xyz="0 0 1"/>
-      <limit lower="-3.14" upper="3.14" effort="0" velocity="0"/>
+      <limit lower="-1.57079632" upper="1.57079632" effort="1000" velocity="0.5"/>
     </joint>
     <!-- rightjoint6 (new joint for end effector extension, Y-axis mirror of leftjoint6) -->
@@ -539,34 +539,34 @@
     </joint>
     <!-- rightjoint2 -->
-    <joint name="${prefix}leftjoint2" type="continuous">
+    <joint name="${prefix}leftjoint2" type="revolute">
       <origin xyz="0.67335 0.10135 0.04" rpy="0 1.5708 0"/>
       <parent link="${prefix}leftjoint1_link"/>
       <child link="${prefix}leftjoint2_link"/>
       <axis xyz="0 0 1"/>
-      <limit lower="-3.14" upper="3.14" effort="0" velocity="0"/>
+      <limit lower="-3.14159265" upper="3.14159265" effort="1000" velocity="0.5"/>
     </joint>
     <!-- rightjoint3 -->
-    <joint name="${prefix}leftjoint3" type="continuous">
+    <joint name="${prefix}leftjoint3" type="revolute">
       <origin xyz="0.01 0.0058 0.098" rpy="-1.5708 -1.5708 0"/>
       <parent link="${prefix}leftjoint2_link"/>
       <child link="${prefix}leftjoint3_link"/>
       <axis xyz="0 0 1"/>
-      <limit lower="-3.14" upper="3.14" effort="0" velocity="0"/>
+      <limit lower="-1.57079632" upper="1.57079632" effort="1000" velocity="0.5"/>
     </joint>
     <!-- rightjoint4 -->
-    <joint name="${prefix}leftjoint4" type="continuous">
+    <joint name="${prefix}leftjoint4" type="revolute">
       <origin xyz="0.3418 -0.01 -0.082" rpy="1.5708 0 1.5708"/>
       <parent link="${prefix}leftjoint3_link"/>
       <child link="${prefix}leftjoint4_link"/>
       <axis xyz="0 0 1"/>
-      <limit lower="-3.14" upper="3.14" effort="0" velocity="0"/>
+      <limit lower="-3.14159265" upper="3.14159265" effort="1000" velocity="0.5"/>
     </joint>
     <!-- leftjoint5 (new joint for 6DOF) -->
-    <joint name="${prefix}leftjoint5" type="continuous">
+    <joint name="${prefix}leftjoint5" type="revolute">
       <origin xyz="0.01 -0.0022 0.098" rpy="-1.5708 -1.5708 0"/>
       <parent link="${prefix}leftjoint4_link"/>
       <child link="${prefix}leftjoint5_link"/>
       <axis xyz="0 0 1"/>
-      <limit lower="-3.14" upper="3.14" effort="0" velocity="0"/>
+      <limit lower="-1.57079632" upper="1.57079632" effort="1000" velocity="0.5"/>
     </joint>
     <!-- leftjoint6 (new joint for end effector extension) -->
