Commit message: feat: 控制器重构为独立三控制器架构并优化MoveIt配置
- 替换dual_arms_controller为left_arm、right_arm、plate独立控制器
- 更新ros2_controllers.yaml和moveit_controllers.yaml
- 修复homing_node.py和joint_states_to_controller_bridge.py脚本
- 更新bringup launch文件支持新控制器架构
- 删除备份文件和临时说明文档

File: src/alfa_robot_moveit_config/config/alfa_robot.ros2_control.xacro (robot description, xacro)
@@ -8,4 +8,46 @@
                 <plugin>mock_components/GenericSystem</plugin>
             </hardware>
+            <joint name="turn">
+                <command_interface name="position"/>
+                <state_interface name="position">
+                  <param name="initial_value">${initial_positions['turn']}</param>
+                </state_interface>
+            </joint>
+            <joint name="updown">
+                <command_interface name="position"/>
+                <state_interface name="position">
+                  <param name="initial_value">${initial_positions['updown']}</param>
+                </state_interface>
+            </joint>
+            <joint name="leftarmbase">
+                <command_interface name="position"/>
+                <state_interface name="position">
+                  <param name="initial_value">${initial_positions['leftarmbase']}</param>
+                </state_interface>
+            </joint>
+            <joint name="leftjoint1">
+                <command_interface name="position"/>
+                <state_interface name="position">
+                  <param name="initial_value">${initial_positions['leftjoint1']}</param>
+                </state_interface>
+            </joint>
+            <joint name="leftjoint2">
+                <command_interface name="position"/>
+                <state_interface name="position">
+                  <param name="initial_value">${initial_positions['leftjoint2']}</param>
+                </state_interface>
+            </joint>
+            <joint name="leftjoint3">
+                <command_interface name="position"/>
+                <state_interface name="position">
+                  <param name="initial_value">${initial_positions['leftjoint3']}</param>
+                </state_interface>
+            </joint>
+            <joint name="leftjoint4">
+                <command_interface name="position"/>
+                <state_interface name="position">
+                  <param name="initial_value">${initial_positions['leftjoint4']}</param>
+                </state_interface>
+            </joint>
             <joint name="rightarmbase">
                 <command_interface name="position"/>
@@ -13,5 +55,4 @@
                   <param name="initial_value">${initial_positions['rightarmbase']}</param>
                 </state_interface>
-                <state_interface name="velocity"/>
             </joint>
             <joint name="rightjoint1">
@@ -20,5 +61,4 @@
                   <param name="initial_value">${initial_positions['rightjoint1']}</param>
                 </state_interface>
-                <state_interface name="velocity"/>
             </joint>
             <joint name="rightjoint2">
@@ -27,5 +67,4 @@
                   <param name="initial_value">${initial_positions['rightjoint2']}</param>
                 </state_interface>
-                <state_interface name="velocity"/>
             </joint>
             <joint name="rightjoint3">
@@ -34,5 +73,4 @@
                   <param name="initial_value">${initial_positions['rightjoint3']}</param>
                 </state_interface>
-                <state_interface name="velocity"/>
             </joint>
             <joint name="rightjoint4">
@@ -41,40 +79,4 @@
                   <param name="initial_value">${initial_positions['rightjoint4']}</param>
                 </state_interface>
-                <state_interface name="velocity"/>
-            </joint>
-            <joint name="leftarmbase">
-                <command_interface name="position"/>
-                <state_interface name="position">
-                  <param name="initial_value">${initial_positions['leftarmbase']}</param>
-                </state_interface>
-                <state_interface name="velocity"/>
-            </joint>
-            <joint name="leftjoint1">
-                <command_interface name="position"/>
-                <state_interface name="position">
-                  <param name="initial_value">${initial_positions['leftjoint1']}</param>
-                </state_interface>
-                <state_interface name="velocity"/>
-            </joint>
-            <joint name="leftjoint2">
-                <command_interface name="position"/>
-                <state_interface name="position">
-                  <param name="initial_value">${initial_positions['leftjoint2']}</param>
-                </state_interface>
-                <state_interface name="velocity"/>
-            </joint>
-            <joint name="leftjoint3">
-                <command_interface name="position"/>
-                <state_interface name="position">
-                  <param name="initial_value">${initial_positions['leftjoint3']}</param>
-                </state_interface>
-                <state_interface name="velocity"/>
-            </joint>
-            <joint name="leftjoint4">
-                <command_interface name="position"/>
-                <state_interface name="position">
-                  <param name="initial_value">${initial_positions['leftjoint4']}</param>
-                </state_interface>
-                <state_interface name="velocity"/>
             </joint>
         </ros2_control>
