Commit message: feat: ros2_control 配置添加 leftjoint5/6
- alfa_robot.ros2_control.xacro: 添加 leftjoint5/6 关节接口
- initial_positions.yaml: 添加 leftjoint5/6 初始位置

Co-Authored-By: Claude Opus 4.7 <noreply@anthropic.com>

File: src/alfa_robot_moveit_config/config/alfa_robot.ros2_control.xacro (robot description, xacro)
@@ -50,4 +50,16 @@
                 </state_interface>
             </joint>
+            <joint name="leftjoint5">
+                <command_interface name="position"/>
+                <state_interface name="position">
+                  <param name="initial_value">${initial_positions['leftjoint5']}</param>
+                </state_interface>
+            </joint>
+            <joint name="leftjoint6">
+                <command_interface name="position"/>
+                <state_interface name="position">
+                  <param name="initial_value">${initial_positions['leftjoint6']}</param>
+                </state_interface>
+            </joint>
             <joint name="rightarmbase">
                 <command_interface name="position"/>
