Commit message: refactor: 移除 leftarmbase/rightarmbase 关节，简化双臂基座结构
- 从 URDF/SRDF/ros2_control/joint_limits 中移除 leftarmbase 和 rightarmbase
- alfa_robot_hardware.cpp buildJoints() 移除对应 CANopen 节点
- controllers/initial_positions/homing_node/joint_states_bridge 适配调整
- 新增 docs/ik_service.md IK 服务接口文档

Co-Authored-By: Claude Opus 4.7 <noreply@anthropic.com>

File: ros2_ws/src/alfa_robot_description/urdf/alfa_robot/alfa_robot_macro.ros2_control.xacro (robot description, xacro)
@@ -39,5 +39,4 @@
           <param name="safe_position_turn">0.0</param>
           <param name="safe_position_updown">0.0</param>
-          <param name="safe_position_leftarmbase">0.0</param>
           <param name="safe_position_leftjoint1">0.0</param>
           <param name="safe_position_leftjoint2">0.0</param>
@@ -46,5 +45,4 @@
           <param name="safe_position_leftjoint5">0.0</param>
           <param name="safe_position_leftjoint6">0.0</param>
-          <param name="safe_position_rightarmbase">0.0</param>
           <param name="safe_position_rightjoint1">0.0</param>
           <param name="safe_position_rightjoint2">0.0</param>
@@ -92,16 +90,4 @@
         <state_interface name="acceleration"/>
       </joint>
-      <!-- rightarmbase (prismatic) -->
-      <joint name="${prefix}rightarmbase">
-        <command_interface name="position">
-          <param name="min">0</param>
-          <param name="max">0.14</param>
-        </command_interface>
-        <state_interface name="position">
-          <param name="initial_value">0.0</param>
-        </state_interface>
-        <state_interface name="velocity"/>
-        <state_interface name="acceleration"/>
-      </joint>
       <!-- rightjoint1 (prismatic) -->
       <joint name="${prefix}rightjoint1">
@@ -169,16 +155,4 @@
           <param name="min">0</param>
           <param name="max">0.15</param>
-        </command_interface>
-        <state_interface name="position">
-          <param name="initial_value">0.0</param>
-        </state_interface>
-        <state_interface name="velocity"/>
-        <state_interface name="acceleration"/>
-      </joint>
-      <!-- leftarmbase (prismatic) -->
-      <joint name="${prefix}leftarmbase">
-        <command_interface name="position">
-          <param name="min">0</param>
-          <param name="max">0.14</param>
         </command_interface>
         <state_interface name="position">

File: ros2_ws/src/alfa_robot_description/urdf/alfa_robot/alfa_robot_macro.xacro (robot description, xacro)
@@ -89,25 +89,4 @@
       </collision>
     </link>
-    <!-- rightarmbase -->
-    <link name="${prefix}rightarmbase_link">
-      <inertial>
-        <origin xyz="0.00858986048699223 0.0287669594345854 0.0499555606572479" rpy="0 0 0"/>
-        <mass value="7.06520786853071"/>
-        <inertia ixx="0.0164730270054181" ixy="-9.84172582142273E-06" ixz="0.000387662666799276" iyy="0.0926777572076808" iyz="-0.0001209391577568" izz="0.091397951636245"/>
-      </inertial>
-      <visual>
-        <origin xyz="0 0 0" rpy="0 0 0"/>
-        <geometry>
-          <mesh filename="package://alfa_robot_description/meshes/alfa_robot/visual/rightarmbase.STL"/>
-        </geometry>
-        <material name="white"/>
-      </visual>
-      <collision>
-        <origin xyz="0 0 0" rpy="0 0 0"/>
-        <geometry>
-          <mesh filename="package://alfa_robot_description/meshes/alfa_robot/collision/rightarmbase.STL"/>
-        </geometry>
-      </collision>
-    </link>
     <!-- rightjoint1 -->
     <link name="${prefix}rightjoint1_link">
@@ -236,26 +215,5 @@
       </collision>
     </link>
-    <!-- rightarmbase (link name differs from joint for GZ compatibility) -->
-    <link name="${prefix}leftarmbase_link">
-      <inertial>
-        <origin xyz="0.00858986048699223 -0.0287669594345854 0.0499555606572479" rpy="0 0 0"/>
-        <mass value="7.06520786853071"/>
-        <inertia ixx="0.0164730270054181" ixy="9.84172582142273E-06" ixz="0.000387662666799276" iyy="0.0926777572076808" iyz="0.0001209391577568" izz="0.091397951636245"/>
-      </inertial>
-      <visual>
-        <origin xyz="0 0 0" rpy="0 0 0"/>
-        <geometry>
-          <mesh filename="package://alfa_robot_description/meshes/alfa_robot/visual/leftarmbase.STL"/>
-        </geometry>
-        <material name="white"/>
-      </visual>
-      <collision>
-        <origin xyz="0 0 0" rpy="0 0 0"/>
-        <geometry>
-          <mesh filename="package://alfa_robot_description/meshes/alfa_robot/collision/leftarmbase.STL"/>
-        </geometry>
-      </collision>
-    </link>
-    <!-- rightjoint1 (link name differs from joint for GZ compatibility) -->
+    <!-- leftjoint1 -->
     <link name="${prefix}leftjoint1_link">
       <inertial>
@@ -460,16 +418,8 @@
       <limit lower="0" upper="0.5" effort="1000" velocity="1000"/>
     </joint>
-    <!-- rightarmbase -->
-    <joint name="${prefix}rightarmbase" type="prismatic">
-      <origin xyz="-0.16145 -0.3282 0.146" rpy="0 0 0"/>
-      <parent link="${prefix}updown_link"/>
-      <child link="${prefix}rightarmbase_link"/>
-      <axis xyz="0 -1 0"/>
-      <limit lower="0" upper="0.14" effort="1000" velocity="0.5"/>
-    </joint>
     <!-- rightjoint1 -->
     <joint name="${prefix}rightjoint1" type="prismatic">
-      <origin xyz="0.15658 0.096099 0.086" rpy="0 0 0"/>
-      <parent link="${prefix}rightarmbase_link"/>
+      <origin xyz="-0.00487 -0.232101 0.232" rpy="0 0 0"/>
+      <parent link="${prefix}updown_link"/>
       <child link="${prefix}rightjoint1_link"/>
       <axis xyz="1 0 0"/>
@@ -522,16 +472,8 @@
       <child link="${prefix}right_ee_link"/>
     </joint>
-    <!-- rightarmbase -->
-    <joint name="${prefix}leftarmbase" type="prismatic">
-      <origin xyz="-0.16145 0.3282 0.146" rpy="0 0 0"/>
+    <!-- leftjoint1 -->
+    <joint name="${prefix}leftjoint1" type="prismatic">
+      <origin xyz="-0.00487 0.232101 0.232" rpy="0 0 0"/>
       <parent link="${prefix}updown_link"/>
-      <child link="${prefix}leftarmbase_link"/>
-      <axis xyz="0 1 0"/>
-      <limit lower="0" upper="0.14" effort="1000" velocity="0.5"/>
-    </joint>
-    <!-- rightjoint1 -->
-    <joint name="${prefix}leftjoint1" type="prismatic">
-      <origin xyz="0.15658 -0.096099 0.086" rpy="0 0 0"/>
-      <parent link="${prefix}leftarmbase_link"/>
       <child link="${prefix}leftjoint1_link"/>
       <axis xyz="1 0 0"/>

File: ros2_ws/src/alfa_robot_moveit_config/config/alfa_robot.ros2_control.xacro (robot description, xacro)
@@ -18,10 +18,4 @@
                 <state_interface name="position">
                   <param name="initial_value">${initial_positions['updown']}</param>
-                </state_interface>
-            </joint>
-            <joint name="leftarmbase">
-                <command_interface name="position"/>
-                <state_interface name="position">
-                  <param name="initial_value">${initial_positions['leftarmbase']}</param>
                 </state_interface>
             </joint>
@@ -60,10 +54,4 @@
                 <state_interface name="position">
                   <param name="initial_value">${initial_positions['leftjoint6']}</param>
-                </state_interface>
-            </joint>
-            <joint name="rightarmbase">
-                <command_interface name="position"/>
-                <state_interface name="position">
-                  <param name="initial_value">${initial_positions['rightarmbase']}</param>
                 </state_interface>
             </joint>
