Commit message: feat: 接入 V3.0.2 双臂模型对比分支
外观与碰撞统一使用 V3.0.2 网格，同步更新七轴关节链并生成严格镜像右臂，保留构建、URDF、镜像 FK 和 MoveIt IK 验证记录。

Refs MOTION-94: 更新 V3 机械臂模型对比基线

File: ros2_ws/src/alfa_robot_description/urdf/alfa_robot/robot_v3_arm.xacro (robot description, xacro)
@@ -1,10 +1,10 @@
 <?xml version="1.0" encoding="UTF-8"?>
 <robot xmlns:xacro="http://wiki.ros.org/xacro">
-  <xacro:macro name="robot_v3_arm_link" params="name visual_mesh collision_mesh collision_xyz collision_rpy">
+  <xacro:macro name="robot_v3_arm_link" params="name mesh">
     <link name="${name}">
       <visual>
         <origin xyz="0 0 0" rpy="0 0 0"/>
         <geometry>
-          <mesh filename="${visual_mesh}"/>
+          <mesh filename="${mesh}"/>
         </geometry>
         <material name="robot_v3_arm_white">
@@ -13,7 +13,7 @@
       </visual>
       <collision>
-        <origin xyz="${collision_xyz}" rpy="${collision_rpy}"/>
+        <origin xyz="0 0 0" rpy="0 0 0"/>
         <geometry>
-          <mesh filename="${collision_mesh}"/>
+          <mesh filename="${mesh}"/>
         </geometry>
       </collision>
@@ -31,7 +31,6 @@
   <xacro:macro name="robot_v3_arm" params="prefix parent mount_xyz mirrored:=false">
     <xacro:property name="variant" value="${'right' if mirrored else 'left'}"/>
-    <xacro:property name="collision_mesh_root" value="package://alfa_robot_description/meshes/robot_v3_0_1/${variant}"/>
-    <xacro:property name="visual_mesh_root" value="package://alfa_robot_description/meshes/robot_v3_0_1/visual/${variant}"/>
-    <xacro:robot_v3_arm_link name="${prefix}_arm_base" visual_mesh="${visual_mesh_root}/base_link.stl" collision_mesh="${collision_mesh_root}/base_link.stl" collision_xyz="0 0 0" collision_rpy="0 0 0"/>
+    <xacro:property name="mesh_root" value="package://alfa_robot_description/meshes/robot_v3_0_2/${variant}"/>
+    <xacro:robot_v3_arm_link name="${prefix}_arm_base" mesh="${mesh_root}/base_link.stl"/>
     <joint name="${prefix}_arm_mount" type="fixed">
       <parent link="${parent}"/>
@@ -40,34 +39,34 @@
     </joint>
     <xacro:unless value="${mirrored}">
-      <xacro:robot_v3_arm_link name="${prefix}_joint1" visual_mesh="${visual_mesh_root}/Link_1.stl" collision_mesh="${collision_mesh_root}/Link_1.stl" collision_xyz="0.000522813 -0.000361729 0.002117818" collision_rpy="-0.000054774 -0.001816128 -0.100210370"/>
-      <xacro:robot_v3_arm_link name="${prefix}_joint2" visual_mesh="${visual_mesh_root}/Link_2.stl" collision_mesh="${collision_mesh_root}/Link_2.stl" collision_xyz="0.000770099 -0.000300398 -0.023978220" collision_rpy="0.001031215 -0.000739591 0.142567923"/>
-      <xacro:robot_v3_arm_link name="${prefix}_joint3" visual_mesh="${visual_mesh_root}/Link_3.stl" collision_mesh="${collision_mesh_root}/Link_3.stl" collision_xyz="0.012124727 0.018730189 0.004397036" collision_rpy="-0.023666759 0.003048467 0.152665621"/>
-      <xacro:robot_v3_arm_link name="${prefix}_joint4" visual_mesh="${visual_mesh_root}/Link_4.stl" collision_mesh="${collision_mesh_root}/Link_4.stl" collision_xyz="-0.004113276 0.000530688 -0.006223374" collision_rpy="-0.015067397 0.031826793 -0.000710309"/>
-      <xacro:robot_v3_arm_link name="${prefix}_joint5" visual_mesh="${visual_mesh_root}/Link_5.stl" collision_mesh="${collision_mesh_root}/Link_5.stl" collision_xyz="0.007248149 0.003483586 0.002682465" collision_rpy="0.018444782 -0.039168674 -0.031123433"/>
-      <xacro:robot_v3_arm_link name="${prefix}_joint6" visual_mesh="${visual_mesh_root}/Link_6.stl" collision_mesh="${collision_mesh_root}/Link_6.stl" collision_xyz="-0.000709350 0.000725282 -0.004991800" collision_rpy="0.002501622 -0.002350798 -0.000022510"/>
-      <xacro:robot_v3_arm_link name="${prefix}_joint7" visual_mesh="${visual_mesh_root}/Link_7.stl" collision_mesh="${collision_mesh_root}/Link_7.stl" collision_xyz="0.009192134 -0.024103896 -0.020348427" collision_rpy="0.001263973 -0.001366502 -0.086546196"/>
-      <xacro:robot_v3_arm_joint name="${prefix}_joint1" parent="${prefix}_arm_base" child="${prefix}_joint1" xyz="0.00001172 0.00004065 0.016" rpy="0 0 3.14159265" axis="0 0 1"/>
-      <xacro:robot_v3_arm_joint name="${prefix}_joint2" parent="${prefix}_joint1" child="${prefix}_joint2" xyz="-0.05925684 -0.00523679 0.112" rpy="1.57079633 0 -1.48265083" axis="0 0 1"/>
-      <xacro:robot_v3_arm_joint name="${prefix}_joint3" parent="${prefix}_joint2" child="${prefix}_joint3" xyz="-0.23925372 0.05721594 -0.06129979" rpy="-1.57079633 -0.0205517 1.33606144" axis="0 0 1"/>
-      <xacro:robot_v3_arm_joint name="${prefix}_joint4" parent="${prefix}_joint3" child="${prefix}_joint4" xyz="-0.15474281 -0.07084206 0.14699994" rpy="1.57079633 1.33563993 0.08156114" axis="0 0 1"/>
-      <xacro:robot_v3_arm_joint name="${prefix}_joint5" parent="${prefix}_joint4" child="${prefix}_joint5" xyz="-0.04593775 -0.00239318 -0.06299914" rpy="1.57079638 -1.51138059 -1.51874803" axis="0 0 1"/>
-      <xacro:robot_v3_arm_joint name="${prefix}_joint6" parent="${prefix}_joint5" child="${prefix}_joint6" xyz="0.04449757 0.000388 0.283" rpy="-1.5707965 1.51883841 -1.56207717" axis="0 0 1"/>
-      <xacro:robot_v3_arm_joint name="${prefix}_joint7" parent="${prefix}_joint6" child="${prefix}_joint7" xyz="-0.00194278 0.06096906 -0.04450033" rpy="-1.57079623 -0.10521384 0.03185501" axis="0 0 1"/>
+      <xacro:robot_v3_arm_link name="${prefix}_joint1" mesh="${mesh_root}/Link_1.stl"/>
+      <xacro:robot_v3_arm_link name="${prefix}_joint2" mesh="${mesh_root}/Link_2.stl"/>
+      <xacro:robot_v3_arm_link name="${prefix}_joint3" mesh="${mesh_root}/Link_3.stl"/>
+      <xacro:robot_v3_arm_link name="${prefix}_joint4" mesh="${mesh_root}/Link_4.stl"/>
+      <xacro:robot_v3_arm_link name="${prefix}_joint5" mesh="${mesh_root}/Link_5.stl"/>
+      <xacro:robot_v3_arm_link name="${prefix}_joint6" mesh="${mesh_root}/Link_6.stl"/>
+      <xacro:robot_v3_arm_link name="${prefix}_joint7" mesh="${mesh_root}/Link_7.stl"/>
+      <xacro:robot_v3_arm_joint name="${prefix}_joint1" parent="${prefix}_arm_base" child="${prefix}_joint1" xyz="0 0 0.018" rpy="0 0 3.14159265" axis="0 0 1"/>
+      <xacro:robot_v3_arm_joint name="${prefix}_joint2" parent="${prefix}_joint1" child="${prefix}_joint2" xyz="-0.03395348 -0.01941469 0.11" rpy="-1.57079633 0 2.09022451" axis="0 0 1"/>
+      <xacro:robot_v3_arm_joint name="${prefix}_joint3" parent="${prefix}_joint2" child="${prefix}_joint3" xyz="-0.23198447 -0.08184869 -0.03729999" rpy="0 1.57079633 -2.80240802" axis="0 0 1"/>
+      <xacro:robot_v3_arm_joint name="${prefix}_joint4" parent="${prefix}_joint3" child="${prefix}_joint4" xyz="-0.07756491 -0.15036183 0.147" rpy="1.57079632 -1.22828075 -1.71595129" axis="0 0 1"/>
+      <xacro:robot_v3_arm_joint name="${prefix}_joint5" parent="${prefix}_joint4" child="${prefix}_joint5" xyz="0.04597995 -0.00135805 -0.05" rpy="-1.57079589 -1.43390621 -1.60032347" axis="0 0 1"/>
+      <xacro:robot_v3_arm_joint name="${prefix}_joint6" parent="${prefix}_joint5" child="${prefix}_joint6" xyz="0.04549984 0.00012564 0.28300003" rpy="-1.57079667 -1.54154524 -1.5680338" axis="0 0 1"/>
+      <xacro:robot_v3_arm_joint name="${prefix}_joint7" parent="${prefix}_joint6" child="${prefix}_joint7" xyz="0.06585468 0.00164675 -0.04498124" rpy="-0.02526825 1.56803419 0" axis="0 0 1"/>
     </xacro:unless>
     <xacro:if value="${mirrored}">
-      <xacro:robot_v3_arm_link name="${prefix}_joint1" visual_mesh="${visual_mesh_root}/Link_1.stl" collision_mesh="${collision_mesh_root}/Link_1.stl" collision_xyz="0.000522813 0.000361729 0.002117818" collision_rpy="0.000054774 -0.001816128 0.100210370"/>
-      <xacro:robot_v3_arm_link name="${prefix}_joint2" visual_mesh="${visual_mesh_root}/Link_2.stl" collision_mesh="${collision_mesh_root}/Link_2.stl" collision_xyz="0.000770099 0.000300398 -0.023978220" collision_rpy="-0.001031215 -0.000739591 -0.142567923"/>
-      <xacro:robot_v3_arm_link name="${prefix}_joint3" visual_mesh="${visual_mesh_root}/Link_3.stl" collision_mesh="${collision_mesh_root}/Link_3.stl" collision_xyz="0.012124727 -0.018730189 0.004397036" collision_rpy="0.023666759 0.003048467 -0.152665621"/>
-      <xacro:robot_v3_arm_link name="${prefix}_joint4" visual_mesh="${visual_mesh_root}/Link_4.stl" collision_mesh="${collision_mesh_root}/Link_4.stl" collision_xyz="-0.004113276 -0.000530688 -0.006223374" collision_rpy="0.015067397 0.031826793 0.000710309"/>
-      <xacro:robot_v3_arm_link name="${prefix}_joint5" visual_mesh="${visual_mesh_root}/Link_5.stl" collision_mesh="${collision_mesh_root}/Link_5.stl" collision_xyz="0.007248149 -0.003483586 0.002682465" collision_rpy="-0.018444782 -0.039168674 0.031123433"/>
-      <xacro:robot_v3_arm_link name="${prefix}_joint6" visual_mesh="${visual_mesh_root}/Link_6.stl" collision_mesh="${collision_mesh_root}/Link_6.stl" collision_xyz="-0.000709350 -0.000725282 -0.004991800" collision_rpy="-0.002501622 -0.002350798 0.000022510"/>
-      <xacro:robot_v3_arm_link name="${prefix}_joint7" visual_mesh="${visual_mesh_root}/Link_7.stl" collision_mesh="${collision_mesh_root}/Link_7.stl" collision_xyz="0.009192134 0.024103896 -0.020348427" collision_rpy="-0.001263973 -0.001366502 0.086546196"/>
-      <xacro:robot_v3_arm_joint name="${prefix}_joint1" parent="${prefix}_arm_base" child="${prefix}_joint1" xyz="0.00001172 -0.00004065 0.016" rpy="0 0 -3.14159265" axis="0 0 -1"/>
-      <xacro:robot_v3_arm_joint name="${prefix}_joint2" parent="${prefix}_joint1" child="${prefix}_joint2" xyz="-0.05925684 0.00523679 0.112" rpy="-1.57079633 0 1.48265083" axis="0 0 -1"/>
-      <xacro:robot_v3_arm_joint name="${prefix}_joint3" parent="${prefix}_joint2" child="${prefix}_joint3" xyz="-0.23925372 -0.05721594 -0.06129979" rpy="1.57079633 -0.0205517 -1.33606144" axis="0 0 -1"/>
-      <xacro:robot_v3_arm_joint name="${prefix}_joint4" parent="${prefix}_joint3" child="${prefix}_joint4" xyz="-0.15474281 0.07084206 0.14699994" rpy="-1.57079633 1.33563993 -0.08156114" axis="0 0 -1"/>
-      <xacro:robot_v3_arm_joint name="${prefix}_joint5" parent="${prefix}_joint4" child="${prefix}_joint5" xyz="-0.04593775 0.00239318 -0.06299914" rpy="-1.57079638 -1.51138059 1.51874803" axis="0 0 -1"/>
-      <xacro:robot_v3_arm_joint name="${prefix}_joint6" parent="${prefix}_joint5" child="${prefix}_joint6" xyz="0.04449757 -0.000388 0.283" rpy="1.5707965 1.51883841 1.56207717" axis="0 0 -1"/>
-      <xacro:robot_v3_arm_joint name="${prefix}_joint7" parent="${prefix}_joint6" child="${prefix}_joint7" xyz="-0.00194278 -0.06096906 -0.04450033" rpy="1.57079623 -0.10521384 -0.03185501" axis="0 0 -1"/>
+      <xacro:robot_v3_arm_link name="${prefix}_joint1" mesh="${mesh_root}/Link_1.stl"/>
+      <xacro:robot_v3_arm_link name="${prefix}_joint2" mesh="${mesh_root}/Link_2.stl"/>
+      <xacro:robot_v3_arm_link name="${prefix}_joint3" mesh="${mesh_root}/Link_3.stl"/>
+      <xacro:robot_v3_arm_link name="${prefix}_joint4" mesh="${mesh_root}/Link_4.stl"/>
+      <xacro:robot_v3_arm_link name="${prefix}_joint5" mesh="${mesh_root}/Link_5.stl"/>
+      <xacro:robot_v3_arm_link name="${prefix}_joint6" mesh="${mesh_root}/Link_6.stl"/>
+      <xacro:robot_v3_arm_link name="${prefix}_joint7" mesh="${mesh_root}/Link_7.stl"/>
+      <xacro:robot_v3_arm_joint name="${prefix}_joint1" parent="${prefix}_arm_base" child="${prefix}_joint1" xyz="0 0 0.018" rpy="0 0 -3.14159265" axis="0 0 -1"/>
+      <xacro:robot_v3_arm_joint name="${prefix}_joint2" parent="${prefix}_joint1" child="${prefix}_joint2" xyz="-0.03395348 0.01941469 0.11" rpy="1.57079633 0 -2.09022451" axis="0 0 -1"/>
+      <xacro:robot_v3_arm_joint name="${prefix}_joint3" parent="${prefix}_joint2" child="${prefix}_joint3" xyz="-0.23198447 0.08184869 -0.03729999" rpy="0 1.57079633 2.80240802" axis="0 0 -1"/>
+      <xacro:robot_v3_arm_joint name="${prefix}_joint4" parent="${prefix}_joint3" child="${prefix}_joint4" xyz="-0.07756491 0.15036183 0.147" rpy="-1.57079632 -1.22828075 1.71595129" axis="0 0 -1"/>
+      <xacro:robot_v3_arm_joint name="${prefix}_joint5" parent="${prefix}_joint4" child="${prefix}_joint5" xyz="0.04597995 0.00135805 -0.05" rpy="1.57079589 -1.43390621 1.60032347" axis="0 0 -1"/>
+      <xacro:robot_v3_arm_joint name="${prefix}_joint6" parent="${prefix}_joint5" child="${prefix}_joint6" xyz="0.04549984 -0.00012564 0.28300003" rpy="1.57079667 -1.54154524 1.5680338" axis="0 0 -1"/>
+      <xacro:robot_v3_arm_joint name="${prefix}_joint7" parent="${prefix}_joint6" child="${prefix}_joint7" xyz="0.06585468 -0.00164675 -0.04498124" rpy="0.02526825 1.56803419 0" axis="0 0 -1"/>
     </xacro:if>
     <link name="${prefix}_tool0"/>
