Commit message: fix(v3): 对齐V3.0.9升降与头部限位 Refs MOTION-94

File: ros2_ws/src/alfa_robot_description/urdf/alfa_robot/robot_v3_0_9.xacro (robot description, xacro)
@@ -759,5 +759,5 @@
     <child link="arm_carriage" />
     <axis xyz="0 0 1" />
-    <limit lower="0" upper="0.7" effort="1000" velocity="0.15" />
+    <limit lower="-0.1" upper="0.1" effort="1000" velocity="0.15" />
   </joint>
   <joint name="head_joint" type="revolute">
@@ -766,5 +766,5 @@
     <child link="head" />
     <axis xyz="0 0 1" />
-    <limit lower="-1.57079633" upper="1.57079633" effort="10" velocity="1" />
+    <limit lower="-1.57" upper="1.57" effort="10" velocity="1" />
   </joint>
   <joint name="left_joint1" type="revolute">

Commit message: fix(v3): 固化一米升降逻辑坐标 Refs MOTION-94

File: ros2_ws/src/alfa_robot_description/urdf/alfa_robot/robot_v3_0_9.xacro (robot description, xacro)
@@ -759,5 +759,6 @@
     <child link="arm_carriage" />
     <axis xyz="0 0 1" />
-    <limit lower="-0.1" upper="0.1" effort="1000" velocity="0.15" />
+    <!-- 逻辑坐标：-1.0m 为升降最低点，0.0m 为从最低点升高 1m 的最高点。 -->
+    <limit lower="-1.0" upper="0.0" effort="1000" velocity="0.15" />
   </joint>
   <joint name="head_joint" type="revolute">
