Commit message: checkpoint: preserve current v4 MoveIt and DH fixes

File: ros2_ws/src/alfa_robot_description/urdf/alfa_robot.urdf.xacro (robot description, xacro)
@@ -109,9 +109,5 @@
     <axis
       xyz="0 1 0" />
-    <limit
-      lower="0"
-      upper="0.26"
-      effort="0"
-      velocity="0" />
+    <limit lower="0" upper="0.26" effort="10" velocity="0.87"/>
   </joint>
   <link
@@ -220,9 +216,5 @@
     <axis
       xyz="0 0 1" />
-    <limit
-      lower="0"
-      upper="0.99"
-      effort="0"
-      velocity="0" />
+    <limit lower="0" upper="1.0" effort="10" velocity="1.0"/>
   </joint>
   <link
@@ -278,9 +270,5 @@
     <axis
       xyz="1 0 0" />
-    <limit
-      lower="0"
-      upper="0.3"
-      effort="0"
-      velocity="0" />
+    <limit lower="0" upper="0.42" effort="10" velocity="1.0"/>
   </joint>
   <link
@@ -326,5 +314,5 @@
   <joint
     name="leftjoint2"
-    type="continuous">
+    type="revolute">
     <origin
       xyz="0.741 0 0.0425"
@@ -336,9 +324,5 @@
     <axis
       xyz="0 0 1" />
-    <limit
-      lower="0"
-      upper="0"
-      effort="0"
-      velocity="0" />
+    <limit lower="-3.14159" upper="3.14159" effort="10" velocity="1.2"/>
   </joint>
   <link
@@ -384,5 +368,5 @@
   <joint
     name="leftjoint3"
-    type="continuous">
+    type="revolute">
     <origin
       xyz="-0.00035108 0.075999 0.058"
@@ -394,9 +378,5 @@
     <axis
       xyz="0 0 1" />
-    <limit
-      lower="0"
-      upper="0"
-      effort="0"
-      velocity="0" />
+    <limit lower="-1.57079632" upper="1.57079632" effort="10" velocity="1.2"/>
   </joint>
   <link
@@ -442,5 +422,5 @@
   <joint
     name="leftjoint4"
-    type="continuous">
+    type="revolute">
     <origin
       xyz="0.311 0 0.058"
@@ -452,9 +432,5 @@
     <axis
       xyz="0 0 1" />
-    <limit
-      lower="0"
-      upper="0"
-      effort="0"
-      velocity="0" />
+    <limit lower="-3.14159" upper="3.14159" effort="10" velocity="1.2"/>
   </joint>
   <link
@@ -500,5 +476,5 @@
   <joint
     name="leftjoint5"
-    type="continuous">
+    type="revolute">
     <origin
       xyz="0 -0.076 0.058"
@@ -510,9 +486,5 @@
     <axis
       xyz="0 0 1" />
-    <limit
-      lower="0"
-      upper="0"
-      effort="0"
-      velocity="0" />
+    <limit lower="-1.57079632" upper="1.57079632" effort="10" velocity="1.2"/>
   </joint>
   <link
@@ -568,9 +540,5 @@
     <axis
       xyz="1 0 0" />
-    <limit
-      lower="0"
-      upper="0.15"
-      effort="0"
-      velocity="0" />
+    <limit lower="0" upper="0.15" effort="1" velocity="0.05"/>
   </joint>
   <link
@@ -626,9 +594,5 @@
     <axis
       xyz="1 0 0" />
-    <limit
-      lower="0"
-      upper="0.3"
-      effort="0"
-      velocity="0" />
+    <limit lower="0" upper="0.42" effort="10" velocity="1.0"/>
   </joint>
   <link
@@ -674,5 +638,5 @@
   <joint
     name="rightjoint2"
-    type="continuous">
+    type="revolute">
     <origin
       xyz="0.741 0 0.0425"
@@ -684,9 +648,5 @@
     <axis
       xyz="0 0 1" />
-    <limit
-      lower="0"
-      upper="0"
-      effort="0"
-      velocity="0" />
+    <limit lower="-3.14159" upper="3.14159" effort="10" velocity="1.2"/>
   </joint>
   <link
@@ -732,5 +692,5 @@
   <joint
     name="rightjoint3"
-    type="continuous">
+    type="revolute">
     <origin
       xyz="0 0.076 0.058"
@@ -742,9 +702,5 @@
     <axis
       xyz="0 0 1" />
-    <limit
-      lower="0"
-      upper="0"
-      effort="0"
-      velocity="0" />
+    <limit lower="-1.57079632" upper="1.57079632" effort="10" velocity="1.2"/>
   </joint>
   <link
@@ -790,5 +746,5 @@
   <joint
     name="rightjoint4"
-    type="continuous">
+    type="revolute">
     <origin
       xyz="0.311 0 0.058"
@@ -800,9 +756,5 @@
     <axis
       xyz="0 0 1" />
-    <limit
-      lower="0"
-      upper="0"
-      effort="0"
-      velocity="0" />
+    <limit lower="-3.14159" upper="3.14159" effort="10" velocity="1.2"/>
   </joint>
   <link
@@ -848,5 +800,5 @@
   <joint
     name="rightjoint5"
-    type="continuous">
+    type="revolute">
     <origin
       xyz="0 -0.0697 0.058"
@@ -858,9 +810,5 @@
     <axis
       xyz="0 0 1" />
-    <limit
-      lower="0"
-      upper="0"
-      effort="0"
-      velocity="0" />
+    <limit lower="-1.57079632" upper="1.57079632" effort="10" velocity="1.2"/>
   </joint>
   <link
@@ -916,9 +864,5 @@
     <axis
       xyz="1 0 0" />
-    <limit
-      lower="0"
-      upper="0.15"
-      effort="0"
-      velocity="0" />
+    <limit lower="0" upper="0.15" effort="1" velocity="0.05"/>
   </joint>
   <link name="left_ee_link"/>

File: ros2_ws/src/alfa_robot_description/urdf/alfa_robot/alfa_robot_macro.ros2_control.xacro (robot description, xacro)
@@ -31,5 +31,4 @@
           <param name="can_interface_canopen">can3</param>
           <param name="can_interface_base">can2</param>
-          <param name="can_interface_plate">can4</param>
           <param name="canopen_profile_velocity">${canopen_profile_velocity}</param>
           <param name="canopen_profile_accel">${canopen_profile_accel}</param>
@@ -51,4 +50,5 @@
           <param name="safe_position_rightjoint5">0.0</param>
           <param name="safe_position_rightjoint6">0.0</param>
+          <param name="safe_position_pitch">0.0</param>
         </xacro:unless>
       </hardware>
@@ -65,7 +65,10 @@
         <state_interface name="acceleration"/>
       </joint>
-      <!-- turn (continuous; no URDF limit tag) -->
+      <!-- turn (continuous) -->
       <joint name="${prefix}turn">
-        <command_interface name="position"/>
+        <command_interface name="position">
+          <param name="min">-3.14159</param>
+          <param name="max">3.14159</param>
+        </command_interface>
         <state_interface name="position">
           <param name="initial_value">0.0</param>
@@ -78,5 +81,5 @@
         <command_interface name="position">
           <param name="min">0</param>
-          <param name="max">0.99</param>
+          <param name="max">1.0</param>
         </command_interface>
         <state_interface name="position">
@@ -90,53 +93,53 @@
         <command_interface name="position">
           <param name="min">0</param>
-          <param name="max">0.3</param>
-        </command_interface>
-        <state_interface name="position">
-          <param name="initial_value">0.0</param>
-        </state_interface>
-        <state_interface name="velocity"/>
-        <state_interface name="acceleration"/>
-      </joint>
-      <!-- rightjoint2 (continuous; URDF limit tag currently 0..0) -->
+          <param name="max">0.42</param>
+        </command_interface>
+        <state_interface name="position">
+          <param name="initial_value">0.0</param>
+        </state_interface>
+        <state_interface name="velocity"/>
+        <state_interface name="acceleration"/>
+      </joint>
+      <!-- rightjoint2 (revolute) -->
       <joint name="${prefix}rightjoint2">
         <command_interface name="position">
-          <param name="min">0</param>
-          <param name="max">0</param>
-        </command_interface>
-        <state_interface name="position">
-          <param name="initial_value">0.0</param>
-        </state_interface>
-        <state_interface name="velocity"/>
-        <state_interface name="acceleration"/>
-      </joint>
-      <!-- rightjoint3 (continuous; URDF limit tag currently 0..0) -->
+          <param name="min">-3.14159</param>
+          <param name="max">3.14159</param>
+        </command_interface>
+        <state_interface name="position">
+          <param name="initial_value">0.0</param>
+        </state_interface>
+        <state_interface name="velocity"/>
+        <state_interface name="acceleration"/>
+      </joint>
+      <!-- rightjoint3 (revolute) -->
       <joint name="${prefix}rightjoint3">
         <command_interface name="position">
-          <param name="min">0</param>
-          <param name="max">0</param>
-        </command_interface>
-        <state_interface name="position">
-          <param name="initial_value">0.0</param>
-        </state_interface>
-        <state_interface name="velocity"/>
-        <state_interface name="acceleration"/>
-      </joint>
-      <!-- rightjoint4 (continuous; URDF limit tag currently 0..0) -->
+          <param name="min">-1.57079632</param>
+          <param name="max">1.57079632</param>
+        </command_interface>
+        <state_interface name="position">
+          <param name="initial_value">0.0</param>
+        </state_interface>
+        <state_interface name="velocity"/>
+        <state_interface name="acceleration"/>
+      </joint>
+      <!-- rightjoint4 (revolute) -->
       <joint name="${prefix}rightjoint4">
         <command_interface name="position">
-          <param name="min">0</param>
-          <param name="max">0</param>
-        </command_interface>
-        <state_interface name="position">
-          <param name="initial_value">0.0</param>
-        </state_interface>
-        <state_interface name="velocity"/>
-        <state_interface name="acceleration"/>
-      </joint>
-      <!-- rightjoint5 (continuous; URDF limit tag currently 0..0) -->
+          <param name="min">-3.14159</param>
+          <param name="max">3.14159</param>
+        </command_interface>
+        <state_interface name="position">
+          <param name="initial_value">0.0</param>
+        </state_interface>
+        <state_interface name="velocity"/>
+        <state_interface name="acceleration"/>
+      </joint>
+      <!-- rightjoint5 (revolute) -->
       <joint name="${prefix}rightjoint5">
         <command_interface name="position">
-          <param name="min">0</param>
-          <param name="max">0</param>
+          <param name="min">-1.57079632</param>
+          <param name="max">1.57079632</param>
         </command_interface>
         <state_interface name="position">
@@ -162,61 +165,61 @@
         <command_interface name="position">
           <param name="min">0</param>
-          <param name="max">0.3</param>
-        </command_interface>
-        <state_interface name="position">
-          <param name="initial_value">0.0</param>
-        </state_interface>
-        <state_interface name="velocity"/>
-        <state_interface name="acceleration"/>
-      </joint>
-      <!-- leftjoint2 (continuous; URDF limit tag currently 0..0) -->
+          <param name="max">0.42</param>
+        </command_interface>
+        <state_interface name="position">
+          <param name="initial_value">0.0</param>
+        </state_interface>
+        <state_interface name="velocity"/>
+        <state_interface name="acceleration"/>
+      </joint>
+      <!-- leftjoint2 (revolute) -->
       <joint name="${prefix}leftjoint2">
         <command_interface name="position">
-          <param name="min">0</param>
-          <param name="max">0</param>
-        </command_interface>
-        <state_interface name="position">
-          <param name="initial_value">0.0</param>
-        </state_interface>
-        <state_interface name="velocity"/>
-        <state_interface name="acceleration"/>
-      </joint>
-      <!-- leftjoint3 (continuous; URDF limit tag currently 0..0) -->
+          <param name="min">-3.14159</param>
+          <param name="max">3.14159</param>
+        </command_interface>
+        <state_interface name="position">
+          <param name="initial_value">0.0</param>
+        </state_interface>
+        <state_interface name="velocity"/>
+        <state_interface name="acceleration"/>
+      </joint>
+      <!-- leftjoint3 (revolute) -->
       <joint name="${prefix}leftjoint3">
         <command_interface name="position">
-          <param name="min">0</param>
-          <param name="max">0</param>
-        </command_interface>
-        <state_interface name="position">
-          <param name="initial_value">0.0</param>
-        </state_interface>
-        <state_interface name="velocity"/>
-        <state_interface name="acceleration"/>
-      </joint>
-      <!-- leftjoint4 (continuous; URDF limit tag currently 0..0) -->
+          <param name="min">-1.57079632</param>
+          <param name="max">1.57079632</param>
+        </command_interface>
+        <state_interface name="position">
+          <param name="initial_value">0.0</param>
+        </state_interface>
+        <state_interface name="velocity"/>
+        <state_interface name="acceleration"/>
+      </joint>
+      <!-- leftjoint4 (revolute) -->
       <joint name="${prefix}leftjoint4">
         <command_interface name="position">
-          <param name="min">0</param>
-          <param name="max">0</param>
-        </command_interface>
-        <state_interface name="position">
-          <param name="initial_value">0.0</param>
-        </state_interface>
-        <state_interface name="velocity"/>
-        <state_interface name="acceleration"/>
-      </joint>
-      <!-- leftjoint5 (continuous; URDF limit tag currently 0..0) -->
+          <param name="min">-3.14159</param>
+          <param name="max">3.14159</param>
+        </command_interface>
+        <state_interface name="position">
+          <param name="initial_value">0.0</param>
+        </state_interface>
+        <state_interface name="velocity"/>
+        <state_interface name="acceleration"/>
+      </joint>
+      <!-- leftjoint5 (revolute) -->
       <joint name="${prefix}leftjoint5">
         <command_interface name="position">
-          <param name="min">0</param>
-          <param name="max">0</param>
-        </command_interface>
-        <state_interface name="position">
-          <param name="initial_value">0.0</param>
-        </state_interface>
-        <state_interface name="velocity"/>
-        <state_interface name="acceleration"/>
-      </joint>
-      <!-- leftjoint6 (prismatic, new end effector extension) -->
+          <param name="min">-1.57079632</param>
+          <param name="max">1.57079632</param>
+        </command_interface>
+        <state_interface name="position">
+          <param name="initial_value">0.0</param>
+        </state_interface>
+        <state_interface name="velocity"/>
+        <state_interface name="acceleration"/>
+      </joint>
+      <!-- leftjoint6 (prismatic) -->
       <joint name="${prefix}leftjoint6">
         <command_interface name="position">
