Commit message: checkpoint: preserve current v4 MoveIt and DH fixes

File: ros2_ws/src/alfa_robot_description/urdf/alfa_robot/alfa_robot_macro.xacro (robot description, xacro)
@@ -1,393 +1,867 @@
 <?xml version="1.0" encoding="UTF-8"?>
 <robot xmlns:xacro="http://wiki.ros.org/xacro">
-  <xacro:include filename="$(find alfa_robot_description)/urdf/common/inertials.xacro"/>
   <xacro:include filename="$(find alfa_robot_description)/urdf/common/materials.xacro"/>
   <xacro:macro name="alfa_robot" params="prefix parent *origin">
-    <!-- LINKS -->
-    <!-- base_link -->
-    <link name="${prefix}base_link">
-      <inertial>
-        <origin xyz="-0.44193110855616 0.000259961331933109 0.176428166472852" rpy="0 0 0"/>
-        <mass value="394.931465036981"/>
-        <inertia ixx="66.5681215725466" ixy="5.74775273893285E-10" ixz="9.85014992290203" iyy="65.6389024339403" iyz="2.76043934386688E-09" izz="112.938477587322"/>
-      </inertial>
-      <visual>
-        <origin xyz="0 0 0" rpy="0 0 0"/>
-        <geometry>
-          <mesh filename="package://alfa_robot_description/meshes/alfa_robot/visual/base_link.STL"/>
-        </geometry>
-        <material name="blue"/>
-      </visual>
-      <collision>
-        <origin xyz="0 0 0" rpy="0 0 0"/>
-        <geometry>
-          <mesh filename="package://alfa_robot_description/meshes/alfa_robot/collision/base_link.STL"/>
-        </geometry>
-      </collision>
-    </link>
-    <!-- turn (link name differs from joint for GZ compatibility) -->
-    <link name="${prefix}turn_link">
-      <inertial>
-        <origin xyz="-0.0697894032768815 -0.00012433244764639 0.982155423971065" rpy="0 0 0"/>
-        <mass value="42.0737844290435"/>
-        <inertia ixx="10.0720353784748" ixy="-1.75362629131178E-06" ixz="5.29823321336754E-05" iyy="10.0937833616587" iyz="1.43589075450652E-06" izz="0.327199381319826"/>
-      </inertial>
-      <visual>
-        <origin xyz="0 0 0" rpy="0 0 0"/>
-        <geometry>
-          <mesh filename="package://alfa_robot_description/meshes/alfa_robot/visual/turn.STL"/>
-        </geometry>
-        <material name="arm_grey"/>
-      </visual>
-      <collision>
-        <origin xyz="0 0 0" rpy="0 0 0"/>
-        <geometry>
-          <mesh filename="package://alfa_robot_description/meshes/alfa_robot/collision/turn.STL"/>
-        </geometry>
-      </collision>
-    </link>
-    <!-- updown (link name differs from joint for GZ compatibility) -->
-    <link name="${prefix}updown_link">
-      <inertial>
-        <origin xyz="-0.196828632659582 0.0148673483555221 0.0956849238503419" rpy="0 0 0"/>
-        <mass value="26.931167747836"/>
-        <inertia ixx="0.231217459750122" ixy="2.93337887014215E-05" ixz="0.000951254936009737" iyy="0.178754005132662" iyz="-1.44830456938328E-05" izz="0.348822965146485"/>
-      </inertial>
-      <visual>
-        <origin xyz="0 0 0" rpy="0 0 0"/>
-        <geometry>
-          <mesh filename="package://alfa_robot_description/meshes/alfa_robot/visual/updown.STL"/>
-        </geometry>
-        <material name="arm_grey"/>
-      </visual>
-      <collision>
-        <origin xyz="0 0 0" rpy="0 0 0"/>
-        <geometry>
-          <mesh filename="package://alfa_robot_description/meshes/alfa_robot/collision/updown.STL"/>
-        </geometry>
-      </collision>
-    </link>
-    <!-- plate (new link) -->
-    <link name="${prefix}plate_link">
-      <inertial>
-        <origin xyz="0.0698918884158706 7.79931674799172E-15 -0.0265000000000004" rpy="0 0 0"/>
-        <mass value="5.63390000000005"/>
-        <inertia ixx="0.0596659645833342" ixy="-9.2486172257981E-16" ixz="-5.64097728970053E-17" iyy="0.0554411298589926" iyz="-2.02970605311345E-14" izz="0.112469490258993"/>
-      </inertial>
-      <visual>
-        <origin xyz="0 0 0" rpy="0 0 0"/>
-        <geometry>
-          <mesh filename="package://alfa_robot_description/meshes/alfa_robot/visual/plate.STL"/>
-        </geometry>
-        <material name="white"/>
-      </visual>
-      <collision>
-        <origin xyz="0 0 0" rpy="0 0 0"/>
-        <geometry>
-          <mesh filename="package://alfa_robot_description/meshes/alfa_robot/collision/plate.STL"/>
-        </geometry>
-      </collision>
-    </link>
-    <!-- rightjoint1 -->
-    <link name="${prefix}rightjoint1_link">
-      <inertial>
-        <origin xyz="0.32398542150288 -0.0675146775051429 -0.0136862113102643" rpy="0 0 0"/>
-        <mass value="2.48077826581444"/>
-        <inertia ixx="0.0026348787049079" ixy="2.78509690352211E-07" ixz="2.27753599606112E-06" iyy="0.0378277422884527" iyz="-3.74055166687532E-05" izz="0.0384178105950815"/>
-      </inertial>
-      <visual>
-        <origin xyz="0 0 0" rpy="0 0 0"/>
-        <geometry>
-          <mesh filename="package://alfa_robot_description/meshes/alfa_robot/visual/rightjoint1.STL"/>
-        </geometry>
-        <material name="white"/>
-      </visual>
-      <collision>
-        <origin xyz="0 0 0" rpy="0 0 0"/>
-        <geometry>
-          <mesh filename="package://alfa_robot_description/meshes/alfa_robot/collision/rightjoint1.STL"/>
-        </geometry>
-      </collision>
-    </link>
-    <!-- rightjoint2 -->
-    <link name="${prefix}rightjoint2_link">
-      <inertial>
-        <origin xyz="0.00998125570987396 0.0501508012211525 0.0836125943851177" rpy="0 0 0"/>
-        <mass value="0.924094586385747"/>
-        <inertia ixx="0.00138886172299487" ixy="9.60798584640597E-07" ixz="-2.47998998359295E-07" iyy="0.00126018297864274" iyz="-6.56045281312999E-07" izz="0.0014853923148985"/>
-      </inertial>
-      <visual>
-        <origin xyz="0 0 0" rpy="0 0 0"/>
-        <geometry>
-          <mesh filename="package://alfa_robot_description/meshes/alfa_robot/visual/rightjoint2.STL"/>
-        </geometry>
-        <material name="white"/>
-      </visual>
-      <collision>
-        <origin xyz="0 0 0" rpy="0 0 0"/>
-        <geometry>
-          <mesh filename="package://alfa_robot_description/meshes/alfa_robot/collision/rightjoint2.STL"/>
-        </geometry>
-      </collision>
-    </link>
-    <!-- rightjoint3 -->
-    <link name="${prefix}rightjoint3_link">
-      <inertial>
-        <origin xyz="0.225299625739963 -1.60107813145238E-05 -0.0720438220450934" rpy="0 0 0"/>
-        <mass value="1.34400405454488"/>
-        <inertia ixx="0.00147896138599604" ixy="-1.09234424169219E-06" ixz="-3.74484328782169E-07" iyy="0.0027517588466101" iyz="1.75900999614053E-08" izz="0.00279083369334524"/>
-      </inertial>
-      <visual>
-        <origin xyz="0 0 0" rpy="0 0 0"/>
-        <geometry>
-          <mesh filename="package://alfa_robot_description/meshes/alfa_robot/visual/rightjoint3.STL"/>
-        </geometry>
-        <material name="white"/>
-      </visual>
-      <collision>
-        <origin xyz="0 0 0" rpy="0 0 0"/>
-        <geometry>
-          <mesh filename="package://alfa_robot_description/meshes/alfa_robot/collision/rightjoint3.STL"/>
-        </geometry>
-      </collision>
-    </link>
-    <!-- rightjoint4 -->
-    <link name="${prefix}rightjoint4_link">
-      <inertial>
-        <origin xyz="0.0100204605383918 0.00985679814963347 0.0840089075623952" rpy="0 0 0"/>
-        <mass value="0.983457322359293"/>
-        <inertia ixx="0.00146324457982104" ixy="1.07921279553368E-06" ixz="2.05978166819893E-07" iyy="0.00136637778648993" iyz="3.51454994521712E-07" izz="0.00151815899256312"/>
-      </inertial>
-      <visual>
-        <origin xyz="0 0 0" rpy="0 0 0"/>
-        <geometry>
-          <mesh filename="package://alfa_robot_description/meshes/alfa_robot/visual/rightjoint4.STL"/>
-        </geometry>
-        <material name="white"/>
-      </visual>
-      <collision>
-        <origin xyz="0 0 0" rpy="0 0 0"/>
-        <geometry>
-          <mesh filename="package://alfa_robot_description/meshes/alfa_robot/collision/rightjoint4.STL"/>
-        </geometry>
-      </collision>
-    </link>
-    <!-- rightjoint5 (new link for 6DOF, Y-axis mirror of leftjoint5) -->
-    <link name="${prefix}rightjoint5_link">
-      <inertial>
-        <origin xyz="0.0101785346040691 -9.30231893336853E-06 0.114866949892092" rpy="0 0 0"/>
-        <mass value="1.05113789872684"/>
-        <inertia ixx="0.00202470522047338" ixy="-1.84484199834478E-08" ixz="-0.000306186752830273" iyy="0.00328579639703018" iyz="-7.17708515637608E-10" izz="0.00340020564373822"/>
-      </inertial>
-      <visual>
-        <origin xyz="0 0 0" rpy="0 0 0"/>
-        <geometry>
-          <mesh filename="package://alfa_robot_description/meshes/alfa_robot/visual/rightjoint5.STL"/>
-        </geometry>
-        <material name="white"/>
-      </visual>
-      <collision>
-        <origin xyz="0 0 0" rpy="0 0 0"/>
-        <geometry>
-          <mesh filename="package://alfa_robot_description/meshes/alfa_robot/collision/rightjoint5.STL"/>
-        </geometry>
-      </collision>
-    </link>
-    <!-- rightjoint6 (new link for end effector extension, Y-axis mirror of leftjoint6) -->
-    <link name="${prefix}rightjoint6_link">
-      <inertial>
-        <origin xyz="0.0338349899428319 -2.18158824338843E-14 1.47522838389591E-09" rpy="0 0 0"/>
-        <mass value="0.763196071605449"/>
-        <inertia ixx="0.00324062849151741" ixy="-6.82020341217245E-19" ixz="-3.87057635370163E-16" iyy="0.0019198659327465" iyz="1.80691312979497E-18" izz="0.00150433027221572"/>
-      </inertial>
-      <visual>
-        <origin xyz="0 0 0" rpy="0 0 0"/>
-        <geometry>
-          <mesh filename="package://alfa_robot_description/meshes/alfa_robot/visual/rightjoint6.STL"/>
-        </geometry>
-        <material name="blue"/>
-      </visual>
-      <collision>
-        <origin xyz="0 0 0" rpy="0 0 0"/>
-        <geometry>
-          <mesh filename="package://alfa_robot_description/meshes/alfa_robot/collision/rightjoint6.STL"/>
-        </geometry>
-      </collision>
-    </link>
-    <!-- leftjoint1 -->
-    <link name="${prefix}leftjoint1_link">
-      <inertial>
-        <origin xyz="0.32398542150288 0.0675146775051429 -0.0136862113102643" rpy="0 0 0"/>
-        <mass value="2.48077826581444"/>
-        <inertia ixx="0.0026348787049079" ixy="-2.78509690352211E-07" ixz="2.27753599606112E-06" iyy="0.0378277422884527" iyz="3.74055166687532E-05" izz="0.0384178105950815"/>
-      </inertial>
-      <visual>
-        <origin xyz="0 0 0" rpy="0 0 0"/>
-        <geometry>
-          <mesh filename="package://alfa_robot_description/meshes/alfa_robot/visual/leftjoint1.STL"/>
-        </geometry>
-        <material name="white"/>
-      </visual>
-      <collision>
-        <origin xyz="0 0 0" rpy="0 0 0"/>
-        <geometry>
-          <mesh filename="package://alfa_robot_description/meshes/alfa_robot/collision/leftjoint1.STL"/>
-        </geometry>
-      </collision>
-    </link>
-    <!-- rightjoint2 (link name differs from joint for GZ compatibility) -->
-    <link name="${prefix}leftjoint2_link">
-      <inertial>
-        <origin xyz="0.00998125570987396 -0.0501508012211525 0.0836125943851177" rpy="0 0 0"/>
-        <mass value="0.924094586385747"/>
-        <inertia ixx="0.00138886172299487" ixy="-9.60798584640597E-07" ixz="-2.47998998359295E-07" iyy="0.00126018297864274" iyz="6.56045281312999E-07" izz="0.0014853923148985"/>
-      </inertial>
-      <visual>
-        <origin xyz="0 0 0" rpy="0 0 0"/>
-        <geometry>
-          <mesh filename="package://alfa_robot_description/meshes/alfa_robot/visual/leftjoint2.STL"/>
-        </geometry>
-        <material name="white"/>
-      </visual>
-      <collision>
-        <origin xyz="0 0 0" rpy="0 0 0"/>
-        <geometry>
-          <mesh filename="package://alfa_robot_description/meshes/alfa_robot/collision/leftjoint2.STL"/>
-        </geometry>
-      </collision>
-    </link>
-    <!-- rightjoint3 (link name differs from joint for GZ compatibility) -->
-    <link name="${prefix}leftjoint3_link">
-      <inertial>
-        <origin xyz="0.225299625739963 1.60107813145238E-05 -0.0720438220450934" rpy="0 0 0"/>
-        <mass value="1.34400405454488"/>
-        <inertia ixx="0.00147896138599604" ixy="1.09234424169219E-06" ixz="-3.74484328782169E-07" iyy="0.0027517586466101" iyz="-1.75900999614053E-08" izz="0.00279083369334524"/>
-      </inertial>
-      <visual>
-        <origin xyz="0 0 0" rpy="0 0 0"/>
-        <geometry>
-          <mesh filename="package://alfa_robot_description/meshes/alfa_robot/visual/leftjoint3.STL"/>
-        </geometry>
-        <material name="white"/>
-      </visual>
-      <collision>
-        <origin xyz="0 0 0" rpy="0 0 0"/>
-        <geometry>
-          <mesh filename="package://alfa_robot_description/meshes/alfa_robot/collision/leftjoint3.STL"/>
-        </geometry>
-      </collision>
-    </link>
-    <!-- rightjoint4 (link name differs from joint for GZ compatibility) -->
-    <link name="${prefix}leftjoint4_link">
-      <inertial>
-        <origin xyz="0.0100204605383918 -0.00985679814963347 0.0840089075623952" rpy="0 0 0"/>
-        <mass value="0.983457322359293"/>
-        <inertia ixx="0.00146324457982104" ixy="-1.07921279553368E-06" ixz="2.05978166819893E-07" iyy="0.00136637778648993" iyz="-3.51454994521712E-07" izz="0.00151815899256312"/>
-      </inertial>
-      <visual>
-        <origin xyz="0 0 0" rpy="0 0 0"/>
-        <geometry>
-          <mesh filename="package://alfa_robot_description/meshes/alfa_robot/visual/leftjoint4.STL"/>
-        </geometry>
-        <material name="white"/>
-      </visual>
-      <collision>
-        <origin xyz="0 0 0" rpy="0 0 0"/>
-        <geometry>
-          <mesh filename="package://alfa_robot_description/meshes/alfa_robot/collision/leftjoint4.STL"/>
-        </geometry>
-      </collision>
-    </link>
-    <!-- leftjoint5 (new link for 6DOF) -->
-    <link name="${prefix}leftjoint5_link">
-      <inertial>
-        <origin xyz="0.0101785346040691 9.30231893336853E-06 0.114866949892092" rpy="0 0 0"/>
-        <mass value="1.05113789872684"/>
-        <inertia ixx="0.00202470522047338" ixy="1.84484199834478E-08" ixz="-0.000306186752830273" iyy="0.00328579639703018" iyz="7.17708515637608E-10" izz="0.00340020564373822"/>
-      </inertial>
-      <visual>
-        <origin xyz="0 0 0" rpy="0 0 0"/>
-        <geometry>
-          <mesh filename="package://alfa_robot_description/meshes/alfa_robot/visual/leftjoint5.STL"/>
-        </geometry>
-        <material name="white"/>
-      </visual>
-      <collision>
-        <origin xyz="0 0 0" rpy="0 0 0"/>
-        <geometry>
-          <mesh filename="package://alfa_robot_description/meshes/alfa_robot/collision/leftjoint5.STL"/>
-        </geometry>
-      </collision>
-    </link>
-    <!-- leftjoint6 (new link for end effector extension) -->
-    <link name="${prefix}leftjoint6_link">
-      <inertial>
-        <origin xyz="0.0338349899428319 2.18158824338843E-14 1.47522838389591E-09" rpy="0 0 0"/>
-        <mass value="0.763196071605449"/>
-        <inertia ixx="0.00324062849151741" ixy="6.82020341217245E-19" ixz="-3.87057635370163E-16" iyy="0.0019198659327465" iyz="-1.80691312979497E-18" izz="0.00150433027221572"/>
-      </inertial>
-      <visual>
-        <origin xyz="0 0 0" rpy="0 0 0"/>
-        <geometry>
-          <mesh filename="package://alfa_robot_description/meshes/alfa_robot/visual/leftjoint6.STL"/>
-        </geometry>
-        <material name="blue"/>
-      </visual>
-      <collision>
-        <origin xyz="0 0 0" rpy="0 0 0"/>
-        <geometry>
-          <mesh filename="package://alfa_robot_description/meshes/alfa_robot/collision/leftjoint6.STL"/>
-        </geometry>
-      </collision>
-    </link>
-    <!-- camera -->
-    <link name="${prefix}camera_link">
-      <inertial>
-        <origin xyz="-0.0129500032830805 3.27763982552187E-08 8.59781135176263E-10" rpy="0 0 0"/>
-        <mass value="0.0884229444440941"/>
-        <inertia ixx="0.000108966100127413" ixy="4.24530017226163E-12" ixz="1.30809093461559E-12" iyy="1.08349581479197E-05" iyz="1.58450016026868E-10" izz="0.000108016955483713"/>
-      </inertial>
-      <visual>
-        <origin xyz="0 0 0" rpy="0 0 0"/>
-        <geometry>
-          <mesh filename="package://alfa_robot_description/meshes/alfa_robot/visual/camera.STL"/>
-        </geometry>
-        <material name="white"/>
-      </visual>
-      <collision>
-        <origin xyz="0 0 0" rpy="0 0 0"/>
-        <geometry>
-          <mesh filename="package://alfa_robot_description/meshes/alfa_robot/collision/camera.STL"/>
-        </geometry>
-      </collision>
-    </link>
-    <!-- lidar -->
-    <link name="${prefix}lidar_link">
-      <inertial>
-        <origin xyz="-0.000765897194240361 5.34294830600857E-16 -0.00285836724227106" rpy="0 0 0"/>
-        <mass value="0.296061195729235"/>
-        <inertia ixx="0.000229195879552691" ixy="-5.34979264059518E-18" ixz="-7.69967406090194E-06" iyy="0.000231259000999259" iyz="8.30310887470795E-18" izz="0.000202523426202246"/>
-      </inertial>
-      <visual>
-        <origin xyz="0 0 0" rpy="0 0 0"/>
-        <geometry>
-          <mesh filename="package://alfa_robot_description/meshes/alfa_robot/visual/lidar.STL"/>
-        </geometry>
-        <material name="arm_grey"/>
-      </visual>
-      <collision>
-        <origin xyz="0 0 0" rpy="0 0 0"/>
-        <geometry>
-          <mesh filename="package://alfa_robot_description/meshes/alfa_robot/collision/lidar.STL"/>
-        </geometry>
-      </collision>
-    </link>
-    <!-- right_ee_link (virtual end effector for MoveIt2 planning) -->
-    <link name="${prefix}right_ee_link"/>
-    <!-- left_ee_link (virtual end effector for MoveIt2 planning) -->
-    <link name="${prefix}left_ee_link"/>
-    <!-- END LINKS -->
-    <!-- JOINTS -->
-    <!-- base_joint fixes base_link to the environment -->
+<link
+    name="${prefix}base_link">
+    <inertial>
+      <origin
+        xyz="-0.00896922200126715 2.35194162193642E-05 0.0179811176086975"
+        rpy="0 0 0" />
+      <mass
+        value="5.21106238092598" />
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