Commit message: feat: v4_dev 分支初始化 — 新增 v2_arm_v4 机械臂模型 + 全链路适配
- 新增 alfa_robot_v2_arm_v4 meshes (collision + visual STL)
- 新增 v2_arm_v4_joint_limits.md 关节限位文档
- URDF xacro 适配 v4 关节结构 (pitch 关节)
- SRDF/joint_limits/ros2_control/controllers 适配 v4 关节配置
- dual_arm_planner/end_effector scripts 适配 v4 末端链接名
- bringup scripts/controllers 适配 v4 关节列表
- ik_solver 适配 v4 关节定义
- MuJoCo 仿真场景适配 v4 模型

Co-Authored-By: Claude Opus 4.7 <noreply@anthropic.com>

File: ros2_ws/src/alfa_robot_description/urdf/alfa_robot.urdf.xacro (robot description, xacro)
@@ -1,5 +1,4 @@
 <?xml version="1.0" encoding="UTF-8"?>
 <robot xmlns:xacro="http://wiki.ros.org/xacro" name="alfa_robot">
-  <!-- Use this if parameters are set from the launch file, otherwise delete -->
   <xacro:arg name="prefix" default=""/>
   <xacro:arg name="use_mock_hardware" default="true"/>
@@ -11,13 +10,876 @@
   <xacro:arg name="canopen_profile_velocity" default="50000"/>
   <xacro:arg name="canopen_profile_accel" default="50000"/>
-  <xacro:include filename="$(find alfa_robot_description)/urdf/alfa_robot/alfa_robot_macro.xacro"/>
   <xacro:include filename="$(find alfa_robot_description)/urdf/alfa_robot/alfa_robot_macro.ros2_control.xacro"/>
-  <!-- create link fixed to the "world" -->
   <link name="world"/>
-  <!-- Load robot's macro with parameters -->
-  <!-- set prefix if multiple robots are used -->
-  <xacro:alfa_robot prefix="$(arg prefix)" parent="world">
-    <origin xyz="0 0 0.09" rpy="0 0 0"/>          <!-- position robot in the world -->
-  </xacro:alfa_robot>
+  <joint name="world_to_base" type="fixed">
+    <parent link="world"/>
+    <child link="base_link"/>
+    <origin xyz="0 0 0.09" rpy="0 0 0"/>
+  </joint>
+  <link
+    name="base_link">
+    <inertial>
+      <origin
+        xyz="-0.00896922200126715 2.35194162190866E-05 0.0179811176086973"
+        rpy="0 0 0" />
+      <mass
+        value="5.21106238092599" />
+      <inertia
+        ixx="0.0633320335254252"
+        ixy="-1.57025952751864E-07"
+        ixz="-3.66796372428847E-07"
+        iyy="0.119212913285128"
+        iyz="6.3371451899133E-07"
+        izz="0.181818429904202" />
+    </inertial>
+    <visual>
+      <origin
+        xyz="0 0 0"
+        rpy="0 0 0" />
+      <geometry>
+        <mesh
+          filename="package://alfa_robot_description/meshes/alfa_robot_v2_arm_v4/visual/base_link.STL" />
+      </geometry>
+      <material
+        name="">
+        <color
+          rgba="1 1 1 1" />
+      </material>
+    </visual>
+    <collision>
+      <origin
+        xyz="0 0 0"
+        rpy="0 0 0" />
+      <geometry>
+        <mesh
+          filename="package://alfa_robot_description/meshes/alfa_robot_v2_arm_v4/collision/base_link.STL" />
+      </geometry>
+    </collision>
+  </link>
+  <link
+    name="pitch">
+    <inertial>
+      <origin
+        xyz="-0.198797876667389 0.0534826037691441 0.0683908156328275"
+        rpy="0 0 0" />
+      <mass
+        value="5.23479125794249" />
+      <inertia
+        ixx="0.0820011779740888"
+        ixy="1.65869971517116E-10"
+        ixz="-8.67361737988404E-18"
+        iyy="0.0820529172807708"
+        iyz="-2.22972698372151E-17"
+        izz="0.163475256832643" />
+    </inertial>
+    <visual>
+      <origin
+        xyz="0 0 0"
+        rpy="0 0 0" />
+      <geometry>
+        <mesh
+          filename="package://alfa_robot_description/meshes/alfa_robot_v2_arm_v4/visual/pitch.STL" />
+      </geometry>
+      <material
+        name="">
+        <color
+          rgba="1 1 1 1" />
+      </material>
+    </visual>
+    <collision>
+      <origin
+        xyz="0 0 0"
+        rpy="0 0 0" />
+      <geometry>
+        <mesh
+          filename="package://alfa_robot_description/meshes/alfa_robot_v2_arm_v4/collision/pitch.STL" />
+      </geometry>
+    </collision>
+  </link>
+  <joint
+    name="pitch"
+    type="revolute">
+    <origin
+      xyz="0.259 -0.0545 0.05"
+      rpy="0 0 0" />
+    <parent
+      link="base_link" />
+    <child
+      link="pitch" />
+    <axis
+      xyz="0 1 0" />
+    <limit
+      lower="0"
+      upper="0.26"
+      effort="0"
+      velocity="0" />
+  </joint>
+  <link
+    name="turn">
+    <inertial>
+      <origin
+        xyz="-0.0279588381716878 3.16554382575607E-05 0.819951711254512"
+        rpy="0 0 0" />
+      <mass
+        value="15.206613319806" />
+      <inertia
+        ixx="1.06710751132169"
+        ixy="5.33982003477675E-06"
+        ixz="0.000444527933425326"
+        iyy="1.0606566000007"
+        iyz="1.02603827456618E-05"
+        izz="0.109926667915607" />
+    </inertial>
+    <visual>
+      <origin
+        xyz="0 0 0"
+        rpy="0 0 0" />
+      <geometry>
+        <mesh
+          filename="package://alfa_robot_description/meshes/alfa_robot_v2_arm_v4/visual/turn.STL" />
+      </geometry>
+      <material
+        name="">
+        <color
+          rgba="1 1 1 1" />
+      </material>
+    </visual>
+    <collision>
+      <origin
+        xyz="0 0 0"
+        rpy="0 0 0" />
+      <geometry>
+        <mesh
+          filename="package://alfa_robot_description/meshes/alfa_robot_v2_arm_v4/collision/turn.STL" />
+      </geometry>
+    </collision>
+  </link>
+  <joint
+    name="turn"
+    type="continuous">
+    <origin
+      xyz="-0.209 0.0545 0.09"
+      rpy="0 0 0" />
+    <parent
+      link="pitch" />
+    <child
+      link="turn" />
+    <axis
+      xyz="0 0 1" />
+  </joint>
+  <link
+    name="updown">
+    <inertial>
+      <origin
+        xyz="0.0212260464062497 -2.11666036081248E-05 0.111174833214802"
+        rpy="0 0 0" />
+      <mass
+        value="8.56370936608539" />
+      <inertia
+        ixx="0.0416436910061337"
+        ixy="-3.48368286367816E-07"
+        ixz="1.03580901428956E-05"
+        iyy="0.151229514328064"
+        iyz="1.21565801733102E-06"
+        izz="0.186025474756556" />
+    </inertial>
+    <visual>
+      <origin
+        xyz="0 0 0"
+        rpy="0 0 0" />
+      <geometry>
+        <mesh
+          filename="package://alfa_robot_description/meshes/alfa_robot_v2_arm_v4/visual/updown.STL" />
+      </geometry>
+      <material
+        name="">
+        <color
+          rgba="1 1 1 1" />
+      </material>
+    </visual>
+    <collision>
+      <origin
+        xyz="0 0 0"
+        rpy="0 0 0" />
+      <geometry>
+        <mesh
+          filename="package://alfa_robot_description/meshes/alfa_robot_v2_arm_v4/collision/updown.STL" />
+      </geometry>
+    </collision>
+  </link>
+  <joint
+    name="updown"
+    type="prismatic">
+    <origin
+      xyz="-0.1 0 0.086"
+      rpy="0 0 0" />
+    <parent
+      link="turn" />
+    <child
+      link="updown" />
+    <axis
+      xyz="0 0 1" />
+    <limit
+      lower="0"
+      upper="0.99"
+      effort="0"
+      velocity="0" />
+  </joint>
+  <link
+    name="leftjoint1">
+    <inertial>
+      <origin
+        xyz="0.319517252158916 -0.00430688057663203 0.029804284492444"
+        rpy="0 0 0" />
+      <mass
+        value="3.32143363177723" />
+      <inertia
+        ixx="0.00335784257897387"
+        ixy="3.85497637875902E-05"
+        ixz="-0.000223384608442736"
+        iyy="0.0875447243413311"
+        iyz="-8.33307395117058E-05"
+        izz="0.0873944733459465" />
+    </inertial>
+    <visual>
+      <origin
+        xyz="0 0 0"
+        rpy="0 0 0" />
+      <geometry>
+        <mesh
+          filename="package://alfa_robot_description/meshes/alfa_robot_v2_arm_v4/visual/leftjoint1.STL" />
+      </geometry>
+      <material
+        name="">
+        <color
+          rgba="1 1 1 1" />
+      </material>
+    </visual>
+    <collision>
+      <origin
+        xyz="0 0 0"
+        rpy="0 0 0" />
+      <geometry>
+        <mesh
+          filename="package://alfa_robot_description/meshes/alfa_robot_v2_arm_v4/collision/leftjoint1.STL" />
+      </geometry>
+    </collision>
+  </link>
+  <joint
+    name="leftjoint1"
+    type="prismatic">
+    <origin
+      xyz="-0.285799999999983 0.269999999999219 0.184500000000939"
+      rpy="0 0 0" />
+    <parent
+      link="updown" />
+    <child
+      link="leftjoint1" />
+    <axis
+      xyz="1 0 0" />
+    <limit
+      lower="0"
+      upper="0.3"
+      effort="0"
+      velocity="0" />
+  </joint>
+  <link
+    name="leftjoint2">
+    <inertial>
+      <origin
+        xyz="1.86514639244351E-05 0.00549008734545911 0.0483192697870322"
+        rpy="0 0 0" />
+      <mass
+        value="1.1434754221004" />
+      <inertia
+        ixx="0.0024543741369995"
+        ixy="1.89450558125154E-06"
+        ixz="-2.45980294088456E-06"
+        iyy="0.00234579099555691"
+        iyz="-7.07026940240241E-05"
+        izz="0.00212775377469202" />
+    </inertial>
+    <visual>
+      <origin
+        xyz="0 0 0"
+        rpy="0 0 0" />
+      <geometry>
+        <mesh
+          filename="package://alfa_robot_description/meshes/alfa_robot_v2_arm_v4/visual/leftjoint2.STL" />
+      </geometry>
+      <material
+        name="">
+        <color
+          rgba="1 1 1 1" />
+      </material>
+    </visual>
+    <collision>
+      <origin
+        xyz="0 0 0"
+        rpy="0 0 0" />
+      <geometry>
+        <mesh
+          filename="package://alfa_robot_description/meshes/alfa_robot_v2_arm_v4/collision/leftjoint2.STL" />
+      </geometry>
+    </collision>
+  </link>
+  <joint
+    name="leftjoint2"
+    type="continuous">
+    <origin
+      xyz="0.716 0 0.1705"
+      rpy="-1.5708 1.5662 -1.5708" />
+    <parent
+      link="leftjoint1" />
+    <child
+      link="leftjoint2" />
+    <axis
+      xyz="0 0 1" />
+  </joint>
+  <link
+    name="leftjoint3">
+    <inertial>
+      <origin
+        xyz="0.0708924301709254 -2.86407864964477E-05 0.0516803522991347"
+        rpy="0 0 0" />
+      <mass
+        value="1.75163255810635" />
+      <inertia
+        ixx="0.00386552461884797"
+        ixy="-1.39559114197398E-06"
+        ixz="-7.06884843737482E-05"
+        iyy="0.00631255855610293"
+        iyz="2.78557081715933E-06"
+        izz="0.00598591407871913" />
+    </inertial>
+    <visual>
+      <origin
+        xyz="0 0 0"
+        rpy="0 0 0" />
+      <geometry>
+        <mesh
+          filename="package://alfa_robot_description/meshes/alfa_robot_v2_arm_v4/visual/leftjoint3.STL" />
+      </geometry>
+      <material
+        name="">
+        <color
+          rgba="1 1 1 1" />
+      </material>
+    </visual>
+    <collision>
+      <origin
+        xyz="0 0 0"
+        rpy="0 0 0" />
+      <geometry>
+        <mesh
+          filename="package://alfa_robot_description/meshes/alfa_robot_v2_arm_v4/collision/leftjoint3.STL" />
+      </geometry>
+    </collision>
+  </link>
+  <joint
+    name="leftjoint3"
+    type="continuous">
+    <origin
+      xyz="-0.00035108 0.075999 0.058"
+      rpy="-1.5754 -1.5708 0" />
+    <parent
+      link="leftjoint2" />
+    <child
+      link="leftjoint3" />
+    <axis
+      xyz="0 0 1" />
+  </joint>
+  <link
+    name="leftjoint4">
+    <inertial>
+      <origin
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
File: ros2_ws/src/alfa_robot_description/urdf/alfa_robot/alfa_robot_macro.ros2_control.xacro (robot description, xacro)
@@ -51,13 +51,21 @@
           <param name="safe_position_rightjoint5">0.0</param>
           <param name="safe_position_rightjoint6">0.0</param>
-          <param name="safe_position_plate">0.0</param>
         </xacro:unless>
       </hardware>
+      <!-- pitch (revolute) -->
+      <joint name="${prefix}pitch">
+        <command_interface name="position">
+          <param name="min">0</param>
+          <param name="max">0.26</param>
+        </command_interface>
+        <state_interface name="position">
+          <param name="initial_value">0.0</param>
+        </state_interface>
+        <state_interface name="velocity"/>
+        <state_interface name="acceleration"/>
+      </joint>
       <!-- turn (continuous) -->
       <joint name="${prefix}turn">
-        <command_interface name="position">
-          <param name="min">-3.14159</param>
-          <param name="max">3.14159</param>
-        </command_interface>
+        <command_interface name="position"/>
         <state_interface name="position">
           <param name="initial_value">0.0</param>
@@ -70,17 +78,5 @@
         <command_interface name="position">
           <param name="min">0</param>
-          <param name="max">1.0</param>
-        </command_interface>
-        <state_interface name="position">
-          <param name="initial_value">0.0</param>
-        </state_interface>
-        <state_interface name="velocity"/>
-        <state_interface name="acceleration"/>
-      </joint>
-      <!-- plate (prismatic, new) -->
-      <joint name="${prefix}plate">
-        <command_interface name="position">
-          <param name="min">0</param>
-          <param name="max">0.5</param>
+          <param name="max">0.99</param>
         </command_interface>
         <state_interface name="position">
@@ -94,5 +90,5 @@
         <command_interface name="position">
           <param name="min">0</param>
-          <param name="max">0.42</param>
+          <param name="max">0.3</param>
         </command_interface>
         <state_interface name="position">
@@ -104,8 +100,5 @@
       <!-- rightjoint2 (continuous) -->
       <joint name="${prefix}rightjoint2">
-        <command_interface name="position">
-          <param name="min">-3.14159</param>
-          <param name="max">3.14159</param>
-        </command_interface>
+        <command_interface name="position"/>
         <state_interface name="position">
           <param name="initial_value">0.0</param>
@@ -116,8 +109,5 @@
       <!-- rightjoint3 (continuous) -->
       <joint name="${prefix}rightjoint3">
-        <command_interface name="position">
-          <param name="min">-3.14159</param>
-          <param name="max">3.14159</param>
-        </command_interface>
+        <command_interface name="position"/>
         <state_interface name="position">
           <param name="initial_value">0.0</param>
@@ -128,8 +118,5 @@
       <!-- rightjoint4 (continuous) -->
       <joint name="${prefix}rightjoint4">
-        <command_interface name="position">
-          <param name="min">-3.14159</param>
-          <param name="max">3.14159</param>
-        </command_interface>
+        <command_interface name="position"/>
         <state_interface name="position">
           <param name="initial_value">0.0</param>
@@ -140,8 +127,5 @@
       <!-- rightjoint5 (continuous) -->
       <joint name="${prefix}rightjoint5">
-        <command_interface name="position">
-          <param name="min">-3.14159</param>
-          <param name="max">3.14159</param>
-        </command_interface>
+        <command_interface name="position"/>
         <state_interface name="position">
           <param name="initial_value">0.0</param>
@@ -166,5 +150,5 @@
         <command_interface name="position">
           <param name="min">0</param>
-          <param name="max">0.42</param>
+          <param name="max">0.3</param>
         </command_interface>
         <state_interface name="position">
@@ -176,8 +160,5 @@
       <!-- leftjoint2 (continuous) -->
       <joint name="${prefix}leftjoint2">
-        <command_interface name="position">
-          <param name="min">-3.14159</param>
-          <param name="max">3.14159</param>
-        </command_interface>
+        <command_interface name="position"/>
         <state_interface name="position">
           <param name="initial_value">0.0</param>
@@ -188,8 +169,5 @@
       <!-- leftjoint3 (continuous) -->
       <joint name="${prefix}leftjoint3">
-        <command_interface name="position">
-          <param name="min">-3.14159</param>
-          <param name="max">3.14159</param>
-        </command_interface>
+        <command_interface name="position"/>
         <state_interface name="position">
           <param name="initial_value">0.0</param>
@@ -200,8 +178,5 @@
       <!-- leftjoint4 (continuous) -->
       <joint name="${prefix}leftjoint4">
-        <command_interface name="position">
-          <param name="min">-3.14159</param>
-          <param name="max">3.14159</param>
-        </command_interface>
+        <command_interface name="position"/>
         <state_interface name="position">
           <param name="initial_value">0.0</param>
@@ -212,8 +187,5 @@
       <!-- leftjoint5 (continuous) -->
       <joint name="${prefix}leftjoint5">
-        <command_interface name="position">
-          <param name="min">-3.14159</param>
-          <param name="max">3.14159</param>
-        </command_interface>
+        <command_interface name="position"/>
         <state_interface name="position">
           <param name="initial_value">0.0</param>

File: ros2_ws/src/alfa_robot_moveit_config/config/alfa_robot.ros2_control.xacro (robot description, xacro)
@@ -8,4 +8,10 @@
                 <plugin>mock_components/GenericSystem</plugin>
             </hardware>
+            <joint name="pitch">
+                <command_interface name="position"/>
+                <state_interface name="position">
+                  <param name="initial_value">${initial_positions['pitch']}</param>
+                </state_interface>
+            </joint>
             <joint name="turn">
                 <command_interface name="position"/>
