Commit message: feat: v2_arm_v4_new 机械臂模型更新 + MoveIt/MuJoCo 配置适配
- 新增 alfa_robot_v2_arm_v4_new meshes（collision + visual STL）
- URDF xacro 更新适配新关节布局
- ros2_control 宏更新对应新关节
- MoveIt: SRDF / kinematics / controllers 配置调整
- MuJoCo alfa_robot.xml 模型同步更新
- debug_mesh_path.py 调试脚本更新
- joint_limits 文档更新

Co-Authored-By: Claude Opus 4.7 <noreply@anthropic.com>

File: ros2_ws/src/alfa_robot_description/urdf/alfa_robot.urdf.xacro (robot description, xacro)
@@ -21,14 +21,14 @@
     <inertial>
       <origin
-        xyz="-0.00896922200126715 2.35194162190866E-05 0.0179811176086973"
-        rpy="0 0 0" />
-      <mass
-        value="5.21106238092599" />
+        xyz="-0.00896922200126715 2.35194162193642E-05 0.0179811176086975"
+        rpy="0 0 0" />
+      <mass
+        value="5.21106238092598" />
       <inertia
         ixx="0.0633320335254252"
-        ixy="-1.57025952751864E-07"
-        ixz="-3.66796372428847E-07"
+        ixy="-1.57025952749484E-07"
+        ixz="-3.66796372424077E-07"
         iyy="0.119212913285128"
-        iyz="6.3371451899133E-07"
+        iyz="6.33714518991059E-07"
         izz="0.181818429904202" />
     </inertial>
@@ -39,19 +39,19 @@
       <geometry>
         <mesh
-          filename="package://alfa_robot_description/meshes/alfa_robot_v2_arm_v4/visual/base_link.STL" />
-      </geometry>
-      <material
-        name="">
-        <color
-          rgba="1 1 1 1" />
-      </material>
-    </visual>
-    <collision>
-      <origin
-        xyz="0 0 0"
-        rpy="0 0 0" />
-      <geometry>
-        <mesh
-          filename="package://alfa_robot_description/meshes/alfa_robot_v2_arm_v4/collision/base_link.STL" />
+          filename="package://alfa_robot_description/meshes/alfa_robot_v2_arm_v4_new/visual/base_link.STL" />
+      </geometry>
+      <material
+        name="">
+        <color
+          rgba="1 1 1 1" />
+      </material>
+    </visual>
+    <collision>
+      <origin
+        xyz="0 0 0"
+        rpy="0 0 0" />
+      <geometry>
+        <mesh
+          filename="package://alfa_robot_description/meshes/alfa_robot_v2_arm_v4_new/collision/base_link.STL" />
       </geometry>
     </collision>
@@ -67,8 +67,8 @@
       <inertia
         ixx="0.0820011779740888"
-        ixy="1.65869971517116E-10"
-        ixz="-8.67361737988404E-18"
+        ixy="1.65869977323853E-10"
+        ixz="-1.12757025938492E-17"
         iyy="0.0820529172807708"
-        iyz="-2.22972698372151E-17"
+        iyz="-2.38941055572563E-17"
         izz="0.163475256832643" />
     </inertial>
@@ -79,19 +79,19 @@
       <geometry>
         <mesh
-          filename="package://alfa_robot_description/meshes/alfa_robot_v2_arm_v4/visual/pitch.STL" />
-      </geometry>
-      <material
-        name="">
-        <color
-          rgba="1 1 1 1" />
-      </material>
-    </visual>
-    <collision>
-      <origin
-        xyz="0 0 0"
-        rpy="0 0 0" />
-      <geometry>
-        <mesh
-          filename="package://alfa_robot_description/meshes/alfa_robot_v2_arm_v4/collision/pitch.STL" />
+          filename="package://alfa_robot_description/meshes/alfa_robot_v2_arm_v4_new/visual/pitch.STL" />
+      </geometry>
+      <material
+        name="">
+        <color
+          rgba="1 1 1 1" />
+      </material>
+    </visual>
+    <collision>
+      <origin
+        xyz="0 0 0"
+        rpy="0 0 0" />
+      <geometry>
+        <mesh
+          filename="package://alfa_robot_description/meshes/alfa_robot_v2_arm_v4_new/collision/pitch.STL" />
       </geometry>
     </collision>
@@ -125,8 +125,8 @@
       <inertia
         ixx="1.06710751132169"
-        ixy="5.33982003477675E-06"
-        ixz="0.000444527933425326"
+        ixy="5.33982003477265E-06"
+        ixz="0.000444527933425444"
         iyy="1.0606566000007"
-        iyz="1.02603827456618E-05"
+        iyz="1.02603827456492E-05"
         izz="0.109926667915607" />
     </inertial>
@@ -137,19 +137,19 @@
       <geometry>
         <mesh
-          filename="package://alfa_robot_description/meshes/alfa_robot_v2_arm_v4/visual/turn.STL" />
-      </geometry>
-      <material
-        name="">
-        <color
-          rgba="1 1 1 1" />
-      </material>
-    </visual>
-    <collision>
-      <origin
-        xyz="0 0 0"
-        rpy="0 0 0" />
-      <geometry>
-        <mesh
-          filename="package://alfa_robot_description/meshes/alfa_robot_v2_arm_v4/collision/turn.STL" />
+          filename="package://alfa_robot_description/meshes/alfa_robot_v2_arm_v4_new/visual/turn.STL" />
+      </geometry>
+      <material
+        name="">
+        <color
+          rgba="1 1 1 1" />
+      </material>
+    </visual>
+    <collision>
+      <origin
+        xyz="0 0 0"
+        rpy="0 0 0" />
+      <geometry>
+        <mesh
+          filename="package://alfa_robot_description/meshes/alfa_robot_v2_arm_v4_new/collision/turn.STL" />
       </geometry>
     </collision>
@@ -172,37 +172,37 @@
     <inertial>
       <origin
-        xyz="0.0212260464062497 -2.11666036081248E-05 0.111174833214802"
-        rpy="0 0 0" />
-      <mass
-        value="8.56370936608539" />
-      <inertia
-        ixx="0.0416436910061337"
-        ixy="-3.48368286367816E-07"
-        ixz="1.03580901428956E-05"
-        iyy="0.151229514328064"
-        iyz="1.21565801733102E-06"
-        izz="0.186025474756556" />
-    </inertial>
-    <visual>
-      <origin
-        xyz="0 0 0"
-        rpy="0 0 0" />
-      <geometry>
-        <mesh
-          filename="package://alfa_robot_description/meshes/alfa_robot_v2_arm_v4/visual/updown.STL" />
-      </geometry>
-      <material
-        name="">
-        <color
-          rgba="1 1 1 1" />
-      </material>
-    </visual>
-    <collision>
-      <origin
-        xyz="0 0 0"
-        rpy="0 0 0" />
-      <geometry>
-        <mesh
-          filename="package://alfa_robot_description/meshes/alfa_robot_v2_arm_v4/collision/updown.STL" />
+        xyz="0.0212260463112321 -2.11665364142077E-05 0.111174833260946"
+        rpy="0 0 0" />
+      <mass
+        value="8.56370936774335" />
+      <inertia
+        ixx="0.0416436910064672"
+        ixy="-3.48369951311999E-07"
+        ixz="1.03580898385951E-05"
+        iyy="0.151229514406379"
+        iyz="1.21565800186775E-06"
+        izz="0.186025474834666" />
+    </inertial>
+    <visual>
+      <origin
+        xyz="0 0 0"
+        rpy="0 0 0" />
+      <geometry>
+        <mesh
+          filename="package://alfa_robot_description/meshes/alfa_robot_v2_arm_v4_new/visual/updown.STL" />
+      </geometry>
+      <material
+        name="">
+        <color
+          rgba="1 1 1 1" />
+      </material>
+    </visual>
+    <collision>
+      <origin
+        xyz="0 0 0"
+        rpy="0 0 0" />
+      <geometry>
+        <mesh
+          filename="package://alfa_robot_description/meshes/alfa_robot_v2_arm_v4_new/collision/updown.STL" />
       </geometry>
     </collision>
@@ -230,37 +230,37 @@
     <inertial>
       <origin
-        xyz="0.319517252158916 -0.00430688057663203 0.029804284492444"
-        rpy="0 0 0" />
-      <mass
-        value="3.32143363177723" />
-      <inertia
-        ixx="0.00335784257897387"
-        ixy="3.85497637875902E-05"
-        ixz="-0.000223384608442736"
-        iyy="0.0875447243413311"
-        iyz="-8.33307395117058E-05"
-        izz="0.0873944733459465" />
-    </inertial>
-    <visual>
-      <origin
-        xyz="0 0 0"
-        rpy="0 0 0" />
-      <geometry>
-        <mesh
-          filename="package://alfa_robot_description/meshes/alfa_robot_v2_arm_v4/visual/leftjoint1.STL" />
-      </geometry>
-      <material
-        name="">
-        <color
-          rgba="1 1 1 1" />
-      </material>
-    </visual>
-    <collision>
-      <origin
-        xyz="0 0 0"
-        rpy="0 0 0" />
-      <geometry>
-        <mesh
-          filename="package://alfa_robot_description/meshes/alfa_robot_v2_arm_v4/collision/leftjoint1.STL" />
+        xyz="0.314153929594229 -0.00440359963042056 0.0239848497114266"
+        rpy="0 0 0" />
+      <mass
+        value="3.24848357477083" />
+      <inertia
+        ixx="0.00295020611494677"
+        ixy="3.85498258135523E-05"
+        ixz="-2.74238134472291E-06"
+        iyy="0.0869139996653311"
+        iyz="-8.33305805370074E-05"
+        izz="0.0868894586798014" />
+    </inertial>
+    <visual>
+      <origin
+        xyz="0 0 0"
+        rpy="0 0 0" />
+      <geometry>
+        <mesh
+          filename="package://alfa_robot_description/meshes/alfa_robot_v2_arm_v4_new/visual/leftjoint1.STL" />
+      </geometry>
+      <material
+        name="">
+        <color
+          rgba="1 1 1 1" />
+      </material>
+    </visual>
+    <collision>
+      <origin
+        xyz="0 0 0"
+        rpy="0 0 0" />
+      <geometry>
+        <mesh
+          filename="package://alfa_robot_description/meshes/alfa_robot_v2_arm_v4_new/collision/leftjoint1.STL" />
       </geometry>
     </collision>
@@ -270,5 +270,5 @@
     type="prismatic">
     <origin
-      xyz="-0.285799999999983 0.269999999999219 0.184500000000939"
+      xyz="-0.2858 0.27 0.1845"
       rpy="0 0 0" />
     <parent
@@ -288,37 +288,37 @@
     <inertial>
       <origin
-        xyz="1.86514639244351E-05 0.00549008734545911 0.0483192697870322"
-        rpy="0 0 0" />
-      <mass
-        value="1.1434754221004" />
-      <inertia
-        ixx="0.0024543741369995"
-        ixy="1.89450558125154E-06"
-        ixz="-2.45980294088456E-06"
-        iyy="0.00234579099555691"
-        iyz="-7.07026940240241E-05"
-        izz="0.00212775377469202" />
-    </inertial>
-    <visual>
-      <origin
-        xyz="0 0 0"
-        rpy="0 0 0" />
-      <geometry>
-        <mesh
-          filename="package://alfa_robot_description/meshes/alfa_robot_v2_arm_v4/visual/leftjoint2.STL" />
-      </geometry>
-      <material
-        name="">
-        <color
-          rgba="1 1 1 1" />
-      </material>
-    </visual>
-    <collision>
-      <origin
-        xyz="0 0 0"
-        rpy="0 0 0" />
-      <geometry>
-        <mesh
-          filename="package://alfa_robot_description/meshes/alfa_robot_v2_arm_v4/collision/leftjoint2.STL" />
+        xyz="1.86514629241241E-05 0.00549008734544698 0.0483192697870418"
+        rpy="0 0 0" />
+      <mass
+        value="1.14347542210027" />
+      <inertia
+        ixx="0.00245437413699915"
+        ixy="1.89450558121563E-06"
+        ixz="-2.45980294098259E-06"
+        iyy="0.00234579099555651"
+        iyz="-7.07026940239687E-05"
+        izz="0.00212775377469186" />
+    </inertial>
+    <visual>
+      <origin
+        xyz="0 0 0"
+        rpy="0 0 0" />
+      <geometry>
+        <mesh
+          filename="package://alfa_robot_description/meshes/alfa_robot_v2_arm_v4_new/visual/leftjoint2.STL" />
+      </geometry>
+      <material
+        name="">
+        <color
+          rgba="1 1 1 1" />
+      </material>
+    </visual>
+    <collision>
+      <origin
+        xyz="0 0 0"
+        rpy="0 0 0" />
+      <geometry>
+        <mesh
+          filename="package://alfa_robot_description/meshes/alfa_robot_v2_arm_v4_new/collision/leftjoint2.STL" />
       </geometry>
     </collision>
@@ -328,5 +328,5 @@
     type="continuous">
     <origin
-      xyz="0.716 0 0.1705"
+      xyz="0.741 0 0.0425"
       rpy="-1.5708 1.5662 -1.5708" />
     <parent
@@ -336,4 +336,9 @@
     <axis
       xyz="0 0 1" />
+    <limit
+      lower="0"
+      upper="0"
+      effort="0"
+      velocity="0" />
   </joint>
   <link
@@ -341,37 +346,37 @@
     <inertial>
       <origin
-        xyz="0.0708924301709254 -2.86407864964477E-05 0.0516803522991347"
-        rpy="0 0 0" />
-      <mass
-        value="1.75163255810635" />
-      <inertia
-        ixx="0.00386552461884797"
-        ixy="-1.39559114197398E-06"
-        ixz="-7.06884843737482E-05"
-        iyy="0.00631255855610293"
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
File: ros2_ws/src/alfa_robot_description/urdf/alfa_robot/alfa_robot_macro.ros2_control.xacro (robot description, xacro)
@@ -65,5 +65,5 @@
         <state_interface name="acceleration"/>
       </joint>
-      <!-- turn (continuous) -->
+      <!-- turn (continuous; no URDF limit tag) -->
       <joint name="${prefix}turn">
         <command_interface name="position"/>
@@ -98,34 +98,46 @@
         <state_interface name="acceleration"/>
       </joint>
-      <!-- rightjoint2 (continuous) -->
+      <!-- rightjoint2 (continuous; URDF limit tag currently 0..0) -->
       <joint name="${prefix}rightjoint2">
-        <command_interface name="position"/>
-        <state_interface name="position">
-          <param name="initial_value">0.0</param>
-        </state_interface>
-        <state_interface name="velocity"/>
-        <state_interface name="acceleration"/>
-      </joint>
-      <!-- rightjoint3 (continuous) -->
+        <command_interface name="position">
+          <param name="min">0</param>
+          <param name="max">0</param>
+        </command_interface>
+        <state_interface name="position">
+          <param name="initial_value">0.0</param>
+        </state_interface>
+        <state_interface name="velocity"/>
+        <state_interface name="acceleration"/>
+      </joint>
+      <!-- rightjoint3 (continuous; URDF limit tag currently 0..0) -->
       <joint name="${prefix}rightjoint3">
-        <command_interface name="position"/>
-        <state_interface name="position">
-          <param name="initial_value">0.0</param>
-        </state_interface>
-        <state_interface name="velocity"/>
-        <state_interface name="acceleration"/>
-      </joint>
-      <!-- rightjoint4 (continuous) -->
+        <command_interface name="position">
+          <param name="min">0</param>
+          <param name="max">0</param>
+        </command_interface>
+        <state_interface name="position">
+          <param name="initial_value">0.0</param>
+        </state_interface>
+        <state_interface name="velocity"/>
+        <state_interface name="acceleration"/>
+      </joint>
+      <!-- rightjoint4 (continuous; URDF limit tag currently 0..0) -->
       <joint name="${prefix}rightjoint4">
-        <command_interface name="position"/>
-        <state_interface name="position">
-          <param name="initial_value">0.0</param>
-        </state_interface>
-        <state_interface name="velocity"/>
-        <state_interface name="acceleration"/>
-      </joint>
-      <!-- rightjoint5 (continuous) -->
+        <command_interface name="position">
+          <param name="min">0</param>
+          <param name="max">0</param>
+        </command_interface>
+        <state_interface name="position">
+          <param name="initial_value">0.0</param>
+        </state_interface>
+        <state_interface name="velocity"/>
+        <state_interface name="acceleration"/>
+      </joint>
+      <!-- rightjoint5 (continuous; URDF limit tag currently 0..0) -->
       <joint name="${prefix}rightjoint5">
-        <command_interface name="position"/>
+        <command_interface name="position">
+          <param name="min">0</param>
+          <param name="max">0</param>
+        </command_interface>
         <state_interface name="position">
           <param name="initial_value">0.0</param>
@@ -158,34 +170,46 @@
         <state_interface name="acceleration"/>
       </joint>
-      <!-- leftjoint2 (continuous) -->
+      <!-- leftjoint2 (continuous; URDF limit tag currently 0..0) -->
       <joint name="${prefix}leftjoint2">
-        <command_interface name="position"/>
-        <state_interface name="position">
-          <param name="initial_value">0.0</param>
-        </state_interface>
-        <state_interface name="velocity"/>
-        <state_interface name="acceleration"/>
-      </joint>
-      <!-- leftjoint3 (continuous) -->
+        <command_interface name="position">
+          <param name="min">0</param>
+          <param name="max">0</param>
+        </command_interface>
+        <state_interface name="position">
+          <param name="initial_value">0.0</param>
+        </state_interface>
+        <state_interface name="velocity"/>
+        <state_interface name="acceleration"/>
+      </joint>
+      <!-- leftjoint3 (continuous; URDF limit tag currently 0..0) -->
       <joint name="${prefix}leftjoint3">
-        <command_interface name="position"/>
-        <state_interface name="position">
-          <param name="initial_value">0.0</param>
-        </state_interface>
-        <state_interface name="velocity"/>
-        <state_interface name="acceleration"/>
-      </joint>
-      <!-- leftjoint4 (continuous) -->
+        <command_interface name="position">
+          <param name="min">0</param>
+          <param name="max">0</param>
+        </command_interface>
+        <state_interface name="position">
+          <param name="initial_value">0.0</param>
+        </state_interface>
+        <state_interface name="velocity"/>
+        <state_interface name="acceleration"/>
+      </joint>
+      <!-- leftjoint4 (continuous; URDF limit tag currently 0..0) -->
       <joint name="${prefix}leftjoint4">
-        <command_interface name="position"/>
-        <state_interface name="position">
-          <param name="initial_value">0.0</param>
-        </state_interface>
-        <state_interface name="velocity"/>
-        <state_interface name="acceleration"/>
-      </joint>
-      <!-- leftjoint5 (continuous) -->
+        <command_interface name="position">
+          <param name="min">0</param>
+          <param name="max">0</param>
+        </command_interface>
+        <state_interface name="position">
+          <param name="initial_value">0.0</param>
+        </state_interface>
+        <state_interface name="velocity"/>
+        <state_interface name="acceleration"/>
+      </joint>
+      <!-- leftjoint5 (continuous; URDF limit tag currently 0..0) -->
       <joint name="${prefix}leftjoint5">
-        <command_interface name="position"/>
+        <command_interface name="position">
+          <param name="min">0</param>
+          <param name="max">0</param>
+        </command_interface>
         <state_interface name="position">
           <param name="initial_value">0.0</param>

Commit message: feat: 添加末端执行器链接 + IK 求解器切换为 KDL
- URDF 新增 left_ee_link / right_ee_link 固定关节（挂载在 joint6 下）
- SRDF vacuum 组末端链接从 joint6 改为 ee_link
- kinematics: left_arm_with_base 求解器从 TRAC-IK 切换为 KDL，超时对齐 0.05s

Co-Authored-By: Claude Opus 4.7 <noreply@anthropic.com>

File: ros2_ws/src/alfa_robot_description/urdf/alfa_robot.urdf.xacro (robot description, xacro)
@@ -922,4 +922,16 @@
       velocity="0" />
   </joint>
+  <link name="left_ee_link"/>
+  <joint name="left_ee_fixed" type="fixed">
+    <parent link="leftjoint6"/>
+    <child link="left_ee_link"/>
+    <origin xyz="0 0 0" rpy="0 0 0"/>
+  </joint>
+  <link name="right_ee_link"/>
+  <joint name="right_ee_fixed" type="fixed">
+    <parent link="rightjoint6"/>
+    <child link="right_ee_link"/>
+    <origin xyz="0 0 0" rpy="0 0 0"/>
+  </joint>
   <xacro:alfa_robot_ros2_control
     name="alfa_robot"
