Commit message: chore: align v4 dev robot simulation state
Co-Authored-By: Codex <codex@openai.com>

File: ros2_ws/src/alfa_robot_description/urdf/alfa_robot.urdf.xacro (robot description, xacro)
@@ -56,4 +56,28 @@
       </geometry>
     </collision>
+    <!-- v3 mobile chassis mesh: keep the v4 arm base, but restore the full moving chassis shell. -->
+    <visual>
+      <origin
+        xyz="0 0 0"
+        rpy="0 0 0" />
+      <geometry>
+        <mesh
+          filename="package://alfa_robot_description/meshes/alfa_robot/visual/base_link.STL" />
+      </geometry>
+      <material
+        name="mobile_chassis_blue">
+        <color
+          rgba="0.2 0.4 0.8 1" />
+      </material>
+    </visual>
+    <collision>
+      <origin
+        xyz="0 0 0"
+        rpy="0 0 0" />
+      <geometry>
+        <mesh
+          filename="package://alfa_robot_description/meshes/alfa_robot/collision/base_link.STL" />
+      </geometry>
+    </collision>
   </link>
   <link

File: scripts/ik_benchmark/models/urdf_versions/v4/alfa_robot.urdf (robot description, URDF)
Before this commit: robot alfa_robot, 19 links, 18 joints
Links:
- link base_link: geometry collision mesh filename=package://alfa_robot_description/meshes/alfa_robot/collisio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; collision mesh filename=package://alfa_robot_description/meshes/alfa_robot_v2_arm_v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
- link leftjoint1: geometry collision mesh filename=package://alfa_robot_description/meshes/alfa_robot_v2_arm_v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; visual mesh filename=package://alfa_robot_description/meshes/alfa_robot_v2_arm_v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
- link leftjoint2: geometry collision mesh filename=package://alfa_robot_description/meshes/alfa_robot_v2_arm_v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; visual mesh filename=package://alfa_robot_description/meshes/alfa_robot_v2_arm_v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
- link leftjoint3: geometry collision mesh filename=package://alfa_robot_description/meshes/alfa_robot_v2_arm_v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; visual mesh filename=package://alfa_robot_description/meshes/alfa_robot_v2_arm_v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
- link leftjoint4: geometry collision mesh filename=package://alfa_robot_description/meshes/alfa_robot_v2_arm_v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; visual mesh filename=package://alfa_robot_description/meshes/alfa_robot_v2_arm_v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
- link leftjoint5: geometry collision mesh filename=package://alfa_robot_description/meshes/alfa_robot_v2_arm_v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; visual mesh filename=package://alfa_robot_description/meshes/alfa_robot_v2_arm_v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
- link leftjoint6: geometry collision mesh filename=package://alfa_robot_description/meshes/alfa_robot_v2_arm_v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; visual mesh filename=package://alfa_robot_description/meshes/alfa_robot_v2_arm_v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
- link pitch: geometry collision mesh filename=package://alfa_robot_description/meshes/alfa_robot_v2_arm_v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; visual mesh filename=package://alfa_robot_description/meshes/alfa_robot_v2_arm_v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
- link rightjoint1: geometry collision mesh filename=package://alfa_robot_description/meshes/alfa_robot_v2_arm_v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; visual mesh filename=package://alfa_robot_description/meshes/alfa_robot_v2_arm_v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
- link rightjoint2: geometry collision mesh filename=package://alfa_robot_description/meshes/alfa_robot_v2_arm_v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; visual mesh filename=package://alfa_robot_description/meshes/alfa_robot_v2_arm_v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
- link rightjoint3: geometry collision mesh filename=package://alfa_robot_description/meshes/alfa_robot_v2_arm_v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; visual mesh filename=package://alfa_robot_description/meshes/alfa_robot_v2_arm_v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
- link rightjoint4: geometry collision mesh filename=package://alfa_robot_description/meshes/alfa_robot_v2_arm_v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; visual mesh filename=package://alfa_robot_description/meshes/alfa_robot_v2_arm_v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
- link rightjoint5: geometry collision mesh filename=package://alfa_robot_description/meshes/alfa_robot_v2_arm_v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; visual mesh filename=package://alfa_robot_description/meshes/alfa_robot_v2_arm_v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
- link rightjoint6: geometry collision mesh filename=package://alfa_robot_description/meshes/alfa_robot_v2_arm_v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; visual mesh filename=package://alfa_robot_description/meshes/alfa_robot_v2_arm_v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
- link turn: geometry collision mesh filename=package://alfa_robot_description/meshes/alfa_robot_v2_arm_v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; visual mesh filename=package://alfa_robot_description/meshes/alfa_robot_v2_arm_v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
- link updown: geometry collision mesh filename=package://alfa_robot_description/meshes/alfa_robot_v2_arm_v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; visual mesh filename=package://alfa_robot_description/meshes/alfa_robot_v2_arm_v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
