Commit message: feat: replace v4 arms with v5 proxy setup
- remove v4 arm links from active URDF/MoveIt/control paths

- add v5 proxy interface docs and dual six-axis arm configuration

- document AI co-author trailer rule for Git operations

Co-Authored-By: Codex <codex@openai.com>

File: ros2_ws/src/alfa_robot_description/urdf/alfa_robot.urdf.xacro (robot description, xacro)
@@ -226,712 +226,185 @@
       velocity="0" />
   </joint>
-  <link
-    name="leftjoint1">
+  <!-- v5 dual six-axis proxy arms.
+       Coordinate convention for this proxy: +Y is forward, +Z is up.
+       User-corrected mounting plane: both mount frames use x=0, so they lie in the same YZ plane as updown.
+       The two proxy arms are separated along +/-Y and use multi-primitive T-motor joint visuals. -->
+  <xacro:property name="v5_mount_y" value="0.32"/>
+  <xacro:property name="v5_mount_z" value="0.18"/>
+  <xacro:property name="v5_upper_arm_length" value="0.65"/>
+  <xacro:property name="v5_forearm_length" value="0.65"/>
+  <xacro:property name="v5_motor_radius" value="0.085"/>
+  <xacro:property name="v5_motor_width" value="0.11"/>
+  <xacro:property name="v5_motor_gap" value="0"/>
+  <xacro:property name="v5_joint1_zero_rpy" value="0 0 -1.5708"/>
+  <xacro:macro name="v5_visual_box" params="size xyz rpy color">
+    <visual>
+      <origin xyz="${xyz}" rpy="${rpy}"/>
+      <geometry><box size="${size}"/></geometry>
+      <material name="v5_box_mat"><color rgba="${color}"/></material>
+    </visual>
+  </xacro:macro>
+  <xacro:macro name="v5_collision_box" params="size xyz rpy">
+    <collision>
+      <origin xyz="${xyz}" rpy="${rpy}"/>
+      <geometry><box size="${size}"/></geometry>
+    </collision>
+  </xacro:macro>
+  <xacro:macro name="v5_visual_cylinder" params="radius length xyz rpy color">
+    <visual>
+      <origin xyz="${xyz}" rpy="${rpy}"/>
+      <geometry><cylinder radius="${radius}" length="${length}"/></geometry>
+      <material name="v5_cylinder_mat"><color rgba="${color}"/></material>
+    </visual>
+  </xacro:macro>
+  <xacro:macro name="v5_collision_cylinder" params="radius length xyz rpy">
+    <collision>
+      <origin xyz="${xyz}" rpy="${rpy}"/>
+      <geometry><cylinder radius="${radius}" length="${length}"/></geometry>
+    </collision>
+  </xacro:macro>
+  <xacro:macro name="v5_simple_inertial" params="mass">
     <inertial>
-      <origin
-        xyz="0.314153929594229 -0.00440359963042056 0.0239848497114266"
-        rpy="0 0 0" />
-      <mass
-        value="3.24848357477083" />
-      <inertia
-        ixx="0.00295020611494677"
-        ixy="3.85498258135523E-05"
-        ixz="-2.74238134472291E-06"
-        iyy="0.0869139996653311"
-        iyz="-8.33305805370074E-05"
-        izz="0.0868894586798014" />
+      <origin xyz="0 0 0" rpy="0 0 0"/>
+      <mass value="${mass}"/>
+      <inertia ixx="0.02" ixy="0" ixz="0" iyy="0.02" iyz="0" izz="0.02"/>
     </inertial>
-    <visual>
-      <origin
-        xyz="0 0 0"
-        rpy="0 0 0" />
-      <geometry>
-        <mesh
-          filename="package://alfa_robot_description/meshes/alfa_robot_v2_arm_v4_new/visual/leftjoint1.STL" />
-      </geometry>
-      <material
-        name="">
-        <color
-          rgba="1 1 1 1" />
-      </material>
-    </visual>
-    <collision>
-      <origin
-        xyz="0 0 0"
-        rpy="0 0 0" />
-      <geometry>
-        <mesh
-          filename="package://alfa_robot_description/meshes/alfa_robot_v2_arm_v4_new/collision/leftjoint1.STL" />
-      </geometry>
-    </collision>
-  </link>
-  <joint
-    name="leftjoint1"
-    type="prismatic">
-    <origin
-      xyz="-0.2858 0.27 0.1845"
-      rpy="0 0 0" />
-    <parent
-      link="updown" />
-    <child
-      link="leftjoint1" />
-    <axis
-      xyz="1 0 0" />
-    <limit
-      lower="0"
-      upper="0.3"
-      effort="0"
-      velocity="0" />
-  </joint>
-  <link
-    name="leftjoint2">
-    <inertial>
-      <origin
-        xyz="1.86514629241241E-05 0.00549008734544698 0.0483192697870418"
-        rpy="0 0 0" />
-      <mass
-        value="1.14347542210027" />
-      <inertia
-        ixx="0.00245437413699915"
-        ixy="1.89450558121563E-06"
-        ixz="-2.45980294098259E-06"
-        iyy="0.00234579099555651"
-        iyz="-7.07026940239687E-05"
-        izz="0.00212775377469186" />
-    </inertial>
-    <visual>
-      <origin
-        xyz="0 0 0"
-        rpy="0 0 0" />
-      <geometry>
-        <mesh
-          filename="package://alfa_robot_description/meshes/alfa_robot_v2_arm_v4_new/visual/leftjoint2.STL" />
-      </geometry>
-      <material
-        name="">
-        <color
-          rgba="1 1 1 1" />
-      </material>
-    </visual>
-    <collision>
-      <origin
-        xyz="0 0 0"
-        rpy="0 0 0" />
-      <geometry>
-        <mesh
-          filename="package://alfa_robot_description/meshes/alfa_robot_v2_arm_v4_new/collision/leftjoint2.STL" />
-      </geometry>
-    </collision>
-  </link>
-  <joint
-    name="leftjoint2"
-    type="continuous">
-    <origin
-      xyz="0.741 0 0.0425"
-      rpy="-1.5708 1.5662 -1.5708" />
-    <parent
-      link="leftjoint1" />
-    <child
-      link="leftjoint2" />
-    <axis
-      xyz="0 0 1" />
-    <limit
-      lower="0"
-      upper="0"
-      effort="0"
-      velocity="0" />
-  </joint>
-  <link
-    name="leftjoint3">
-    <inertial>
-      <origin
-        xyz="0.0708924301709439 -2.86407864120708E-05 0.0516803523003164"
-        rpy="0 0 0" />
-      <mass
-        value="1.75163255810626" />
-      <inertia
-        ixx="0.00386552461884768"
-        ixy="-1.39559114195796E-06"
-        ixz="-7.06884843736434E-05"
-        iyy="0.0063125585561027"
-        iyz="2.78557081723717E-06"
-        izz="0.005985914078719" />
-    </inertial>
-    <visual>
-      <origin
-        xyz="0 0 0"
-        rpy="0 0 0" />
-      <geometry>
-        <mesh
-          filename="package://alfa_robot_description/meshes/alfa_robot_v2_arm_v4_new/visual/leftjoint3.STL" />
-      </geometry>
-      <material
-        name="">
-        <color
-          rgba="1 1 1 1" />
-      </material>
-    </visual>
-    <collision>
-      <origin
-        xyz="0 0 0"
-        rpy="0 0 0" />
-      <geometry>
-        <mesh
-          filename="package://alfa_robot_description/meshes/alfa_robot_v2_arm_v4_new/collision/leftjoint3.STL" />
-      </geometry>
-    </collision>
-  </link>
-  <joint
-    name="leftjoint3"
-    type="continuous">
-    <origin
-      xyz="-0.00035108 0.075999 0.058"
-      rpy="-1.5754 -1.5708 0" />
-    <parent
-      link="leftjoint2" />
-    <child
-      link="leftjoint3" />
-    <axis
-      xyz="0 0 1" />
-    <limit
-      lower="0"
-      upper="0"
-      effort="0"
-      velocity="0" />
-  </joint>
-  <link
-    name="leftjoint4">
-    <inertial>
-      <origin
-        xyz="-4.39524881128417E-05 -0.00548991615501886 0.0483192628631884"
-        rpy="0 0 0" />
-      <mass
-        value="1.14347490195887" />
-      <inertia
-        ixx="0.00245438876124795"
-        ixy="1.3933232810866E-06"
-        ixz="2.78611892667967E-06"
-        iyy="0.00234577612781096"
-        iyz="7.06904868831907E-05"
-        izz="0.00212775390428859" />
-    </inertial>
-    <visual>
-      <origin
-        xyz="0 0 0"
-        rpy="0 0 0" />
-      <geometry>
-        <mesh
-          filename="package://alfa_robot_description/meshes/alfa_robot_v2_arm_v4_new/visual/leftjoint4.STL" />
-      </geometry>
-      <material
-        name="">
-        <color
-          rgba="1 1 1 1" />
-      </material>
-    </visual>
-    <collision>
-      <origin
-        xyz="0 0 0"
-        rpy="0 0 0" />
-      <geometry>
-        <mesh
-          filename="package://alfa_robot_description/meshes/alfa_robot_v2_arm_v4_new/collision/leftjoint4.STL" />
-      </geometry>
-    </collision>
-  </link>
-  <joint
-    name="leftjoint4"
-    type="continuous">
-    <origin
-      xyz="0.311 0 0.058"
-      rpy="1.5708 0 1.5708" />
-    <parent
-      link="leftjoint3" />
-    <child
-      link="leftjoint4" />
-    <axis
-      xyz="0 0 1" />
-    <limit
-      lower="0"
-      upper="0"
-      effort="0"
-      velocity="0" />
-  </joint>
-  <link
-    name="leftjoint5">
-    <inertial>
-      <origin
-        xyz="-0.0101973263914319 0.0354519575077605 0.0525851030184155"
-        rpy="0 0 0" />
-      <mass
-        value="2.04610954463043" />
-      <inertia
-        ixx="0.00370756754827538"
-        ixy="-5.97979164598911E-06"
-        ixz="-7.07123942208118E-05"
-        iyy="0.00475856066836737"
-        iyz="2.78433906406734E-06"
-        izz="0.00439564074712178" />
-    </inertial>
-    <visual>
-      <origin
-        xyz="0 0 0"
-        rpy="0 0 0" />
-      <geometry>
-        <mesh
-          filename="package://alfa_robot_description/meshes/alfa_robot_v2_arm_v4_new/visual/leftjoint5.STL" />
-      </geometry>
-      <material
-        name="">
-        <color
-          rgba="0.792156862745098 0.819607843137255 0.933333333333333 1" />
-      </material>
-    </visual>
-    <collision>
-      <origin
-        xyz="0 0 0"
-        rpy="0 0 0" />
-      <geometry>
-        <mesh
-          filename="package://alfa_robot_description/meshes/alfa_robot_v2_arm_v4_new/collision/leftjoint5.STL" />
-      </geometry>
-    </collision>
-  </link>
-  <joint
-    name="leftjoint5"
-    type="continuous">
-    <origin
-      xyz="0 -0.076 0.058"
-      rpy="-1.4138 -1.5708 2.9829" />
-    <parent
-      link="leftjoint4" />
-    <child
-      link="leftjoint5" />
-    <axis
-      xyz="0 0 1" />
-    <limit
-      lower="0"
-      upper="0"
-      effort="0"
-      velocity="0" />
-  </joint>
-  <link
-    name="leftjoint6">
-    <inertial>
-      <origin
-        xyz="0.00399999999999223 -1.06858966120171E-14 1.00341956965622E-12"
-        rpy="0 0 0" />
-      <mass
-        value="0.383392154077702" />
-      <inertia
-        ixx="0.00308153252550287"
-        ixy="6.65285003011356E-20"
-        ixz="-2.71050543121376E-20"
-        iyy="0.00133504319064112"
-        iyz="-6.87175958398818E-19"
-        izz="0.00175057885117191" />
-    </inertial>
-    <visual>
-      <origin
-        xyz="0 0 0"
-        rpy="0 0 0" />
-      <geometry>
-        <mesh
-          filename="package://alfa_robot_description/meshes/alfa_robot_v2_arm_v4_new/visual/leftjoint6.STL" />
-      </geometry>
-      <material
-        name="">
-        <color
-          rgba="0.792156862745098 0.819607843137255 0.933333333333333 1" />
-      </material>
-    </visual>
-    <collision>
-      <origin
-        xyz="0 0 0"
-        rpy="0 0 0" />
-      <geometry>
-        <mesh
-          filename="package://alfa_robot_description/meshes/alfa_robot_v2_arm_v4_new/collision/leftjoint6.STL" />
-      </geometry>
-    </collision>
-  </link>
-  <joint
-    name="leftjoint6"
-    type="prismatic">
-    <origin
-      xyz="0.102 0.0898 0.058"
-      rpy="-1.5708 0 0" />
-    <parent
-      link="leftjoint5" />
-    <child
-      link="leftjoint6" />
-    <axis
-      xyz="1 0 0" />
-    <limit
-      lower="0"
-      upper="0.15"
-      effort="0"
-      velocity="0" />
-  </joint>
-  <link
-    name="rightjoint1">
-    <inertial>
-      <origin
-        xyz="0.316321020532001 1.67392358475515E-05 0.0261312896149528"
-        rpy="0 0 0" />
-      <mass
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
File: ros2_ws/src/alfa_robot_description/urdf/alfa_robot/alfa_robot_macro.ros2_control.xacro (robot description, xacro)
@@ -39,16 +39,4 @@
           <param name="safe_position_turn">0.0</param>
           <param name="safe_position_updown">0.0</param>
-          <param name="safe_position_leftjoint1">0.0</param>
-          <param name="safe_position_leftjoint2">0.0</param>
-          <param name="safe_position_leftjoint3">0.0</param>
-          <param name="safe_position_leftjoint4">0.0</param>
-          <param name="safe_position_leftjoint5">0.0</param>
-          <param name="safe_position_leftjoint6">0.0</param>
-          <param name="safe_position_rightjoint1">0.0</param>
-          <param name="safe_position_rightjoint2">0.0</param>
-          <param name="safe_position_rightjoint3">0.0</param>
-          <param name="safe_position_rightjoint4">0.0</param>
-          <param name="safe_position_rightjoint5">0.0</param>
-          <param name="safe_position_rightjoint6">0.0</param>
         </xacro:unless>
       </hardware>
@@ -86,148 +74,30 @@
         <state_interface name="acceleration"/>
       </joint>
-      <!-- rightjoint1 (prismatic) -->
-      <joint name="${prefix}rightjoint1">
-        <command_interface name="position">
-          <param name="min">0</param>
-          <param name="max">0.3</param>
-        </command_interface>
-        <state_interface name="position">
-          <param name="initial_value">0.0</param>
-        </state_interface>
-        <state_interface name="velocity"/>
-        <state_interface name="acceleration"/>
-      </joint>
-      <!-- rightjoint2 (continuous; URDF limit tag currently 0..0) -->
-      <joint name="${prefix}rightjoint2">
-        <command_interface name="position">
-          <param name="min">0</param>
-          <param name="max">0</param>
-        </command_interface>
-        <state_interface name="position">
-          <param name="initial_value">0.0</param>
-        </state_interface>
-        <state_interface name="velocity"/>
-        <state_interface name="acceleration"/>
-      </joint>
-      <!-- rightjoint3 (continuous; URDF limit tag currently 0..0) -->
-      <joint name="${prefix}rightjoint3">
-        <command_interface name="position">
-          <param name="min">0</param>
-          <param name="max">0</param>
-        </command_interface>
-        <state_interface name="position">
-          <param name="initial_value">0.0</param>
-        </state_interface>
-        <state_interface name="velocity"/>
-        <state_interface name="acceleration"/>
-      </joint>
-      <!-- rightjoint4 (continuous; URDF limit tag currently 0..0) -->
-      <joint name="${prefix}rightjoint4">
-        <command_interface name="position">
-          <param name="min">0</param>
-          <param name="max">0</param>
-        </command_interface>
-        <state_interface name="position">
-          <param name="initial_value">0.0</param>
-        </state_interface>
-        <state_interface name="velocity"/>
-        <state_interface name="acceleration"/>
-      </joint>
-      <!-- rightjoint5 (continuous; URDF limit tag currently 0..0) -->
-      <joint name="${prefix}rightjoint5">
-        <command_interface name="position">
-          <param name="min">0</param>
-          <param name="max">0</param>
-        </command_interface>
-        <state_interface name="position">
-          <param name="initial_value">0.0</param>
-        </state_interface>
-        <state_interface name="velocity"/>
-        <state_interface name="acceleration"/>
-      </joint>
-      <!-- rightjoint6 (prismatic) -->
-      <joint name="${prefix}rightjoint6">
-        <command_interface name="position">
-          <param name="min">0</param>
-          <param name="max">0.15</param>
-        </command_interface>
-        <state_interface name="position">
-          <param name="initial_value">0.0</param>
-        </state_interface>
-        <state_interface name="velocity"/>
-        <state_interface name="acceleration"/>
-      </joint>
-      <!-- leftjoint1 (prismatic) -->
-      <joint name="${prefix}leftjoint1">
-        <command_interface name="position">
-          <param name="min">0</param>
-          <param name="max">0.3</param>
-        </command_interface>
-        <state_interface name="position">
-          <param name="initial_value">0.0</param>
-        </state_interface>
-        <state_interface name="velocity"/>
-        <state_interface name="acceleration"/>
-      </joint>
-      <!-- leftjoint2 (continuous; URDF limit tag currently 0..0) -->
-      <joint name="${prefix}leftjoint2">
-        <command_interface name="position">
-          <param name="min">0</param>
-          <param name="max">0</param>
-        </command_interface>
-        <state_interface name="position">
-          <param name="initial_value">0.0</param>
-        </state_interface>
-        <state_interface name="velocity"/>
-        <state_interface name="acceleration"/>
-      </joint>
-      <!-- leftjoint3 (continuous; URDF limit tag currently 0..0) -->
-      <joint name="${prefix}leftjoint3">
-        <command_interface name="position">
-          <param name="min">0</param>
-          <param name="max">0</param>
-        </command_interface>
-        <state_interface name="position">
-          <param name="initial_value">0.0</param>
-        </state_interface>
-        <state_interface name="velocity"/>
-        <state_interface name="acceleration"/>
-      </joint>
-      <!-- leftjoint4 (continuous; URDF limit tag currently 0..0) -->
-      <joint name="${prefix}leftjoint4">
-        <command_interface name="position">
-          <param name="min">0</param>
-          <param name="max">0</param>
-        </command_interface>
-        <state_interface name="position">
-          <param name="initial_value">0.0</param>
-        </state_interface>
-        <state_interface name="velocity"/>
-        <state_interface name="acceleration"/>
-      </joint>
-      <!-- leftjoint5 (continuous; URDF limit tag currently 0..0) -->
-      <joint name="${prefix}leftjoint5">
-        <command_interface name="position">
-          <param name="min">0</param>
-          <param name="max">0</param>
-        </command_interface>
-        <state_interface name="position">
-          <param name="initial_value">0.0</param>
-        </state_interface>
-        <state_interface name="velocity"/>
-        <state_interface name="acceleration"/>
-      </joint>
-      <!-- leftjoint6 (prismatic, new end effector extension) -->
-      <joint name="${prefix}leftjoint6">
-        <command_interface name="position">
-          <param name="min">0</param>
-          <param name="max">0.15</param>
-        </command_interface>
-        <state_interface name="position">
-          <param name="initial_value">0.0</param>
-        </state_interface>
-        <state_interface name="velocity"/>
-        <state_interface name="acceleration"/>
-      </joint>
+      <!-- v5 proxy arms (position controlled) -->
+      <xacro:macro name="v5_proxy_control_joint" params="joint_name lower upper velocity">
+        <joint name="${prefix}${joint_name}">
+          <command_interface name="position">
+            <param name="min">${lower}</param>
+            <param name="max">${upper}</param>
+          </command_interface>
+          <state_interface name="position">
+            <param name="initial_value">0.0</param>
+          </state_interface>
+          <state_interface name="velocity"/>
+          <state_interface name="acceleration"/>
+        </joint>
+      </xacro:macro>
+      <xacro:v5_proxy_control_joint joint_name="left_v5_joint1" lower="-3.14159265" upper="3.14159265" velocity="1.2"/>
+      <xacro:v5_proxy_control_joint joint_name="left_v5_joint2" lower="-1.57079632" upper="1.57079632" velocity="1.2"/>
+      <xacro:v5_proxy_control_joint joint_name="left_v5_joint3" lower="-2.35619449" upper="2.35619449" velocity="1.2"/>
+      <xacro:v5_proxy_control_joint joint_name="left_v5_joint4" lower="-3.14159265" upper="3.14159265" velocity="1.5"/>
+      <xacro:v5_proxy_control_joint joint_name="left_v5_joint5" lower="-1.57079632" upper="1.57079632" velocity="1.5"/>
+      <xacro:v5_proxy_control_joint joint_name="left_v5_joint6" lower="-3.14159265" upper="3.14159265" velocity="1.5"/>
+      <xacro:v5_proxy_control_joint joint_name="right_v5_joint1" lower="-3.14159265" upper="3.14159265" velocity="1.2"/>
+      <xacro:v5_proxy_control_joint joint_name="right_v5_joint2" lower="-1.57079632" upper="1.57079632" velocity="1.2"/>
+      <xacro:v5_proxy_control_joint joint_name="right_v5_joint3" lower="-2.35619449" upper="2.35619449" velocity="1.2"/>
+      <xacro:v5_proxy_control_joint joint_name="right_v5_joint4" lower="-3.14159265" upper="3.14159265" velocity="1.5"/>
+      <xacro:v5_proxy_control_joint joint_name="right_v5_joint5" lower="-1.57079632" upper="1.57079632" velocity="1.5"/>
+      <xacro:v5_proxy_control_joint joint_name="right_v5_joint6" lower="-3.14159265" upper="3.14159265" velocity="1.5"/>
     </ros2_control>
     <xacro:if value="$(arg sim_gazebo_classic)">
