Commit message: fix: add collision-aware v5 IK and refresh arm meshes
- add PlanningScene validity callback to the dual-arm BioIK setFromIK path

- refresh v5 arm meshes from the v5_1 SolidWorks export and mirrored right meshes

- remove the temporary root export package after copying assets into alfa_robot_description

Co-Authored-By: Codex <codex@openai.com>

File: ros2_ws/src/alfa_robot_description/urdf/alfa_robot.urdf.xacro (robot description, xacro)
@@ -259,7 +259,7 @@
       <xacro:if value="${motor == 'motor1'}">
         <inertial>
-          <origin xyz="0.00549007475138907 ${mirror_y * -4.41381777807892E-05} 0.0638192668274469" rpy="0 0 0"/>
-          <mass value="1.14347753856634"/>
-          <inertia ixx="0.00234577755868115" ixy="${mirror_y * -1.39193363061916E-06}" ixz="-7.06941578932414E-05" iyy="0.00245440035038314" iyz="${mirror_y * 2.78529148686552E-06}" izz="0.00212775140786364"/>
+          <origin xyz="-0.00549007480040076 ${mirror_y * 4.41384348585649E-05} 0.0638192670583628" rpy="0 0 0"/>
+          <mass value="1.14347754183273"/>
+          <inertia ixx="0.00234577756970447" ixy="${mirror_y * -1.39192053258421E-06}" ixz="7.06941577680902E-05" iyy="0.00245440034346279" iyz="${mirror_y * -2.78529246638655E-06}" izz="0.00212775141233719"/>
         </inertial>
         <xacro:v5_visual_mesh mesh_dir="${visual_dir}" mesh="motor1.STL" origin_xyz="0 0 0" origin_rpy="0 0 0" color="${color}"/>
@@ -268,7 +268,7 @@
       <xacro:if value="${motor == 'motor2'}">
         <inertial>
-          <origin xyz="2.093E-05 ${mirror_y * 0.3} 0.074" rpy="0 0 0"/>
-          <mass value="4.8059"/>
-          <inertia ixx="0.051414" ixy="${mirror_y * 1.1107E-09}" ixz="7.002E-10" iyy="0.010931" iyz="${mirror_y * -0.00014138}" izz="0.050761"/>
+          <origin xyz="-2.09300645109267E-05 ${mirror_y * 0.300000037733846} -0.0739999978650945" rpy="0 0 0"/>
+          <mass value="4.80591024170092"/>
+          <inertia ixx="0.0514140216022789" ixy="${mirror_y * -1.11071009974064E-09}" ixz="7.00200352560243E-10" iyy="0.0109314943608357" iyz="${mirror_y * 0.000141378481768625}" izz="0.0507607430231609"/>
         </inertial>
         <xacro:v5_visual_mesh mesh_dir="${visual_dir}" mesh="motor2.STL" origin_xyz="0 0 0" origin_rpy="0 0 0" color="${color}"/>
@@ -277,7 +277,7 @@
       <xacro:if value="${motor == 'motor3'}">
         <inertial>
-          <origin xyz="-2.8361E-05 ${mirror_y * -0.33834} -0.043469" rpy="0 0 0"/>
-          <mass value="1.766"/>
-          <inertia ixx="0.016132" ixy="${mirror_y * 2.7853E-06}" ixz="-1.3961E-06" iyy="0.002789" iyz="${mirror_y * -0.0001017}" izz="0.01667"/>
+          <origin xyz="-8.86583279652298E-06 ${mirror_y * -0.191421080971033} -0.0611928334493207" rpy="0 0 0"/>
+          <mass value="5.53739421393496"/>
+          <inertia ixx="0.0659171393206471" ixy="${mirror_y * -1.40894015322047E-06}" ixz="-2.83298512105713E-06" iyy="0.0102087351820484" iyz="${mirror_y * -0.00128557192119225}" izz="0.0652938482117856"/>
         </inertial>
         <xacro:v5_visual_mesh mesh_dir="${visual_dir}" mesh="motor3.STL" origin_xyz="0 0 0" origin_rpy="0 0 0" color="${color}"/>
@@ -286,7 +286,7 @@
       <xacro:if value="${motor == 'motor4'}">
         <inertial>
-          <origin xyz="-0.0096807 ${mirror_y * -4.4024E-05} 0.05401" rpy="0 0 0"/>
-          <mass value="1.1435"/>
-          <inertia ixx="0.0021278" ixy="${mirror_y * 2.7864E-06}" ixz="7.0691E-05" iyy="0.0024544" iyz="${mirror_y * 1.3934E-06}" izz="0.0023458"/>
+          <origin xyz="0.054010017525899 ${mirror_y * -0.00968074438612282} -4.38885459771443E-05" rpy="0 0 0"/>
+          <mass value="1.14347527972143"/>
+          <inertia ixx="0.00234577526969165" ixy="${mirror_y * 7.06887224662317E-05}" ixz="1.39432827945232E-06" iyy="0.00212775138988867" iyz="${mirror_y * 2.78555789689753E-06}" izz="0.00245439599558472"/>
         </inertial>
         <xacro:v5_visual_mesh mesh_dir="${visual_dir}" mesh="motor4.STL" origin_xyz="0 0 0" origin_rpy="0 0 0" color="${color}"/>
@@ -295,7 +295,7 @@
       <xacro:if value="${motor == 'motor5'}">
         <inertial>
-          <origin xyz="4.3802E-05 ${mirror_y * -0.0096808} 0.05451" rpy="0 0 0"/>
-          <mass value="1.1435"/>
-          <inertia ixx="0.0024544" ixy="${mirror_y * -2.7853E-06}" ixz="-1.3961E-06" iyy="0.0021278" iyz="${mirror_y * 7.0689E-05}" izz="0.0023458"/>
+          <origin xyz="-0.0545098970073398 ${mirror_y * -0.00968076621990099} 4.3968113340731E-05" rpy="0 0 0"/>
+          <mass value="1.14347708247491"/>
+          <inertia ixx="0.00234577450108908" ixy="${mirror_y * -7.0688725031574E-05}" ixz="1.39442681307563E-06" iyy="0.00212775140409106" iyz="${mirror_y * -2.78654985483454E-06}" izz="0.00245439718636663"/>
         </inertial>
         <xacro:v5_visual_mesh mesh_dir="${visual_dir}" mesh="motor5.STL" origin_xyz="0 0 0" origin_rpy="0 0 0" color="${color}"/>
@@ -304,7 +304,7 @@
       <xacro:if value="${motor == 'motor6'}">
         <inertial>
-          <origin xyz="0 0 0.027325" rpy="0 0 0"/>
-          <mass value="1.9452"/>
-          <inertia ixx="0.0066307" ixy="0" ixz="0" iyy="0.0044221" iyz="0" izz="0.010447"/>
+          <origin xyz="0 0 0.056752" rpy="0 0 0"/>
+          <mass value="8.2851"/>
+          <inertia ixx="0.041557" ixy="0" ixz="0" iyy="0.063474" iyz="0" izz="0.099371"/>
         </inertial>
         <xacro:v5_visual_mesh mesh_dir="${visual_dir}" mesh="motor6.STL" origin_xyz="0 0 0" origin_rpy="0 0 0" color="${color}"/>
@@ -334,6 +334,6 @@
       <parent link="${side}_v5_link1"/>
       <child link="${side}_v5_link2"/>
-      <origin xyz="0.0595 0 0.0735" rpy="${mirror_y * 1.5708} 0 ${mirror_y * 1.5708}"/>
-      <axis xyz="0 0 1"/>
+      <origin xyz="-0.0595 0 0.0735" rpy="${mirror_y * 1.5708} 0 ${mirror_y * 1.5708}"/>
+      <axis xyz="0 0 -1"/>
       <limit lower="-3.14159265" upper="3.14159265" effort="120" velocity="1.2"/>
     </joint>
@@ -342,6 +342,6 @@
       <parent link="${side}_v5_link2"/>
       <child link="${side}_v5_link3"/>
-      <origin xyz="0 ${mirror_y * 0.6} 0.148" rpy="0 0 ${mirror_y * 3.1416}"/>
-      <axis xyz="0 0 -1"/>
+      <origin xyz="0 ${mirror_y * 0.6} -0.148" rpy="0 0 ${mirror_y * 3.1416}"/>
+      <axis xyz="0 0 1"/>
       <limit lower="-3.14159265" upper="3.14159265" effort="100" velocity="1.2"/>
     </joint>
@@ -350,6 +350,6 @@
       <parent link="${side}_v5_link3"/>
       <child link="${side}_v5_link4"/>
-      <origin xyz="0 ${mirror_y * -0.47402} -0.075" rpy="${mirror_y * 1.5708} -1.5708 0"/>
-      <axis xyz="0 0 -1"/>
+      <origin xyz="0 ${mirror_y * -0.412} 0.009" rpy="${mirror_y * 1.5708} -1.5708 0"/>
+      <axis xyz="-1 0 0"/>
       <limit lower="-3.14159265" upper="3.14159265" effort="60" velocity="1.5"/>
     </joint>
@@ -358,6 +358,6 @@
       <parent link="${side}_v5_link4"/>
       <child link="${side}_v5_link5"/>
-      <origin xyz="-0.074 0 0.0595" rpy="${mirror_y * -1.5708} 0 ${mirror_y * 1.5708}"/>
-      <axis xyz="0 0 -1"/>
+      <origin xyz="0.0595 ${mirror_y * -0.074} 0" rpy="${mirror_y * -1.5708} 0 ${mirror_y * 1.5708}"/>
+      <axis xyz="1 0 0"/>
       <limit lower="-3.14159265" upper="3.14159265" effort="60" velocity="1.5"/>
     </joint>
@@ -366,5 +366,5 @@
       <parent link="${side}_v5_link5"/>
       <child link="${side}_v5_link6"/>
-      <origin xyz="0 ${mirror_y * -0.074} 0.06" rpy="${mirror_y * 1.5708} 1.5708 0"/>
+      <origin xyz="-0.06 ${mirror_y * -0.074} 0" rpy="${mirror_y * 1.5708} 0 0"/>
       <axis xyz="0 0 -1"/>
       <limit lower="-3.14159265" upper="3.14159265" effort="40" velocity="1.5"/>

Commit message: fix: remove v5 mount collision artifacts
- hide the old updown STL visual and collision while keeping the lift link and joints

- remove the small internal connector block from motor1 meshes and mirrored right meshes

- record T-0012 completion notes

Co-Authored-By: Codex <codex@openai.com>

File: ros2_ws/src/alfa_robot_description/urdf/alfa_robot.urdf.xacro (robot description, xacro)
@@ -184,27 +184,5 @@
         izz="0.186025474834666" />
     </inertial>
-    <visual>
-      <origin
-        xyz="0 0 0"
-        rpy="0 0 0" />
-      <geometry>
-        <mesh
-          filename="package://alfa_robot_description/meshes/alfa_robot_v2_arm_v4_new/visual/updown.STL" />
-      </geometry>
-      <material
-        name="">
-        <color
-          rgba="1 1 1 1" />
-      </material>
-    </visual>
-    <collision>
-      <origin
-        xyz="0 0 0"
-        rpy="0 0 0" />
-      <geometry>
-        <mesh
-          filename="package://alfa_robot_description/meshes/alfa_robot_v2_arm_v4_new/collision/updown.STL" />
-      </geometry>
-    </collision>
+    <!-- updown link remains the lift/mount frame, but its metal STL is intentionally hidden and non-colliding. -->
   </link>
   <joint
@@ -255,5 +233,5 @@
     </collision>
   </xacro:macro>
-  <xacro:macro name="v5_imported_motor_link" params="name motor color visual_dir collision_dir mirror_y:=1">
+  <xacro:macro name="v5_imported_motor_link" params="name motor color visual_dir collision_dir mirror_y:=1 include_visual:=true include_collision:=true">
     <link name="${name}">
       <xacro:if value="${motor == 'motor1'}">
@@ -263,6 +241,10 @@
           <inertia ixx="0.00234577756970447" ixy="${mirror_y * -1.39192053258421E-06}" ixz="7.06941577680902E-05" iyy="0.00245440034346279" iyz="${mirror_y * -2.78529246638655E-06}" izz="0.00212775141233719"/>
         </inertial>
-        <xacro:v5_visual_mesh mesh_dir="${visual_dir}" mesh="motor1.STL" origin_xyz="0 0 0" origin_rpy="0 0 0" color="${color}"/>
-        <xacro:v5_collision_mesh mesh_dir="${collision_dir}" mesh="motor1.STL" origin_xyz="0 0 0" origin_rpy="0 0 0"/>
+        <xacro:if value="${include_visual}">
+          <xacro:v5_visual_mesh mesh_dir="${visual_dir}" mesh="motor1.STL" origin_xyz="0 0 0" origin_rpy="0 0 0" color="${color}"/>
+        </xacro:if>
+        <xacro:if value="${include_collision}">
+          <xacro:v5_collision_mesh mesh_dir="${collision_dir}" mesh="motor1.STL" origin_xyz="0 0 0" origin_rpy="0 0 0"/>
+        </xacro:if>
       </xacro:if>
       <xacro:if value="${motor == 'motor2'}">
@@ -272,6 +254,10 @@
           <inertia ixx="0.0514140216022789" ixy="${mirror_y * -1.11071009974064E-09}" ixz="7.00200352560243E-10" iyy="0.0109314943608357" iyz="${mirror_y * 0.000141378481768625}" izz="0.0507607430231609"/>
         </inertial>
-        <xacro:v5_visual_mesh mesh_dir="${visual_dir}" mesh="motor2.STL" origin_xyz="0 0 0" origin_rpy="0 0 0" color="${color}"/>
-        <xacro:v5_collision_mesh mesh_dir="${collision_dir}" mesh="motor2.STL" origin_xyz="0 0 0" origin_rpy="0 0 0"/>
+        <xacro:if value="${include_visual}">
+          <xacro:v5_visual_mesh mesh_dir="${visual_dir}" mesh="motor2.STL" origin_xyz="0 0 0" origin_rpy="0 0 0" color="${color}"/>
+        </xacro:if>
+        <xacro:if value="${include_collision}">
+          <xacro:v5_collision_mesh mesh_dir="${collision_dir}" mesh="motor2.STL" origin_xyz="0 0 0" origin_rpy="0 0 0"/>
+        </xacro:if>
       </xacro:if>
       <xacro:if value="${motor == 'motor3'}">
@@ -281,6 +267,10 @@
           <inertia ixx="0.0659171393206471" ixy="${mirror_y * -1.40894015322047E-06}" ixz="-2.83298512105713E-06" iyy="0.0102087351820484" iyz="${mirror_y * -0.00128557192119225}" izz="0.0652938482117856"/>
         </inertial>
-        <xacro:v5_visual_mesh mesh_dir="${visual_dir}" mesh="motor3.STL" origin_xyz="0 0 0" origin_rpy="0 0 0" color="${color}"/>
-        <xacro:v5_collision_mesh mesh_dir="${collision_dir}" mesh="motor3.STL" origin_xyz="0 0 0" origin_rpy="0 0 0"/>
+        <xacro:if value="${include_visual}">
+          <xacro:v5_visual_mesh mesh_dir="${visual_dir}" mesh="motor3.STL" origin_xyz="0 0 0" origin_rpy="0 0 0" color="${color}"/>
+        </xacro:if>
+        <xacro:if value="${include_collision}">
+          <xacro:v5_collision_mesh mesh_dir="${collision_dir}" mesh="motor3.STL" origin_xyz="0 0 0" origin_rpy="0 0 0"/>
+        </xacro:if>
       </xacro:if>
       <xacro:if value="${motor == 'motor4'}">
@@ -290,6 +280,10 @@
           <inertia ixx="0.00234577526969165" ixy="${mirror_y * 7.06887224662317E-05}" ixz="1.39432827945232E-06" iyy="0.00212775138988867" iyz="${mirror_y * 2.78555789689753E-06}" izz="0.00245439599558472"/>
         </inertial>
-        <xacro:v5_visual_mesh mesh_dir="${visual_dir}" mesh="motor4.STL" origin_xyz="0 0 0" origin_rpy="0 0 0" color="${color}"/>
-        <xacro:v5_collision_mesh mesh_dir="${collision_dir}" mesh="motor4.STL" origin_xyz="0 0 0" origin_rpy="0 0 0"/>
+        <xacro:if value="${include_visual}">
+          <xacro:v5_visual_mesh mesh_dir="${visual_dir}" mesh="motor4.STL" origin_xyz="0 0 0" origin_rpy="0 0 0" color="${color}"/>
+        </xacro:if>
+        <xacro:if value="${include_collision}">
+          <xacro:v5_collision_mesh mesh_dir="${collision_dir}" mesh="motor4.STL" origin_xyz="0 0 0" origin_rpy="0 0 0"/>
+        </xacro:if>
       </xacro:if>
       <xacro:if value="${motor == 'motor5'}">
@@ -299,6 +293,10 @@
           <inertia ixx="0.00234577450108908" ixy="${mirror_y * -7.0688725031574E-05}" ixz="1.39442681307563E-06" iyy="0.00212775140409106" iyz="${mirror_y * -2.78654985483454E-06}" izz="0.00245439718636663"/>
         </inertial>
-        <xacro:v5_visual_mesh mesh_dir="${visual_dir}" mesh="motor5.STL" origin_xyz="0 0 0" origin_rpy="0 0 0" color="${color}"/>
-        <xacro:v5_collision_mesh mesh_dir="${collision_dir}" mesh="motor5.STL" origin_xyz="0 0 0" origin_rpy="0 0 0"/>
+        <xacro:if value="${include_visual}">
+          <xacro:v5_visual_mesh mesh_dir="${visual_dir}" mesh="motor5.STL" origin_xyz="0 0 0" origin_rpy="0 0 0" color="${color}"/>
+        </xacro:if>
+        <xacro:if value="${include_collision}">
+          <xacro:v5_collision_mesh mesh_dir="${collision_dir}" mesh="motor5.STL" origin_xyz="0 0 0" origin_rpy="0 0 0"/>
+        </xacro:if>
       </xacro:if>
       <xacro:if value="${motor == 'motor6'}">
@@ -308,6 +306,10 @@
           <inertia ixx="0.041557" ixy="0" ixz="0" iyy="0.063474" iyz="0" izz="0.099371"/>
         </inertial>
-        <xacro:v5_visual_mesh mesh_dir="${visual_dir}" mesh="motor6.STL" origin_xyz="0 0 0" origin_rpy="0 0 0" color="${color}"/>
-        <xacro:v5_collision_mesh mesh_dir="${collision_dir}" mesh="motor6.STL" origin_xyz="0 0 0" origin_rpy="0 0 0"/>
+        <xacro:if value="${include_visual}">
+          <xacro:v5_visual_mesh mesh_dir="${visual_dir}" mesh="motor6.STL" origin_xyz="0 0 0" origin_rpy="0 0 0" color="${color}"/>
+        </xacro:if>
+        <xacro:if value="${include_collision}">
+          <xacro:v5_collision_mesh mesh_dir="${collision_dir}" mesh="motor6.STL" origin_xyz="0 0 0" origin_rpy="0 0 0"/>
+        </xacro:if>
       </xacro:if>
     </link>
