Commit message: feat: integrate v5_5 arm URDF and v1 chassis base
Replace the previous v5 arm definition with the new v5_5 SolidWorks
export, which adds big_arm, big_arm_2, and little_arm fixed sub-links
between motor2→motor3 and motor3→motor4. Also swap base_link, turn,
and updown to use the v1 (alfa_robot) chassis mesh and inertial data,
with pitch joint origin adjusted to match v1 chassis geometry.

Co-Authored-By: Claude Opus 4.7 <noreply@anthropic.com>

File: ros2_ws/src/alfa_robot_moveit_config/config/alfa_robot.ros2_control.xacro (robot description, xacro)
@@ -5,6 +5,6 @@
         <ros2_control name="${name}" type="system">
             <hardware>
-                <!-- By default, set up controllers for simulation. This won't work on real hardware -->
                 <plugin>mock_components/GenericSystem</plugin>
+                <param name="mock_sensor_commands">true</param>
             </hardware>
             <joint name="pitch">
@@ -13,4 +13,5 @@
                   <param name="initial_value">${initial_positions['pitch']}</param>
                 </state_interface>
+                <state_interface name="velocity"/>
             </joint>
             <joint name="turn">
@@ -19,4 +20,5 @@
                   <param name="initial_value">${initial_positions['turn']}</param>
                 </state_interface>
+                <state_interface name="velocity"/>
             </joint>
             <joint name="updown">
@@ -25,4 +27,5 @@
                   <param name="initial_value">${initial_positions['updown']}</param>
                 </state_interface>
+                <state_interface name="velocity"/>
             </joint>
             <joint name="left_v5_joint1">
@@ -31,7 +34,9 @@
                   <param name="initial_value">${initial_positions['left_v5_joint1']}</param>
                 </state_interface>
+                <state_interface name="velocity"/>
             </joint>
             <joint name="left_v5_joint2">
                 <command_interface name="position"/>
+                <state_interface name="velocity"/>
                 <state_interface name="position">
                   <param name="initial_value">${initial_positions['left_v5_joint2']}</param>
@@ -43,4 +48,5 @@
                   <param name="initial_value">${initial_positions['left_v5_joint3']}</param>
                 </state_interface>
+                <state_interface name="velocity"/>
             </joint>
             <joint name="left_v5_joint4">
@@ -49,4 +55,5 @@
                   <param name="initial_value">${initial_positions['left_v5_joint4']}</param>
                 </state_interface>
+                <state_interface name="velocity"/>
             </joint>
             <joint name="left_v5_joint5">
@@ -55,4 +62,5 @@
                   <param name="initial_value">${initial_positions['left_v5_joint5']}</param>
                 </state_interface>
+                <state_interface name="velocity"/>
             </joint>
             <joint name="left_v5_joint6">
@@ -61,4 +69,5 @@
                   <param name="initial_value">${initial_positions['left_v5_joint6']}</param>
                 </state_interface>
+                <state_interface name="velocity"/>
             </joint>
             <joint name="right_v5_joint1">
@@ -67,4 +76,5 @@
                   <param name="initial_value">${initial_positions['right_v5_joint1']}</param>
                 </state_interface>
+                <state_interface name="velocity"/>
             </joint>
             <joint name="right_v5_joint2">
@@ -73,4 +83,5 @@
                   <param name="initial_value">${initial_positions['right_v5_joint2']}</param>
                 </state_interface>
+                <state_interface name="velocity"/>
             </joint>
             <joint name="right_v5_joint3">
@@ -79,4 +90,5 @@
                   <param name="initial_value">${initial_positions['right_v5_joint3']}</param>
                 </state_interface>
+                <state_interface name="velocity"/>
             </joint>
             <joint name="right_v5_joint4">
@@ -85,4 +97,5 @@
                   <param name="initial_value">${initial_positions['right_v5_joint4']}</param>
                 </state_interface>
+                <state_interface name="velocity"/>
             </joint>
             <joint name="right_v5_joint5">
@@ -91,4 +104,5 @@
                   <param name="initial_value">${initial_positions['right_v5_joint5']}</param>
                 </state_interface>
+                <state_interface name="velocity"/>
             </joint>
             <joint name="right_v5_joint6">
@@ -97,4 +111,5 @@
                   <param name="initial_value">${initial_positions['right_v5_joint6']}</param>
                 </state_interface>
+                <state_interface name="velocity"/>
             </joint>
         </ros2_control>

Commit message: feat: v5 双臂完整 MoveIt 配置 + 分支重命名
- RViz 修复双机器人显示 bug：禁用 Query Goal State 和 Planned Path 可视
- pick_place_demo.py IK group 修正为 dual_v5_arm_with_base
- v1 底盘恢复：base_link/turn/updown mesh 和惯性参数
- 吸盘碰撞体积完全忽略：SRDF SuctionVsArm 扩展到 link6
- 左右臂差异化关节限位（URDF + ros2_control + joint_limits）
- SRDF 新增 dual_v5_arm/dual_v5_arm_with_base/empty_group 及碰撞规则
- kinematics.yaml 新增 bio_ik solver 配置
- 双控制器配置（torso + dual_v5_arm）
- updown.STL mesh 优化 19MB→5MB
- 清理 get_end_effector_pose.py
- 分支重命名：v3_dev→alfa_v3, v4_dev→alfa_v4, v4_dev_1→alfa_v4_beta, v5_dev_p→v5_dev_beta

Co-Authored-By: Claude <claude@anthropic.com>

File: ros2_ws/src/alfa_robot_description/urdf/alfa_robot.urdf.xacro (robot description, xacro)
@@ -3,5 +3,5 @@
   <xacro:arg name="prefix" default=""/>
   <xacro:arg name="use_mock_hardware" default="true"/>
-  <xacro:arg name="mock_sensor_commands" default="false"/>
+  <xacro:arg name="mock_sensor_commands" default="true"/>
   <xacro:arg name="sim_gazebo_classic" default="false"/>
   <xacro:arg name="sim_gazebo" default="false"/>
@@ -21,15 +21,15 @@
     <inertial>
       <origin
-        xyz="-0.00896922200126715 2.35194162193642E-05 0.0179811176086975"
+        xyz="-0.44193110855616 0.000259961331933109 0.176428166472852"
         rpy="0 0 0" />
       <mass
-        value="5.21106238092598" />
+        value="394.931465036981" />
       <inertia
-        ixx="0.0633320335254252"
-        ixy="-1.57025952749484E-07"
-        ixz="-3.66796372424077E-07"
-        iyy="0.119212913285128"
-        iyz="6.33714518991059E-07"
-        izz="0.181818429904202" />
+        ixx="66.5681215725466"
+        ixy="5.74775273893285E-10"
+        ixz="9.85014992290203"
+        iyy="65.6389024339403"
+        iyz="2.76043934386688E-09"
+        izz="112.938477587322" />
     </inertial>
     <visual>
@@ -39,10 +39,10 @@
       <geometry>
         <mesh
-          filename="package://alfa_robot_description/meshes/alfa_robot_v2_arm_v4_new/visual/base_link.STL" />
+          filename="package://alfa_robot_description/meshes/alfa_robot/visual/base_link.STL" />
       </geometry>
       <material
-        name="">
+        name="blue">
         <color
-          rgba="1 1 1 1" />
+          rgba="0 0 1 1" />
       </material>
     </visual>
@@ -53,5 +53,5 @@
       <geometry>
         <mesh
-          filename="package://alfa_robot_description/meshes/alfa_robot_v2_arm_v4_new/collision/base_link.STL" />
+          filename="package://alfa_robot_description/meshes/alfa_robot/collision/base_link.STL" />
       </geometry>
     </collision>
@@ -101,5 +101,5 @@
     type="revolute">
     <origin
-      xyz="0.259 -0.0545 0.05"
+      xyz="-0.007937 0 0.129"
       rpy="0 0 0" />
     <parent
@@ -119,15 +119,15 @@
     <inertial>
       <origin
-        xyz="-0.0279588381716878 3.16554382575607E-05 0.819951711254512"
+        xyz="-0.0697894032768815 -0.00012433244764639 0.982155423971065"
         rpy="0 0 0" />
       <mass
-        value="15.206613319806" />
+        value="42.0737844290435" />
       <inertia
-        ixx="1.06710751132169"
-        ixy="5.33982003477265E-06"
-        ixz="0.000444527933425444"
-        iyy="1.0606566000007"
-        iyz="1.02603827456492E-05"
-        izz="0.109926667915607" />
+        ixx="10.0720353784748"
+        ixy="-1.75362629131178E-06"
+        ixz="5.29823321336754E-05"
+        iyy="10.0937833616587"
+        iyz="1.43589075450652E-06"
+        izz="0.327199381319826" />
     </inertial>
     <visual>
@@ -137,10 +137,10 @@
       <geometry>
         <mesh
-          filename="package://alfa_robot_description/meshes/alfa_robot_v2_arm_v4_new/visual/turn.STL" />
+          filename="package://alfa_robot_description/meshes/alfa_robot/visual/turn.STL" />
       </geometry>
       <material
-        name="">
+        name="arm_grey">
         <color
-          rgba="1 1 1 1" />
+          rgba="0.5 0.5 0.5 1" />
       </material>
     </visual>
@@ -151,5 +151,5 @@
       <geometry>
         <mesh
-          filename="package://alfa_robot_description/meshes/alfa_robot_v2_arm_v4_new/collision/turn.STL" />
+          filename="package://alfa_robot_description/meshes/alfa_robot/collision/turn.STL" />
       </geometry>
     </collision>
@@ -159,5 +159,5 @@
     type="continuous">
     <origin
-      xyz="-0.209 0.0545 0.09"
+      xyz="0 0 0"
       rpy="0 0 0" />
     <parent
@@ -172,17 +172,39 @@
     <inertial>
       <origin
-        xyz="0.0212260463112321 -2.11665364142077E-05 0.111174833260946"
+        xyz="-0.196828632659582 0.0148673483555221 0.0956849238503419"
         rpy="0 0 0" />
       <mass
-        value="8.56370936774335" />
+        value="26.931167747836" />
       <inertia
-        ixx="0.0416436910064672"
-        ixy="-3.48369951311999E-07"
-        ixz="1.03580898385951E-05"
-        iyy="0.151229514406379"
-        iyz="1.21565800186775E-06"
-        izz="0.186025474834666" />
+        ixx="0.231217459750122"
+        ixy="2.93337887014215E-05"
+        ixz="0.000951254936009737"
+        iyy="0.178754005132662"
+        iyz="-1.44830456938328E-05"
+        izz="0.348822965146485" />
     </inertial>
-    <!-- updown link remains the lift/mount frame, but its metal STL is intentionally hidden and non-colliding. -->
+    <visual>
+      <origin
+        xyz="0 0 0"
+        rpy="0 0 0" />
+      <geometry>
+        <mesh
+          filename="package://alfa_robot_description/meshes/alfa_robot/visual/updown.STL" />
+      </geometry>
+      <material
+        name="arm_grey">
+        <color
+          rgba="0.5 0.5 0.5 1" />
+      </material>
+    </visual>
+    <collision>
+      <origin
+        xyz="0 0 0"
+        rpy="0 0 0" />
+      <geometry>
+        <mesh
+          filename="package://alfa_robot_description/meshes/alfa_robot/collision/updown.STL" />
+      </geometry>
+    </collision>
   </link>
   <joint
@@ -190,5 +212,5 @@
     type="prismatic">
     <origin
-      xyz="-0.1 0 0.086"
+      xyz="-0.23547 0 0.57771"
       rpy="0 0 0" />
     <parent
@@ -315,5 +337,6 @@
     </link>
   </xacro:macro>
-  <xacro:macro name="v5_imported_arm" params="side mount_y mirror_y color visual_dir collision_dir">
+  <xacro:macro name="v5_imported_arm" params="side mount_y mirror_y color visual_dir collision_dir
+    j1_lo j1_hi j2_lo j2_hi j3_lo j3_hi j4_lo j4_hi j5_lo j5_hi j6_lo j6_hi">
     <link name="${side}_v5_link0">
       <xacro:v5_simple_inertial mass="0.5"/>
@@ -330,5 +353,5 @@
       <origin xyz="0 0 0" rpy="0 0 0"/>
       <axis xyz="0 0 1"/>
-      <limit lower="-3.14159265" upper="3.14159265" effort="120" velocity="1.2"/>
+      <limit lower="${j1_lo}" upper="${j1_hi}" effort="120" velocity="1.2"/>
     </joint>
     <xacro:v5_imported_motor_link name="${side}_v5_link2" motor="motor2" color="${color}" visual_dir="${visual_dir}" collision_dir="${collision_dir}" mirror_y="${mirror_y}"/>
@@ -338,5 +361,5 @@
       <origin xyz="-0.0595 0 0.0735" rpy="${mirror_y * 1.5708} 0 ${mirror_y * 1.5708}"/>
       <axis xyz="0 0 -1"/>
-      <limit lower="-3.14159265" upper="3.14159265" effort="120" velocity="1.2"/>
+      <limit lower="${j2_lo}" upper="${j2_hi}" effort="120" velocity="1.2"/>
     </joint>
     <xacro:v5_imported_motor_link name="${side}_v5_link3" motor="motor3" color="${color}" visual_dir="${visual_dir}" collision_dir="${collision_dir}" mirror_y="${mirror_y}"/>
@@ -346,5 +369,5 @@
       <origin xyz="0 ${mirror_y * 0.6} -0.148" rpy="0 0 ${mirror_y * 3.1416}"/>
       <axis xyz="0 0 1"/>
-      <limit lower="-3.14159265" upper="3.14159265" effort="100" velocity="1.2"/>
+      <limit lower="${j3_lo}" upper="${j3_hi}" effort="100" velocity="1.2"/>
     </joint>
     <xacro:v5_imported_motor_link name="${side}_v5_link4" motor="motor4" color="${color}" visual_dir="${visual_dir}" collision_dir="${collision_dir}" mirror_y="${mirror_y}"/>
@@ -354,5 +377,5 @@
       <origin xyz="0 ${mirror_y * -0.412} 0.009" rpy="${mirror_y * 1.5708} -1.5708 0"/>
       <axis xyz="-1 0 0"/>
-      <limit lower="-3.14159265" upper="3.14159265" effort="60" velocity="1.5"/>
+      <limit lower="${j4_lo}" upper="${j4_hi}" effort="60" velocity="1.5"/>
     </joint>
     <xacro:v5_imported_motor_link name="${side}_v5_link5" motor="motor5" color="${color}" visual_dir="${visual_dir}" collision_dir="${collision_dir}" mirror_y="${mirror_y}"/>
@@ -362,5 +385,5 @@
       <origin xyz="0.0595 ${mirror_y * -0.074} 0" rpy="${mirror_y * -1.5708} 0 ${mirror_y * 1.5708}"/>
       <axis xyz="1 0 0"/>
-      <limit lower="-3.14159265" upper="3.14159265" effort="60" velocity="1.5"/>
+      <limit lower="${j5_lo}" upper="${j5_hi}" effort="60" velocity="1.5"/>
     </joint>
     <xacro:v5_imported_motor_link name="${side}_v5_link6" motor="motor6" color="${color}" visual_dir="${visual_dir}" collision_dir="${collision_dir}" mirror_y="${mirror_y}"/>
@@ -370,5 +393,5 @@
       <origin xyz="-0.06 ${mirror_y * -0.074} 0" rpy="${mirror_y * 1.5708} 0 0"/>
       <axis xyz="0 0 -1"/>
-      <limit lower="-3.14159265" upper="3.14159265" effort="40" velocity="1.5"/>
+      <limit lower="${j6_lo}" upper="${j6_hi}" effort="40" velocity="1.5"/>
     </joint>
     <link name="${side}_v5_tool0">
@@ -381,6 +404,20 @@
     </joint>
   </xacro:macro>
-  <xacro:v5_imported_arm side="left" mount_y="${v5_mount_y}" mirror_y="1" color="0.2 0.55 1.0 1" visual_dir="visual" collision_dir="collision"/>
-  <xacro:v5_imported_arm side="right" mount_y="${-v5_mount_y}" mirror_y="-1" color="1.0 0.55 0.2 1" visual_dir="visual_right" collision_dir="collision_right"/>
+  <!-- 左臂: j1 -180~0, j2 ±180, j3 ±180, j4 -90~270, j5 0~180, j6 ±180 -->
+  <xacro:v5_imported_arm side="left" mount_y="${v5_mount_y}" mirror_y="1" color="0.2 0.55 1.0 1" visual_dir="visual" collision_dir="collision"
+    j1_lo="-3.14159265" j1_hi="0"
+    j2_lo="-3.14159265" j2_hi="3.14159265"
+    j3_lo="-3.14159265" j3_hi="3.14159265"
+    j4_lo="-1.57079633" j4_hi="4.71238898"
+    j5_lo="-1.57079633" j5_hi="4.71238898"
+    j6_lo="-3.14159265" j6_hi="3.14159265"/>
+  <!-- 右臂: j1 0~180, j2 ±180, j3 ±180, j4 -270~90, j5 -180~0, j6 ±180 -->
+  <xacro:v5_imported_arm side="right" mount_y="${-v5_mount_y}" mirror_y="-1" color="1.0 0.55 0.2 1" visual_dir="visual_right" collision_dir="collision_right"
+    j1_lo="0" j1_hi="3.14159265"
+    j2_lo="-3.14159265" j2_hi="3.14159265"
+    j3_lo="-3.14159265" j3_hi="3.14159265"
+    j4_lo="-4.71238898" j4_hi="1.57079633"
+    j5_lo="-4.71238898" j5_hi="1.57079633"
+    j6_lo="-3.14159265" j6_hi="3.14159265"/>
   <xacro:alfa_robot_ros2_control
     name="alfa_robot"

File: ros2_ws/src/alfa_robot_description/urdf/alfa_robot/alfa_robot_macro.ros2_control.xacro (robot description, xacro)
@@ -88,15 +88,15 @@
         </joint>
       </xacro:macro>
-      <xacro:v5_proxy_control_joint joint_name="left_v5_joint1" lower="-3.14159265" upper="3.14159265" velocity="1.2"/>
-      <xacro:v5_proxy_control_joint joint_name="left_v5_joint2" lower="-1.57079632" upper="1.57079632" velocity="1.2"/>
-      <xacro:v5_proxy_control_joint joint_name="left_v5_joint3" lower="-2.35619449" upper="2.35619449" velocity="1.2"/>
-      <xacro:v5_proxy_control_joint joint_name="left_v5_joint4" lower="-3.14159265" upper="3.14159265" velocity="1.5"/>
-      <xacro:v5_proxy_control_joint joint_name="left_v5_joint5" lower="-1.57079632" upper="1.57079632" velocity="1.5"/>
+      <xacro:v5_proxy_control_joint joint_name="left_v5_joint1" lower="-3.14159265" upper="0" velocity="1.2"/>
+      <xacro:v5_proxy_control_joint joint_name="left_v5_joint2" lower="-3.14159265" upper="3.14159265" velocity="1.2"/>
+      <xacro:v5_proxy_control_joint joint_name="left_v5_joint3" lower="-3.14159265" upper="3.14159265" velocity="1.2"/>
+      <xacro:v5_proxy_control_joint joint_name="left_v5_joint4" lower="-1.57079633" upper="4.71238898" velocity="1.5"/>
+      <xacro:v5_proxy_control_joint joint_name="left_v5_joint5" lower="-1.57079633" upper="4.71238898" velocity="1.5"/>
       <xacro:v5_proxy_control_joint joint_name="left_v5_joint6" lower="-3.14159265" upper="3.14159265" velocity="1.5"/>
-      <xacro:v5_proxy_control_joint joint_name="right_v5_joint1" lower="-3.14159265" upper="3.14159265" velocity="1.2"/>
-      <xacro:v5_proxy_control_joint joint_name="right_v5_joint2" lower="-1.57079632" upper="1.57079632" velocity="1.2"/>
-      <xacro:v5_proxy_control_joint joint_name="right_v5_joint3" lower="-2.35619449" upper="2.35619449" velocity="1.2"/>
-      <xacro:v5_proxy_control_joint joint_name="right_v5_joint4" lower="-3.14159265" upper="3.14159265" velocity="1.5"/>
-      <xacro:v5_proxy_control_joint joint_name="right_v5_joint5" lower="-1.57079632" upper="1.57079632" velocity="1.5"/>
+      <xacro:v5_proxy_control_joint joint_name="right_v5_joint1" lower="0" upper="3.14159265" velocity="1.2"/>
+      <xacro:v5_proxy_control_joint joint_name="right_v5_joint2" lower="-3.14159265" upper="3.14159265" velocity="1.2"/>
+      <xacro:v5_proxy_control_joint joint_name="right_v5_joint3" lower="-3.14159265" upper="3.14159265" velocity="1.2"/>
+      <xacro:v5_proxy_control_joint joint_name="right_v5_joint4" lower="-4.71238898" upper="1.57079633" velocity="1.5"/>
+      <xacro:v5_proxy_control_joint joint_name="right_v5_joint5" lower="-4.71238898" upper="1.57079633" velocity="1.5"/>
       <xacro:v5_proxy_control_joint joint_name="right_v5_joint6" lower="-3.14159265" upper="3.14159265" velocity="1.5"/>
     </ros2_control>

File: ros2_ws/src/alfa_robot_moveit_config/config/alfa_robot.ros2_control.xacro (robot description, xacro)
@@ -7,4 +7,5 @@
                 <!-- By default, set up controllers for simulation. This won't work on real hardware -->
                 <plugin>mock_components/GenericSystem</plugin>
+                <param name="mock_sensor_commands">true</param>
             </hardware>
             <joint name="pitch">

Commit message: feat: v5 机械臂简化碰撞模型 + SRDF end_effector 完善
- 大臂/小臂改为圆柱体碰撞几何（radius=0.05, length 对应实际长度）
- 调整 inertial origin 和 joint offset 以匹配简化模型
- SRDF 移除 turn关节，增加 left/right_suction_with_base、dual_left/right_suction end_effector
- 刷新 v5 机械臂 visual/collision mesh 文件

Co-Authored-By: Claude Opus 4.7 <noreply@anthropic.com>

File: ros2_ws/src/alfa_robot_description/urdf/alfa_robot.urdf.xacro (robot description, xacro)
@@ -301,19 +301,19 @@
       <limit lower="-3.14159265" upper="3.14159265" effort="120" velocity="1.2"/>
     </joint>
-    <!-- ========== big_arm (fixed from link2) ========== -->
+    <!-- ========== big_arm (fixed from link2, straight cylinder along its local Z) ========== -->
     <link name="${side}_v5_big_arm">
       <inertial>
-        <origin xyz="1.66533453693773E-16 ${mirror_y * 1.66533453693773E-16} 0.192" rpy="0 0 0"/>
+        <origin xyz="0 0 0.1785" rpy="0 0 0"/>
         <mass value="1.15977547674044"/>
         <inertia ixx="0.0245288914447722" ixy="${mirror_y * 5.00652940690442E-18}" ixz="-1.04636466228108E-17" iyy="0.0245288914447722" iyz="${mirror_y * -2.19397400103325E-17}" izz="0.00328554236419837"/>
       </inertial>
       <visual>
-        <origin xyz="0 0 0" rpy="0 0 0"/>
-        <geometry><mesh filename="${v5_mesh_base}/${visual_dir}/big_arm.STL"/></geometry>
-        <material name="v5_imported_mesh_mat"><color rgba="${color}"/></material>
-      </visual>
-      <collision>
-        <origin xyz="0 0 0" rpy="0 0 0"/>
-        <geometry><mesh filename="${v5_mesh_base}/${collision_dir}/big_arm.STL"/></geometry>
+        <origin xyz="0 0 0.1785" rpy="0 0 0"/>
+        <geometry><cylinder radius="0.05" length="0.3570"/></geometry>
+        <material name="v5_arm_mat"><color rgba="${color}"/></material>
+      </visual>
+      <collision>
+        <origin xyz="0 0 0.1785" rpy="0 0 0"/>
+        <geometry><cylinder radius="0.05" length="0.3570"/></geometry>
       </collision>
     </link>
@@ -343,5 +343,5 @@
       <parent link="${side}_v5_big_arm"/>
       <child link="${side}_v5_big_arm_2"/>
-      <origin xyz="0 0 0.384" rpy="0 0 0"/>
+      <origin xyz="0 0 0.3570" rpy="0 0 0"/>
     </joint>
     <!-- ========== link3 (motor3) ========== -->
@@ -372,16 +372,16 @@
     <link name="${side}_v5_little_arm">
       <inertial>
-        <origin xyz="3.12250225675825E-17 ${mirror_y * 4.5102810375397E-17} 0.0807664410058027" rpy="0 0 0"/>
+        <origin xyz="0 ${mirror_y * 0} 0.1190" rpy="0 0 0"/>
         <mass value="0.819573036601734"/>
         <inertia ixx="0.00487621643874643" ixy="${mirror_y * -6.941435002749E-19}" ixz="-1.40385385199839E-18" iyy="0.00487621643874643" iyz="${mirror_y * -2.99487714303266E-18}" izz="0.00230784421862048"/>
       </inertial>
       <visual>
-        <origin xyz="0 0 0" rpy="0 0 0"/>
-        <geometry><mesh filename="${v5_mesh_base}/${visual_dir}/little_arm.STL"/></geometry>
-        <material name="v5_imported_mesh_mat"><color rgba="${color}"/></material>
-      </visual>
-      <collision>
-        <origin xyz="0 0 0" rpy="0 0 0"/>
-        <geometry><mesh filename="${v5_mesh_base}/${collision_dir}/little_arm.STL"/></geometry>
+        <origin xyz="0 0 0.1190" rpy="0 0 0"/>
+        <geometry><cylinder radius="0.05" length="0.2380"/></geometry>
+        <material name="v5_arm_mat"><color rgba="${color}"/></material>
+      </visual>
+      <collision>
+        <origin xyz="0 0 0.1190" rpy="0 0 0"/>
+        <geometry><cylinder radius="0.05" length="0.2380"/></geometry>
       </collision>
     </link>
@@ -411,5 +411,5 @@
       <parent link="${side}_v5_little_arm"/>
       <child link="${side}_v5_link4"/>
-      <origin xyz="0 0 0.211" rpy="0 0 0"/>
+      <origin xyz="0 0 0.2380" rpy="0 0 0"/>
       <axis xyz="0 0 1"/>
       <limit lower="-3.14159265" upper="3.14159265" effort="60" velocity="1.5"/>
