Commit message: fix: 调整 v5 单圈关节限位和预览初始姿态
- 将 v5 六轴关节按单圈 revolute 限位同步到 URDF 和 MoveIt 配置

- 为 description 预览 launch 增加 v5 初始角注入，匹配 remap 后姿态

- 修正 right_v5_joint1 和 right_v5_joint4 的直观零位语义

Co-Authored-By: Codex <codex@openai.com>

File: ros2_ws/src/alfa_robot_description/urdf/alfa_robot.urdf.xacro (robot description, xacro)
@@ -263,5 +263,5 @@
     <child link="left_v5_link1"/>
     <axis xyz="0 0 1"/>
-    <limit lower="-3.14159265" upper="0" effort="120" velocity="1.2"/>
+    <limit lower="-3.14159265" upper="3.14159265" effort="120" velocity="1.2"/>
   </joint>
   <link name="left_v5_link2">
@@ -287,5 +287,5 @@
     <child link="left_v5_link2"/>
     <axis xyz="0 0 1"/>
-    <limit lower="-3.14159265" upper="3.14159265" effort="120" velocity="1.2"/>
+    <limit lower="-1.57079633" upper="4.71238898" effort="120" velocity="1.2"/>
   </joint>
   <link name="left_v5_link3">
@@ -311,5 +311,5 @@
     <child link="left_v5_link3"/>
     <axis xyz="0 0 1"/>
-    <limit lower="0" upper="6.28318530" effort="100" velocity="1.2"/>
+    <limit lower="3.14159265" upper="9.42477795" effort="100" velocity="1.2"/>
   </joint>
   <link name="left_v5_link4">
@@ -335,5 +335,5 @@
     <child link="left_v5_link4"/>
     <axis xyz="0 0 1"/>
-    <limit lower="-1.57079633" upper="4.71238898" effort="60" velocity="1.5"/>
+    <limit lower="-3.14159265" upper="3.14159265" effort="60" velocity="1.5"/>
   </joint>
   <link name="left_v5_link5">
@@ -359,5 +359,5 @@
     <child link="left_v5_link5"/>
     <axis xyz="0 0 1"/>
-    <limit lower="-1.57079633" upper="4.71238898" effort="60" velocity="1.5"/>
+    <limit lower="3.14159265" upper="9.42477795" effort="60" velocity="1.5"/>
   </joint>
   <link name="left_v5_link6">
@@ -433,5 +433,5 @@
     <child link="right_v5_link1"/>
     <axis xyz="0 0 1"/>
-    <limit lower="0" upper="3.14159265" effort="120" velocity="1.2"/>
+    <limit lower="-3.14159265" upper="3.14159265" effort="120" velocity="1.2"/>
   </joint>
   <link name="right_v5_link2">
@@ -457,5 +457,5 @@
     <child link="right_v5_link2"/>
     <axis xyz="0 0 1"/>
-    <limit lower="-3.14159265" upper="3.14159265" effort="120" velocity="1.2"/>
+    <limit lower="-1.57079633" upper="4.71238898" effort="120" velocity="1.2"/>
   </joint>
   <link name="right_v5_link3">
@@ -505,5 +505,5 @@
     <child link="right_v5_link4"/>
     <axis xyz="0 0 1"/>
-    <limit lower="-4.71238898" upper="1.57079633" effort="60" velocity="1.5"/>
+    <limit lower="-3.14159265" upper="3.14159265" effort="60" velocity="1.5"/>
   </joint>
   <link name="right_v5_link5">
@@ -529,5 +529,5 @@
     <child link="right_v5_link5"/>
     <axis xyz="0 0 1"/>
-    <limit lower="-4.71238898" upper="1.57079633" effort="60" velocity="1.5"/>
+    <limit lower="-3.14159265" upper="3.14159265" effort="60" velocity="1.5"/>
   </joint>
   <link name="right_v5_link6">

Commit message: Refs MOTION-30: 同步 v5 上半身模型状态
- 复刻 8f911db 的 v5 上半身 mesh 来源和安装位姿同步

- 更新 ROS description 与 MuJoCo alfa_robot.xml，保持 IK/仿真机器人状态一致

Co-Authored-By: Codex <codex@openai.com>

File: ros2_ws/src/alfa_robot_description/urdf/alfa_robot.urdf.xacro (robot description, xacro)
@@ -79,5 +79,5 @@
       <geometry>
         <mesh
-          filename="package://alfa_robot_description/meshes/alfa_robot_v2_arm_v4_new/visual/pitch.STL" />
+          filename="package://alfa_robot_description/meshes/alfa_robot_v2_arm_v5/visual/pitch.STL" />
       </geometry>
       <material
@@ -93,5 +93,5 @@
       <geometry>
         <mesh
-          filename="package://alfa_robot_description/meshes/alfa_robot_v2_arm_v4_new/collision/pitch.STL" />
+          filename="package://alfa_robot_description/meshes/alfa_robot_v2_arm_v5/collision/pitch.STL" />
       </geometry>
     </collision>
@@ -137,5 +137,5 @@
       <geometry>
         <mesh
-          filename="package://alfa_robot_description/meshes/alfa_robot/visual/turn.STL" />
+          filename="package://alfa_robot_description/meshes/alfa_robot_v2_arm_v5/visual/turn.STL" />
       </geometry>
       <material
@@ -151,5 +151,5 @@
       <geometry>
         <mesh
-          filename="package://alfa_robot_description/meshes/alfa_robot/collision/turn.STL" />
+          filename="package://alfa_robot_description/meshes/alfa_robot_v2_arm_v5/collision/turn.STL" />
       </geometry>
     </collision>
@@ -159,5 +159,5 @@
     type="continuous">
     <origin
-      xyz="0 0 0"
+      xyz="-0.189 0.0545 0.12"
       rpy="0 0 0" />
     <parent
@@ -190,5 +190,5 @@
       <geometry>
         <mesh
-          filename="package://alfa_robot_description/meshes/alfa_robot/visual/updown.STL" />
+          filename="package://alfa_robot_description/meshes/alfa_robot_v2_arm_v5/visual/updown.STL" />
       </geometry>
       <material
@@ -204,5 +204,5 @@
       <geometry>
         <mesh
-          filename="package://alfa_robot_description/meshes/alfa_robot/collision/updown.STL" />
+          filename="package://alfa_robot_description/meshes/alfa_robot_v2_arm_v5/collision/updown.STL" />
       </geometry>
     </collision>
@@ -212,5 +212,5 @@
     type="prismatic">
     <origin
-      xyz="-0.23547 0 0.57771"
+      xyz="-0.07 0.0005 0.0645"
       rpy="0 0 0" />
     <parent
@@ -239,5 +239,5 @@
     <parent link="updown"/>
     <child link="left_v5_link0"/>
-    <origin xyz="0 0.20 0.18" rpy="0 0 0"/>
+    <origin xyz="0.105 0.26 0.2" rpy="0 0 0"/>
   </joint>
   <link name="left_v5_link1">
@@ -409,5 +409,5 @@
     <parent link="updown"/>
     <child link="right_v5_link0"/>
-    <origin xyz="0 -0.20 0.18" rpy="0 0 0"/>
+    <origin xyz="0.105 -0.26 0.2" rpy="0 0 0"/>
   </joint>
   <link name="right_v5_link1">
