Commit message: fix(motion): 对齐 v5 零位与 tool0 末端语义
- 将 joint1 的 30° 机械姿态烘进 URDF origin，使控制和 MoveIt 中 joint1=0 呈现正确姿态。

- 将 SRDF end_effector parent_link 对齐到左右 tool0，并同步 home、initial_positions 与 ros2_control 初始值。

- 调整 IK benchmark 的 tool0_offset 为 0.0，恢复固定 64 次候选 smoke 成功。

Refs MOTION-33

Co-Authored-By: Codex <codex@openai.com>

File: ros2_ws/src/alfa_robot_description/urdf/alfa_robot.urdf.xacro (robot description, xacro)
@@ -235,13 +235,4 @@
       <inertia ixx="0.000741163324579453" ixy="0" ixz="6.73482801154554E-20" iyy="0.000741163324579453" iyz="0" izz="0.00132016293912598"/>
     </inertial>
-    <visual>
-      <origin xyz="0 0 0" rpy="0 0 0"/>
-      <geometry><mesh filename="${mesh_base}/visual_mirrored_y/base.STL"/></geometry>
-      <material name=""><color rgba="0.2 0.55 1.0 1"/></material>
-    </visual>
-    <collision>
-      <origin xyz="0 0 0" rpy="0 0 0"/>
-      <geometry><mesh filename="${mesh_base}/collision_mirrored_y/base.STL"/></geometry>
-    </collision>
   </link>
   <joint name="left_v5_mount" type="fixed">
@@ -267,5 +258,5 @@
   </link>
   <joint name="left_v5_joint1" type="revolute">
-    <origin xyz="0 0 0.056" rpy="0 0 0"/>
+    <origin xyz="0 0 0" rpy="0 0 -0.52359878"/>
     <parent link="left_v5_link0"/>
     <child link="left_v5_link1"/>
@@ -398,5 +389,5 @@
     <parent link="left_v5_link6"/>
     <child link="left_v5_tool0"/>
-    <origin xyz="0 0 0.1" rpy="0 0 0"/>
+    <origin xyz="0 0 0.1" rpy="0.00000188634799516 0.00363531907027 0.523587766715"/>
   </joint>
   <!-- ========== RIGHT ARM (right_v5_joint1-6) ========== -->
@@ -407,13 +398,4 @@
       <inertia ixx="0.000741163324579453" ixy="-1.92778886435101E-35" ixz="6.73482801154554E-20" iyy="0.000741163324579453" iyz="7.56724488341848E-35" izz="0.00132016293912598"/>
     </inertial>
-    <visual>
-      <origin xyz="0 0 0" rpy="0 0 0"/>
-      <geometry><mesh filename="${mesh_base}/visual/base.STL"/></geometry>
-      <material name=""><color rgba="1.0 0.55 0.2 1"/></material>
-    </visual>
-    <collision>
-      <origin xyz="0 0 0" rpy="0 0 0"/>
-      <geometry><mesh filename="${mesh_base}/collision/base.STL"/></geometry>
-    </collision>
   </link>
   <joint name="right_v5_mount" type="fixed">
@@ -439,5 +421,5 @@
   </link>
   <joint name="right_v5_joint1" type="revolute">
-    <origin xyz="0 0 0.056" rpy="0 0 0"/>
+    <origin xyz="0 0 0" rpy="0 0 0.52359878"/>
     <parent link="right_v5_link0"/>
     <child link="right_v5_link1"/>
@@ -570,5 +552,5 @@
     <parent link="right_v5_link6"/>
     <child link="right_v5_tool0"/>
-    <origin xyz="0 0 0.1" rpy="0 0 0"/>
+    <origin xyz="0 0 0.1" rpy="-0.00000188633751216 0.00363531853545 -0.523587767584"/>
   </joint>
   <xacro:alfa_robot_ros2_control

File: ros2_ws/src/alfa_robot_description/urdf/alfa_robot/alfa_robot_macro.ros2_control.xacro (robot description, xacro)
@@ -11,5 +11,7 @@
                real_hardware_plugin:=alfa_robot_hardware/AlfaRobotHW
                canopen_profile_velocity:=50000
-               canopen_profile_accel:=50000"
+               canopen_profile_accel:=50000
+               left_v5_joint1_initial:=0.0
+               right_v5_joint1_initial:=0.0"
                >
     <ros2_control name="${name}" type="system">
@@ -75,5 +77,5 @@
       </joint>
       <!-- v5 proxy arms (position controlled) -->
-      <xacro:macro name="v5_proxy_control_joint" params="joint_name lower upper velocity">
+      <xacro:macro name="v5_proxy_control_joint" params="joint_name lower upper velocity initial_value:=0.0">
         <joint name="${prefix}${joint_name}">
           <command_interface name="position">
@@ -82,5 +84,5 @@
           </command_interface>
           <state_interface name="position">
-            <param name="initial_value">0.0</param>
+            <param name="initial_value">${initial_value}</param>
           </state_interface>
           <state_interface name="velocity"/>
@@ -88,5 +90,5 @@
         </joint>
       </xacro:macro>
-      <xacro:v5_proxy_control_joint joint_name="left_v5_joint1" lower="-3.14159265" upper="3.14159265" velocity="1.2"/>
+      <xacro:v5_proxy_control_joint joint_name="left_v5_joint1" lower="-3.14159265" upper="3.14159265" velocity="1.2" initial_value="${left_v5_joint1_initial}"/>
       <xacro:v5_proxy_control_joint joint_name="left_v5_joint2" lower="-1.57079633" upper="4.71238898" velocity="1.2"/>
       <xacro:v5_proxy_control_joint joint_name="left_v5_joint3" lower="-3.14159265" upper="3.14159265" velocity="1.2"/>
@@ -94,5 +96,5 @@
       <xacro:v5_proxy_control_joint joint_name="left_v5_joint5" lower="-3.14159265" upper="3.14159265" velocity="1.5"/>
       <xacro:v5_proxy_control_joint joint_name="left_v5_joint6" lower="-3.14159265" upper="3.14159265" velocity="1.5"/>
-      <xacro:v5_proxy_control_joint joint_name="right_v5_joint1" lower="-3.14159265" upper="3.14159265" velocity="1.2"/>
+      <xacro:v5_proxy_control_joint joint_name="right_v5_joint1" lower="-3.14159265" upper="3.14159265" velocity="1.2" initial_value="${right_v5_joint1_initial}"/>
       <xacro:v5_proxy_control_joint joint_name="right_v5_joint2" lower="-1.57079633" upper="4.71238898" velocity="1.2"/>
       <xacro:v5_proxy_control_joint joint_name="right_v5_joint3" lower="-3.14159265" upper="3.14159265" velocity="1.2"/>

Commit message: feat(description): 接入 v6 机械臂模型资产
- 新增 v6 视觉/碰撞网格和原始 URDF 参考文件。

- 将主 URDF 映射到 v6 模型并同步 ros2_control 初始配置。

- 更新 MoveIt 初始姿态说明与 joint2 关节限位。

Co-Authored-By: Codex <codex@openai.com>

File: ros2_ws/src/alfa_robot_description/urdf/alfa_robot.urdf.xacro (robot description, xacro)
@@ -17,221 +17,118 @@
     <origin xyz="0 0 0.09" rpy="0 0 0"/>
   </joint>
-  <link
-    name="base_link">
-    <inertial>
-      <origin
-        xyz="-0.44193110855616 0.000259961331933109 0.176428166472852"
-        rpy="0 0 0" />
-      <mass
-        value="394.931465036981" />
-      <inertia
-        ixx="66.5681215725466"
-        ixy="5.74775273893285E-10"
-        ixz="9.85014992290203"
-        iyy="65.6389024339403"
-        iyz="2.76043934386688E-09"
-        izz="112.938477587322" />
-    </inertial>
-    <visual>
-      <origin
-        xyz="0 0 0"
-        rpy="0 0 0" />
-      <geometry>
-        <mesh
-          filename="package://alfa_robot_description/meshes/alfa_robot/visual/base_link.STL" />
-      </geometry>
-      <material
-        name="blue">
-        <color
-          rgba="0 0 1 1" />
-      </material>
-    </visual>
-    <collision>
-      <origin
-        xyz="0 0 0"
-        rpy="0 0 0" />
-      <geometry>
-        <mesh
-          filename="package://alfa_robot_description/meshes/alfa_robot/collision/base_link.STL" />
-      </geometry>
-    </collision>
-  </link>
-  <link
-    name="pitch">
-    <inertial>
-      <origin
-        xyz="-0.198797876667389 0.0534826037691441 0.0683908156328275"
-        rpy="0 0 0" />
-      <mass
-        value="5.23479125794249" />
-      <inertia
-        ixx="0.0820011779740888"
-        ixy="1.65869977323853E-10"
-        ixz="-1.12757025938492E-17"
-        iyy="0.0820529172807708"
-        iyz="-2.38941055572563E-17"
-        izz="0.163475256832643" />
-    </inertial>
-    <visual>
-      <origin
-        xyz="0 0 0"
-        rpy="0 0 0" />
-      <geometry>
-        <mesh
-          filename="package://alfa_robot_description/meshes/alfa_robot_v2_arm_v5/visual/pitch.STL" />
-      </geometry>
-      <material
-        name="">
-        <color
-          rgba="1 1 1 1" />
-      </material>
-    </visual>
-    <collision>
-      <origin
-        xyz="0 0 0"
-        rpy="0 0 0" />
-      <geometry>
-        <mesh
-          filename="package://alfa_robot_description/meshes/alfa_robot_v2_arm_v5/collision/pitch.STL" />
-      </geometry>
-    </collision>
-  </link>
-  <joint
-    name="pitch"
-    type="revolute">
-    <origin
-      xyz="0.3 -0.05 0.129"
-      rpy="0 0 0" />
-    <parent
-      link="base_link" />
-    <child
-      link="pitch" />
-    <axis
-      xyz="0 1 0" />
-    <limit
-      lower="0"
-      upper="0.26"
-      effort="0"
-      velocity="0" />
-  </joint>
-  <link
-    name="turn">
-    <inertial>
-      <origin
-        xyz="-0.0697894032768815 -0.00012433244764639 0.982155423971065"
-        rpy="0 0 0" />
-      <mass
-        value="42.0737844290435" />
-      <inertia
-        ixx="10.0720353784748"
-        ixy="-1.75362629131178E-06"
-        ixz="5.29823321336754E-05"
-        iyy="10.0937833616587"
-        iyz="1.43589075450652E-06"
-        izz="0.327199381319826" />
-    </inertial>
-    <visual>
-      <origin
-        xyz="0 0 0"
-        rpy="0 0 0" />
-      <geometry>
-        <mesh
-          filename="package://alfa_robot_description/meshes/alfa_robot_v2_arm_v5/visual/turn.STL" />
-      </geometry>
-      <material
-        name="arm_grey">
-        <color
-          rgba="0.5 0.5 0.5 1" />
-      </material>
-    </visual>
-    <collision>
-      <origin
-        xyz="0 0 0"
-        rpy="0 0 0" />
-      <geometry>
-        <mesh
-          filename="package://alfa_robot_description/meshes/alfa_robot_v2_arm_v5/collision/turn.STL" />
-      </geometry>
-    </collision>
-  </link>
-  <joint
-    name="turn"
-    type="continuous">
-    <origin
-      xyz="-0.189 0.0545 0.12"
-      rpy="0 0 0" />
-    <parent
-      link="pitch" />
-    <child
-      link="turn" />
-    <axis
-      xyz="0 0 1" />
-  </joint>
-  <link
-    name="updown">
-    <inertial>
-      <origin
-        xyz="-0.196828632659582 0.0148673483555221 0.0956849238503419"
-        rpy="0 0 0" />
-      <mass
-        value="26.931167747836" />
-      <inertia
-        ixx="0.231217459750122"
-        ixy="2.93337887014215E-05"
-        ixz="0.000951254936009737"
-        iyy="0.178754005132662"
-        iyz="-1.44830456938328E-05"
-        izz="0.348822965146485" />
-    </inertial>
-    <visual>
-      <origin
-        xyz="0 0 0"
-        rpy="0 0 0" />
-      <geometry>
-        <mesh
-          filename="package://alfa_robot_description/meshes/alfa_robot_v2_arm_v5/visual/updown.STL" />
-      </geometry>
-      <material
-        name="arm_grey">
-        <color
-          rgba="0.5 0.5 0.5 1" />
-      </material>
-    </visual>
-    <collision>
-      <origin
-        xyz="0 0 0"
-        rpy="0 0 0" />
-      <geometry>
-        <mesh
-          filename="package://alfa_robot_description/meshes/alfa_robot_v2_arm_v5/collision/updown.STL" />
-      </geometry>
-    </collision>
-  </link>
-  <joint
-    name="updown"
-    type="prismatic">
-    <origin
-      xyz="-0.07 0.0005 0.0645"
-      rpy="0 0 0" />
-    <parent
-      link="turn" />
-    <child
-      link="updown" />
-    <axis
-      xyz="0 0 1" />
-    <limit
-      lower="0"
-      upper="0.99"
-      effort="0"
-      velocity="0" />
-  </joint>
-  <!-- Mesh base path for latest single-arm v5_6 model -->
-  <xacro:property name="mesh_base" value="package://alfa_robot_description/meshes/alfa_robot_arm_v5_6"/>
-  <!-- ========== LEFT ARM (left_v5_joint1-6) ========== -->
+<link name="base_link">
+    <inertial>
+      <origin xyz="-0.230864859994365 -3.59465059753261E-05 0.00982453569098829" rpy="0 0 0" />
+      <mass value="452.254374649793" />
+      <inertia ixx="42.2528118012676" ixy="2.90433873726581E-05" ixz="5.29862244779797" iyy="45.7334828734001" iyz="-7.53976926824646E-07" izz="73.6321595788915" />
+    </inertial>
+    <visual>
+      <origin xyz="0 0 0" rpy="0 0 0" />
+      <geometry>
+        <mesh filename="package://alfa_robot_description/meshes/alfa_robot_v2_arm_v6/visual/base_link.STL" />
+      </geometry>
+      <material name="">
+        <color rgba="0.752941176470588 0.752941176470588 0.752941176470588 1" />
+      </material>
+    </visual>
+    <collision>
+      <origin xyz="0 0 0" rpy="0 0 0" />
+      <geometry>
+        <mesh filename="package://alfa_robot_description/meshes/alfa_robot_v2_arm_v6/collision/base_link.STL" />
+      </geometry>
+    </collision>
+  </link>
+<link name="pitch">
+    <inertial>
+      <origin xyz="-0.197037068600063 0.0545002757388739 0.0847212210627051" rpy="0 0 0" />
+      <mass value="31.6067905352622" />
+      <inertia ixx="0.518725062034511" ixy="2.02803901410849E-08" ixz="-0.00603915225902053" iyy="0.579528262067602" iyz="3.22538967579058E-07" izz="1.06221345040969" />
+    </inertial>
+    <visual>
+      <origin xyz="0 0 0" rpy="0 0 0" />
+      <geometry>
+        <mesh filename="package://alfa_robot_description/meshes/alfa_robot_v2_arm_v6/visual/pitch.STL" />
+      </geometry>
+      <material name="">
+        <color rgba="0.752941176470588 0.752941176470588 0.752941176470588 1" />
+      </material>
+    </visual>
+    <collision>
+      <origin xyz="0 0 0" rpy="0 0 0" />
+      <geometry>
+        <mesh filename="package://alfa_robot_description/meshes/alfa_robot_v2_arm_v6/collision/pitch.STL" />
+      </geometry>
+    </collision>
+  </link>
+<joint name="pitch" type="revolute">
+    <origin xyz="0.25918 -0.0545 0.05" rpy="0 0 0" />
+    <parent link="base_link" />
+    <child link="pitch" />
+    <axis xyz="0 1 0" />
+    <limit lower="0" upper="0.26" effort="0" velocity="0" />
+  </joint>
+<link name="turn">
+    <inertial>
+      <origin xyz="-0.00579960525321255 -7.81089694046333E-06 1.06475532040538" rpy="0 0 0" />
+      <mass value="52.9957329420753" />
+      <inertia ixx="7.51064439986969" ixy="5.95969545267824E-06" ixz="0.221612834319679" iyy="7.73162717719144" iyz="-8.94723713424965E-06" izz="0.725095105907374" />
+    </inertial>
+    <visual>
+      <origin xyz="0 0 0" rpy="0 0 0" />
+      <geometry>
+        <mesh filename="package://alfa_robot_description/meshes/alfa_robot_v2_arm_v6/visual/turn.STL" />
+      </geometry>
+      <material name="">
+        <color rgba="0.752941176470588 0.752941176470588 0.752941176470588 1" />
+      </material>
+    </visual>
+    <collision>
+      <origin xyz="0 0 0" rpy="0 0 0" />
+      <geometry>
+        <mesh filename="package://alfa_robot_description/meshes/alfa_robot_v2_arm_v6/collision/turn.STL" />
+      </geometry>
+    </collision>
+  </link>
+<joint name="turn" type="continuous">
+    <origin xyz="-0.18924 0.0545 0.135" rpy="0 0 0" />
+    <parent link="pitch" />
+    <child link="turn" />
+    <axis xyz="0 0 1" />
+  </joint>
+<link name="updown">
+    <inertial>
+      <origin xyz="0.0601856186326954 3.82033426615802E-07 0.101233179160814" rpy="0 0 0" />
+      <mass value="28.1491686567643" />
+      <inertia ixx="1.18481506897735" ixy="-3.87618830042902E-08" ixz="-0.00404701824967137" iyy="0.266184937066632" iyz="7.22041694632457E-11" izz="1.39675046484991" />
+    </inertial>
+    <visual>
+      <origin xyz="0 0 0" rpy="0 0 0" />
+      <geometry>
+        <mesh filename="package://alfa_robot_description/meshes/alfa_robot_v2_arm_v6/visual/updown.STL" />
+      </geometry>
+      <material name="">
+        <color rgba="0.752941176470588 0.752941176470588 0.752941176470588 1" />
+      </material>
+    </visual>
+    <collision>
+      <origin xyz="0 0 0" rpy="0 0 0" />
+      <geometry>
+        <mesh filename="package://alfa_robot_description/meshes/alfa_robot_v2_arm_v6/collision/updown.STL" />
+      </geometry>
+    </collision>
+  </link>
+<joint name="updown" type="prismatic">
+    <origin xyz="-0.079765 0 0.038925" rpy="0 0 0" />
+    <parent link="turn" />
+    <child link="updown" />
+    <axis xyz="0 0 1" />
+    <limit lower="0" upper="0.99" effort="0" velocity="0" />
+  </joint>
+  <!-- ========== LEFT ARM v6 mapped to left_v5_* names ========== -->
   <link name="left_v5_link0">
     <inertial>
-      <origin xyz="0 0 0.01670398103" rpy="0 0 0"/>
-      <mass value="0.310084776766906"/>
-      <inertia ixx="0.000741163324579453" ixy="0" ixz="6.73482801154554E-20" iyy="0.000741163324579453" iyz="0" izz="0.00132016293912598"/>
+      <origin xyz="0 0 0" rpy="0 0 0"/>
+      <mass value="0.001"/>
+      <inertia ixx="1e-6" ixy="0" ixz="0" iyy="1e-6" iyz="0" izz="1e-6"/>
     </inertial>
   </link>
@@ -239,143 +136,179 @@
     <parent link="updown"/>
     <child link="left_v5_link0"/>
-    <origin xyz="0.105 0.26 0.2" rpy="0 0 0"/>
-  </joint>
-  <link name="left_v5_link1">
-    <inertial>
-      <origin xyz="-0.004752553966 0.008497713108 0.05815985177" rpy="0 0 0"/>
-      <mass value="1.74726890834066"/>
-      <inertia ixx="0.00457134350611956" ixy="0.0002288805479" ixz="1.99526917072982E-05" iyy="0.00429016337003855" iyz="-3.566115088e-05" izz="0.00359307936517085"/>
-    </inertial>
-    <visual>
-      <origin xyz="0 0 0" rpy="0 0 0"/>
-      <geometry><mesh filename="${mesh_base}/visual_mirrored_y/link1.STL"/></geometry>
-      <material name=""><color rgba="0.2 0.55 1.0 1"/></material>
-    </visual>
-    <collision>
-      <origin xyz="0 0 0" rpy="0 0 0"/>
-      <geometry><mesh filename="${mesh_base}/collision_mirrored_y/link1.STL"/></geometry>
-    </collision>
-  </link>
-  <joint name="left_v5_joint1" type="revolute">
-    <origin xyz="0 0 0" rpy="0 0 -0.52359878"/>
-    <parent link="left_v5_link0"/>
-    <child link="left_v5_link1"/>
-    <axis xyz="0 0 -1"/>
-    <limit lower="-3.14159265" upper="3.14159265" effort="120" velocity="1.2"/>
-  </joint>
-  <link name="left_v5_link2">
-    <inertial>
-      <origin xyz="-0.1999998828 -0.0002164972132 0.04318701696" rpy="0 0 0"/>
-      <mass value="6.19241787742505"/>
-      <inertia ixx="0.017665290529847" ixy="-3.290895014e-05" ixz="-8.38471642040595E-17" iyy="0.048066506145401" iyz="0" izz="0.0543426112488358"/>
-    </inertial>
-    <visual>
-      <origin xyz="0 0 0" rpy="0 0 0"/>
-      <geometry><mesh filename="${mesh_base}/visual_mirrored_y/link2.STL"/></geometry>
-      <material name=""><color rgba="0.2 0.55 1.0 1"/></material>
-    </visual>
-    <collision>
-      <origin xyz="0 0 0" rpy="0 0 0"/>
-      <geometry><mesh filename="${mesh_base}/collision_mirrored_y/link2.STL"/></geometry>
-    </collision>
-  </link>
-  <joint name="left_v5_joint2" type="revolute">
-    <origin xyz="-0.048573 0.086838 0.058" rpy="1.060792654 1.570792654 3.141592654"/>
-    <parent link="left_v5_link1"/>
-    <child link="left_v5_link2"/>
-    <axis xyz="0 0 1"/>
-    <limit lower="-1.57079633" upper="4.71238898" effort="120" velocity="1.2"/>
-  </joint>
-  <link name="left_v5_link3">
-    <inertial>
-      <origin xyz="0.07409140733 -1.001705375e-09 0.07364765219" rpy="0 0 0"/>
-      <mass value="1.90258780164428"/>
-      <inertia ixx="0.00411572596862418" ixy="3.019111472e-09" ixz="-0.00120850135091154" iyy="0.00644066810590579" iyz="2.228072963e-09" izz="0.0058105765548736"/>
-    </inertial>
-    <visual>
-      <origin xyz="0 0 0" rpy="0 0 0"/>
-      <geometry><mesh filename="${mesh_base}/visual_mirrored_y/link3.STL"/></geometry>
-      <material name=""><color rgba="0.2 0.55 1.0 1"/></material>
-    </visual>
-    <collision>
-      <origin xyz="0 0 0" rpy="0 0 0"/>
-      <geometry><mesh filename="${mesh_base}/collision_mirrored_y/link3.STL"/></geometry>
-    </collision>
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
File: ros2_ws/src/alfa_robot_description/urdf/alfa_robot/alfa_robot_macro.ros2_control.xacro (robot description, xacro)
@@ -104,5 +104,5 @@
       </xacro:macro>
       <xacro:v5_proxy_control_joint joint_name="left_v5_joint1" lower="-3.14159265" upper="3.14159265" velocity="1.2" initial_value="${left_v5_joint1_initial}"/>
-      <xacro:v5_proxy_control_joint joint_name="left_v5_joint2" lower="-1.57079633" upper="4.71238898" velocity="1.2" initial_value="${left_v5_joint2_initial}"/>
+      <xacro:v5_proxy_control_joint joint_name="left_v5_joint2" lower="-3.14" upper="3.14" velocity="1.2" initial_value="${left_v5_joint2_initial}"/>
       <xacro:v5_proxy_control_joint joint_name="left_v5_joint3" lower="-3.14159265" upper="3.14159265" velocity="1.2" initial_value="${left_v5_joint3_initial}"/>
       <xacro:v5_proxy_control_joint joint_name="left_v5_joint4" lower="-3.14159265" upper="3.14159265" velocity="1.5" initial_value="${left_v5_joint4_initial}"/>
@@ -110,5 +110,5 @@
       <xacro:v5_proxy_control_joint joint_name="left_v5_joint6" lower="-3.14159265" upper="3.14159265" velocity="1.5" initial_value="${left_v5_joint6_initial}"/>
       <xacro:v5_proxy_control_joint joint_name="right_v5_joint1" lower="-3.14159265" upper="3.14159265" velocity="1.2" initial_value="${right_v5_joint1_initial}"/>
-      <xacro:v5_proxy_control_joint joint_name="right_v5_joint2" lower="-1.57079633" upper="4.71238898" velocity="1.2" initial_value="${right_v5_joint2_initial}"/>
+      <xacro:v5_proxy_control_joint joint_name="right_v5_joint2" lower="-3.14" upper="3.14" velocity="1.2" initial_value="${right_v5_joint2_initial}"/>
       <xacro:v5_proxy_control_joint joint_name="right_v5_joint3" lower="-3.14159265" upper="3.14159265" velocity="1.2" initial_value="${right_v5_joint3_initial}"/>
       <xacro:v5_proxy_control_joint joint_name="right_v5_joint4" lower="-3.14159265" upper="3.14159265" velocity="1.5" initial_value="${right_v5_joint4_initial}"/>
