Commit message: fix(motion): 校准 v6 箱垛 IK 坐标与关节约束
- 修正 world/base 坐标转换、tool0 TCP 延伸和箱垛目标可视化。

- 同步 v6 双臂关节限位到 URDF、ros2_control 与 MoveIt 配置。

- 扩展 updown 感知 IK 的顶吸模式与箱垛基准记录。

Co-Authored-By: Codex <codex@openai.com>

File: ros2_ws/src/alfa_robot_description/urdf/alfa_robot.urdf.xacro (robot description, xacro)
@@ -15,5 +15,5 @@
     <parent link="world"/>
     <child link="base_link"/>
-    <origin xyz="0 0 0.09" rpy="0 0 0"/>
+    <origin xyz="0 0 0.202094" rpy="0 0 0"/>
   </joint>
 <link name="base_link">
@@ -165,5 +165,5 @@
     <child link="left_v5_link1" />
     <axis xyz="0 0 1" />
-    <limit lower="-3.14" upper="3.14" effort="120" velocity="1.2" />
+    <limit lower="-2.35619449" upper="2.35619449" effort="120" velocity="1.2" />
   </joint>
 <link name="left_v5_link2">
@@ -194,5 +194,5 @@
     <child link="left_v5_link2" />
     <axis xyz="0 0 1" />
-    <limit lower="-3.14" upper="3.14" effort="120" velocity="1.2" />
+    <limit lower="-3.14159265" upper="3.14159265" effort="120" velocity="1.2" />
   </joint>
 <link name="left_v5_link3">
@@ -223,5 +223,5 @@
     <child link="left_v5_link3" />
     <axis xyz="0 0 1" />
-    <limit lower="-3.14" upper="3.14" effort="100" velocity="1.2" />
+    <limit lower="-3.14159265" upper="3.14159265" effort="100" velocity="1.2" />
   </joint>
 <link name="left_v5_link4">
@@ -252,5 +252,5 @@
     <child link="left_v5_link4" />
     <axis xyz="0 0 1" />
-    <limit lower="-3.14" upper="3.14" effort="60" velocity="1.5" />
+    <limit lower="-3.14159265" upper="3.14159265" effort="60" velocity="1.5" />
   </joint>
 <link name="left_v5_link5">
@@ -281,5 +281,5 @@
     <child link="left_v5_link5" />
     <axis xyz="0 0 -1" />
-    <limit lower="-3.14" upper="3.14" effort="60" velocity="1.5" />
+    <limit lower="-2.53072742" upper="2.53072742" effort="60" velocity="1.5" />
   </joint>
 <link name="left_v5_link6">
@@ -310,5 +310,5 @@
     <child link="left_v5_link6" />
     <axis xyz="0 0 1" />
-    <limit lower="-3.14" upper="3.14" effort="40" velocity="1.5" />
+    <limit lower="-3.14159265" upper="3.14159265" effort="40" velocity="1.5" />
   </joint>
   <link name="left_v5_tool0">
@@ -322,5 +322,5 @@
     <parent link="left_v5_link6"/>
     <child link="left_v5_tool0"/>
-    <origin xyz="0 0 0.1" rpy="0 0 0"/>
+    <origin xyz="0 0 0.159" rpy="0 0 0"/>
   </joint>
   <!-- ========== RIGHT ARM v6 mapped to right_v5_* names ========== -->
@@ -364,5 +364,5 @@
     <child link="right_v5_link1" />
     <axis xyz="0 0 1" />
-    <limit lower="-3.14" upper="3.14" effort="120" velocity="1.2" />
+    <limit lower="-2.35619449" upper="2.35619449" effort="120" velocity="1.2" />
   </joint>
 <link name="right_v5_link2">
@@ -393,5 +393,5 @@
     <child link="right_v5_link2" />
     <axis xyz="0 0 1" />
-    <limit lower="-3.14" upper="3.14" effort="120" velocity="1.2" />
+    <limit lower="-3.14159265" upper="3.14159265" effort="120" velocity="1.2" />
   </joint>
 <link name="right_v5_link3">
@@ -422,5 +422,5 @@
     <child link="right_v5_link3" />
     <axis xyz="0 0 1" />
-    <limit lower="-3.14" upper="3.14" effort="100" velocity="1.2" />
+    <limit lower="-3.14159265" upper="3.14159265" effort="100" velocity="1.2" />
   </joint>
 <link name="right_v5_link4">
@@ -451,5 +451,5 @@
     <child link="right_v5_link4" />
     <axis xyz="0 0 1" />
-    <limit lower="-3.14" upper="3.14" effort="60" velocity="1.5" />
+    <limit lower="-3.14159265" upper="3.14159265" effort="60" velocity="1.5" />
   </joint>
 <link name="right_v5_link5">
@@ -480,5 +480,5 @@
     <child link="right_v5_link5" />
     <axis xyz="0 0 -1" />
-    <limit lower="-3.14" upper="3.14" effort="60" velocity="1.5" />
+    <limit lower="-2.53072742" upper="2.53072742" effort="60" velocity="1.5" />
   </joint>
 <link name="right_v5_link6">
@@ -509,5 +509,5 @@
     <child link="right_v5_link6" />
     <axis xyz="0 0 1" />
-    <limit lower="-3.14" upper="3.14" effort="40" velocity="1.5" />
+    <limit lower="-3.14159265" upper="3.14159265" effort="40" velocity="1.5" />
   </joint>
   <link name="right_v5_tool0">
@@ -521,5 +521,5 @@
     <parent link="right_v5_link6"/>
     <child link="right_v5_tool0"/>
-    <origin xyz="0 0 0.1" rpy="0 0 0"/>
+    <origin xyz="0 0 0.159" rpy="0 0 0"/>
   </joint>
   <xacro:alfa_robot_ros2_control

File: ros2_ws/src/alfa_robot_description/urdf/alfa_robot/alfa_robot_macro.ros2_control.xacro (robot description, xacro)
@@ -103,15 +103,15 @@
         </joint>
       </xacro:macro>
-      <xacro:v5_proxy_control_joint joint_name="left_v5_joint1" lower="-3.14159265" upper="3.14159265" velocity="1.2" initial_value="${left_v5_joint1_initial}"/>
-      <xacro:v5_proxy_control_joint joint_name="left_v5_joint2" lower="-3.14" upper="3.14" velocity="1.2" initial_value="${left_v5_joint2_initial}"/>
+      <xacro:v5_proxy_control_joint joint_name="left_v5_joint1" lower="-2.35619449" upper="2.35619449" velocity="1.2" initial_value="${left_v5_joint1_initial}"/>
+      <xacro:v5_proxy_control_joint joint_name="left_v5_joint2" lower="-3.14159265" upper="3.14159265" velocity="1.2" initial_value="${left_v5_joint2_initial}"/>
       <xacro:v5_proxy_control_joint joint_name="left_v5_joint3" lower="-3.14159265" upper="3.14159265" velocity="1.2" initial_value="${left_v5_joint3_initial}"/>
       <xacro:v5_proxy_control_joint joint_name="left_v5_joint4" lower="-3.14159265" upper="3.14159265" velocity="1.5" initial_value="${left_v5_joint4_initial}"/>
-      <xacro:v5_proxy_control_joint joint_name="left_v5_joint5" lower="-3.14159265" upper="3.14159265" velocity="1.5" initial_value="${left_v5_joint5_initial}"/>
+      <xacro:v5_proxy_control_joint joint_name="left_v5_joint5" lower="-2.53072742" upper="2.53072742" velocity="1.5" initial_value="${left_v5_joint5_initial}"/>
       <xacro:v5_proxy_control_joint joint_name="left_v5_joint6" lower="-3.14159265" upper="3.14159265" velocity="1.5" initial_value="${left_v5_joint6_initial}"/>
-      <xacro:v5_proxy_control_joint joint_name="right_v5_joint1" lower="-3.14159265" upper="3.14159265" velocity="1.2" initial_value="${right_v5_joint1_initial}"/>
-      <xacro:v5_proxy_control_joint joint_name="right_v5_joint2" lower="-3.14" upper="3.14" velocity="1.2" initial_value="${right_v5_joint2_initial}"/>
+      <xacro:v5_proxy_control_joint joint_name="right_v5_joint1" lower="-2.35619449" upper="2.35619449" velocity="1.2" initial_value="${right_v5_joint1_initial}"/>
+      <xacro:v5_proxy_control_joint joint_name="right_v5_joint2" lower="-3.14159265" upper="3.14159265" velocity="1.2" initial_value="${right_v5_joint2_initial}"/>
       <xacro:v5_proxy_control_joint joint_name="right_v5_joint3" lower="-3.14159265" upper="3.14159265" velocity="1.2" initial_value="${right_v5_joint3_initial}"/>
       <xacro:v5_proxy_control_joint joint_name="right_v5_joint4" lower="-3.14159265" upper="3.14159265" velocity="1.5" initial_value="${right_v5_joint4_initial}"/>
-      <xacro:v5_proxy_control_joint joint_name="right_v5_joint5" lower="-3.14159265" upper="3.14159265" velocity="1.5" initial_value="${right_v5_joint5_initial}"/>
+      <xacro:v5_proxy_control_joint joint_name="right_v5_joint5" lower="-2.53072742" upper="2.53072742" velocity="1.5" initial_value="${right_v5_joint5_initial}"/>
       <xacro:v5_proxy_control_joint joint_name="right_v5_joint6" lower="-3.14159265" upper="3.14159265" velocity="1.5" initial_value="${right_v5_joint6_initial}"/>
     </ros2_control>

Commit message: fix(motion): 放宽顶吸 IK 验收并记录重试
- 将 v6 双臂 tool0 延伸调整到 0.209m。

- 为顶吸模式单独设置位置和姿态误差容差。

- 箱垛双臂 IK 基准增加失败后 updown 抖动重试与审计字段。

Co-Authored-By: Codex <codex@openai.com>

File: ros2_ws/src/alfa_robot_description/urdf/alfa_robot.urdf.xacro (robot description, xacro)
@@ -322,5 +322,5 @@
     <parent link="left_v5_link6"/>
     <child link="left_v5_tool0"/>
-    <origin xyz="0 0 0.159" rpy="0 0 0"/>
+    <origin xyz="0 0 0.209" rpy="0 0 0"/>
   </joint>
   <!-- ========== RIGHT ARM v6 mapped to right_v5_* names ========== -->
@@ -521,5 +521,5 @@
     <parent link="right_v5_link6"/>
     <child link="right_v5_tool0"/>
-    <origin xyz="0 0 0.159" rpy="0 0 0"/>
+    <origin xyz="0 0 0.209" rpy="0 0 0"/>
   </joint>
   <xacro:alfa_robot_ros2_control

Commit message: feat(motion): 验证三平行机械结构代理模型
- 将 joint4 外观件固定为连接件，并新增 link4_axis 承接可动 joint4。

- 使用 joint5 STL 代理可见的 1234556 三平行结构接续。

- 同步 SRDF 相邻禁碰关系并记录轴向验证结论。

Co-Authored-By: Codex <codex@openai.com>

Refs MOTION-49

File: ros2_ws/src/alfa_robot_description/urdf/alfa_robot.urdf.xacro (robot description, xacro)
@@ -247,8 +247,35 @@
     </collision>
   </link>
-<joint name="left_v5_joint4" type="revolute">
+<joint name="left_v5_joint4_connector_fixed" type="fixed">
     <origin xyz="0.0010609 -0.239 -0.077993" rpy="1.5708 0 0" />
     <parent link="left_v5_link3" />
     <child link="left_v5_link4" />
+  </joint>
+  <link name="left_v5_link4_axis">
+    <inertial>
+      <origin xyz="0 0 0" rpy="0 0 0"/>
+      <mass value="0.001"/>
+      <inertia ixx="1e-6" ixy="0" ixz="0" iyy="1e-6" iyz="0" izz="1e-6"/>
+    </inertial>
+    <visual>
+      <origin xyz="0 0 0" rpy="0 0 0" />
+      <geometry>
+        <mesh filename="package://alfa_robot_description/meshes/alfa_robot_v2_arm_v6/visual/leftjoint5.STL" />
+      </geometry>
+      <material name="">
+        <color rgba="0.752941176470588 0.752941176470588 0.752941176470588 1" />
+      </material>
+    </visual>
+    <collision>
+      <origin xyz="0 0 0" rpy="0 0 0" />
+      <geometry>
+        <mesh filename="package://alfa_robot_description/meshes/alfa_robot_v2_arm_v6/collision/leftjoint5.STL" />
+      </geometry>
+    </collision>
+  </link>
+  <joint name="left_v5_joint4" type="revolute">
+    <origin xyz="-0.0010337 0.075993 0.058" rpy="-1.5708 0 0" />
+    <parent link="left_v5_link4" />
+    <child link="left_v5_link4_axis" />
     <axis xyz="0 0 1" />
     <limit lower="-3.14159265" upper="3.14159265" effort="60" velocity="1.5" />
@@ -277,6 +304,6 @@
   </link>
 <joint name="left_v5_joint5" type="revolute">
-    <origin xyz="-0.0010337 0.075993 0.058" rpy="-1.5708 0 0" />
-    <parent link="left_v5_link4" />
+    <origin xyz="-0.00078891 -0.083 0.057995" rpy="1.5708 -0.013602 0" />
+    <parent link="left_v5_link4_axis" />
     <child link="left_v5_link5" />
     <axis xyz="0 0 -1" />
@@ -446,8 +473,35 @@
     </collision>
   </link>
-<joint name="right_v5_joint4" type="revolute">
+<joint name="right_v5_joint4_connector_fixed" type="fixed">
     <origin xyz="-0.0010609 -0.239 0.077993" rpy="1.5708 0 0" />
     <parent link="right_v5_link3" />
     <child link="right_v5_link4" />
+  </joint>
+  <link name="right_v5_link4_axis">
+    <inertial>
+      <origin xyz="0 0 0" rpy="0 0 0"/>
+      <mass value="0.001"/>
+      <inertia ixx="1e-6" ixy="0" ixz="0" iyy="1e-6" iyz="0" izz="1e-6"/>
+    </inertial>
+    <visual>
+      <origin xyz="0 0 0" rpy="0 0 0" />
+      <geometry>
+        <mesh filename="package://alfa_robot_description/meshes/alfa_robot_v2_arm_v6/visual/rightjoint5.STL" />
+      </geometry>
+      <material name="">
+        <color rgba="0.752941176470588 0.752941176470588 0.752941176470588 1" />
+      </material>
+    </visual>
+    <collision>
+      <origin xyz="0 0 0" rpy="0 0 0" />
+      <geometry>
+        <mesh filename="package://alfa_robot_description/meshes/alfa_robot_v2_arm_v6/collision/rightjoint5.STL" />
+      </geometry>
+    </collision>
+  </link>
+  <joint name="right_v5_joint4" type="revolute">
+    <origin xyz="0.0010337 -0.075993 0.058" rpy="-1.5708 0 0" />
+    <parent link="right_v5_link4" />
+    <child link="right_v5_link4_axis" />
     <axis xyz="0 0 1" />
     <limit lower="-3.14159265" upper="3.14159265" effort="60" velocity="1.5" />
@@ -476,6 +530,6 @@
   </link>
 <joint name="right_v5_joint5" type="revolute">
-    <origin xyz="0.0010337 -0.075993 0.058" rpy="-1.5708 0 0" />
-    <parent link="right_v5_link4" />
+    <origin xyz="0.00078891 -0.083 -0.057995" rpy="1.5708 -0.013602 0" />
+    <parent link="right_v5_link4_axis" />
     <child link="right_v5_link5" />
     <axis xyz="0 0 -1" />

Commit message: fix(motion): 统一三平行代理模型零位初始化
- 将 description、MoveIt、ros2_control 与 MuJoCo 默认启动姿态统一为零位。

- 修正右臂 55 代理件偏移，避免两个 T 型件重合。

- 补充协作日志中的验证结论与后续注意事项。

Co-Authored-By: Codex <codex@openai.com>

Refs MOTION-49

File: ros2_ws/src/alfa_robot_description/urdf/alfa_robot.urdf.xacro (robot description, xacro)
@@ -530,5 +530,5 @@
   </link>
 <joint name="right_v5_joint5" type="revolute">
-    <origin xyz="0.00078891 -0.083 -0.057995" rpy="1.5708 -0.013602 0" />
+    <origin xyz="0.00078891 0.083 -0.057995" rpy="1.5708 -0.013602 0" />
     <parent link="right_v5_link4_axis" />
     <child link="right_v5_link5" />

File: ros2_ws/src/alfa_robot_description/urdf/alfa_robot/alfa_robot_macro.ros2_control.xacro (robot description, xacro)
@@ -14,16 +14,16 @@
                pitch_initial:=0.0
                turn_initial:=0.0
-               updown_initial:=0.45
+               updown_initial:=0.0
                left_v5_joint1_initial:=0.0
-               left_v5_joint2_initial:=0.26179939
-               left_v5_joint3_initial:=2.35619449
+               left_v5_joint2_initial:=0.0
+               left_v5_joint3_initial:=0.0
                left_v5_joint4_initial:=0.0
-               left_v5_joint5_initial:=1.04719755
+               left_v5_joint5_initial:=0.0
                left_v5_joint6_initial:=0.0
                right_v5_joint1_initial:=0.0
-               right_v5_joint2_initial:=0.26179939
-               right_v5_joint3_initial:=2.35619449
+               right_v5_joint2_initial:=0.0
+               right_v5_joint3_initial:=0.0
                right_v5_joint4_initial:=0.0
-               right_v5_joint5_initial:=1.04719755
+               right_v5_joint5_initial:=0.0
                right_v5_joint6_initial:=0.0"
                >

Commit message: fix(motion): 镜像右臂三平行后段结构
- 将右臂 joint4 到 joint6 后段按左臂中线镜像反解局部 origin。

- 将 joint5 零位烘入旧 -90° 姿态，并同步左右 joint5 限位为 ±π。

- 记录右臂 5 外观排查与严格镜像验证结论。

Co-Authored-By: Codex <codex@openai.com>

Refs MOTION-49

File: ros2_ws/src/alfa_robot_description/urdf/alfa_robot.urdf.xacro (robot description, xacro)
@@ -304,9 +304,9 @@
   </link>
 <joint name="left_v5_joint5" type="revolute">
-    <origin xyz="-0.00078891 -0.083 0.057995" rpy="1.5708 -0.013602 0" />
+    <origin xyz="-0.00078891 -0.083 0.057995" rpy="-1.57106636 -1.55719433 -3.14132260" />
     <parent link="left_v5_link4_axis" />
     <child link="left_v5_link5" />
     <axis xyz="0 0 -1" />
-    <limit lower="-2.53072742" upper="2.53072742" effort="60" velocity="1.5" />
+    <limit lower="-3.14159265" upper="3.14159265" effort="60" velocity="1.5" />
   </joint>
 <link name="left_v5_link6">
@@ -474,5 +474,5 @@
   </link>
 <joint name="right_v5_joint4_connector_fixed" type="fixed">
-    <origin xyz="-0.0010609 -0.239 0.077993" rpy="1.5708 0 0" />
+    <origin xyz="-0.00226694 -0.23900051 0.07798831" rpy="1.5708 0 0" />
     <parent link="right_v5_link3" />
     <child link="right_v5_link4" />
@@ -501,5 +501,5 @@
   </link>
   <joint name="right_v5_joint4" type="revolute">
-    <origin xyz="0.0010337 -0.075993 0.058" rpy="-1.5708 0 0" />
+    <origin xyz="-0.00103370 -0.07599300 0.05800000" rpy="1.5708 0 0" />
     <parent link="right_v5_link4" />
     <child link="right_v5_link4_axis" />
@@ -530,9 +530,9 @@
   </link>
 <joint name="right_v5_joint5" type="revolute">
-    <origin xyz="0.00078891 0.083 -0.057995" rpy="1.5708 -0.013602 0" />
+    <origin xyz="-0.00078891 0.08300000 0.05799500" rpy="1.57106636 -1.55719433 3.14132260" />
     <parent link="right_v5_link4_axis" />
     <child link="right_v5_link5" />
     <axis xyz="0 0 -1" />
-    <limit lower="-2.53072742" upper="2.53072742" effort="60" velocity="1.5" />
+    <limit lower="-3.14159265" upper="3.14159265" effort="60" velocity="1.5" />
   </joint>
 <link name="right_v5_link6">
@@ -559,5 +559,5 @@
   </link>
 <joint name="right_v5_joint6" type="revolute">
-    <origin xyz="0.00078891 -0.083 -0.057995" rpy="1.5708 -0.013602 0" />
+    <origin xyz="-0.00078891 0.08300000 0.05799500" rpy="-1.5708 -0.013602 0" />
     <parent link="right_v5_link5" />
     <child link="right_v5_link6" />

File: ros2_ws/src/alfa_robot_description/urdf/alfa_robot/alfa_robot_macro.ros2_control.xacro (robot description, xacro)
@@ -107,5 +107,5 @@
       <xacro:v5_proxy_control_joint joint_name="left_v5_joint3" lower="-3.14159265" upper="3.14159265" velocity="1.2" initial_value="${left_v5_joint3_initial}"/>
       <xacro:v5_proxy_control_joint joint_name="left_v5_joint4" lower="-3.14159265" upper="3.14159265" velocity="1.5" initial_value="${left_v5_joint4_initial}"/>
-      <xacro:v5_proxy_control_joint joint_name="left_v5_joint5" lower="-2.53072742" upper="2.53072742" velocity="1.5" initial_value="${left_v5_joint5_initial}"/>
+      <xacro:v5_proxy_control_joint joint_name="left_v5_joint5" lower="-3.14159265" upper="3.14159265" velocity="1.5" initial_value="${left_v5_joint5_initial}"/>
       <xacro:v5_proxy_control_joint joint_name="left_v5_joint6" lower="-3.14159265" upper="3.14159265" velocity="1.5" initial_value="${left_v5_joint6_initial}"/>
       <xacro:v5_proxy_control_joint joint_name="right_v5_joint1" lower="-2.35619449" upper="2.35619449" velocity="1.2" initial_value="${right_v5_joint1_initial}"/>
@@ -113,5 +113,5 @@
       <xacro:v5_proxy_control_joint joint_name="right_v5_joint3" lower="-3.14159265" upper="3.14159265" velocity="1.2" initial_value="${right_v5_joint3_initial}"/>
       <xacro:v5_proxy_control_joint joint_name="right_v5_joint4" lower="-3.14159265" upper="3.14159265" velocity="1.5" initial_value="${right_v5_joint4_initial}"/>
-      <xacro:v5_proxy_control_joint joint_name="right_v5_joint5" lower="-2.53072742" upper="2.53072742" velocity="1.5" initial_value="${right_v5_joint5_initial}"/>
+      <xacro:v5_proxy_control_joint joint_name="right_v5_joint5" lower="-3.14159265" upper="3.14159265" velocity="1.5" initial_value="${right_v5_joint5_initial}"/>
       <xacro:v5_proxy_control_joint joint_name="right_v5_joint6" lower="-3.14159265" upper="3.14159265" velocity="1.5" initial_value="${right_v5_joint6_initial}"/>
     </ros2_control>
