Commit message: MOTION-59 新机械臂模型迁移与命名资产收口 (#10)
* feat(motion): 支持左臂连续可达性验证

- 增强 top suction 抽离、IK target order 与 yaw 采样诊断，支持左臂连续可达性探索。

- 将实机方向映射收敛到 execution bridge joints 真相源，并补充方向契约测试。

- 新增初始 yaw/turn Rerun 预览工具，补充安全检查和诊断输出。

Co-Authored-By: Codex <codex@openai.com>

* chore(motion): 增加工程化护栏基线

- 新增 motion baseline manifest 与生成脚本，绑定模型、场景和核心策略版本。

- 将执行关节方向映射收敛到 execution bridge joints 真相源，并补充契约检查。

- 补充工程化护栏文档和 Rerun 显示参数，明确 AABB 仅作诊断默认。

Co-Authored-By: Codex <codex@openai.com>

* feat(motion): 迁移新机械臂初版模型

- 迁入 v9 机械臂 visual/collision mesh 资产，并切换 URDF 关节原点、惯量和 mesh 引用。
- 同步 ros2_control、MoveIt SRDF、初始姿态、关节限制和 MuJoCo 初始姿态配置。
- 保留既有 left_v5/right_v5/tool0 对外接口名，记录后续 TCP 与自碰撞矩阵复核风险。

验证：
- xacro + check_urdf 通过 description 与 MoveIt wrapper。
- colcon build --packages-select alfa_robot_description alfa_robot_moveit_config --symlink-install --cmake-args -DBUILD_TESTING=OFF 通过。

Co-Authored-By: Codex <codex@openai.com>

Refs MOTION-59

* refactor(robot): 收口新机械臂命名与仓库资产

- 将当前机械臂模型收口到 current_robot mesh 和无版本语义的关节、group、controller 命名。
- 同步 description、MoveIt、bringup、execution bridge、scene service、MuJoCo 与 benchmark 脚本中的新命名。
- 移除旧代际 mesh、废弃 URDF 入口、pick_ik/trac_ik 依赖包和旧 IK 安装脚本。
- 更新 IK 服务口径、命名护栏文档和协作日志，保留当前 BioIK/KDL 主线能力。

验证：
- git diff --cached --check 通过。
- colcon build --packages-select alfa_robot_description robot_motion_scene_service alfa_robot_moveit_config alfa_robot_bringup alfa_robot_execution_bridge alfa_robot_benchmarks --symlink-install --cmake-args -DBUILD_TESTING=OFF 通过。
- colcon build --packages-select robot_motion_scene_service alfa_robot_moveit_config --symlink-install --cmake-args -DBUILD_TESTING=ON 通过。
- colcon test --packages-select robot_motion_scene_service alfa_robot_moveit_config --return-code-on-test-failure 通过；colcon test-result --verbose 显示 15 tests, 0 errors, 0 failures。

Co-Authored-By: Codex <codex@openai.com>

---------

Co-authored-by: Codex <codex@openai.com>

File: ros2_ws/src/alfa_robot_description/urdf/alfa_robot.urdf.xacro (robot description, xacro)
@@ -17,49 +17,577 @@
     <origin xyz="0 0 0.202094" rpy="0 0 0"/>
   </joint>
-<link name="base_link">
-    <inertial>
-      <origin xyz="-0.230864859994365 -3.59465059753261E-05 0.00982453569098829" rpy="0 0 0" />
-      <mass value="452.254374649793" />
-      <inertia ixx="42.2528118012676" ixy="2.90433873726581E-05" ixz="5.29862244779797" iyy="45.7334828734001" iyz="-7.53976926824646E-07" izz="73.6321595788915" />
-    </inertial>
-    <visual>
-      <origin xyz="0 0 0" rpy="0 0 0" />
-      <geometry>
-        <mesh filename="package://alfa_robot_description/meshes/alfa_robot_v2_arm_v6/visual/base_link.STL" />
-      </geometry>
-      <material name="">
-        <color rgba="0.752941176470588 0.752941176470588 0.752941176470588 1" />
-      </material>
-    </visual>
-    <collision>
-      <origin xyz="0 0 0" rpy="0 0 0" />
-      <geometry>
-        <mesh filename="package://alfa_robot_description/meshes/alfa_robot_v2_arm_v6/collision/base_link.STL" />
-      </geometry>
-    </collision>
-  </link>
-<link name="pitch">
-    <inertial>
-      <origin xyz="-0.197037068600063 0.0545002757388739 0.0847212210627051" rpy="0 0 0" />
-      <mass value="31.6067905352622" />
-      <inertia ixx="0.518725062034511" ixy="2.02803901410849E-08" ixz="-0.00603915225902053" iyy="0.579528262067602" iyz="3.22538967579058E-07" izz="1.06221345040969" />
-    </inertial>
-    <visual>
-      <origin xyz="0 0 0" rpy="0 0 0" />
-      <geometry>
-        <mesh filename="package://alfa_robot_description/meshes/alfa_robot_v2_arm_v6/visual/pitch.STL" />
-      </geometry>
-      <material name="">
-        <color rgba="0.752941176470588 0.752941176470588 0.752941176470588 1" />
-      </material>
-    </visual>
-    <collision>
-      <origin xyz="0 0 0" rpy="0 0 0" />
-      <geometry>
-        <mesh filename="package://alfa_robot_description/meshes/alfa_robot_v2_arm_v6/collision/pitch.STL" />
-      </geometry>
-    </collision>
-  </link>
-<joint name="pitch" type="revolute">
+  <link name="base_link">
+    <inertial>
+      <origin xyz="-0.230884916297589 -3.59403635404876E-05 0.0098300335923569" rpy="0 0 0" />
+      <mass value="452.331665683053" />
+      <inertia ixx="42.2528214496965" ixy="2.90433873714437E-05" ixz="5.298622447798" iyy="45.7349589120892" iyz="-7.53976926582118E-07" izz="73.6336356175808" />
+    </inertial>
+    <visual>
+      <origin xyz="0 0 0" rpy="0 0 0" />
+      <geometry>
+        <mesh filename="package://alfa_robot_description/meshes/current_robot/visual/base_link.STL" />
+      </geometry>
+      <material name="">
+        <color rgba="0.752941176470588 0.752941176470588 0.752941176470588 1" />
+      </material>
+    </visual>
+    <collision>
+      <origin xyz="0 0 0" rpy="0 0 0" />
+      <geometry>
+        <mesh filename="package://alfa_robot_description/meshes/current_robot/collision/base_link.STL" />
+      </geometry>
+    </collision>
+  </link>
+  <link name="pitch">
+    <inertial>
+      <origin xyz="-0.197223755735604 0.0545002751304142 0.0848583683408171" rpy="0 0 0" />
+      <mass value="31.6766900042973" />
+      <inertia ixx="0.518885879634885" ixy="2.02803902282039E-08" ixz="-0.0059164248689273" iyy="0.580169083875299" iyz="3.22538967435459E-07" izz="1.06295541093974" />
+    </inertial>
+    <visual>
+      <origin xyz="0 0 0" rpy="0 0 0" />
+      <geometry>
+        <mesh filename="package://alfa_robot_description/meshes/current_robot/visual/pitch.STL" />
+      </geometry>
+      <material name="">
+        <color rgba="0.752941176470588 0.752941176470588 0.752941176470588 1" />
+      </material>
+    </visual>
+    <collision>
+      <origin xyz="0 0 0" rpy="0 0 0" />
+      <geometry>
+        <mesh filename="package://alfa_robot_description/meshes/current_robot/collision/pitch.STL" />
+      </geometry>
+    </collision>
+  </link>
+  <link name="turn">
+    <inertial>
+      <origin xyz="-0.0095811094528917 -7.73859721447945E-06 1.06018839944043" rpy="0 0 0" />
+      <mass value="53.4681885650186" />
+      <inertia ixx="7.9404350019494" ixy="5.99860879539091E-06" ixz="0.185339515626497" iyy="8.17240800709107" iyz="-8.94803411825732E-06" izz="0.75519185821394" />
+    </inertial>
+    <visual>
+      <origin xyz="0 0 0" rpy="0 0 0" />
+      <geometry>
+        <mesh filename="package://alfa_robot_description/meshes/current_robot/visual/turn.STL" />
+      </geometry>
+      <material name="">
+        <color rgba="0.752941176470588 0.752941176470588 0.752941176470588 1" />
+      </material>
+    </visual>
+    <collision>
+      <origin xyz="0 0 0" rpy="0 0 0" />
+      <geometry>
+        <mesh filename="package://alfa_robot_description/meshes/current_robot/collision/turn.STL" />
+      </geometry>
+    </collision>
+  </link>
+  <link name="updown">
+    <inertial>
+      <origin xyz="0.0637333774739139 -2.92604740437241E-09 0.104211014753682" rpy="0 0 0" />
+      <mass value="24.4167257440598" />
+      <inertia ixx="1.07967195604977" ixy="-1.55435028640832E-08" ixz="-0.00582099906204058" iyy="0.231957862842844" iyz="9.04966113481007E-11" izz="1.26737556353379" />
+    </inertial>
+    <visual>
+      <origin xyz="0 0 0" rpy="0 0 0" />
+      <geometry>
+        <mesh filename="package://alfa_robot_description/meshes/current_robot/visual/updown.STL" />
+      </geometry>
+      <material name="">
+        <color rgba="0.752941176470588 0.752941176470588 0.752941176470588 1" />
+      </material>
+    </visual>
+    <collision>
+      <origin xyz="0 0 0" rpy="0 0 0" />
+      <geometry>
+        <mesh filename="package://alfa_robot_description/meshes/current_robot/collision/updown.STL" />
+      </geometry>
+    </collision>
+  </link>
+  <!-- ========== LEFT ARM mapped to project names ========== -->
+  <link name="left_arm_base">
+    <inertial>
+      <origin xyz="0 0 0" rpy="0 0 0"/>
+      <mass value="0.001"/>
+      <inertia ixx="1e-6" ixy="0" ixz="0" iyy="1e-6" iyz="0" izz="1e-6"/>
+    </inertial>
+  </link>
+  <joint name="left_arm_mount" type="fixed">
+    <parent link="updown"/>
+    <child link="left_arm_base"/>
+    <origin xyz="0.095 0.26 0.2" rpy="0 0 0"/>
+  </joint>
+  <link name="leftjoint1">
+    <inertial>
+      <origin xyz="1.98132632578396E-05 0.0024729821757461 0.0580356323599247" rpy="0 0 0" />
+      <mass value="2.53849365971092" />
+      <inertia ixx="0.00565316591359222" ixy="1.39299660382164E-06" ixz="-2.78630772107311E-06" iyy="0.00554455173094155" iyz="-7.06906283259906E-05" izz="0.00447417412424819" />
+    </inertial>
+    <visual>
+      <origin xyz="0 0 0" rpy="0 0 0" />
+      <geometry>
+        <mesh filename="package://alfa_robot_description/meshes/current_robot/visual/leftjoint1.STL" />
+      </geometry>
+      <material name="">
+        <color rgba="0.752941176470588 0.752941176470588 0.752941176470588 1" />
+      </material>
+    </visual>
+    <collision>
+      <origin xyz="0 0 0" rpy="0 0 0" />
+      <geometry>
+        <mesh filename="package://alfa_robot_description/meshes/current_robot/collision/leftjoint1.STL" />
+      </geometry>
+    </collision>
+  </link>
+  <joint name="leftjoint1" type="revolute">
+    <origin xyz="0 0 0" rpy="0 0 0" />
+    <parent link="left_arm_base" />
+    <child link="leftjoint1" />
+    <axis xyz="0 0 1" />
+    <limit lower="-2.35619449" upper="2.35619449" effort="120" velocity="1.2" />
+  </joint>
+  <link name="leftjoint2">
+    <inertial>
+      <origin xyz="-3.91993260073775E-09 -0.198242241905537 0.0685963634370466" rpy="0 0 0" />
+      <mass value="13.5734229269593" />
+      <inertia ixx="0.347009291103137" ixy="1.79329294469621E-12" ixz="2.19848376530362E-12" iyy="0.0505989087942828" iyz="4.33552705015945E-12" izz="0.367314390536816" />
+    </inertial>
+    <visual>
+      <origin xyz="0 0 0" rpy="0 0 0" />
+      <geometry>
+        <mesh filename="package://alfa_robot_description/meshes/current_robot/visual/leftjoint2.STL" />
+      </geometry>
+      <material name="">
+        <color rgba="0.752941176470588 0.752941176470588 0.752941176470588 1" />
+      </material>
+    </visual>
+    <collision>
+      <origin xyz="0 0 0" rpy="0 0 0" />
+      <geometry>
+        <mesh filename="package://alfa_robot_description/meshes/current_robot/collision/leftjoint2.STL" />
+      </geometry>
+    </collision>
+  </link>
+  <joint name="leftjoint2" type="revolute">
+    <origin xyz="0 0.0825 0.058" rpy="-1.5708 0 0" />
+    <parent link="leftjoint1" />
+    <child link="leftjoint2" />
+    <axis xyz="0 0 1" />
+    <limit lower="-3.14159265" upper="3.14159265" effort="120" velocity="1.2" />
+  </joint>
+  <link name="leftjoint3">
+    <inertial>
+      <origin xyz="2.86018788653308E-08 -0.174995964436896 -0.0214654505916678" rpy="0 0 0" />
+      <mass value="5.46918956371602" />
+      <inertia ixx="0.102635037762556" ixy="1.82331494669218E-08" ixz="3.03709958770067E-09" iyy="0.0138225294833702" iyz="4.39575520960004E-05" izz="0.114289616262011" />
+    </inertial>
+    <visual>
+      <origin xyz="0 0 0" rpy="0 0 0" />
+      <geometry>
+        <mesh filename="package://alfa_robot_description/meshes/current_robot/visual/leftjoint3.STL" />
+      </geometry>
+      <material name="">
+        <color rgba="0.752941176470588 0.752941176470588 0.752941176470588 1" />
+      </material>
+    </visual>
+    <collision>
+      <origin xyz="0 0 0" rpy="0 0 0" />
+      <geometry>
+        <mesh filename="package://alfa_robot_description/meshes/current_robot/collision/leftjoint3.STL" />
+      </geometry>
+    </collision>
+  </link>
+  <joint name="leftjoint3" type="revolute">
+    <origin xyz="0 -0.4 0.008" rpy="0 0 0" />
+    <parent link="leftjoint2" />
+    <child link="leftjoint3" />
+    <axis xyz="0 0 1" />
+    <limit lower="-3.14159265" upper="3.14159265" effort="100" velocity="1.2" />
+  </joint>
+  <link name="leftjoint4">
+    <inertial>
+      <origin xyz="1.79301766545237E-05 0.0022398818670486 0.0513862987308302" rpy="0 0 0" />
+      <mass value="2.80270206383319" />
+      <inertia ixx="0.00725799360950605" ixy="1.39369533421895E-06" ixz="-2.78625386086696E-06" iyy="0.00714937209205323" iyz="-7.06885588698108E-05" izz="0.00491856957816283" />
+    </inertial>
+    <visual>
+      <origin xyz="0 0 0" rpy="0 0 0" />
+      <geometry>
+        <mesh filename="package://alfa_robot_description/meshes/current_robot/visual/leftjoint4.STL" />
+      </geometry>
+      <material name="">
+        <color rgba="0.752941176470588 0.752941176470588 0.752941176470588 1" />
+      </material>
+    </visual>
+    <collision>
+      <origin xyz="0 0 0" rpy="0 0 0" />
+      <geometry>
+        <mesh filename="package://alfa_robot_description/meshes/current_robot/collision/leftjoint4.STL" />
+      </geometry>
+    </collision>
+  </link>
+  <joint name="leftjoint4" type="revolute">
+    <origin xyz="0 -0.34 0.036" rpy="0 0 3.14159265" />
+    <parent link="leftjoint3" />
+    <child link="leftjoint4" />
+    <axis xyz="0 0 1" />
+    <limit lower="-3.14159265" upper="3.14159265" effort="60" velocity="1.5" />
+  </joint>
+  <link name="leftjoint5">
+    <inertial>
+      <origin xyz="0.00232761885815957 1.86282466611079E-05 -0.0541835932362768" rpy="0 0 0" />
+      <mass value="2.69701788961683" />
+      <inertia ixx="0.00644984661938273" ixy="1.39391456329041E-06" ixz="7.06885192213968E-05" iyy="0.00655846677979015" iyz="2.78593765647904E-06" izz="0.00474081002137964" />
+    </inertial>
+    <visual>
+      <origin xyz="0 0 0" rpy="0 0 0" />
+      <geometry>
+        <mesh filename="package://alfa_robot_description/meshes/current_robot/visual/leftjoint5.STL" />
+      </geometry>
+      <material name="">
+        <color rgba="0.752941176470588 0.752941176470588 0.752941176470588 1" />
+      </material>
+    </visual>
+    <collision>
+      <origin xyz="0 0 0" rpy="0 0 0" />
+      <geometry>
+        <mesh filename="package://alfa_robot_description/meshes/current_robot/collision/leftjoint5.STL" />
+      </geometry>
+    </collision>
+  </link>
+  <joint name="leftjoint5" type="revolute">
+    <origin xyz="0 0.076 0.058" rpy="-1.5708 0 3.14159265" />
+    <parent link="leftjoint4" />
+    <child link="leftjoint5" />
+    <axis xyz="0 0 1" />
+    <limit lower="-3.14159265" upper="3.14159265" effort="60" velocity="1.5" />
+  </joint>
+  <link name="leftjoint6">
+    <inertial>
+      <origin xyz="0.000656912040293556 0.000831354479587647 0.143020209405828" rpy="0 0 0" />
+      <mass value="9.66858880038425" />
+      <inertia ixx="0.0956031747008674" ixy="2.07680535688619E-07" ixz="-3.59179174235467E-07" iyy="0.073686444653942" iyz="-1.65114179069294E-07" izz="0.104451818743786" />
+    </inertial>
+    <visual>
+      <origin xyz="0 0 0" rpy="0 0 0" />
+      <geometry>
+        <mesh filename="package://alfa_robot_description/meshes/current_robot/visual/leftjoint6.STL" />
+      </geometry>
+      <material name="">
+        <color rgba="0.752941176470588 0.752941176470588 0.752941176470588 1" />
+      </material>
+    </visual>
+    <collision>
+      <origin xyz="0 0 0" rpy="0 0 0" />
+      <geometry>
+        <mesh filename="package://alfa_robot_description/meshes/current_robot/collision/leftjoint6.STL" />
+      </geometry>
+    </collision>
+  </link>
+  <joint name="leftjoint6" type="revolute">
+    <origin xyz="0.0825 0 -0.058" rpy="0 1.5708 0" />
+    <parent link="leftjoint5" />
+    <child link="leftjoint6" />
+    <axis xyz="0 0 1" />
+    <limit lower="-3.14159265" upper="3.14159265" effort="40" velocity="1.5" />
+  </joint>
+  <!-- ========== RIGHT ARM mapped to project names ========== -->
+  <link name="right_arm_base">
+    <inertial>
+      <origin xyz="0 0 0" rpy="0 0 0"/>
+      <mass value="0.001"/>
+      <inertia ixx="1e-6" ixy="0" ixz="0" iyy="1e-6" iyz="0" izz="1e-6"/>
+    </inertial>
+  </link>
+  <joint name="right_arm_mount" type="fixed">
+    <parent link="updown"/>
+    <child link="right_arm_base"/>
+    <origin xyz="0.095 -0.26 0.2" rpy="0 0 0"/>
+  </joint>
+  <link name="rightjoint1">
+    <inertial>
+      <origin xyz="-1.97935614578704E-05 -0.00247298310211252 0.0580356306667533" rpy="0 0 0" />
+      <mass value="2.53849328920251" />
+      <inertia ixx="0.00565316574735245" ixy="1.3934599584903E-06" ixz="2.78607721450309E-06" iyy="0.00554455177196281" iyz="7.06907347564618E-05" izz="0.00447417409155335" />
+    </inertial>
+    <visual>
+      <origin xyz="0 0 0" rpy="0 0 0" />
+      <geometry>
+        <mesh filename="package://alfa_robot_description/meshes/current_robot/visual/rightjoint1.STL" />
+      </geometry>
+      <material name="">
+        <color rgba="0.752941176470588 0.752941176470588 0.752941176470588 1" />
+      </material>
+    </visual>
+    <collision>
+      <origin xyz="0 0 0" rpy="0 0 0" />
+      <geometry>
+        <mesh filename="package://alfa_robot_description/meshes/current_robot/collision/rightjoint1.STL" />
+      </geometry>
+    </collision>
+  </link>
+  <joint name="rightjoint1" type="revolute">
+    <origin xyz="0 0 0" rpy="0 0 0" />
+    <parent link="right_arm_base" />
+    <child link="rightjoint1" />
+    <axis xyz="0 0 1" />
+    <limit lower="-2.35619449" upper="2.35619449" effort="120" velocity="1.2" />
+  </joint>
+  <link name="rightjoint2">
+    <inertial>
+      <origin xyz="-3.93094157224994E-09 -0.198242241906288 -0.0685963669555529" rpy="0 0 0" />
+      <mass value="13.573422926924" />
+      <inertia ixx="0.347009291103142" ixy="-1.77065393597298E-12" ixz="2.09998863566369E-12" iyy="0.0505989087942401" iyz="-4.27592541614651E-12" izz="0.367314390536786" />
+    </inertial>
+    <visual>
+      <origin xyz="0 0 0" rpy="0 0 0" />
+      <geometry>
+        <mesh filename="package://alfa_robot_description/meshes/current_robot/visual/rightjoint2.STL" />
+      </geometry>
+      <material name="">
+        <color rgba="0.752941176470588 0.752941176470588 0.752941176470588 1" />
+      </material>
+    </visual>
+    <collision>
+      <origin xyz="0 0 0" rpy="0 0 0" />
+      <geometry>
+        <mesh filename="package://alfa_robot_description/meshes/current_robot/collision/rightjoint2.STL" />
+      </geometry>
+    </collision>
+  </link>
+  <joint name="rightjoint2" type="revolute">
+    <origin xyz="0 -0.0825 0.058" rpy="-1.5708 0 0" />
+    <parent link="rightjoint1" />
+    <child link="rightjoint2" />
+    <axis xyz="0 0 1" />
+    <limit lower="-3.14159265" upper="3.14159265" effort="120" velocity="1.2" />
+  </joint>
+  <link name="rightjoint3">
+    <inertial>
+      <origin xyz="-2.19745741603106E-08 -0.174995898002215 0.0214654414595061" rpy="0 0 0" />
+      <mass value="5.4691844498613" />
+      <inertia ixx="0.102634928752236" ixy="5.65369033783247E-09" ixz="4.23974883669152E-09" iyy="0.0138225144033142" iyz="-4.3961229805213E-05" izz="0.114289495613127" />
+    </inertial>
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