Commit message: MOTION-59 新机械臂模型迁移与命名资产收口 (#10)
* feat(motion): 支持左臂连续可达性验证

- 增强 top suction 抽离、IK target order 与 yaw 采样诊断，支持左臂连续可达性探索。

- 将实机方向映射收敛到 execution bridge joints 真相源，并补充方向契约测试。

- 新增初始 yaw/turn Rerun 预览工具，补充安全检查和诊断输出。

Co-Authored-By: Codex <codex@openai.com>

* chore(motion): 增加工程化护栏基线

- 新增 motion baseline manifest 与生成脚本，绑定模型、场景和核心策略版本。

- 将执行关节方向映射收敛到 execution bridge joints 真相源，并补充契约检查。

- 补充工程化护栏文档和 Rerun 显示参数，明确 AABB 仅作诊断默认。

Co-Authored-By: Codex <codex@openai.com>

* feat(motion): 迁移新机械臂初版模型

- 迁入 v9 机械臂 visual/collision mesh 资产，并切换 URDF 关节原点、惯量和 mesh 引用。
- 同步 ros2_control、MoveIt SRDF、初始姿态、关节限制和 MuJoCo 初始姿态配置。
- 保留既有 left_v5/right_v5/tool0 对外接口名，记录后续 TCP 与自碰撞矩阵复核风险。

验证：
- xacro + check_urdf 通过 description 与 MoveIt wrapper。
- colcon build --packages-select alfa_robot_description alfa_robot_moveit_config --symlink-install --cmake-args -DBUILD_TESTING=OFF 通过。

Co-Authored-By: Codex <codex@openai.com>

Refs MOTION-59

* refactor(robot): 收口新机械臂命名与仓库资产

- 将当前机械臂模型收口到 current_robot mesh 和无版本语义的关节、group、controller 命名。
- 同步 description、MoveIt、bringup、execution bridge、scene service、MuJoCo 与 benchmark 脚本中的新命名。
- 移除旧代际 mesh、废弃 URDF 入口、pick_ik/trac_ik 依赖包和旧 IK 安装脚本。
- 更新 IK 服务口径、命名护栏文档和协作日志，保留当前 BioIK/KDL 主线能力。

验证：
- git diff --cached --check 通过。
- colcon build --packages-select alfa_robot_description robot_motion_scene_service alfa_robot_moveit_config alfa_robot_bringup alfa_robot_execution_bridge alfa_robot_benchmarks --symlink-install --cmake-args -DBUILD_TESTING=OFF 通过。
- colcon build --packages-select robot_motion_scene_service alfa_robot_moveit_config --symlink-install --cmake-args -DBUILD_TESTING=ON 通过。
- colcon test --packages-select robot_motion_scene_service alfa_robot_moveit_config --return-code-on-test-failure 通过；colcon test-result --verbose 显示 15 tests, 0 errors, 0 failures。

Co-Authored-By: Codex <codex@openai.com>

---------

Co-authored-by: Codex <codex@openai.com>

File: ros2_ws/src/alfa_robot_description/urdf/alfa_robot/alfa_robot_macro.ros2_control.xacro (robot description, xacro)
@@ -14,17 +14,17 @@
                pitch_initial:=0.0
                turn_initial:=0.0
-               updown_initial:=0.45
-               left_v5_joint1_initial:=0.0
-               left_v5_joint2_initial:=0.26179939
-               left_v5_joint3_initial:=2.35619449
-               left_v5_joint4_initial:=0.0
-               left_v5_joint5_initial:=1.04719755
-               left_v5_joint6_initial:=0.0
-               right_v5_joint1_initial:=0.0
-               right_v5_joint2_initial:=0.26179939
-               right_v5_joint3_initial:=2.35619449
-               right_v5_joint4_initial:=0.0
-               right_v5_joint5_initial:=1.04719755
-               right_v5_joint6_initial:=0.0"
+               updown_initial:=0.0
+               leftjoint1_initial:=0.0
+               leftjoint2_initial:=0.0
+               leftjoint3_initial:=0.0
+               leftjoint4_initial:=0.0
+               leftjoint5_initial:=0.0
+               leftjoint6_initial:=0.0
+               rightjoint1_initial:=0.0
+               rightjoint2_initial:=0.0
+               rightjoint3_initial:=0.0
+               rightjoint4_initial:=0.0
+               rightjoint5_initial:=0.0
+               rightjoint6_initial:=0.0"
                >
     <ros2_control name="${name}" type="system">
@@ -81,5 +81,5 @@
         <command_interface name="position">
           <param name="min">0</param>
-          <param name="max">0.99</param>
+          <param name="max">0.92</param>
         </command_interface>
         <state_interface name="position">
@@ -89,6 +89,6 @@
         <state_interface name="acceleration"/>
       </joint>
-      <!-- v5 proxy arms (position controlled) -->
-      <xacro:macro name="v5_proxy_control_joint" params="joint_name lower upper velocity initial_value:=0.0">
+      <!-- dual arms (position controlled) -->
+      <xacro:macro name="arm_control_joint" params="joint_name lower upper velocity initial_value:=0.0">
         <joint name="${prefix}${joint_name}">
           <command_interface name="position">
@@ -103,16 +103,16 @@
         </joint>
       </xacro:macro>
-      <xacro:v5_proxy_control_joint joint_name="left_v5_joint1" lower="-2.35619449" upper="2.35619449" velocity="1.2" initial_value="${left_v5_joint1_initial}"/>
-      <xacro:v5_proxy_control_joint joint_name="left_v5_joint2" lower="-3.14159265" upper="3.14159265" velocity="1.2" initial_value="${left_v5_joint2_initial}"/>
-      <xacro:v5_proxy_control_joint joint_name="left_v5_joint3" lower="-3.14159265" upper="3.14159265" velocity="1.2" initial_value="${left_v5_joint3_initial}"/>
-      <xacro:v5_proxy_control_joint joint_name="left_v5_joint4" lower="-3.14159265" upper="3.14159265" velocity="1.5" initial_value="${left_v5_joint4_initial}"/>
-      <xacro:v5_proxy_control_joint joint_name="left_v5_joint5" lower="-2.53072742" upper="2.53072742" velocity="1.5" initial_value="${left_v5_joint5_initial}"/>
-      <xacro:v5_proxy_control_joint joint_name="left_v5_joint6" lower="-3.14159265" upper="3.14159265" velocity="1.5" initial_value="${left_v5_joint6_initial}"/>
-      <xacro:v5_proxy_control_joint joint_name="right_v5_joint1" lower="-2.35619449" upper="2.35619449" velocity="1.2" initial_value="${right_v5_joint1_initial}"/>
-      <xacro:v5_proxy_control_joint joint_name="right_v5_joint2" lower="-3.14159265" upper="3.14159265" velocity="1.2" initial_value="${right_v5_joint2_initial}"/>
-      <xacro:v5_proxy_control_joint joint_name="right_v5_joint3" lower="-3.14159265" upper="3.14159265" velocity="1.2" initial_value="${right_v5_joint3_initial}"/>
-      <xacro:v5_proxy_control_joint joint_name="right_v5_joint4" lower="-3.14159265" upper="3.14159265" velocity="1.5" initial_value="${right_v5_joint4_initial}"/>
-      <xacro:v5_proxy_control_joint joint_name="right_v5_joint5" lower="-2.53072742" upper="2.53072742" velocity="1.5" initial_value="${right_v5_joint5_initial}"/>
-      <xacro:v5_proxy_control_joint joint_name="right_v5_joint6" lower="-3.14159265" upper="3.14159265" velocity="1.5" initial_value="${right_v5_joint6_initial}"/>
+      <xacro:arm_control_joint joint_name="leftjoint1" lower="-0.0" upper="0.0" velocity="1.2" initial_value="${leftjoint1_initial}"/>
+      <xacro:arm_control_joint joint_name="leftjoint2" lower="-3.14159265" upper="3.14159265" velocity="1.2" initial_value="${leftjoint2_initial}"/>
+      <xacro:arm_control_joint joint_name="leftjoint3" lower="-3.14159265" upper="3.14159265" velocity="1.2" initial_value="${leftjoint3_initial}"/>
+      <xacro:arm_control_joint joint_name="leftjoint4" lower="-3.14159265" upper="3.14159265" velocity="1.5" initial_value="${leftjoint4_initial}"/>
+      <xacro:arm_control_joint joint_name="leftjoint5" lower="-3.14159265" upper="3.14159265" velocity="1.5" initial_value="${leftjoint5_initial}"/>
+      <xacro:arm_control_joint joint_name="leftjoint6" lower="-3.14159265" upper="3.14159265" velocity="1.5" initial_value="${leftjoint6_initial}"/>
+      <xacro:arm_control_joint joint_name="rightjoint1" lower="-0.0" upper="0.0" velocity="1.2" initial_value="${rightjoint1_initial}"/>
+      <xacro:arm_control_joint joint_name="rightjoint2" lower="-3.14159265" upper="3.14159265" velocity="1.2" initial_value="${rightjoint2_initial}"/>
+      <xacro:arm_control_joint joint_name="rightjoint3" lower="-3.14159265" upper="3.14159265" velocity="1.2" initial_value="${rightjoint3_initial}"/>
+      <xacro:arm_control_joint joint_name="rightjoint4" lower="-3.14159265" upper="3.14159265" velocity="1.5" initial_value="${rightjoint4_initial}"/>
+      <xacro:arm_control_joint joint_name="rightjoint5" lower="-3.14159265" upper="3.14159265" velocity="1.5" initial_value="${rightjoint5_initial}"/>
+      <xacro:arm_control_joint joint_name="rightjoint6" lower="-3.14159265" upper="3.14159265" velocity="1.5" initial_value="${rightjoint6_initial}"/>
     </ros2_control>
     <xacro:if value="$(arg sim_gazebo_classic)">

File: ros2_ws/src/alfa_robot_moveit_config/config/alfa_robot.ros2_control.xacro (robot description, xacro)
@@ -27,74 +27,74 @@
                 </state_interface>
             </joint>
-            <joint name="left_v5_joint1">
+            <joint name="leftjoint1">
                 <command_interface name="position"/>
                 <state_interface name="position">
-                  <param name="initial_value">${initial_positions['left_v5_joint1']}</param>
+                  <param name="initial_value">${initial_positions['leftjoint1']}</param>
                 </state_interface>
             </joint>
-            <joint name="left_v5_joint2">
+            <joint name="leftjoint2">
                 <command_interface name="position"/>
                 <state_interface name="position">
-                  <param name="initial_value">${initial_positions['left_v5_joint2']}</param>
+                  <param name="initial_value">${initial_positions['leftjoint2']}</param>
                 </state_interface>
             </joint>
-            <joint name="left_v5_joint3">
+            <joint name="leftjoint3">
                 <command_interface name="position"/>
                 <state_interface name="position">
-                  <param name="initial_value">${initial_positions['left_v5_joint3']}</param>
+                  <param name="initial_value">${initial_positions['leftjoint3']}</param>
                 </state_interface>
             </joint>
-            <joint name="left_v5_joint4">
+            <joint name="leftjoint4">
                 <command_interface name="position"/>
                 <state_interface name="position">
-                  <param name="initial_value">${initial_positions['left_v5_joint4']}</param>
+                  <param name="initial_value">${initial_positions['leftjoint4']}</param>
                 </state_interface>
             </joint>
-            <joint name="left_v5_joint5">
+            <joint name="leftjoint5">
                 <command_interface name="position"/>
                 <state_interface name="position">
-                  <param name="initial_value">${initial_positions['left_v5_joint5']}</param>
+                  <param name="initial_value">${initial_positions['leftjoint5']}</param>
                 </state_interface>
             </joint>
-            <joint name="left_v5_joint6">
+            <joint name="leftjoint6">
                 <command_interface name="position"/>
                 <state_interface name="position">
-                  <param name="initial_value">${initial_positions['left_v5_joint6']}</param>
+                  <param name="initial_value">${initial_positions['leftjoint6']}</param>
                 </state_interface>
             </joint>
-            <joint name="right_v5_joint1">
+            <joint name="rightjoint1">
                 <command_interface name="position"/>
                 <state_interface name="position">
-                  <param name="initial_value">${initial_positions['right_v5_joint1']}</param>
+                  <param name="initial_value">${initial_positions['rightjoint1']}</param>
                 </state_interface>
             </joint>
-            <joint name="right_v5_joint2">
+            <joint name="rightjoint2">
                 <command_interface name="position"/>
                 <state_interface name="position">
-                  <param name="initial_value">${initial_positions['right_v5_joint2']}</param>
+                  <param name="initial_value">${initial_positions['rightjoint2']}</param>
                 </state_interface>
             </joint>
-            <joint name="right_v5_joint3">
+            <joint name="rightjoint3">
                 <command_interface name="position"/>
                 <state_interface name="position">
-                  <param name="initial_value">${initial_positions['right_v5_joint3']}</param>
+                  <param name="initial_value">${initial_positions['rightjoint3']}</param>
                 </state_interface>
             </joint>
-            <joint name="right_v5_joint4">
+            <joint name="rightjoint4">
                 <command_interface name="position"/>
                 <state_interface name="position">
-                  <param name="initial_value">${initial_positions['right_v5_joint4']}</param>
+                  <param name="initial_value">${initial_positions['rightjoint4']}</param>
                 </state_interface>
             </joint>
-            <joint name="right_v5_joint5">
+            <joint name="rightjoint5">
                 <command_interface name="position"/>
                 <state_interface name="position">
-                  <param name="initial_value">${initial_positions['right_v5_joint5']}</param>
+                  <param name="initial_value">${initial_positions['rightjoint5']}</param>
                 </state_interface>
             </joint>
-            <joint name="right_v5_joint6">
+            <joint name="rightjoint6">
                 <command_interface name="position"/>
                 <state_interface name="position">
-                  <param name="initial_value">${initial_positions['right_v5_joint6']}</param>
+                  <param name="initial_value">${initial_positions['rightjoint6']}</param>
                 </state_interface>
             </joint>

Commit message: feat(motion): 对齐生产执行接口与孪生轨迹
- 将 runtime 默认执行 action 对齐生产 /dual_arm_trajectory_controller/follow_joint_trajectory，并保留旧 /alfa_execution/execute_joint_trajectory 兼容入口。
- 执行 service 将模型关节名适配为生产 13 轴顺序，10Hz 重采样后转发；检测到 updown 等不可转发关节发生变化时直接拒绝。
- 仿真执行器支持生产 action、轨迹 topic、updown command topic、真实/模型关节 alias 和 250Hz 内部插值。
- 抽离/负重过渡轨迹按最大关节速度重新定时，并改进局部 RRT patch 回滚拼接。
- 将运行时全流程默认 fixed_updown 调整为 0.0，匹配当前新机械臂基线。
- 补充三平行六轴闭式解析解说明和抽离快照验证脚本。

验证：
- git diff --cached --check 通过。
- python3 -m py_compile 相关脚本和 runtime 节点通过。
- xacro 生成 URDF 通过，check_urdf 通过。
- colcon build --packages-select alfa_robot_analytic_ik alfa_robot_description robot_motion_core robot_motion_interfaces robot_motion_scene_service alfa_robot_moveit_config robot_motion_runtime 通过。
- colcon test --packages-select robot_motion_core robot_motion_scene_service alfa_robot_moveit_config robot_motion_runtime 通过；30 tests, 0 errors, 0 failures。

Co-Authored-By: Codex <codex@openai.com>

File: ros2_ws/src/alfa_robot_description/urdf/alfa_robot.urdf.xacro (robot description, xacro)
@@ -600,9 +600,9 @@
   </joint>
   <joint name="updown" type="prismatic">
-    <origin xyz="-0.081156 0 0.127" rpy="0 0 0" />
+    <origin xyz="-0.081156 0 0.207" rpy="0 0 0" />
     <parent link="turn" />
     <child link="updown" />
     <axis xyz="0 0 1" />
-    <limit lower="0" upper="0.92" effort="0" velocity="0" />
+    <limit lower="0" upper="0.7" effort="0" velocity="0" />
   </joint>
   <joint name="front_sensor" type="fixed">

File: ros2_ws/src/alfa_robot_description/urdf/alfa_robot/alfa_robot_macro.ros2_control.xacro (robot description, xacro)
@@ -71,6 +71,6 @@
       <joint name="${prefix}updown">
         <command_interface name="position">
-          <param name="min">0</param>
-          <param name="max">0.92</param>
+          <param name="min">0.0</param>
+          <param name="max">0.7</param>
         </command_interface>
         <state_interface name="position">
