Commit message: feat(description): 接入 V3 双吸盘主动悬挂整机模型
Co-Authored-By: Codex <codex@openai.com>

File: ros2_ws/src/alfa_robot_description/urdf/alfa_robot.urdf.xacro (robot description, xacro)
@@ -4,38 +4,62 @@
   <xacro:arg name="use_mock_hardware" default="true"/>
   <xacro:arg name="mock_sensor_commands" default="true"/>
-  <!-- Demo grounding calibration; default preserves existing model coordinates. -->
+  <xacro:arg name="end_effector" default="suction"/>
+  <!-- Optional scene calibration; zero keeps base_footprint on world ground. -->
   <xacro:arg name="model_ground_offset" default="0"/>
   <xacro:arg name="arm_mount_forward_offset" default="0"/>
   <xacro:arg name="updown_initial" default="0.0"/>
   <xacro:arg name="head_joint_initial" default="0.0"/>
-  <xacro:arg name="left_joint1_initial" default="-1.57079632679"/>
-  <xacro:arg name="left_joint2_initial" default="-1.57079632679"/>
-  <xacro:arg name="left_joint3_initial" default="0.0"/>
-  <xacro:arg name="left_joint4_initial" default="-1.57079632679"/>
+  <xacro:arg name="head_pitch_joint_initial" default="0.0"/>
+  <xacro:arg name="left_joint1_initial" default="2.61799387799"/>
+  <xacro:arg name="left_joint2_initial" default="1.57079632679"/>
+  <xacro:arg name="left_joint3_initial" default="-0.0872664625997"/>
+  <xacro:arg name="left_joint4_initial" default="2.09439510239"/>
   <xacro:arg name="left_joint5_initial" default="0.0"/>
   <xacro:arg name="left_joint6_initial" default="0.0"/>
   <xacro:arg name="left_joint7_initial" default="0.0"/>
-  <xacro:arg name="right_joint1_initial" default="-1.57079632679"/>
+  <xacro:arg name="right_joint1_initial" default="-2.61799387799"/>
   <xacro:arg name="right_joint2_initial" default="-1.57079632679"/>
-  <xacro:arg name="right_joint3_initial" default="0.0"/>
-  <xacro:arg name="right_joint4_initial" default="-1.57079632679"/>
+  <xacro:arg name="right_joint3_initial" default="0.0872664625997"/>
+  <xacro:arg name="right_joint4_initial" default="-2.09439510239"/>
   <xacro:arg name="right_joint5_initial" default="0.0"/>
   <xacro:arg name="right_joint6_initial" default="0.0"/>
   <xacro:arg name="right_joint7_initial" default="0.0"/>
+  <xacro:arg name="left_moving_jaw_initial" default="0.0"/>
+  <xacro:arg name="right_moving_jaw_initial" default="0.0"/>
+  <xacro:arg name="active_suspension_joint_initial" default="0.0"/>
+  <xacro:arg name="caster01_joint_initial" default="0.0"/>
+  <xacro:arg name="wheel01_joint_initial" default="0.0"/>
+  <xacro:arg name="caster02_joint_initial" default="0.0"/>
+  <xacro:arg name="wheel02_joint_initial" default="0.0"/>
+  <xacro:arg name="caster03_joint_initial" default="0.0"/>
+  <xacro:arg name="wheel03_joint_initial" default="0.0"/>
+  <xacro:arg name="caster04_joint_initial" default="0.0"/>
+  <xacro:arg name="wheel04_joint_initial" default="0.0"/>
   <xacro:include filename="$(find alfa_robot_description)/urdf/alfa_robot/alfa_robot_macro.ros2_control.xacro"/>
-  <xacro:property name="arm_mount_forward_offset_value" value="$(arg arm_mount_forward_offset)"/>
   <xacro:include filename="$(find alfa_robot_description)/urdf/alfa_robot/robot_v3_0_9.xacro"/>
+  <xacro:include filename="$(find alfa_robot_description)/urdf/alfa_robot/robot_v3_chassis.xacro"/>
   <link name="world"/>
   <joint name="world_to_base" type="fixed">
     <parent link="world"/>
+    <child link="base_footprint"/>
+    <origin xyz="0 0 $(arg model_ground_offset)" rpy="0 0 0"/>
+  </joint>
+  <link name="base_footprint"/>
+  <joint name="base_footprint_to_base_link" type="fixed">
+    <parent link="base_footprint"/>
     <child link="base_link"/>
-    <origin xyz="0 0 0" rpy="0 0 0"/>
+    <origin xyz="0.195 0.015 0.400" rpy="0 0 0"/>
   </joint>
   <link name="base_link"/>
+  <joint name="base_to_chassis" type="fixed">
+    <parent link="base_link"/>
+    <child link="chassis_base"/>
+    <origin xyz="-0.19 0 -0.034415142" rpy="0 0 0"/>
+  </joint>
   <joint name="base_to_model" type="fixed">
     <parent link="base_link"/>
     <child link="model_base"/>
     <origin
-      xyz="${-0.190000017371 + float(arm_mount_forward_offset_value)} 6.50500004219e-09 ${0.648299964909 + float(xacro.arg('model_ground_offset'))}"
+      xyz="${-0.190000017371 + float(xacro.arg('arm_mount_forward_offset'))} 6.50500004219e-09 0.662499964909"
       rpy="1.5707963 0 1.57079632679"/>
   </joint>
@@ -45,6 +69,8 @@
     use_mock_hardware="$(arg use_mock_hardware)"
     mock_sensor_commands="$(arg mock_sensor_commands)"
+    end_effector="$(arg end_effector)"
     updown_initial="$(arg updown_initial)"
     head_joint_initial="$(arg head_joint_initial)"
+    head_pitch_joint_initial="$(arg head_pitch_joint_initial)"
     left_joint1_initial="$(arg left_joint1_initial)"
     left_joint2_initial="$(arg left_joint2_initial)"
@@ -60,4 +86,15 @@
     right_joint5_initial="$(arg right_joint5_initial)"
     right_joint6_initial="$(arg right_joint6_initial)"
-    right_joint7_initial="$(arg right_joint7_initial)"/>
+    right_joint7_initial="$(arg right_joint7_initial)"
+    left_moving_jaw_initial="$(arg left_moving_jaw_initial)"
+    right_moving_jaw_initial="$(arg right_moving_jaw_initial)"
+    active_suspension_joint_initial="$(arg active_suspension_joint_initial)"
+    caster01_joint_initial="$(arg caster01_joint_initial)"
+    wheel01_joint_initial="$(arg wheel01_joint_initial)"
+    caster02_joint_initial="$(arg caster02_joint_initial)"
+    wheel02_joint_initial="$(arg wheel02_joint_initial)"
+    caster03_joint_initial="$(arg caster03_joint_initial)"
+    wheel03_joint_initial="$(arg wheel03_joint_initial)"
+    caster04_joint_initial="$(arg caster04_joint_initial)"
+    wheel04_joint_initial="$(arg wheel04_joint_initial)"/>
 </robot>

File: ros2_ws/src/alfa_robot_description/urdf/alfa_robot/alfa_robot_macro.ros2_control.xacro (robot description, xacro)
@@ -6,20 +6,33 @@
                use_mock_hardware:=true
                mock_sensor_commands:=true
+               end_effector:=suction
                updown_initial:=0.0
                head_joint_initial:=0.0
-               left_joint1_initial:=-1.57079632679
-               left_joint2_initial:=-1.57079632679
-               left_joint3_initial:=0.0
-               left_joint4_initial:=-1.57079632679
+               head_pitch_joint_initial:=0.0
+               left_joint1_initial:=2.61799387799
+               left_joint2_initial:=1.57079632679
+               left_joint3_initial:=-0.0872664625997
+               left_joint4_initial:=2.09439510239
                left_joint5_initial:=0.0
                left_joint6_initial:=0.0
                left_joint7_initial:=0.0
-               right_joint1_initial:=-1.57079632679
+               right_joint1_initial:=-2.61799387799
                right_joint2_initial:=-1.57079632679
-               right_joint3_initial:=0.0
-               right_joint4_initial:=-1.57079632679
+               right_joint3_initial:=0.0872664625997
+               right_joint4_initial:=-2.09439510239
                right_joint5_initial:=0.0
                right_joint6_initial:=0.0
-               right_joint7_initial:=0.0">
+               right_joint7_initial:=0.0
+               left_moving_jaw_initial:=0.0
+               right_moving_jaw_initial:=0.0
+               active_suspension_joint_initial:=0.0
+               caster01_joint_initial:=0.0
+               wheel01_joint_initial:=0.0
+               caster02_joint_initial:=0.0
+               wheel02_joint_initial:=0.0
+               caster03_joint_initial:=0.0
+               wheel03_joint_initial:=0.0
+               caster04_joint_initial:=0.0
+               wheel04_joint_initial:=0.0">
     <ros2_control name="${name}" type="system">
       <hardware>
@@ -27,5 +40,5 @@
         <param name="mock_sensor_commands">${mock_sensor_commands}</param>
       </hardware>
-      <xacro:macro name="arm_control_joint" params="joint_name initial_value lower upper">
+      <xacro:macro name="control_joint" params="joint_name initial_value lower upper">
         <joint name="${prefix}${joint_name}">
           <command_interface name="position">
@@ -39,20 +52,34 @@
         </joint>
       </xacro:macro>
-      <xacro:arm_control_joint joint_name="updown" initial_value="${updown_initial}" lower="-1.0" upper="0.0"/>
-      <xacro:arm_control_joint joint_name="head_joint" initial_value="${head_joint_initial}" lower="-1.57" upper="1.57"/>
-      <xacro:arm_control_joint joint_name="left_joint1" initial_value="${left_joint1_initial}" lower="-3.14159265" upper="3.14159265"/>
-      <xacro:arm_control_joint joint_name="left_joint2" initial_value="${left_joint2_initial}" lower="-1.83259571" upper="1.83259571"/>
-      <xacro:arm_control_joint joint_name="left_joint3" initial_value="${left_joint3_initial}" lower="-3.14159265" upper="3.14159265"/>
-      <xacro:arm_control_joint joint_name="left_joint4" initial_value="${left_joint4_initial}" lower="-2.53072742" upper="2.53072742"/>
-      <xacro:arm_control_joint joint_name="left_joint5" initial_value="${left_joint5_initial}" lower="-3.14159265" upper="3.14159265"/>
-      <xacro:arm_control_joint joint_name="left_joint6" initial_value="${left_joint6_initial}" lower="-1.91986218" upper="1.91986218"/>
-      <xacro:arm_control_joint joint_name="left_joint7" initial_value="${left_joint7_initial}" lower="-3.14159265" upper="3.14159265"/>
-      <xacro:arm_control_joint joint_name="right_joint1" initial_value="${right_joint1_initial}" lower="-3.14159265" upper="3.14159265"/>
-      <xacro:arm_control_joint joint_name="right_joint2" initial_value="${right_joint2_initial}" lower="-1.83259571" upper="1.83259571"/>
-      <xacro:arm_control_joint joint_name="right_joint3" initial_value="${right_joint3_initial}" lower="-3.14159265" upper="3.14159265"/>
-      <xacro:arm_control_joint joint_name="right_joint4" initial_value="${right_joint4_initial}" lower="-2.53072742" upper="2.53072742"/>
-      <xacro:arm_control_joint joint_name="right_joint5" initial_value="${right_joint5_initial}" lower="-3.14159265" upper="3.14159265"/>
-      <xacro:arm_control_joint joint_name="right_joint6" initial_value="${right_joint6_initial}" lower="-1.91986218" upper="1.91986218"/>
-      <xacro:arm_control_joint joint_name="right_joint7" initial_value="${right_joint7_initial}" lower="-3.14159265" upper="3.14159265"/>
+      <xacro:control_joint joint_name="updown" initial_value="${updown_initial}" lower="-0.5" upper="0.5"/>
+      <xacro:control_joint joint_name="head_joint" initial_value="${head_joint_initial}" lower="-1.57" upper="1.57"/>
+      <xacro:control_joint joint_name="head_pitch_joint" initial_value="${head_pitch_joint_initial}" lower="-1.57" upper="1.57"/>
+      <xacro:control_joint joint_name="left_joint1" initial_value="${left_joint1_initial}" lower="-3.14159265" upper="3.14159265"/>
+      <xacro:control_joint joint_name="left_joint2" initial_value="${left_joint2_initial}" lower="-1.8325957145940461" upper="1.8325957145940461"/>
+      <xacro:control_joint joint_name="left_joint3" initial_value="${left_joint3_initial}" lower="-3.14159265" upper="3.14159265"/>
+      <xacro:control_joint joint_name="left_joint4" initial_value="${left_joint4_initial}" lower="-2.53072742" upper="2.53072742"/>
+      <xacro:control_joint joint_name="left_joint5" initial_value="${left_joint5_initial}" lower="-3.14159265" upper="3.14159265"/>
+      <xacro:control_joint joint_name="left_joint6" initial_value="${left_joint6_initial}" lower="-1.91986218" upper="1.91986218"/>
+      <xacro:control_joint joint_name="left_joint7" initial_value="${left_joint7_initial}" lower="-3.14159265" upper="3.14159265"/>
+      <xacro:control_joint joint_name="right_joint1" initial_value="${right_joint1_initial}" lower="-3.14159265" upper="3.14159265"/>
+      <xacro:control_joint joint_name="right_joint2" initial_value="${right_joint2_initial}" lower="-1.8325957145940461" upper="1.8325957145940461"/>
+      <xacro:control_joint joint_name="right_joint3" initial_value="${right_joint3_initial}" lower="-3.14159265" upper="3.14159265"/>
+      <xacro:control_joint joint_name="right_joint4" initial_value="${right_joint4_initial}" lower="-2.53072742" upper="2.53072742"/>
+      <xacro:control_joint joint_name="right_joint5" initial_value="${right_joint5_initial}" lower="-3.14159265" upper="3.14159265"/>
+      <xacro:control_joint joint_name="right_joint6" initial_value="${right_joint6_initial}" lower="-1.91986218" upper="1.91986218"/>
+      <xacro:control_joint joint_name="right_joint7" initial_value="${right_joint7_initial}" lower="-3.14159265" upper="3.14159265"/>
+      <xacro:if value="${end_effector == 'gripper'}">
+        <xacro:control_joint joint_name="left_moving_jaw_joint" initial_value="${left_moving_jaw_initial}" lower="0.0" upper="0.08"/>
+        <xacro:control_joint joint_name="right_moving_jaw_joint" initial_value="${right_moving_jaw_initial}" lower="0.0" upper="0.08"/>
+      </xacro:if>
+      <xacro:control_joint joint_name="active_suspension_joint" initial_value="${active_suspension_joint_initial}" lower="-0.15" upper="0.0"/>
+      <xacro:control_joint joint_name="caster01_joint" initial_value="${caster01_joint_initial}" lower="-3.14159" upper="3.14159"/>
+      <xacro:control_joint joint_name="wheel01_joint" initial_value="${wheel01_joint_initial}" lower="-3.14159" upper="3.14159"/>
+      <xacro:control_joint joint_name="caster02_joint" initial_value="${caster02_joint_initial}" lower="-3.14159" upper="3.14159"/>
+      <xacro:control_joint joint_name="wheel02_joint" initial_value="${wheel02_joint_initial}" lower="-3.14159" upper="3.14159"/>
+      <xacro:control_joint joint_name="caster03_joint" initial_value="${caster03_joint_initial}" lower="-3.14159" upper="3.14159"/>
+      <xacro:control_joint joint_name="wheel03_joint" initial_value="${wheel03_joint_initial}" lower="-3.14159" upper="3.14159"/>
+      <xacro:control_joint joint_name="caster04_joint" initial_value="${caster04_joint_initial}" lower="-3.14159" upper="3.14159"/>
+      <xacro:control_joint joint_name="wheel04_joint" initial_value="${wheel04_joint_initial}" lower="-3.14159" upper="3.14159"/>
     </ros2_control>
   </xacro:macro>
