Commit message: feat(description): 接入 V3 双吸盘主动悬挂整机模型
Co-Authored-By: Codex <codex@openai.com>

File: ros2_ws/src/alfa_robot_description/urdf/alfa_robot/robot_v3_0_9.xacro (robot description, xacro)
@@ -1,97 +1,20 @@
 <?xml version="1.0" encoding="UTF-8"?>
 <!--
-  V3.0.9 与 V3.0.8 上游导出的 URDF/STL 内容逐字节一致。
-  本模型复用相同网格，只恢复上游已有但 V3.0.8 集成时固定的升降和头部自由度。
+  机身与机械臂沿用已校核的 V3.0.9 坐标、零位和限位。
+  末端支持双夹爪和双吸盘；上游 left/right 按 ROS 物理侧交换命名。
 -->
-<robot name="robot_v3_0_9_model">
+<robot xmlns:xacro="http://wiki.ros.org/xacro" name="robot_v3_0_9_model">
+  <xacro:arg name="end_effector" default="suction" />
+  <xacro:include filename="$(find alfa_robot_description)/urdf/alfa_robot/robot_v3_end_effectors.xacro" />
+  <xacro:include filename="$(find alfa_robot_description)/urdf/alfa_robot/robot_v3_head.xacro" />
   <link name="model_base">
-    <inertial>
-      <origin xyz="1.1416073e-07 -0.56016512 0.080972761" rpy="0 0 0" />
-      <mass value="79.116973" />
-      <inertia ixx="26.948925" iyy="11.135143" izz="26.372598" ixy="5.0161807e-07" ixz="0.00011324089" iyz="-3.143916" />
-    </inertial>
-    <visual>
-      <material name="robot_v3_0_8_gray">
-        <color rgba="0.82 0.82 0.82 1" />
-      </material>
-      <origin xyz="0.22515633 0.1942373 0.11" rpy="0 0 0" />
-      <geometry>
-        <mesh filename="package://alfa_robot_description/meshes/robot_v3_0_8/part_043_solid_043.stl" scale="0.001 0.001 0.001" />
-      </geometry>
-    </visual>
-    <visual>
-      <material name="robot_v3_0_8_gray">
-        <color rgba="0.82 0.82 0.82 1" />
-      </material>
-      <origin xyz="0.22515633 0.1942373 0.11" rpy="0 0 0" />
-      <geometry>
-        <mesh filename="package://alfa_robot_description/meshes/robot_v3_0_8/part_040_solid_040.stl" scale="0.001 0.001 0.001" />
-      </geometry>
-    </visual>
-    <visual>
-      <material name="robot_v3_0_8_gray">
-        <color rgba="0.82 0.82 0.82 1" />
-      </material>
-      <origin xyz="0.22515633 0.1942373 0.11" rpy="0 0 0" />
-      <geometry>
-        <mesh filename="package://alfa_robot_description/meshes/robot_v3_0_8/part_038_solid_038.stl" scale="0.001 0.001 0.001" />
-      </geometry>
-    </visual>
-    <visual>
-      <material name="robot_v3_0_8_gray">
-        <color rgba="0.82 0.82 0.82 1" />
-      </material>
-      <origin xyz="0.22515633 0.1942373 0.11" rpy="0 0 0" />
-      <geometry>
-        <mesh filename="package://alfa_robot_description/meshes/robot_v3_0_8/part_039_solid_039.stl" scale="0.001 0.001 0.001" />
-      </geometry>
-    </visual>
-    <visual>
-      <material name="robot_v3_0_8_gray">
-        <color rgba="0.82 0.82 0.82 1" />
-      </material>
-      <origin xyz="0.22515633 0.1942373 0.11" rpy="0 0 0" />
-      <geometry>
-        <mesh filename="package://alfa_robot_description/meshes/robot_v3_0_8/part_044_solid_044.stl" scale="0.001 0.001 0.001" />
-      </geometry>
-    </visual>
-    <visual>
-      <material name="robot_v3_0_8_gray">
-        <color rgba="0.82 0.82 0.82 1" />
-      </material>
-      <origin xyz="0.22515633 0.1942373 0.11" rpy="0 0 0" />
-      <geometry>
-        <mesh filename="package://alfa_robot_description/meshes/robot_v3_0_8/part_046_solid_046.stl" scale="0.001 0.001 0.001" />
-      </geometry>
-    </visual>
-    <visual>
-      <material name="robot_v3_0_8_gray">
-        <color rgba="0.82 0.82 0.82 1" />
-      </material>
-      <origin xyz="0.22515633 0.1942373 0.11" rpy="0 0 0" />
-      <geometry>
-        <mesh filename="package://alfa_robot_description/meshes/robot_v3_0_8/part_045_solid_045.stl" scale="0.001 0.001 0.001" />
-      </geometry>
-    </visual>
-    <visual>
-      <material name="robot_v3_0_8_gray">
-        <color rgba="0.82 0.82 0.82 1" />
-      </material>
-      <origin xyz="0.22515633 0.1942373 0.11" rpy="0 0 0" />
-      <geometry>
-        <mesh filename="package://alfa_robot_description/meshes/robot_v3_0_8/part_041_solid_041.stl" scale="0.001 0.001 0.001" />
-      </geometry>
-    </visual>
-    <visual>
-      <material name="robot_v3_0_8_gray">
-        <color rgba="0.82 0.82 0.82 1" />
-      </material>
-      <origin xyz="0.22515633 0.1942373 0.11" rpy="0 0 0" />
-      <geometry>
-        <mesh filename="package://alfa_robot_description/meshes/robot_v3_0_8/part_042_solid_042.stl" scale="0.001 0.001 0.001" />
-      </geometry>
-    </visual>
-    <visual>
-      <material name="robot_v3_0_8_gray">
+    <!-- Subtract the legacy chassis (parts 038-046) from the source aggregate. -->
+    <inertial>
+      <origin xyz="3.29536501166e-07 -0.0749149604820 0.212516887943" rpy="0 0 0" />
+      <mass value="30.1449868854" />
+      <inertia ixx="9.34604656910" iyy="0.775485502676" izz="9.63693915058" ixy="5.60440224250e-06" ixz="-2.85802943049e-07" iyz="-0.0352490739796" />
+    </inertial>
+    <visual>
+      <material name="robot_v3_gray">
         <color rgba="0.82 0.82 0.82 1" />
       </material>
@@ -102,5 +25,5 @@
     </visual>
     <visual>
-      <material name="robot_v3_0_8_gray">
+      <material name="robot_v3_gray">
         <color rgba="0.82 0.82 0.82 1" />
       </material>
@@ -111,5 +34,5 @@
     </visual>
     <visual>
-      <material name="robot_v3_0_8_gray">
+      <material name="robot_v3_gray">
         <color rgba="0.82 0.82 0.82 1" />
       </material>
@@ -120,5 +43,5 @@
     </visual>
     <visual>
-      <material name="robot_v3_0_8_gray">
+      <material name="robot_v3_gray">
         <color rgba="0.82 0.82 0.82 1" />
       </material>
@@ -129,5 +52,5 @@
     </visual>
     <visual>
-      <material name="robot_v3_0_8_gray">
+      <material name="robot_v3_gray">
         <color rgba="0.82 0.82 0.82 1" />
       </material>
@@ -138,5 +61,5 @@
     </visual>
     <visual>
-      <material name="robot_v3_0_8_gray">
+      <material name="robot_v3_gray">
         <color rgba="0.82 0.82 0.82 1" />
       </material>
@@ -147,5 +70,5 @@
     </visual>
     <visual>
-      <material name="robot_v3_0_8_gray">
+      <material name="robot_v3_gray">
         <color rgba="0.82 0.82 0.82 1" />
       </material>
@@ -156,5 +79,5 @@
     </visual>
     <visual>
-      <material name="robot_v3_0_8_gray">
+      <material name="robot_v3_gray">
         <color rgba="0.82 0.82 0.82 1" />
       </material>
@@ -165,5 +88,5 @@
     </visual>
     <visual>
-      <material name="robot_v3_0_8_gray">
+      <material name="robot_v3_gray">
         <color rgba="0.82 0.82 0.82 1" />
       </material>
@@ -174,5 +97,5 @@
     </visual>
     <visual>
-      <material name="robot_v3_0_8_gray">
+      <material name="robot_v3_gray">
         <color rgba="0.82 0.82 0.82 1" />
       </material>
@@ -182,58 +105,4 @@
       </geometry>
     </visual>
-    <collision>
-      <origin xyz="0.22515633 0.1942373 0.11" rpy="0 0 0" />
-      <geometry>
-        <mesh filename="package://alfa_robot_description/meshes/robot_v3_0_8/part_043_solid_043.stl" scale="0.001 0.001 0.001" />
-      </geometry>
-    </collision>
-    <collision>
-      <origin xyz="0.22515633 0.1942373 0.11" rpy="0 0 0" />
-      <geometry>
-        <mesh filename="package://alfa_robot_description/meshes/robot_v3_0_8/part_040_solid_040.stl" scale="0.001 0.001 0.001" />
-      </geometry>
-    </collision>
-    <collision>
-      <origin xyz="0.22515633 0.1942373 0.11" rpy="0 0 0" />
-      <geometry>
-        <mesh filename="package://alfa_robot_description/meshes/robot_v3_0_8/part_038_solid_038.stl" scale="0.001 0.001 0.001" />
-      </geometry>
-    </collision>
-    <collision>
-      <origin xyz="0.22515633 0.1942373 0.11" rpy="0 0 0" />
-      <geometry>
-        <mesh filename="package://alfa_robot_description/meshes/robot_v3_0_8/part_039_solid_039.stl" scale="0.001 0.001 0.001" />
-      </geometry>
-    </collision>
-    <collision>
-      <origin xyz="0.22515633 0.1942373 0.11" rpy="0 0 0" />
-      <geometry>
-        <mesh filename="package://alfa_robot_description/meshes/robot_v3_0_8/part_044_solid_044.stl" scale="0.001 0.001 0.001" />
-      </geometry>
-    </collision>
-    <collision>
-      <origin xyz="0.22515633 0.1942373 0.11" rpy="0 0 0" />
-      <geometry>
-        <mesh filename="package://alfa_robot_description/meshes/robot_v3_0_8/part_046_solid_046.stl" scale="0.001 0.001 0.001" />
-      </geometry>
-    </collision>
-    <collision>
-      <origin xyz="0.22515633 0.1942373 0.11" rpy="0 0 0" />
-      <geometry>
-        <mesh filename="package://alfa_robot_description/meshes/robot_v3_0_8/part_045_solid_045.stl" scale="0.001 0.001 0.001" />
-      </geometry>
-    </collision>
-    <collision>
-      <origin xyz="0.22515633 0.1942373 0.11" rpy="0 0 0" />
-      <geometry>
-        <mesh filename="package://alfa_robot_description/meshes/robot_v3_0_8/part_041_solid_041.stl" scale="0.001 0.001 0.001" />
-      </geometry>
-    </collision>
-    <collision>
-      <origin xyz="0.22515633 0.1942373 0.11" rpy="0 0 0" />
-      <geometry>
-        <mesh filename="package://alfa_robot_description/meshes/robot_v3_0_8/part_042_solid_042.stl" scale="0.001 0.001 0.001" />
-      </geometry>
-    </collision>
     <collision>
       <origin xyz="0.22515633 0.1942373 0.11" rpy="0 0 0" />
@@ -304,5 +173,5 @@
     </inertial>
     <visual>
-      <material name="robot_v3_0_8_gray">
+      <material name="robot_v3_gray">
         <color rgba="0.82 0.82 0.82 1" />
       </material>
@@ -313,5 +182,5 @@
     </visual>
     <visual>
-      <material name="robot_v3_0_8_gray">
+      <material name="robot_v3_gray">
         <color rgba="0.82 0.82 0.82 1" />
       </material>
@@ -322,5 +191,5 @@
     </visual>
     <visual>
-      <material name="robot_v3_0_8_gray">
+      <material name="robot_v3_gray">
         <color rgba="0.82 0.82 0.82 1" />
       </material>
@@ -331,5 +200,5 @@
     </visual>
     <visual>
-      <material name="robot_v3_0_8_gray">
+      <material name="robot_v3_gray">
         <color rgba="0.82 0.82 0.82 1" />
       </material>
@@ -340,5 +209,5 @@
     </visual>
     <visual>
-      <material name="robot_v3_0_8_gray">
+      <material name="robot_v3_gray">
         <color rgba="0.82 0.82 0.82 1" />
       </material>
@@ -349,5 +218,5 @@
     </visual>
     <visual>
-      <material name="robot_v3_0_8_gray">
+      <material name="robot_v3_gray">
         <color rgba="0.82 0.82 0.82 1" />
       </material>
@@ -358,5 +227,5 @@
     </visual>
     <visual>
-      <material name="robot_v3_0_8_gray">
+      <material name="robot_v3_gray">
         <color rgba="0.82 0.82 0.82 1" />
       </material>
@@ -367,5 +236,5 @@
     </visual>
     <visual>
-      <material name="robot_v3_0_8_gray">
+      <material name="robot_v3_gray">
         <color rgba="0.82 0.82 0.82 1" />
       </material>
@@ -424,27 +293,5 @@
     </collision>
   </link>
-  <link name="head">
-    <inertial>
-      <origin xyz="-2.3829891e-10 -0.028936597 0.10499576" rpy="0 0 0" />
-      <mass value="10.239801" />
-      <inertia ixx="0.080256221" iyy="0.059651585" izz="0.07120189" ixy="1.3644813e-10" ixz="-1.6398701e-09" iyz="-0.00029037379" />
-    </inertial>
-    <visual>
-      <material name="robot_v3_0_8_gray">
-        <color rgba="0.82 0.82 0.82 1" />
-      </material>
-      <origin xyz="0.22515633 0.306 -0.53310388" rpy="1.5707963 0 0" />
-      <geometry>
-        <mesh filename="package://alfa_robot_description/meshes/robot_v3_0_8/part_021_solid_021.stl" scale="0.001 0.001 0.001" />
-      </geometry>
-    </visual>
-    <collision>
-      <origin xyz="0.22515633 0.306 -0.53310388" rpy="1.5707963 0 0" />
-      <geometry>
-        <mesh filename="package://alfa_robot_description/meshes/robot_v3_0_8/part_021_solid_021.stl" scale="0.001 0.001 0.001" />
-      </geometry>
-    </collision>
-  </link>
-  <link name="left_joint1">
+  <link name="right_joint1">
     <inertial>
       <origin xyz="0.026713084 -0.00035041447 0.12770383" rpy="0 0 0" />
@@ -453,5 +300,5 @@
     </inertial>
     <visual>
-      <material name="robot_v3_0_8_gray">
+      <material name="robot_v3_gray">
         <color rgba="0.82 0.82 0.82 1" />
       </material>
@@ -468,5 +315,5 @@
     </collision>
   </link>
-  <link name="left_joint2">
+  <link name="right_joint2">
     <inertial>
       <origin xyz="-0.16099656 2.2026045e-08 0.040000128" rpy="0 0 0" />
@@ -475,5 +322,5 @@
     </inertial>
     <visual>
-      <material name="robot_v3_0_8_gray">
+      <material name="robot_v3_gray">
         <color rgba="0.82 0.82 0.82 1" />
       </material>
@@ -490,5 +337,5 @@
     </collision>
   </link>
-  <link name="left_joint3">
+  <link name="right_joint3">
     <inertial>
       <origin xyz="-5.6955242e-08 9.0900244e-10 0.23006341" rpy="0 0 0" />
@@ -497,5 +344,5 @@
     </inertial>
     <visual>
-      <material name="robot_v3_0_8_gray">
+      <material name="robot_v3_gray">
         <color rgba="0.82 0.82 0.82 1" />
       </material>
@@ -512,5 +359,5 @@
     </collision>
   </link>
-  <link name="left_joint4">
+  <link name="right_joint4">
     <inertial>
       <origin xyz="-0.12628065 0.033836795 -0.068004734" rpy="0 0 0" />
@@ -519,5 +366,5 @@
     </inertial>
     <visual>
-      <material name="robot_v3_0_8_gray">
+      <material name="robot_v3_gray">
         <color rgba="0.82 0.82 0.82 1" />
       </material>
@@ -534,5 +381,5 @@
     </collision>
   </link>
-  <link name="left_joint5">
+  <link name="right_joint5">
     <inertial>
       <origin xyz="-0.026243466 5.8789419e-10 0.12878599" rpy="0 0 0" />
@@ -541,5 +388,5 @@
     </inertial>
     <visual>
-      <material name="robot_v3_0_8_gray">
+      <material name="robot_v3_gray">
         <color rgba="0.82 0.82 0.82 1" />
       </material>
@@ -556,5 +403,5 @@
     </collision>
   </link>
-  <link name="left_joint6">
+  <link name="right_joint6">
     <inertial>
       <origin xyz="-0.055950548 -3.659148e-10 -0.061500003" rpy="0 0 0" />
@@ -563,5 +410,5 @@
     </inertial>
     <visual>
-      <material name="robot_v3_0_8_gray">
+      <material name="robot_v3_gray">
         <color rgba="0.82 0.82 0.82 1" />
       </material>
@@ -578,27 +425,6 @@
     </collision>
   </link>
-  <link name="left_joint7">
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
Commit message: [feat][description] 接入 V3 双吸盘主动悬挂整机模型 (#26)
* feat(motion): 冻结距离输入单箱抓取与双臂仿真演示

复用旧架构单臂演示，新增距离与箱号服务、双臂规划反馈及RViz/Rerun回放。修复启动残留和14号箱体数值接触问题，补齐回归及操作指南。

Issue经核对无明确对应项，按用户授权留空；仅仿真，不接入实机。

Co-Authored-By: Codex <codex@openai.com>

* feat(motion): 单箱抓取前按箱高调整升降轴

基于冻结抓取版新增25cm可调肩箱高度对齐、升降限位和碰撞检查，传播下降后的IK/RRT状态并补齐双视图及回归测试。严格记录低两排实际覆盖范围，保留固定高度兼容模式。

Co-Authored-By: Codex <codex@openai.com>

* feat(motion): 加入单开口仓库碰撞并统一默认起终姿态与零地面

距离抓取演示读取SRDF home，携箱返回后恢复升降零位；统一底盘、箱墙及地面基准，加入4×2.38×2.35米单开口仓库全流程碰撞。同步双视图、配置校验、回归测试和操作指南。

依赖前序PR #20、#21；当前任务无明确对应Linear Issue，沿用前序约定留空。仅仿真，未接实机，不混入独立冗余IK修复。

Co-Authored-By: Codex <codex@openai.com>

* feat(motion): 增加单次舒适高度实验并集中Demo启动说明

基于肩心到吸取TCP的几何距离一次选高，保留固定偏移默认、完整仓库碰撞及原规划预算。补充实验冻结、独立验证和七个Demo启动/二次操作速查。独立验证未证实优势舒适区间，不宣称动作更自然。

依赖前序PR #20、#21、#22；无明确对应Linear Issue，沿用前序约定留空。仅仿真，不混入独立冗余IK启动修复与其他未归属修改。

Co-Authored-By: Codex <codex@openai.com>

* fix(motion): 将舒适选高限制在初态可达的升降区间

先检查固定双臂姿态下的升降碰撞边界，再取最接近候选舒适区间的高度；补齐请求诊断与6/7号及中途阻挡回归。保留关节限位、完整碰撞、单高度和原规划预算。7号仍在接触IK阶段失败，不宣称完整搬运已修复。

无明确对应Linear Issue，沿用前序约定留空；追加至PR #23，不混入独立交互IK改动。

Co-Authored-By: Codex <codex@openai.com>

* feat(motion): 完成箱墙连续搬运与Rerun全量时间轴诊断

5×5自上而下搬运，非底排正吸失败后顶吸、底排顶吸；携箱后放释放并继承末姿态，保留全量碰撞与连续失败前缀。Rerun取消播放等待，全帧写入时间轴，保留吸附、消失和失败末帧；RViz不采用该批量写入逻辑。

实际暂存树独立构建2包，CTest20/20、解析IK2/2、8类失败冻结及Rerun完整54830帧读回通过，写入23.6816秒。依赖PR #20至#23；无明确关联Issue，沿用留空约定。不包含独立IK启动修复等未归属工作。

Co-Authored-By: Codex <codex@openai.com>

* feat(motion): Rerun按箱完整规划结果增量追加时间轴

每箱完整规划和碰撞检查后发布独立分段，按连续帧范围批量写入；保留最终完整快照补齐缺段、去重与失败末帧。RViz播放、规划顺序与碰撞精度不变。

25箱51154帧逐段与最终结果一致，RRD全帧场景回读、原生UI追帧/暂停、故障与乱序恢复通过；CTest20/20。依赖PR #20至#23，无明确关联Issue。

Co-Authored-By: Codex <codex@openai.com>

* feat(motion): 箱墙序列支持双臂同步搬运与自然姿态约束

每排按外侧双箱、内侧双箱、中心单箱执行；双臂轨迹按阶段同步并重新检查整机、双负载、环境及帧间碰撞，失败保留原因并降级单箱。

IK与RRT限制肩肘分支跳变、腕部冗余空转和明显绕远；Rerun按箱号分别回放双负载。确定性仿真25/25、双臂10/10、无降级，CTest20/20。

仅限仿真几何验证，不包含吸盘保持力、箱体惯量或执行器动态验证。无明确关联Issue。

Co-Authored-By: Codex <codex@openai.com>

* feat(description): 接入 V3 双吸盘主动悬挂整机模型

Co-Authored-By: Codex <codex@openai.com>

* fix(moveit): 适配 V3 双臂几何与底盘碰撞基准

Co-Authored-By: Codex <codex@openai.com>

---------

Co-authored-by: Codex <codex@openai.com>

File: ros2_ws/src/alfa_robot_description/urdf/alfa_robot.urdf.xacro (robot description, xacro)
@@ -4,36 +4,62 @@
   <xacro:arg name="use_mock_hardware" default="true"/>
   <xacro:arg name="mock_sensor_commands" default="true"/>
+  <xacro:arg name="end_effector" default="suction"/>
+  <!-- Optional scene calibration; zero keeps base_footprint on world ground. -->
+  <xacro:arg name="model_ground_offset" default="0"/>
   <xacro:arg name="arm_mount_forward_offset" default="0"/>
   <xacro:arg name="updown_initial" default="0.0"/>
   <xacro:arg name="head_joint_initial" default="0.0"/>
-  <xacro:arg name="left_joint1_initial" default="-1.57079632679"/>
-  <xacro:arg name="left_joint2_initial" default="-1.57079632679"/>
-  <xacro:arg name="left_joint3_initial" default="0.0"/>
-  <xacro:arg name="left_joint4_initial" default="-1.57079632679"/>
+  <xacro:arg name="head_pitch_joint_initial" default="0.0"/>
+  <xacro:arg name="left_joint1_initial" default="2.61799387799"/>
+  <xacro:arg name="left_joint2_initial" default="1.57079632679"/>
+  <xacro:arg name="left_joint3_initial" default="-0.0872664625997"/>
+  <xacro:arg name="left_joint4_initial" default="2.09439510239"/>
   <xacro:arg name="left_joint5_initial" default="0.0"/>
   <xacro:arg name="left_joint6_initial" default="0.0"/>
   <xacro:arg name="left_joint7_initial" default="0.0"/>
-  <xacro:arg name="right_joint1_initial" default="-1.57079632679"/>
+  <xacro:arg name="right_joint1_initial" default="-2.61799387799"/>
   <xacro:arg name="right_joint2_initial" default="-1.57079632679"/>
-  <xacro:arg name="right_joint3_initial" default="0.0"/>
-  <xacro:arg name="right_joint4_initial" default="-1.57079632679"/>
+  <xacro:arg name="right_joint3_initial" default="0.0872664625997"/>
+  <xacro:arg name="right_joint4_initial" default="-2.09439510239"/>
   <xacro:arg name="right_joint5_initial" default="0.0"/>
   <xacro:arg name="right_joint6_initial" default="0.0"/>
   <xacro:arg name="right_joint7_initial" default="0.0"/>
+  <xacro:arg name="left_moving_jaw_initial" default="0.0"/>
+  <xacro:arg name="right_moving_jaw_initial" default="0.0"/>
+  <xacro:arg name="active_suspension_joint_initial" default="0.0"/>
+  <xacro:arg name="caster01_joint_initial" default="0.0"/>
+  <xacro:arg name="wheel01_joint_initial" default="0.0"/>
+  <xacro:arg name="caster02_joint_initial" default="0.0"/>
+  <xacro:arg name="wheel02_joint_initial" default="0.0"/>
+  <xacro:arg name="caster03_joint_initial" default="0.0"/>
+  <xacro:arg name="wheel03_joint_initial" default="0.0"/>
+  <xacro:arg name="caster04_joint_initial" default="0.0"/>
+  <xacro:arg name="wheel04_joint_initial" default="0.0"/>
   <xacro:include filename="$(find alfa_robot_description)/urdf/alfa_robot/alfa_robot_macro.ros2_control.xacro"/>
-  <xacro:property name="arm_mount_forward_offset_value" value="$(arg arm_mount_forward_offset)"/>
   <xacro:include filename="$(find alfa_robot_description)/urdf/alfa_robot/robot_v3_0_9.xacro"/>
+  <xacro:include filename="$(find alfa_robot_description)/urdf/alfa_robot/robot_v3_chassis.xacro"/>
   <link name="world"/>
   <joint name="world_to_base" type="fixed">
     <parent link="world"/>
+    <child link="base_footprint"/>
+    <origin xyz="0 0 $(arg model_ground_offset)" rpy="0 0 0"/>
+  </joint>
+  <link name="base_footprint"/>
+  <joint name="base_footprint_to_base_link" type="fixed">
+    <parent link="base_footprint"/>
     <child link="base_link"/>
-    <origin xyz="0 0 0" rpy="0 0 0"/>
+    <origin xyz="0.195 0.015 0.400" rpy="0 0 0"/>
   </joint>
   <link name="base_link"/>
+  <joint name="base_to_chassis" type="fixed">
+    <parent link="base_link"/>
+    <child link="chassis_base"/>
+    <origin xyz="-0.19 0 -0.034415142" rpy="0 0 0"/>
+  </joint>
   <joint name="base_to_model" type="fixed">
     <parent link="base_link"/>
     <child link="model_base"/>
     <origin
-      xyz="${-0.190000017371 + float(arm_mount_forward_offset_value)} 6.50500004219e-09 0.648299964909"
+      xyz="${-0.190000017371 + float(xacro.arg('arm_mount_forward_offset'))} 6.50500004219e-09 0.662499964909"
       rpy="1.5707963 0 1.57079632679"/>
   </joint>
@@ -43,6 +69,8 @@
     use_mock_hardware="$(arg use_mock_hardware)"
     mock_sensor_commands="$(arg mock_sensor_commands)"
+    end_effector="$(arg end_effector)"
     updown_initial="$(arg updown_initial)"
     head_joint_initial="$(arg head_joint_initial)"
+    head_pitch_joint_initial="$(arg head_pitch_joint_initial)"
     left_joint1_initial="$(arg left_joint1_initial)"
     left_joint2_initial="$(arg left_joint2_initial)"
@@ -58,4 +86,15 @@
     right_joint5_initial="$(arg right_joint5_initial)"
     right_joint6_initial="$(arg right_joint6_initial)"
-    right_joint7_initial="$(arg right_joint7_initial)"/>
+    right_joint7_initial="$(arg right_joint7_initial)"
+    left_moving_jaw_initial="$(arg left_moving_jaw_initial)"
+    right_moving_jaw_initial="$(arg right_moving_jaw_initial)"
+    active_suspension_joint_initial="$(arg active_suspension_joint_initial)"
+    caster01_joint_initial="$(arg caster01_joint_initial)"
+    wheel01_joint_initial="$(arg wheel01_joint_initial)"
+    caster02_joint_initial="$(arg caster02_joint_initial)"
+    wheel02_joint_initial="$(arg wheel02_joint_initial)"
+    caster03_joint_initial="$(arg caster03_joint_initial)"
+    wheel03_joint_initial="$(arg wheel03_joint_initial)"
+    caster04_joint_initial="$(arg caster04_joint_initial)"
+    wheel04_joint_initial="$(arg wheel04_joint_initial)"/>
 </robot>
