Commit message: feat(motion): 将完整碰撞检查接入抽离RRT扩树

File: ros2_ws/src/alfa_robot_description/urdf/alfa_robot.urdf.xacro (robot description, xacro)
@@ -171,5 +171,5 @@
     <child link="leftjoint2" />
     <axis xyz="0 0 1" />
-    <limit lower="-3.14159265" upper="3.14159265" effort="120" velocity="1.2" />
+    <limit lower="-1.57079633" upper="1.57079633" effort="120" velocity="1.2" />
   </joint>
   <link name="leftjoint3">
@@ -358,5 +358,5 @@
     <child link="rightjoint2" />
     <axis xyz="0 0 1" />
-    <limit lower="-3.14159265" upper="3.14159265" effort="120" velocity="1.2" />
+    <limit lower="-1.57079633" upper="1.57079633" effort="120" velocity="1.2" />
   </joint>
   <link name="rightjoint3">

File: ros2_ws/src/alfa_robot_description/urdf/alfa_robot/alfa_robot_macro.ros2_control.xacro (robot description, xacro)
@@ -95,5 +95,5 @@
       </xacro:macro>
       <xacro:arm_control_joint joint_name="leftjoint1" lower="-0.0" upper="0.0" velocity="1.2" initial_value="${leftjoint1_initial}"/>
-      <xacro:arm_control_joint joint_name="leftjoint2" lower="-3.14159265" upper="3.14159265" velocity="1.2" initial_value="${leftjoint2_initial}"/>
+      <xacro:arm_control_joint joint_name="leftjoint2" lower="-1.57079633" upper="1.57079633" velocity="1.2" initial_value="${leftjoint2_initial}"/>
       <xacro:arm_control_joint joint_name="leftjoint3" lower="-3.14159265" upper="3.14159265" velocity="1.2" initial_value="${leftjoint3_initial}"/>
       <xacro:arm_control_joint joint_name="leftjoint4" lower="-3.14159265" upper="3.14159265" velocity="1.5" initial_value="${leftjoint4_initial}"/>
@@ -101,5 +101,5 @@
       <xacro:arm_control_joint joint_name="leftjoint6" lower="-3.14159265" upper="3.14159265" velocity="1.5" initial_value="${leftjoint6_initial}"/>
       <xacro:arm_control_joint joint_name="rightjoint1" lower="-0.0" upper="0.0" velocity="1.2" initial_value="${rightjoint1_initial}"/>
-      <xacro:arm_control_joint joint_name="rightjoint2" lower="-3.14159265" upper="3.14159265" velocity="1.2" initial_value="${rightjoint2_initial}"/>
+      <xacro:arm_control_joint joint_name="rightjoint2" lower="-1.57079633" upper="1.57079633" velocity="1.2" initial_value="${rightjoint2_initial}"/>
       <xacro:arm_control_joint joint_name="rightjoint3" lower="-3.14159265" upper="3.14159265" velocity="1.2" initial_value="${rightjoint3_initial}"/>
       <xacro:arm_control_joint joint_name="rightjoint4" lower="-3.14159265" upper="3.14159265" velocity="1.5" initial_value="${rightjoint4_initial}"/>

Commit message: feat(motion): 箱体位姿RRT抽离策略与执行链路对齐 Refs MOTION-52
汇总本轮双臂抽离运动规划迭代（30个commit squash）：

- 新增箱体位姿RRT抽离规划器（box_pose_rrt_extract_planner / box_pose_extract_rrt），
  支持自由状态空间侧吸抽离、失败候选全量回放、首碰撞帧诊断
- 抽离候选扩展参数化，收紧默认范围并加入best-first回退搜索
- 缓存箱体RRT边验证，提升抽离规划性能
- 插入吸附前预接触与平滑抽离轨迹，对齐生产执行接口与孪生轨迹
- model<->hardware joint 命名转换收敛到 common.py，加固 planner-live 实机执行安全机制
- 修正 updown 定点读取来源 topic（CANopen /canopen/joint_states 与 EtherCAT /joint_states 分离）
- 补充 scene_geometry / trajectory_plan_utils / pose_math 相关单测

File: ros2_ws/src/alfa_robot_description/urdf/alfa_robot.urdf.xacro (robot description, xacro)
@@ -171,5 +171,5 @@
     <child link="leftjoint2" />
     <axis xyz="0 0 1" />
-    <limit lower="-3.14159265" upper="3.14159265" effort="120" velocity="1.2" />
+    <limit lower="-1.57079633" upper="1.57079633" effort="120" velocity="1.2" />
   </joint>
   <link name="leftjoint3">
@@ -358,5 +358,5 @@
     <child link="rightjoint2" />
     <axis xyz="0 0 1" />
-    <limit lower="-3.14159265" upper="3.14159265" effort="120" velocity="1.2" />
+    <limit lower="-1.57079633" upper="1.57079633" effort="120" velocity="1.2" />
   </joint>
   <link name="rightjoint3">
@@ -600,9 +600,9 @@
   </joint>
   <joint name="updown" type="prismatic">
-    <origin xyz="-0.081156 0 0.127" rpy="0 0 0" />
+    <origin xyz="-0.081156 0 0.207" rpy="0 0 0" />
     <parent link="turn" />
     <child link="updown" />
     <axis xyz="0 0 1" />
-    <limit lower="0" upper="0.92" effort="0" velocity="0" />
+    <limit lower="0" upper="0.7" effort="0" velocity="0" />
   </joint>
   <joint name="front_sensor" type="fixed">

File: ros2_ws/src/alfa_robot_description/urdf/alfa_robot/alfa_robot_macro.ros2_control.xacro (robot description, xacro)
@@ -71,6 +71,6 @@
       <joint name="${prefix}updown">
         <command_interface name="position">
-          <param name="min">0</param>
-          <param name="max">0.92</param>
+          <param name="min">0.0</param>
+          <param name="max">0.7</param>
         </command_interface>
         <state_interface name="position">
@@ -95,5 +95,5 @@
       </xacro:macro>
       <xacro:arm_control_joint joint_name="leftjoint1" lower="-0.0" upper="0.0" velocity="1.2" initial_value="${leftjoint1_initial}"/>
-      <xacro:arm_control_joint joint_name="leftjoint2" lower="-3.14159265" upper="3.14159265" velocity="1.2" initial_value="${leftjoint2_initial}"/>
+      <xacro:arm_control_joint joint_name="leftjoint2" lower="-1.57079633" upper="1.57079633" velocity="1.2" initial_value="${leftjoint2_initial}"/>
       <xacro:arm_control_joint joint_name="leftjoint3" lower="-3.14159265" upper="3.14159265" velocity="1.2" initial_value="${leftjoint3_initial}"/>
       <xacro:arm_control_joint joint_name="leftjoint4" lower="-3.14159265" upper="3.14159265" velocity="1.5" initial_value="${leftjoint4_initial}"/>
@@ -101,5 +101,5 @@
       <xacro:arm_control_joint joint_name="leftjoint6" lower="-3.14159265" upper="3.14159265" velocity="1.5" initial_value="${leftjoint6_initial}"/>
       <xacro:arm_control_joint joint_name="rightjoint1" lower="-0.0" upper="0.0" velocity="1.2" initial_value="${rightjoint1_initial}"/>
-      <xacro:arm_control_joint joint_name="rightjoint2" lower="-3.14159265" upper="3.14159265" velocity="1.2" initial_value="${rightjoint2_initial}"/>
+      <xacro:arm_control_joint joint_name="rightjoint2" lower="-1.57079633" upper="1.57079633" velocity="1.2" initial_value="${rightjoint2_initial}"/>
       <xacro:arm_control_joint joint_name="rightjoint3" lower="-3.14159265" upper="3.14159265" velocity="1.2" initial_value="${rightjoint3_initial}"/>
       <xacro:arm_control_joint joint_name="rightjoint4" lower="-3.14159265" upper="3.14159265" velocity="1.5" initial_value="${rightjoint4_initial}"/>

Commit message: feat(motion): 集装箱动态刷新健壮性 + updown规划域收紧到[0.08,0.78] Refs MOTION-72 MOTION-73
squash 合并 feature/container-refresh-updown-align-20260717(5 commits)。

集装箱动态位姿健壮性(MOTION-72):
- container_pose_dynamic 自动启用漂移刷新(vehicle_pose_tracking_active=track_drift
  ||pose_dynamic 统一 gate timer/provider/drift-check),修复只开 pose_dynamic 时
  集装箱几何静默冻结。
- lookup_vehicle_pose 加 tf_ok 出参;TF 失败时不用 identity 兜底覆盖缓存,沿用上次
  成功值或退回静态默认,避免集装箱跳到错误位置。

updown 规划域整体收紧到 [0.08,0.78](MOTION-73):
- 换算方向修正: physical(电机)=logical(URDF)-0.08,收口到 joints.py 单一来源,
  电机行程硬夹紧 [0,0.7]。
- URDF limit / joint_limits.yaml / IK h 采样范围(launch+C++默认) 统一 [0.08,0.78],
  在采样阶段就限死,不生成越界候选再拒;逻辑域与电机满行程 [0,0.7] 精确一一对应。
- execute_l6_r8 收发对称走 joints.py 换算;RunDualGraspTask 两个 adapter 的
  fixed_updown 喂规划前 clamp;loaded 抬升上限 0.99->0.78。
- ros2_control command_interface 有意保持电机物理 [0,0.7](非生产执行路径)。

新增 generate_test_report.py 生成自包含测试结果可视化 HTML。

验证: 5 包编译通过; test_scene_geometry/test_task_geometry/joint 契约测试全通过;
xacro 展开确认 URDF updown limit=[0.08,0.78]; 独立代码审查发现的 4 处残留已修复。

File: ros2_ws/src/alfa_robot_description/urdf/alfa_robot.urdf.xacro (robot description, xacro)
@@ -604,5 +604,7 @@
     <child link="updown" />
     <axis xyz="0 0 1" />
-    <limit lower="0" upper="0.7" effort="0" velocity="0" />
+    <!-- updown 逻辑/URDF 规划范围 [0.08, 0.78]，对应电机物理满行程 [0, 0.7]
+         (physical = logical - 0.08，换算与夹紧收口在 alfa_robot_execution_bridge/joints.py)。 -->
+    <limit lower="0.08" upper="0.78" effort="0" velocity="0" />
   </joint>
   <joint name="front_sensor" type="fixed">
