Commit message: refactor(motion): 统一关节命名为下划线风格 left_joint3,消灭 leftjoint3 双命名 Refs MOTION-73
真机全流程排查发现关节命名不统一是深层根因:/joint_states(robot_driver ethercat
驱动)用下划线 left_joint3,而本仓库 MoveIt 模型(URDF/SRDF)用无下划线 leftjoint3,
靠适配层来回翻译。dual_arm_planner_node 直接 ingest /joint_states 当 IK seed 时
hasJointModel("left_joint3") 因名字对不上返回 false,12 个手臂关节被整段跳过退回零位,
planner 从错误 seed 出发导致 RRT 慢/姿态错/假自碰撞。

全仓库统一为下划线风格(right_joint1..6/left_joint1..6/turn/updown),让模型命名与
/joint_states、与工控机 robot_driver 一致,不再需要适配层翻译。48 文件:
- URDF/xacro: link/joint/parent/child 名改下划线;mesh filename 路径保留 leftjoint3.STL
  不动(mesh 文件名不属于关节命名合同,磁盘文件未改名),避免指向不存在的文件。
- SRDF: disable_collisions/group 的 link 名改下划线(跟随 URDF)。
- 控制器/限位/初始位 yaml(9个)、C++ src+test 硬编码 joint/link/touch_links、
  Python(common.py DEFAULT_MOTION_JOINTS/别名表等)、moveit.rviz/文档 全部改下划线。
- 适配层(alfaToMoveItJointName/HARDWARE_TO_MODEL_JOINT_ALIASES/moveit_to_execution_name)
  映射自然收敛为 identity,函数保留不删以稳定 API。
- 方向符号表 ROS_TO_ETHERCAT_SIGN_BY_JOINT key 本就是下划线风格,不受影响;上一轮
  读/发方向校准逻辑保留(命名合同与方向合同是两件独立的事)。

验证: xacro 展开成功(joint名下划线、mesh路径仍 leftjoint3.STL);SRDF 所有 link 名
在 URDF 存在;6 包 colcon build 通过;test_scene_geometry/task_geometry/joint 契约/
runtime common(8)全过;全仓库 grep 无非 mesh 的无下划线残留。唯一失败 check_l6_r8_real_safety
是历史遗留的 EtherCAT 方向快照哨兵(与命名无关)。

File: ros2_ws/src/alfa_robot_description/urdf/alfa_robot.urdf.xacro (robot description, xacro)
@@ -115,5 +115,5 @@
     <origin xyz="0.095 0.26 0.2" rpy="0 0 0"/>
   </joint>
-  <link name="leftjoint1">
+  <link name="left_joint1">
     <inertial>
       <origin xyz="1.98132632578396E-05 0.0024729821757461 0.0580356323599247" rpy="0 0 0" />
@@ -137,12 +137,12 @@
     </collision>
   </link>
-  <joint name="leftjoint1" type="revolute">
+  <joint name="left_joint1" type="revolute">
     <origin xyz="0 0 0" rpy="0 0 0" />
     <parent link="left_arm_base" />
-    <child link="leftjoint1" />
+    <child link="left_joint1" />
     <axis xyz="0 0 1" />
     <limit lower="-2.35619449" upper="2.35619449" effort="120" velocity="1.2" />
   </joint>
-  <link name="leftjoint2">
+  <link name="left_joint2">
     <inertial>
       <origin xyz="-3.91993260073775E-09 -0.198242241905537 0.0685963634370466" rpy="0 0 0" />
@@ -166,12 +166,12 @@
     </collision>
   </link>
-  <joint name="leftjoint2" type="revolute">
+  <joint name="left_joint2" type="revolute">
     <origin xyz="0 0.0825 0.058" rpy="-1.5708 0 0" />
-    <parent link="leftjoint1" />
-    <child link="leftjoint2" />
+    <parent link="left_joint1" />
+    <child link="left_joint2" />
     <axis xyz="0 0 1" />
     <limit lower="-1.57079633" upper="1.57079633" effort="120" velocity="1.2" />
   </joint>
-  <link name="leftjoint3">
+  <link name="left_joint3">
     <inertial>
       <origin xyz="2.86018788653308E-08 -0.174995964436896 -0.0214654505916678" rpy="0 0 0" />
@@ -195,12 +195,12 @@
     </collision>
   </link>
-  <joint name="leftjoint3" type="revolute">
+  <joint name="left_joint3" type="revolute">
     <origin xyz="0 -0.4 0.008" rpy="0 0 0" />
-    <parent link="leftjoint2" />
-    <child link="leftjoint3" />
+    <parent link="left_joint2" />
+    <child link="left_joint3" />
     <axis xyz="0 0 1" />
     <limit lower="-3.14159265" upper="3.14159265" effort="100" velocity="1.2" />
   </joint>
-  <link name="leftjoint4">
+  <link name="left_joint4">
     <inertial>
       <origin xyz="1.79301766545237E-05 0.0022398818670486 0.0513862987308302" rpy="0 0 0" />
@@ -224,12 +224,12 @@
     </collision>
   </link>
-  <joint name="leftjoint4" type="revolute">
+  <joint name="left_joint4" type="revolute">
     <origin xyz="0 -0.34 0.036" rpy="0 0 3.14159265" />
-    <parent link="leftjoint3" />
-    <child link="leftjoint4" />
+    <parent link="left_joint3" />
+    <child link="left_joint4" />
     <axis xyz="0 0 1" />
     <limit lower="-3.14159265" upper="3.14159265" effort="60" velocity="1.5" />
   </joint>
-  <link name="leftjoint5">
+  <link name="left_joint5">
     <inertial>
       <origin xyz="0.00232761885815957 1.86282466611079E-05 -0.0541835932362768" rpy="0 0 0" />
@@ -253,12 +253,12 @@
     </collision>
   </link>
-  <joint name="leftjoint5" type="revolute">
+  <joint name="left_joint5" type="revolute">
     <origin xyz="0 0.076 0.058" rpy="-1.5708 0 3.14159265" />
-    <parent link="leftjoint4" />
-    <child link="leftjoint5" />
+    <parent link="left_joint4" />
+    <child link="left_joint5" />
     <axis xyz="0 0 1" />
     <limit lower="-3.14159265" upper="3.14159265" effort="60" velocity="1.5" />
   </joint>
-  <link name="leftjoint6">
+  <link name="left_joint6">
     <inertial>
       <origin xyz="0.000656912040293556 0.000831354479587647 0.143020209405828" rpy="0 0 0" />
@@ -282,8 +282,8 @@
     </collision>
   </link>
-  <joint name="leftjoint6" type="revolute">
+  <joint name="left_joint6" type="revolute">
     <origin xyz="0.0825 0 -0.058" rpy="0 1.5708 0" />
-    <parent link="leftjoint5" />
-    <child link="leftjoint6" />
+    <parent link="left_joint5" />
+    <child link="left_joint6" />
     <axis xyz="0 0 1" />
     <limit lower="-3.14159265" upper="3.14159265" effort="40" velocity="1.5" />
@@ -302,5 +302,5 @@
     <origin xyz="0.095 -0.26 0.2" rpy="0 0 0"/>
   </joint>
-  <link name="rightjoint1">
+  <link name="right_joint1">
     <inertial>
       <origin xyz="-1.97935614578704E-05 -0.00247298310211252 0.0580356306667533" rpy="0 0 0" />
@@ -324,12 +324,12 @@
     </collision>
   </link>
-  <joint name="rightjoint1" type="revolute">
+  <joint name="right_joint1" type="revolute">
     <origin xyz="0 0 0" rpy="0 0 0" />
     <parent link="right_arm_base" />
-    <child link="rightjoint1" />
+    <child link="right_joint1" />
     <axis xyz="0 0 1" />
     <limit lower="-2.35619449" upper="2.35619449" effort="120" velocity="1.2" />
   </joint>
-  <link name="rightjoint2">
+  <link name="right_joint2">
     <inertial>
       <origin xyz="-3.93094157224994E-09 -0.198242241906288 -0.0685963669555529" rpy="0 0 0" />
@@ -353,12 +353,12 @@
     </collision>
   </link>
-  <joint name="rightjoint2" type="revolute">
+  <joint name="right_joint2" type="revolute">
     <origin xyz="0 -0.0825 0.058" rpy="-1.5708 0 0" />
-    <parent link="rightjoint1" />
-    <child link="rightjoint2" />
+    <parent link="right_joint1" />
+    <child link="right_joint2" />
     <axis xyz="0 0 1" />
     <limit lower="-1.57079633" upper="1.57079633" effort="120" velocity="1.2" />
   </joint>
-  <link name="rightjoint3">
+  <link name="right_joint3">
     <inertial>
       <origin xyz="-2.19745741603106E-08 -0.174995898002215 0.0214654414595061" rpy="0 0 0" />
@@ -382,12 +382,12 @@
     </collision>
   </link>
-  <joint name="rightjoint3" type="revolute">
+  <joint name="right_joint3" type="revolute">
     <origin xyz="0 -0.4 -0.008" rpy="0 0 0" />
-    <parent link="rightjoint2" />
-    <child link="rightjoint3" />
+    <parent link="right_joint2" />
+    <child link="right_joint3" />
     <axis xyz="0 0 1" />
     <limit lower="-3.14159265" upper="3.14159265" effort="100" velocity="1.2" />
   </joint>
-  <link name="rightjoint4">
+  <link name="right_joint4">
     <inertial>
       <origin xyz="-1.79645036204601E-05 0.0022398851924712 -0.051386302023446" rpy="0 0 0" />
@@ -411,12 +411,12 @@
     </collision>
   </link>
-  <joint name="rightjoint4" type="revolute">
+  <joint name="right_joint4" type="revolute">
     <origin xyz="0 -0.34 -0.036" rpy="0 0 3.14159265" />
-    <parent link="rightjoint3" />
-    <child link="rightjoint4" />
+    <parent link="right_joint3" />
+    <child link="right_joint4" />
     <axis xyz="0 0 1" />
     <limit lower="-3.14159265" upper="3.14159265" effort="60" velocity="1.5" />
   </joint>
-  <link name="rightjoint5">
+  <link name="right_joint5">
     <inertial>
       <origin xyz="0.00247297487810383 1.97916984613355E-05 -0.0580356333661171" rpy="0 0 0" />
@@ -440,12 +440,12 @@
     </collision>
   </link>
-  <joint name="rightjoint5" type="revolute">
+  <joint name="right_joint5" type="revolute">
     <origin xyz="0 0.076 -0.058" rpy="-1.5708 0 3.14159265" />
-    <parent link="rightjoint4" />
-    <child link="rightjoint5" />
+    <parent link="right_joint4" />
+    <child link="right_joint5" />
     <axis xyz="0 0 1" />
     <limit lower="-3.14159265" upper="3.14159265" effort="60" velocity="1.5" />
   </joint>
-  <link name="rightjoint6">
+  <link name="right_joint6">
     <inertial>
       <origin xyz="0.000634748756222159 -0.000892103298974378 0.142311014574405" rpy="0 0 0" />
@@ -469,8 +469,8 @@
     </collision>
   </link>
-  <joint name="rightjoint6" type="revolute">
+  <joint name="right_joint6" type="revolute">
     <origin xyz="0.0825 0 -0.058" rpy="0 1.5708 0" />
-    <parent link="rightjoint5" />
-    <child link="rightjoint6" />
+    <parent link="right_joint5" />
+    <child link="right_joint6" />
     <axis xyz="0 0 1" />
     <limit lower="-3.14159265" upper="3.14159265" effort="40" velocity="1.5" />
@@ -646,5 +646,5 @@
   </link>
   <joint name="left_tool0_fixed" type="fixed">
-    <parent link="leftjoint6"/>
+    <parent link="left_joint6"/>
     <child link="left_tool0"/>
     <origin xyz="0 0 0.209" rpy="0 0 0"/>
@@ -658,5 +658,5 @@
   </link>
   <joint name="right_tool0_fixed" type="fixed">
-    <parent link="rightjoint6"/>
+    <parent link="right_joint6"/>
     <child link="right_tool0"/>
     <origin xyz="0 0 0.209" rpy="0 0 0"/>

File: ros2_ws/src/alfa_robot_description/urdf/alfa_robot/alfa_robot_macro.ros2_control.xacro (robot description, xacro)
@@ -12,16 +12,16 @@
                turn_initial:=0.0
                updown_initial:=0.0
-               leftjoint1_initial:=0.0
-               leftjoint2_initial:=0.0
-               leftjoint3_initial:=0.0
-               leftjoint4_initial:=0.0
-               leftjoint5_initial:=0.0
-               leftjoint6_initial:=0.0
-               rightjoint1_initial:=0.0
-               rightjoint2_initial:=0.0
-               rightjoint3_initial:=0.0
-               rightjoint4_initial:=0.0
-               rightjoint5_initial:=0.0
-               rightjoint6_initial:=0.0"
+               left_joint1_initial:=0.0
+               left_joint2_initial:=0.0
+               left_joint3_initial:=0.0
+               left_joint4_initial:=0.0
+               left_joint5_initial:=0.0
+               left_joint6_initial:=0.0
+               right_joint1_initial:=0.0
+               right_joint2_initial:=0.0
+               right_joint3_initial:=0.0
+               right_joint4_initial:=0.0
+               right_joint5_initial:=0.0
+               right_joint6_initial:=0.0"
                >
     <ros2_control name="${name}" type="system">
@@ -94,16 +94,16 @@
         </joint>
       </xacro:macro>
-      <xacro:arm_control_joint joint_name="leftjoint1" lower="-0.0" upper="0.0" velocity="1.2" initial_value="${leftjoint1_initial}"/>
-      <xacro:arm_control_joint joint_name="leftjoint2" lower="-1.57079633" upper="1.57079633" velocity="1.2" initial_value="${leftjoint2_initial}"/>
-      <xacro:arm_control_joint joint_name="leftjoint3" lower="-3.14159265" upper="3.14159265" velocity="1.2" initial_value="${leftjoint3_initial}"/>
-      <xacro:arm_control_joint joint_name="leftjoint4" lower="-3.14159265" upper="3.14159265" velocity="1.5" initial_value="${leftjoint4_initial}"/>
-      <xacro:arm_control_joint joint_name="leftjoint5" lower="-3.14159265" upper="3.14159265" velocity="1.5" initial_value="${leftjoint5_initial}"/>
-      <xacro:arm_control_joint joint_name="leftjoint6" lower="-3.14159265" upper="3.14159265" velocity="1.5" initial_value="${leftjoint6_initial}"/>
-      <xacro:arm_control_joint joint_name="rightjoint1" lower="-0.0" upper="0.0" velocity="1.2" initial_value="${rightjoint1_initial}"/>
-      <xacro:arm_control_joint joint_name="rightjoint2" lower="-1.57079633" upper="1.57079633" velocity="1.2" initial_value="${rightjoint2_initial}"/>
-      <xacro:arm_control_joint joint_name="rightjoint3" lower="-3.14159265" upper="3.14159265" velocity="1.2" initial_value="${rightjoint3_initial}"/>
-      <xacro:arm_control_joint joint_name="rightjoint4" lower="-3.14159265" upper="3.14159265" velocity="1.5" initial_value="${rightjoint4_initial}"/>
-      <xacro:arm_control_joint joint_name="rightjoint5" lower="-3.14159265" upper="3.14159265" velocity="1.5" initial_value="${rightjoint5_initial}"/>
-      <xacro:arm_control_joint joint_name="rightjoint6" lower="-3.14159265" upper="3.14159265" velocity="1.5" initial_value="${rightjoint6_initial}"/>
+      <xacro:arm_control_joint joint_name="left_joint1" lower="-0.0" upper="0.0" velocity="1.2" initial_value="${left_joint1_initial}"/>
+      <xacro:arm_control_joint joint_name="left_joint2" lower="-1.57079633" upper="1.57079633" velocity="1.2" initial_value="${left_joint2_initial}"/>
+      <xacro:arm_control_joint joint_name="left_joint3" lower="-3.14159265" upper="3.14159265" velocity="1.2" initial_value="${left_joint3_initial}"/>
+      <xacro:arm_control_joint joint_name="left_joint4" lower="-3.14159265" upper="3.14159265" velocity="1.5" initial_value="${left_joint4_initial}"/>
+      <xacro:arm_control_joint joint_name="left_joint5" lower="-3.14159265" upper="3.14159265" velocity="1.5" initial_value="${left_joint5_initial}"/>
+      <xacro:arm_control_joint joint_name="left_joint6" lower="-3.14159265" upper="3.14159265" velocity="1.5" initial_value="${left_joint6_initial}"/>
+      <xacro:arm_control_joint joint_name="right_joint1" lower="-0.0" upper="0.0" velocity="1.2" initial_value="${right_joint1_initial}"/>
+      <xacro:arm_control_joint joint_name="right_joint2" lower="-1.57079633" upper="1.57079633" velocity="1.2" initial_value="${right_joint2_initial}"/>
+      <xacro:arm_control_joint joint_name="right_joint3" lower="-3.14159265" upper="3.14159265" velocity="1.2" initial_value="${right_joint3_initial}"/>
+      <xacro:arm_control_joint joint_name="right_joint4" lower="-3.14159265" upper="3.14159265" velocity="1.5" initial_value="${right_joint4_initial}"/>
+      <xacro:arm_control_joint joint_name="right_joint5" lower="-3.14159265" upper="3.14159265" velocity="1.5" initial_value="${right_joint5_initial}"/>
+      <xacro:arm_control_joint joint_name="right_joint6" lower="-3.14159265" upper="3.14159265" velocity="1.5" initial_value="${right_joint6_initial}"/>
     </ros2_control>
   </xacro:macro>

File: ros2_ws/src/alfa_robot_moveit_config/config/alfa_robot.ros2_control.xacro (robot description, xacro)
@@ -27,74 +27,74 @@
                 </state_interface>
             </joint>
-            <joint name="leftjoint1">
+            <joint name="left_joint1">
                 <command_interface name="position"/>
                 <state_interface name="position">
-                  <param name="initial_value">${initial_positions['leftjoint1']}</param>
+                  <param name="initial_value">${initial_positions['left_joint1']}</param>
                 </state_interface>
             </joint>
-            <joint name="leftjoint2">
+            <joint name="left_joint2">
                 <command_interface name="position"/>
                 <state_interface name="position">
-                  <param name="initial_value">${initial_positions['leftjoint2']}</param>
+                  <param name="initial_value">${initial_positions['left_joint2']}</param>
                 </state_interface>
             </joint>
-            <joint name="leftjoint3">
+            <joint name="left_joint3">
                 <command_interface name="position"/>
                 <state_interface name="position">
-                  <param name="initial_value">${initial_positions['leftjoint3']}</param>
+                  <param name="initial_value">${initial_positions['left_joint3']}</param>
                 </state_interface>
             </joint>
-            <joint name="leftjoint4">
+            <joint name="left_joint4">
                 <command_interface name="position"/>
                 <state_interface name="position">
-                  <param name="initial_value">${initial_positions['leftjoint4']}</param>
+                  <param name="initial_value">${initial_positions['left_joint4']}</param>
                 </state_interface>
             </joint>
-            <joint name="leftjoint5">
+            <joint name="left_joint5">
                 <command_interface name="position"/>
                 <state_interface name="position">
-                  <param name="initial_value">${initial_positions['leftjoint5']}</param>
+                  <param name="initial_value">${initial_positions['left_joint5']}</param>
                 </state_interface>
             </joint>
-            <joint name="leftjoint6">
+            <joint name="left_joint6">
                 <command_interface name="position"/>
                 <state_interface name="position">
-                  <param name="initial_value">${initial_positions['leftjoint6']}</param>
+                  <param name="initial_value">${initial_positions['left_joint6']}</param>
                 </state_interface>
             </joint>
-            <joint name="rightjoint1">
+            <joint name="right_joint1">
                 <command_interface name="position"/>
                 <state_interface name="position">
-                  <param name="initial_value">${initial_positions['rightjoint1']}</param>
+                  <param name="initial_value">${initial_positions['right_joint1']}</param>
                 </state_interface>
             </joint>
-            <joint name="rightjoint2">
+            <joint name="right_joint2">
                 <command_interface name="position"/>
                 <state_interface name="position">
-                  <param name="initial_value">${initial_positions['rightjoint2']}</param>
+                  <param name="initial_value">${initial_positions['right_joint2']}</param>
                 </state_interface>
             </joint>
-            <joint name="rightjoint3">
+            <joint name="right_joint3">
                 <command_interface name="position"/>
                 <state_interface name="position">
-                  <param name="initial_value">${initial_positions['rightjoint3']}</param>
+                  <param name="initial_value">${initial_positions['right_joint3']}</param>
                 </state_interface>
             </joint>
-            <joint name="rightjoint4">
+            <joint name="right_joint4">
                 <command_interface name="position"/>
                 <state_interface name="position">
-                  <param name="initial_value">${initial_positions['rightjoint4']}</param>
+                  <param name="initial_value">${initial_positions['right_joint4']}</param>
                 </state_interface>
             </joint>
-            <joint name="rightjoint5">
+            <joint name="right_joint5">
                 <command_interface name="position"/>
                 <state_interface name="position">
-                  <param name="initial_value">${initial_positions['rightjoint5']}</param>
+                  <param name="initial_value">${initial_positions['right_joint5']}</param>
                 </state_interface>
             </joint>
-            <joint name="rightjoint6">
+            <joint name="right_joint6">
                 <command_interface name="position"/>
                 <state_interface name="position">
-                  <param name="initial_value">${initial_positions['rightjoint6']}</param>
+                  <param name="initial_value">${initial_positions['right_joint6']}</param>
                 </state_interface>
             </joint>
