Commit message: feat(motion): 统一接口分层与中央契约 Refs MOTION-123
统一 Motion 域间/域内接口边界，固定中央 robot_interfaces 依赖并补齐结构化回执、readiness、QoS、部署与回滚验证。

File: ros2_ws/src/alfa_robot_description/urdf/alfa_robot.urdf.xacro (robot description, xacro)
@@ -143,5 +143,5 @@
     <child link="left_joint1" />
     <axis xyz="0 0 1" />
-    <limit lower="-2.35619449" upper="2.35619449" effort="120" velocity="1.2" />
+    <limit lower="-1.57079632679" upper="1.57079632679" effort="120" velocity="1.2" />
   </joint>
   <link name="left_joint2">
@@ -172,5 +172,5 @@
     <child link="left_joint2" />
     <axis xyz="0 0 1" />
-    <limit lower="-1.57079633" upper="1.57079633" effort="120" velocity="1.2" />
+    <limit lower="-1.57079632679" upper="1.57079632679" effort="120" velocity="1.2" />
   </joint>
   <link name="left_joint3">
@@ -201,5 +201,5 @@
     <child link="left_joint3" />
     <axis xyz="0 0 1" />
-    <limit lower="-3.14159265" upper="3.14159265" effort="100" velocity="1.2" />
+    <limit lower="-2.44346095279" upper="2.44346095279" effort="100" velocity="1.2" />
   </joint>
   <link name="left_joint4">
@@ -230,5 +230,5 @@
     <child link="left_joint4" />
     <axis xyz="0 0 1" />
-    <limit lower="-3.14159265" upper="3.14159265" effort="60" velocity="1.5" />
+    <limit lower="-3.14159265359" upper="3.14159265359" effort="60" velocity="1.5" />
   </joint>
   <link name="left_joint5">
@@ -259,5 +259,5 @@
     <child link="left_joint5" />
     <axis xyz="0 0 1" />
-    <limit lower="-3.14159265" upper="3.14159265" effort="60" velocity="1.5" />
+    <limit lower="-2.18166156499" upper="2.18166156499" effort="60" velocity="1.5" />
   </joint>
   <link name="left_joint6">
@@ -288,5 +288,5 @@
     <child link="left_joint6" />
     <axis xyz="0 0 1" />
-    <limit lower="-3.14159265" upper="3.14159265" effort="40" velocity="1.5" />
+    <limit lower="-3.12413936107" upper="3.12413936107" effort="40" velocity="1.5" />
   </joint>
   <!-- ========== RIGHT ARM mapped to project names ========== -->
@@ -330,5 +330,5 @@
     <child link="right_joint1" />
     <axis xyz="0 0 1" />
-    <limit lower="-2.35619449" upper="2.35619449" effort="120" velocity="1.2" />
+    <limit lower="-1.57079632679" upper="1.57079632679" effort="120" velocity="1.2" />
   </joint>
   <link name="right_joint2">
@@ -359,5 +359,5 @@
     <child link="right_joint2" />
     <axis xyz="0 0 1" />
-    <limit lower="-1.57079633" upper="1.57079633" effort="120" velocity="1.2" />
+    <limit lower="-1.57079632679" upper="1.57079632679" effort="120" velocity="1.2" />
   </joint>
   <link name="right_joint3">
@@ -388,5 +388,5 @@
     <child link="right_joint3" />
     <axis xyz="0 0 1" />
-    <limit lower="-3.14159265" upper="3.14159265" effort="100" velocity="1.2" />
+    <limit lower="-2.44346095279" upper="2.44346095279" effort="100" velocity="1.2" />
   </joint>
   <link name="right_joint4">
@@ -417,5 +417,5 @@
     <child link="right_joint4" />
     <axis xyz="0 0 1" />
-    <limit lower="-3.14159265" upper="3.14159265" effort="60" velocity="1.5" />
+    <limit lower="-3.14159265359" upper="3.14159265359" effort="60" velocity="1.5" />
   </joint>
   <link name="right_joint5">
@@ -446,5 +446,5 @@
     <child link="right_joint5" />
     <axis xyz="0 0 1" />
-    <limit lower="-3.14159265" upper="3.14159265" effort="60" velocity="1.5" />
+    <limit lower="-2.18166156499" upper="2.18166156499" effort="60" velocity="1.5" />
   </joint>
   <link name="right_joint6">
@@ -475,5 +475,5 @@
     <child link="right_joint6" />
     <axis xyz="0 0 1" />
-    <limit lower="-3.14159265" upper="3.14159265" effort="40" velocity="1.5" />
+    <limit lower="-3.12413936107" upper="3.12413936107" effort="40" velocity="1.5" />
   </joint>
   <link name="front_sensor">

File: ros2_ws/src/alfa_robot_description/urdf/alfa_robot/alfa_robot_macro.ros2_control.xacro (robot description, xacro)
@@ -94,16 +94,16 @@
         </joint>
       </xacro:macro>
-      <xacro:arm_control_joint joint_name="left_joint1" lower="-0.0" upper="0.0" velocity="1.2" initial_value="${left_joint1_initial}"/>
-      <xacro:arm_control_joint joint_name="left_joint2" lower="-1.57079633" upper="1.57079633" velocity="1.2" initial_value="${left_joint2_initial}"/>
-      <xacro:arm_control_joint joint_name="left_joint3" lower="-3.14159265" upper="3.14159265" velocity="1.2" initial_value="${left_joint3_initial}"/>
-      <xacro:arm_control_joint joint_name="left_joint4" lower="-3.14159265" upper="3.14159265" velocity="1.5" initial_value="${left_joint4_initial}"/>
-      <xacro:arm_control_joint joint_name="left_joint5" lower="-3.14159265" upper="3.14159265" velocity="1.5" initial_value="${left_joint5_initial}"/>
-      <xacro:arm_control_joint joint_name="left_joint6" lower="-3.14159265" upper="3.14159265" velocity="1.5" initial_value="${left_joint6_initial}"/>
-      <xacro:arm_control_joint joint_name="right_joint1" lower="-0.0" upper="0.0" velocity="1.2" initial_value="${right_joint1_initial}"/>
-      <xacro:arm_control_joint joint_name="right_joint2" lower="-1.57079633" upper="1.57079633" velocity="1.2" initial_value="${right_joint2_initial}"/>
-      <xacro:arm_control_joint joint_name="right_joint3" lower="-3.14159265" upper="3.14159265" velocity="1.2" initial_value="${right_joint3_initial}"/>
-      <xacro:arm_control_joint joint_name="right_joint4" lower="-3.14159265" upper="3.14159265" velocity="1.5" initial_value="${right_joint4_initial}"/>
-      <xacro:arm_control_joint joint_name="right_joint5" lower="-3.14159265" upper="3.14159265" velocity="1.5" initial_value="${right_joint5_initial}"/>
-      <xacro:arm_control_joint joint_name="right_joint6" lower="-3.14159265" upper="3.14159265" velocity="1.5" initial_value="${right_joint6_initial}"/>
+      <xacro:arm_control_joint joint_name="left_joint1" lower="-1.57079632679" upper="1.57079632679" velocity="1.2" initial_value="${left_joint1_initial}"/>
+      <xacro:arm_control_joint joint_name="left_joint2" lower="-1.57079632679" upper="1.57079632679" velocity="1.2" initial_value="${left_joint2_initial}"/>
+      <xacro:arm_control_joint joint_name="left_joint3" lower="-2.44346095279" upper="2.44346095279" velocity="1.2" initial_value="${left_joint3_initial}"/>
+      <xacro:arm_control_joint joint_name="left_joint4" lower="-3.14159265359" upper="3.14159265359" velocity="1.5" initial_value="${left_joint4_initial}"/>
+      <xacro:arm_control_joint joint_name="left_joint5" lower="-2.18166156499" upper="2.18166156499" velocity="1.5" initial_value="${left_joint5_initial}"/>
+      <xacro:arm_control_joint joint_name="left_joint6" lower="-3.12413936107" upper="3.12413936107" velocity="1.5" initial_value="${left_joint6_initial}"/>
+      <xacro:arm_control_joint joint_name="right_joint1" lower="-1.57079632679" upper="1.57079632679" velocity="1.2" initial_value="${right_joint1_initial}"/>
+      <xacro:arm_control_joint joint_name="right_joint2" lower="-1.57079632679" upper="1.57079632679" velocity="1.2" initial_value="${right_joint2_initial}"/>
+      <xacro:arm_control_joint joint_name="right_joint3" lower="-2.44346095279" upper="2.44346095279" velocity="1.2" initial_value="${right_joint3_initial}"/>
+      <xacro:arm_control_joint joint_name="right_joint4" lower="-3.14159265359" upper="3.14159265359" velocity="1.5" initial_value="${right_joint4_initial}"/>
+      <xacro:arm_control_joint joint_name="right_joint5" lower="-2.18166156499" upper="2.18166156499" velocity="1.5" initial_value="${right_joint5_initial}"/>
+      <xacro:arm_control_joint joint_name="right_joint6" lower="-3.12413936107" upper="3.12413936107" velocity="1.5" initial_value="${right_joint6_initial}"/>
     </ros2_control>
   </xacro:macro>

Commit message: feat(description): 接入V3.0.5整机双臂与解析IK Refs MOTION-94

File: ros2_ws/src/alfa_robot_description/urdf/alfa_robot.urdf.xacro (robot description, xacro)
@@ -4,4 +4,5 @@
   <xacro:arg name="use_mock_hardware" default="true"/>
   <xacro:arg name="mock_sensor_commands" default="true"/>
+  <xacro:arg name="arm_mount_forward_offset" default="0"/>
   <xacro:arg name="left_joint1_initial" default="0.0"/>
   <xacro:arg name="left_joint2_initial" default="0.0"/>
@@ -19,45 +20,20 @@
   <xacro:arg name="right_joint7_initial" default="0.0"/>
   <xacro:include filename="$(find alfa_robot_description)/urdf/alfa_robot/alfa_robot_macro.ros2_control.xacro"/>
-  <xacro:include filename="$(find alfa_robot_description)/urdf/alfa_robot/robot_v3_arm.xacro"/>
+  <xacro:property name="arm_mount_forward_offset_value" value="$(arg arm_mount_forward_offset)"/>
+  <xacro:include filename="$(find alfa_robot_description)/urdf/alfa_robot/robot_v3_0_5.xacro"/>
   <link name="world"/>
   <joint name="world_to_base" type="fixed">
     <parent link="world"/>
     <child link="base_link"/>
-    <origin xyz="0 0 0" rpy="0 0 0"/>
+    <origin xyz="-0.055 0 0" rpy="0 0 0"/>
   </joint>
-  <link name="base_link">
-    <inertial>
-      <origin xyz="0 0 0.25" rpy="0 0 0"/>
-      <mass value="25"/>
-      <inertia ixx="1.041667" ixy="0" ixz="0" iyy="0.854167" iyz="0" izz="0.854167"/>
-    </inertial>
-    <visual>
-      <origin xyz="0 0 0.25" rpy="0 0 0"/>
-      <geometry>
-        <box size="0.4 0.5 0.5"/>
-      </geometry>
-      <material name="cube_base_blue">
-        <color rgba="0.16 0.34 0.55 1"/>
-      </material>
-    </visual>
-    <collision>
-      <origin xyz="0 0 0.25" rpy="0 0 0"/>
-      <geometry>
-        <box size="0.4 0.5 0.5"/>
-      </geometry>
-    </collision>
-  </link>
-  <!--
-    V3.0.4 单臂复制为左右两臂，安装在立方体的左右侧面。
-    两臂局部 Y 轴均朝机器人前方；joint1 局部 Z 轴分别朝左右外侧。
-  -->
-  <xacro:robot_v3_arm
-    prefix="left" parent="base_link"
-    mount_xyz="0 0.255 0.25"
-    mount_rpy="-1.57079633 -1.57079633 0"/>
-  <xacro:robot_v3_arm
-    prefix="right" parent="base_link"
-    mount_xyz="0 -0.255 0.25"
-    mount_rpy="1.57079633 1.57079633 0"/>
+  <link name="base_link"/>
+  <joint name="base_to_model" type="fixed">
+    <parent link="base_link"/>
+    <child link="model_base"/>
+    <origin
+      xyz="${0.13899334 + float(arm_mount_forward_offset_value)} 0 -0.50669703"
+      rpy="1.57079632679 0.22548136 0"/>
+  </joint>
   <xacro:alfa_robot_ros2_control
     name="alfa_robot"

File: ros2_ws/src/alfa_robot_description/urdf/alfa_robot/alfa_robot_macro.ros2_control.xacro (robot description, xacro)
@@ -40,5 +40,5 @@
       <xacro:arm_control_joint joint_name="left_joint2" initial_value="${left_joint2_initial}" lower="-1.83259571" upper="1.83259571"/>
       <xacro:arm_control_joint joint_name="left_joint3" initial_value="${left_joint3_initial}" lower="-3.14159265" upper="3.14159265"/>
-      <xacro:arm_control_joint joint_name="left_joint4" initial_value="${left_joint4_initial}" lower="-2.61799388" upper="2.61799388"/>
+      <xacro:arm_control_joint joint_name="left_joint4" initial_value="${left_joint4_initial}" lower="-2.53072742" upper="2.53072742"/>
       <xacro:arm_control_joint joint_name="left_joint5" initial_value="${left_joint5_initial}" lower="-3.14159265" upper="3.14159265"/>
       <xacro:arm_control_joint joint_name="left_joint6" initial_value="${left_joint6_initial}" lower="-2.09439510" upper="2.09439510"/>
@@ -47,5 +47,5 @@
       <xacro:arm_control_joint joint_name="right_joint2" initial_value="${right_joint2_initial}" lower="-1.83259571" upper="1.83259571"/>
       <xacro:arm_control_joint joint_name="right_joint3" initial_value="${right_joint3_initial}" lower="-3.14159265" upper="3.14159265"/>
-      <xacro:arm_control_joint joint_name="right_joint4" initial_value="${right_joint4_initial}" lower="-2.61799388" upper="2.61799388"/>
+      <xacro:arm_control_joint joint_name="right_joint4" initial_value="${right_joint4_initial}" lower="-2.53072742" upper="2.53072742"/>
       <xacro:arm_control_joint joint_name="right_joint5" initial_value="${right_joint5_initial}" lower="-3.14159265" upper="3.14159265"/>
       <xacro:arm_control_joint joint_name="right_joint6" initial_value="${right_joint6_initial}" lower="-2.09439510" upper="2.09439510"/>

Commit message: feat(motion): 校准末端长度并重建轨迹缓存
统一URDF、解析IK和MoveIt FK的243mm工具长度，重建75至82厘米、2厘米横向分辨率的五排轨迹缓存，并更新运行时命中与统计工具。

Refs MOTION-52

File: ros2_ws/src/alfa_robot_description/urdf/alfa_robot.urdf.xacro (robot description, xacro)
@@ -649,5 +649,5 @@
     <parent link="left_joint6"/>
     <child link="left_tool0"/>
-    <origin xyz="0 0 0.259" rpy="0 0 0"/>
+    <origin xyz="0 0 0.243" rpy="0 0 0"/>
   </joint>
   <link name="right_tool0">
@@ -661,5 +661,5 @@
     <parent link="right_joint6"/>
     <child link="right_tool0"/>
-    <origin xyz="0 0 0.259" rpy="0 0 0"/>
+    <origin xyz="0 0 0.243" rpy="0 0 0"/>
   </joint>
   <xacro:alfa_robot_ros2_control

Commit message: feat(ik): 完善V3解析验证并接入V3.0.7整机模型 Refs MOTION-94

File: ros2_ws/src/alfa_robot_description/urdf/alfa_robot.urdf.xacro (robot description, xacro)
@@ -21,10 +21,10 @@
   <xacro:include filename="$(find alfa_robot_description)/urdf/alfa_robot/alfa_robot_macro.ros2_control.xacro"/>
   <xacro:property name="arm_mount_forward_offset_value" value="$(arg arm_mount_forward_offset)"/>
-  <xacro:include filename="$(find alfa_robot_description)/urdf/alfa_robot/robot_v3_0_5.xacro"/>
+  <xacro:include filename="$(find alfa_robot_description)/urdf/alfa_robot/robot_v3_0_7.xacro"/>
   <link name="world"/>
   <joint name="world_to_base" type="fixed">
     <parent link="world"/>
     <child link="base_link"/>
-    <origin xyz="-0.055 0 0" rpy="0 0 0"/>
+    <origin xyz="0 0 0" rpy="0 0 0"/>
   </joint>
   <link name="base_link"/>
@@ -33,5 +33,5 @@
     <child link="model_base"/>
     <origin
-      xyz="${0.13899334 + float(arm_mount_forward_offset_value)} 0 -0.50669703"
+      xyz="${0.319993084526 + float(arm_mount_forward_offset_value)} -1.343e-08 0.566102751502"
       rpy="1.57079632679 0.22548136 0"/>
   </joint>

File: ros2_ws/src/alfa_robot_description/urdf/alfa_robot/alfa_robot_macro.ros2_control.xacro (robot description, xacro)
@@ -42,5 +42,5 @@
       <xacro:arm_control_joint joint_name="left_joint4" initial_value="${left_joint4_initial}" lower="-2.53072742" upper="2.53072742"/>
       <xacro:arm_control_joint joint_name="left_joint5" initial_value="${left_joint5_initial}" lower="-3.14159265" upper="3.14159265"/>
-      <xacro:arm_control_joint joint_name="left_joint6" initial_value="${left_joint6_initial}" lower="-2.09439510" upper="2.09439510"/>
+      <xacro:arm_control_joint joint_name="left_joint6" initial_value="${left_joint6_initial}" lower="-1.91986218" upper="1.91986218"/>
       <xacro:arm_control_joint joint_name="left_joint7" initial_value="${left_joint7_initial}" lower="-3.14159265" upper="3.14159265"/>
       <xacro:arm_control_joint joint_name="right_joint1" initial_value="${right_joint1_initial}" lower="-3.14159265" upper="3.14159265"/>
@@ -49,5 +49,5 @@
       <xacro:arm_control_joint joint_name="right_joint4" initial_value="${right_joint4_initial}" lower="-2.53072742" upper="2.53072742"/>
       <xacro:arm_control_joint joint_name="right_joint5" initial_value="${right_joint5_initial}" lower="-3.14159265" upper="3.14159265"/>
-      <xacro:arm_control_joint joint_name="right_joint6" initial_value="${right_joint6_initial}" lower="-2.09439510" upper="2.09439510"/>
+      <xacro:arm_control_joint joint_name="right_joint6" initial_value="${right_joint6_initial}" lower="-1.91986218" upper="1.91986218"/>
       <xacro:arm_control_joint joint_name="right_joint7" initial_value="${right_joint7_initial}" lower="-3.14159265" upper="3.14159265"/>
     </ros2_control>

File: ros2_ws/src/alfa_robot_description/urdf/alfa_robot/robot_v3_0_5.xacro (robot description, xacro)
@@ -465,4 +465,10 @@
     </collision>
   </link>
+  <joint name="arm_carriage_joint" type="fixed">
+    <origin xyz="0.065760636 -0.66236699 -2.021e-08" rpy="1.5707963 0 0.22548136" />
+    <parent link="model_base" />
+    <child link="arm_carriage" />
+  </joint>
+  <xacro:if value="false">
   <link name="right_joint1">
     <inertial>
@@ -888,3 +894,4 @@
     <origin xyz="0 0 0.1895" rpy="0 0 0" />
   </joint>
+  </xacro:if>
 </robot>

Commit message: [feat][v3] 接入 V3.1.1 模型并对齐解析规划流程 (#27)
整合远端 V3 主流程、权威 V3.1.1 description、解析 IK 与本地诊断能力。保留远端主编排，并以显式研究策略保留携箱回 Home 能力。\n\nRefs MOTION-94

File: ros2_ws/src/alfa_robot_description/urdf/alfa_robot.urdf.xacro (robot description, xacro)
@@ -37,5 +37,5 @@
   <xacro:arg name="wheel04_joint_initial" default="0.0"/>
   <xacro:include filename="$(find alfa_robot_description)/urdf/alfa_robot/alfa_robot_macro.ros2_control.xacro"/>
-  <xacro:include filename="$(find alfa_robot_description)/urdf/alfa_robot/robot_v3_0_9.xacro"/>
+  <xacro:include filename="$(find alfa_robot_description)/urdf/alfa_robot/robot_v3_1_1.xacro"/>
   <xacro:include filename="$(find alfa_robot_description)/urdf/alfa_robot/robot_v3_chassis.xacro"/>
   <link name="world"/>
@@ -49,5 +49,5 @@
     <parent link="base_footprint"/>
     <child link="base_link"/>
-    <origin xyz="0.195 0.015 0.400" rpy="0 0 0"/>
+    <origin xyz="0.190000002779484 -0.0000442724271391554 0.40000250599116" rpy="0 0 0"/>
   </joint>
   <link name="base_link"/>

File: ros2_ws/src/alfa_robot_description/urdf/alfa_robot/alfa_robot_macro.ros2_control.xacro (robot description, xacro)
@@ -52,5 +52,5 @@
         </joint>
       </xacro:macro>
-      <xacro:control_joint joint_name="updown" initial_value="${updown_initial}" lower="-0.5" upper="0.5"/>
+      <xacro:control_joint joint_name="updown" initial_value="${updown_initial}" lower="-1.0" upper="0.0"/>
       <xacro:control_joint joint_name="head_joint" initial_value="${head_joint_initial}" lower="-1.57" upper="1.57"/>
       <xacro:control_joint joint_name="head_pitch_joint" initial_value="${head_pitch_joint_initial}" lower="-1.57" upper="1.57"/>
