Commit message: feat: integrate v5 arm meshes and RViz goal monitor
- add SolidWorks-exported alfa_robot_arm_v5 model assets and mirrored right-arm meshes

- replace the active v5 arm URDF with imported motor meshes while preserving v5 interfaces

- add RViz dual end-effector goal pose monitor and update teamwork task records

Co-Authored-By: Codex <codex@openai.com>

File: ros2_ws/src/alfa_robot_description/urdf/alfa_robot_v5_proxy_backup.urdf.xacro (robot description, xacro)
@@ -226,13 +226,42 @@
       velocity="0" />
   </joint>
-  <!-- v5 dual six-axis arms from the imported SolidWorks URDF.
-       Source package snapshot: /mnt/mydisk/ALFA/alfa_robot/alfa_robot_arm_v5
-       Current v5 proxy before replacement is preserved at:
-       urdf/alfa_robot_v5_proxy_backup.urdf.xacro
-       Naming is kept as left_v5_joint1..6 / right_v5_joint1..6 for MoveIt and ros2_control compatibility.
-       The imported single-arm URDF contains motor1..motor6 and 5 internal joints; the mount joint is the added joint1. -->
+  <!-- v5 dual six-axis proxy arms.
+       Coordinate convention for this proxy: +Y is forward, +Z is up.
+       User-corrected mounting plane: both mount frames use x=0, so they lie in the same YZ plane as updown.
+       The two proxy arms are separated along +/-Y and use multi-primitive T-motor joint visuals. -->
   <xacro:property name="v5_mount_y" value="0.32"/>
   <xacro:property name="v5_mount_z" value="0.18"/>
-  <xacro:property name="v5_mesh_base" value="package://alfa_robot_description/meshes/alfa_robot_arm_v5"/>
+  <xacro:property name="v5_upper_arm_length" value="0.65"/>
+  <xacro:property name="v5_forearm_length" value="0.65"/>
+  <xacro:property name="v5_motor_radius" value="0.085"/>
+  <xacro:property name="v5_motor_width" value="0.11"/>
+  <xacro:property name="v5_motor_gap" value="0"/>
+  <xacro:property name="v5_joint1_zero_rpy" value="0 0 -1.5708"/>
+  <xacro:macro name="v5_visual_box" params="size xyz rpy color">
+    <visual>
+      <origin xyz="${xyz}" rpy="${rpy}"/>
+      <geometry><box size="${size}"/></geometry>
+      <material name="v5_box_mat"><color rgba="${color}"/></material>
+    </visual>
+  </xacro:macro>
+  <xacro:macro name="v5_collision_box" params="size xyz rpy">
+    <collision>
+      <origin xyz="${xyz}" rpy="${rpy}"/>
+      <geometry><box size="${size}"/></geometry>
+    </collision>
+  </xacro:macro>
+  <xacro:macro name="v5_visual_cylinder" params="radius length xyz rpy color">
+    <visual>
+      <origin xyz="${xyz}" rpy="${rpy}"/>
+      <geometry><cylinder radius="${radius}" length="${length}"/></geometry>
+      <material name="v5_cylinder_mat"><color rgba="${color}"/></material>
+    </visual>
+  </xacro:macro>
+  <xacro:macro name="v5_collision_cylinder" params="radius length xyz rpy">
+    <collision>
+      <origin xyz="${xyz}" rpy="${rpy}"/>
+      <geometry><cylinder radius="${radius}" length="${length}"/></geometry>
+    </collision>
+  </xacro:macro>
   <xacro:macro name="v5_simple_inertial" params="mass">
     <inertial>
@@ -242,79 +271,67 @@
     </inertial>
   </xacro:macro>
-  <xacro:macro name="v5_visual_mesh" params="mesh_dir mesh origin_xyz origin_rpy color">
-    <visual>
-      <origin xyz="${origin_xyz}" rpy="${origin_rpy}"/>
-      <geometry><mesh filename="${v5_mesh_base}/${mesh_dir}/${mesh}"/></geometry>
-      <material name="v5_imported_mesh_mat"><color rgba="${color}"/></material>
-    </visual>
-  </xacro:macro>
-  <xacro:macro name="v5_collision_mesh" params="mesh_dir mesh origin_xyz origin_rpy">
-    <collision>
-      <origin xyz="${origin_xyz}" rpy="${origin_rpy}"/>
-      <geometry><mesh filename="${v5_mesh_base}/${mesh_dir}/${mesh}"/></geometry>
-    </collision>
-  </xacro:macro>
-  <xacro:macro name="v5_imported_motor_link" params="name motor color visual_dir collision_dir mirror_y:=1">
+  <xacro:macro name="v5_t_motor_mesh_visual" params="mesh xyz rpy color">
+    <visual>
+      <origin xyz="${xyz}" rpy="${rpy}"/>
+      <geometry>
+        <mesh filename="${mesh}"/>
+      </geometry>
+      <material name="v5_t_motor_mesh_mat"><color rgba="${color}"/></material>
+    </visual>
+  </xacro:macro>
+  <xacro:macro name="v5_t_motor_link" params="name axis mass color mesh mirror_y:=1">
     <link name="${name}">
-      <xacro:if value="${motor == 'motor1'}">
-        <inertial>
-          <origin xyz="0.00549007475138907 ${mirror_y * -4.41381777807892E-05} 0.0638192668274469" rpy="0 0 0"/>
-          <mass value="1.14347753856634"/>
-          <inertia ixx="0.00234577755868115" ixy="${mirror_y * -1.39193363061916E-06}" ixz="-7.06941578932414E-05" iyy="0.00245440035038314" iyz="${mirror_y * 2.78529148686552E-06}" izz="0.00212775140786364"/>
-        </inertial>
-        <xacro:v5_visual_mesh mesh_dir="${visual_dir}" mesh="motor1.STL" origin_xyz="0 0 0" origin_rpy="0 0 0" color="${color}"/>
-        <xacro:v5_collision_mesh mesh_dir="${collision_dir}" mesh="motor1.STL" origin_xyz="0 0 0" origin_rpy="0 0 0"/>
+      <xacro:v5_simple_inertial mass="${mass}"/>
+      <xacro:if value="${axis == 'z'}">
+        <!-- Visual uses leftjoint4.STL as the T-motor template; collision stays primitive for MoveIt stability. -->
+        <xacro:v5_t_motor_mesh_visual mesh="${mesh}" xyz="0 0 0" rpy="0 0 0" color="${color}"/>
+        <xacro:v5_collision_cylinder radius="${v5_motor_radius}" length="${v5_motor_width}" xyz="0 0 0.05" rpy="0 0 0"/>
       </xacro:if>
-      <xacro:if value="${motor == 'motor2'}">
-        <inertial>
-          <origin xyz="2.093E-05 ${mirror_y * 0.3} 0.074" rpy="0 0 0"/>
-          <mass value="4.8059"/>
-          <inertia ixx="0.051414" ixy="${mirror_y * 1.1107E-09}" ixz="7.002E-10" iyy="0.010931" iyz="${mirror_y * -0.00014138}" izz="0.050761"/>
-        </inertial>
-        <xacro:v5_visual_mesh mesh_dir="${visual_dir}" mesh="motor2.STL" origin_xyz="0 0 0" origin_rpy="0 0 0" color="${color}"/>
-        <xacro:v5_collision_mesh mesh_dir="${collision_dir}" mesh="motor2.STL" origin_xyz="0 0 0" origin_rpy="0 0 0"/>
+      <xacro:if value="${axis == 'x'}">
+        <xacro:v5_t_motor_mesh_visual mesh="${mesh}" xyz="0 0 0" rpy="0 1.5708 0" color="${color}"/>
+        <xacro:v5_collision_cylinder radius="${v5_motor_radius}" length="${v5_motor_width}" xyz="0.05 0 0" rpy="0 1.5708 0"/>
       </xacro:if>
-      <xacro:if value="${motor == 'motor3'}">
-        <inertial>
-          <origin xyz="-2.8361E-05 ${mirror_y * -0.33834} -0.043469" rpy="0 0 0"/>
-          <mass value="1.766"/>
-          <inertia ixx="0.016132" ixy="${mirror_y * 2.7853E-06}" ixz="-1.3961E-06" iyy="0.002789" iyz="${mirror_y * -0.0001017}" izz="0.01667"/>
-        </inertial>
-        <xacro:v5_visual_mesh mesh_dir="${visual_dir}" mesh="motor3.STL" origin_xyz="0 0 0" origin_rpy="0 0 0" color="${color}"/>
-        <xacro:v5_collision_mesh mesh_dir="${collision_dir}" mesh="motor3.STL" origin_xyz="0 0 0" origin_rpy="0 0 0"/>
-      </xacro:if>
-      <xacro:if value="${motor == 'motor4'}">
-        <inertial>
-          <origin xyz="-0.0096807 ${mirror_y * -4.4024E-05} 0.05401" rpy="0 0 0"/>
-          <mass value="1.1435"/>
-          <inertia ixx="0.0021278" ixy="${mirror_y * 2.7864E-06}" ixz="7.0691E-05" iyy="0.0024544" iyz="${mirror_y * 1.3934E-06}" izz="0.0023458"/>
-        </inertial>
-        <xacro:v5_visual_mesh mesh_dir="${visual_dir}" mesh="motor4.STL" origin_xyz="0 0 0" origin_rpy="0 0 0" color="${color}"/>
-        <xacro:v5_collision_mesh mesh_dir="${collision_dir}" mesh="motor4.STL" origin_xyz="0 0 0" origin_rpy="0 0 0"/>
-      </xacro:if>
-      <xacro:if value="${motor == 'motor5'}">
-        <inertial>
-          <origin xyz="4.3802E-05 ${mirror_y * -0.0096808} 0.05451" rpy="0 0 0"/>
-          <mass value="1.1435"/>
-          <inertia ixx="0.0024544" ixy="${mirror_y * -2.7853E-06}" ixz="-1.3961E-06" iyy="0.0021278" iyz="${mirror_y * 7.0689E-05}" izz="0.0023458"/>
-        </inertial>
-        <xacro:v5_visual_mesh mesh_dir="${visual_dir}" mesh="motor5.STL" origin_xyz="0 0 0" origin_rpy="0 0 0" color="${color}"/>
-        <xacro:v5_collision_mesh mesh_dir="${collision_dir}" mesh="motor5.STL" origin_xyz="0 0 0" origin_rpy="0 0 0"/>
-      </xacro:if>
-      <xacro:if value="${motor == 'motor6'}">
-        <inertial>
-          <origin xyz="0 0 0.027325" rpy="0 0 0"/>
-          <mass value="1.9452"/>
-          <inertia ixx="0.0066307" ixy="0" ixz="0" iyy="0.0044221" iyz="0" izz="0.010447"/>
-        </inertial>
-        <xacro:v5_visual_mesh mesh_dir="${visual_dir}" mesh="motor6.STL" origin_xyz="0 0 0" origin_rpy="0 0 0" color="${color}"/>
-        <xacro:v5_collision_mesh mesh_dir="${collision_dir}" mesh="motor6.STL" origin_xyz="0 0 0" origin_rpy="0 0 0"/>
+      <xacro:if value="${axis == 'y'}">
+        <xacro:v5_t_motor_mesh_visual mesh="${mesh}" xyz="0 0 0" rpy="${mirror_y * 1.5708} 0 0" color="${color}"/>
+        <xacro:v5_collision_cylinder radius="${v5_motor_radius}" length="${v5_motor_width}" xyz="0 ${mirror_y * 0.05} 0" rpy="${mirror_y * 1.5708} 0 0"/>
       </xacro:if>
     </link>
   </xacro:macro>
-  <xacro:macro name="v5_imported_arm" params="side mount_y mirror_y color visual_dir collision_dir">
-    <link name="${side}_v5_link0">
-      <xacro:v5_simple_inertial mass="0.5"/>
+  <xacro:macro name="v5_t_motor_with_bar_link" params="name axis bar_length bar_radius mass color mesh mirror_y:=1">
+    <link name="${name}">
+      <xacro:v5_simple_inertial mass="${mass}"/>
+      <xacro:if value="${axis == 'x'}">
+        <xacro:v5_t_motor_mesh_visual mesh="${mesh}" xyz="0.06 0 0" rpy="${(mirror_y + 1) * 1.570796327} 1.5708 ${(1 - mirror_y) * 1.570796327}" color="${color}"/>
+        <xacro:v5_collision_cylinder radius="${v5_motor_radius}" length="${v5_motor_width}" xyz="0.05 0 0" rpy="0 1.5708 0"/>
+      </xacro:if>
+      <xacro:if value="${axis == 'y'}">
+        <xacro:v5_t_motor_mesh_visual mesh="${mesh}" xyz="0 0 0" rpy="${mirror_y * 1.5708} 0 0" color="${color}"/>
+        <xacro:v5_collision_cylinder radius="${v5_motor_radius}" length="${v5_motor_width}" xyz="0 ${mirror_y * 0.05} 0" rpy="${mirror_y * 1.5708} 0 0"/>
+      </xacro:if>
+      <!-- Single cylindrical arm segment starts at this joint and ends at the next joint. -->
+      <xacro:v5_visual_cylinder radius="${bar_radius}" length="${bar_length}" xyz="0 ${mirror_y * bar_length / 2.0} 0" rpy="${mirror_y * 1.5708} 0 0" color="${color}"/>
+      <xacro:v5_collision_cylinder radius="${bar_radius}" length="${bar_length}" xyz="0 ${mirror_y * bar_length / 2.0} 0" rpy="${mirror_y * 1.5708} 0 0"/>
     </link>
+  </xacro:macro>
+  <xacro:macro name="v5_fixed_t_support" params="name color mesh mirror_y:=1">
+    <link name="${name}">
+      <xacro:v5_simple_inertial mass="1.0"/>
+      <!-- Passive T-shaped motor/bracket: visual reference only, no active DOF. -->
+      <xacro:v5_t_motor_mesh_visual mesh="${mesh}" xyz="0 0 0" rpy="0 1.5708 0" color="${color}"/>
+      <xacro:v5_collision_cylinder radius="${v5_motor_radius}" length="${v5_motor_width}" xyz="0.05 0 0" rpy="0 1.5708 0"/>
+    </link>
+  </xacro:macro>
+  <xacro:macro name="v5_mount_link" params="name color">
+    <link name="${name}">
+      <xacro:v5_simple_inertial mass="3.0"/>
+      <!-- Explicit mounting bracket: not a point mount. -->
+      <xacro:v5_visual_box size="0.30 0.18 0.08" xyz="0 0 0" rpy="0 0 0" color="0.18 0.18 0.18 1"/>
+      <xacro:v5_visual_box size="0.22 0.06 0.18" xyz="0 0 0.08" rpy="0 0 0" color="${color}"/>
+      <xacro:v5_visual_cylinder radius="0.025" length="0.32" xyz="0 0 0.12" rpy="0 1.5708 0" color="0.03 0.03 0.03 1"/>
+      <xacro:v5_collision_box size="0.30 0.18 0.18" xyz="0 0 0.05" rpy="0 0 0"/>
+    </link>
+  </xacro:macro>
+  <xacro:macro name="v5_proxy_arm" params="side mount_y mirror_y color mesh">
+    <xacro:v5_mount_link name="${side}_v5_link0" color="${color}"/>
     <joint name="${side}_v5_mount" type="fixed">
       <parent link="updown"/>
@@ -322,63 +339,72 @@
       <origin xyz="0 ${mount_y} ${v5_mount_z}" rpy="0 0 0"/>
     </joint>
-    <xacro:v5_imported_motor_link name="${side}_v5_link1" motor="motor1" color="${color}" visual_dir="${visual_dir}" collision_dir="${collision_dir}" mirror_y="${mirror_y}"/>
+    <xacro:v5_t_motor_link name="${side}_v5_link1" axis="z" mass="2.0" color="${color}" mesh="${mesh}" mirror_y="${mirror_y}"/>
     <joint name="${side}_v5_joint1" type="revolute">
       <parent link="${side}_v5_link0"/>
       <child link="${side}_v5_link1"/>
-      <origin xyz="0 0 0" rpy="0 0 0"/>
+      <origin xyz="0 0 0.16" rpy="0 0 ${mirror_y * 3.141592654}"/>
       <axis xyz="0 0 1"/>
       <limit lower="-3.14159265" upper="3.14159265" effort="120" velocity="1.2"/>
     </joint>
-    <xacro:v5_imported_motor_link name="${side}_v5_link2" motor="motor2" color="${color}" visual_dir="${visual_dir}" collision_dir="${collision_dir}" mirror_y="${mirror_y}"/>
+    <xacro:v5_t_motor_with_bar_link name="${side}_v5_link2" axis="x" bar_length="${v5_upper_arm_length}" bar_radius="0.055" mass="4.5" color="${color}" mesh="${mesh}" mirror_y="${mirror_y}"/>
     <joint name="${side}_v5_joint2" type="revolute">
       <parent link="${side}_v5_link1"/>
       <child link="${side}_v5_link2"/>
-      <origin xyz="0.0595 0 0.0735" rpy="${mirror_y * 1.5708} 0 ${mirror_y * 1.5708}"/>
-      <axis xyz="0 0 1"/>
-      <limit lower="-3.14159265" upper="3.14159265" effort="120" velocity="1.2"/>
-    </joint>
-    <xacro:v5_imported_motor_link name="${side}_v5_link3" motor="motor3" color="${color}" visual_dir="${visual_dir}" collision_dir="${collision_dir}" mirror_y="${mirror_y}"/>
+      <origin xyz="0 ${mirror_y * -0.1} 0.06" rpy="${mirror_y * 3.141592654} 0 ${mirror_y * 1.57079632}"/>
+      <axis xyz="1 0 0"/>
+      <limit lower="-1.57079632" upper="1.57079632" effort="120" velocity="1.2"/>
+    </joint>
+    <xacro:v5_t_motor_with_bar_link name="${side}_v5_link3" axis="x" bar_length="${v5_forearm_length}" bar_radius="0.05" mass="3.6" color="${color}" mesh="${mesh}" mirror_y="${mirror_y}"/>
     <joint name="${side}_v5_joint3" type="revolute">
       <parent link="${side}_v5_link2"/>
       <child link="${side}_v5_link3"/>
-      <origin xyz="0 ${mirror_y * 0.6} 0.148" rpy="0 0 ${mirror_y * 3.1416}"/>
-      <axis xyz="0 0 -1"/>
-      <limit lower="-3.14159265" upper="3.14159265" effort="100" velocity="1.2"/>
-    </joint>
-    <xacro:v5_imported_motor_link name="${side}_v5_link4" motor="motor4" color="${color}" visual_dir="${visual_dir}" collision_dir="${collision_dir}" mirror_y="${mirror_y}"/>
+      <!-- Elbow joint is at the end of upper arm, separated from shoulder J2. -->
+      <origin xyz="-0.14 ${mirror_y * 0.7} 0" rpy="0 0 0"/>
+      <axis xyz="1 0 0"/>
+      <limit lower="-2.35619449" upper="2.35619449" effort="100" velocity="1.2"/>
+    </joint>
+    <xacro:v5_fixed_t_support name="${side}_v5_link3_passive_t" color="${color}" mesh="${mesh}" mirror_y="${mirror_y}"/>
+    <joint name="${side}_v5_joint3_passive_t" type="fixed">
+      <parent link="${side}_v5_link3"/>
+      <child link="${side}_v5_link3_passive_t"/>
+      <origin xyz="0.08 ${mirror_y * v5_motor_gap} 0" rpy="0 0 0"/>
+    </joint>
+    <xacro:v5_t_motor_link name="${side}_v5_link4" axis="y" mass="1.4" color="${color}" mesh="${mesh}" mirror_y="${mirror_y}"/>
     <joint name="${side}_v5_joint4" type="revolute">
       <parent link="${side}_v5_link3"/>
       <child link="${side}_v5_link4"/>
-      <origin xyz="0 ${mirror_y * -0.47402} -0.075" rpy="${mirror_y * 1.5708} -1.5708 0"/>
-      <axis xyz="0 0 -1"/>
+      <!-- Wrist joint4 is at the end of forearm, separated from elbow J3. -->
+      <origin xyz="0 ${mirror_y * v5_forearm_length} ${v5_motor_gap}" rpy="${mirror_y * 3.141592654} 0 0"/>
+      <axis xyz="0 ${mirror_y} 0"/>
       <limit lower="-3.14159265" upper="3.14159265" effort="60" velocity="1.5"/>
     </joint>
-    <xacro:v5_imported_motor_link name="${side}_v5_link5" motor="motor5" color="${color}" visual_dir="${visual_dir}" collision_dir="${collision_dir}" mirror_y="${mirror_y}"/>
+    <xacro:v5_t_motor_link name="${side}_v5_link5" axis="x" mass="1.0" color="${color}" mesh="${mesh}" mirror_y="${mirror_y}"/>
     <joint name="${side}_v5_joint5" type="revolute">
       <parent link="${side}_v5_link4"/>
       <child link="${side}_v5_link5"/>
-      <origin xyz="-0.074 0 0.0595" rpy="${mirror_y * -1.5708} 0 ${mirror_y * 1.5708}"/>
-      <axis xyz="0 0 -1"/>
-      <limit lower="-3.14159265" upper="3.14159265" effort="60" velocity="1.5"/>
-    </joint>
-    <xacro:v5_imported_motor_link name="${side}_v5_link6" motor="motor6" color="${color}" visual_dir="${visual_dir}" collision_dir="${collision_dir}" mirror_y="${mirror_y}"/>
+      <origin xyz="0.0 ${mirror_y * -0.06} -0.08" rpy="0 1.57079632 0"/>
+      <axis xyz="1 0 0"/>
+      <limit lower="-1.57079632" upper="1.57079632" effort="60" velocity="1.5"/>
+    </joint>
+    <xacro:v5_t_motor_link name="${side}_v5_link6" axis="z" mass="1.0" color="${color}" mesh="${mesh}" mirror_y="${mirror_y}"/>
     <joint name="${side}_v5_joint6" type="revolute">
       <parent link="${side}_v5_link5"/>
       <child link="${side}_v5_link6"/>
-      <origin xyz="0 ${mirror_y * -0.074} 0.06" rpy="${mirror_y * 1.5708} 1.5708 0"/>
-      <axis xyz="0 0 -1"/>
+      <origin xyz="0.06 ${mirror_y * -0.08} 0" rpy="${mirror_y * 1.57079632} 0 0"/>
+      <axis xyz="0 0 1"/>
       <limit lower="-3.14159265" upper="3.14159265" effort="40" velocity="1.5"/>
     </joint>
     <link name="${side}_v5_tool0">
       <xacro:v5_simple_inertial mass="0.2"/>
+      <xacro:v5_visual_box size="0.10 0.10 0.04" xyz="0 ${mirror_y * 0.05} 0" rpy="0 0 0" color="0.9 0.9 0.1 1"/>
     </link>
     <joint name="${side}_v5_tool0_fixed" type="fixed">
       <parent link="${side}_v5_link6"/>
       <child link="${side}_v5_tool0"/>
-      <origin xyz="0 0 0.08" rpy="0 0 0"/>
-    </joint>
-  </xacro:macro>
-  <xacro:v5_imported_arm side="left" mount_y="${v5_mount_y}" mirror_y="1" color="0.2 0.55 1.0 1" visual_dir="visual" collision_dir="collision"/>
-  <xacro:v5_imported_arm side="right" mount_y="${-v5_mount_y}" mirror_y="-1" color="1.0 0.55 0.2 1" visual_dir="visual_right" collision_dir="collision_right"/>
+      <origin xyz="0 ${mirror_y * 0.12} 0" rpy="0 0 0"/>
+    </joint>
+  </xacro:macro>
+  <xacro:v5_proxy_arm side="left" mount_y="${v5_mount_y}" mirror_y="1" color="0.2 0.55 1.0 1" mesh="package://alfa_robot_description/meshes/alfa_robot_v2_arm_v4_new/visual/leftjoint4.STL"/>
+  <xacro:v5_proxy_arm side="right" mount_y="${-v5_mount_y}" mirror_y="-1" color="1.0 0.55 0.2 1" mesh="package://alfa_robot_description/meshes/alfa_robot_v2_arm_v4_new/visual/rightjoint4.STL"/>
   <xacro:alfa_robot_ros2_control
     name="alfa_robot"
