Commit message: Apply conservative arm motion limits

File: research/curobo_v3/generated/v3_analytic_071cb95/mobile18/model/robot_meter_meshes_mobile18.urdf (robot description, URDF)
Before this commit: robot alfa_robot_v3, 24 links, 23 joints
Joints:
- joint left_joint1: limit lower=-3.14159265 upper=3.14159265 effort=647 velocity=1.309 -> lower=-3.14159265 upper=3.14159265 effort=647 velocity=0.261799387799149
- joint left_joint2: limit lower=-1.8325957145940461 upper=1.8325957145940461 effort=647 velocity=1.309 -> lower=-1.8325957145940461 upper=1.8325957145940461 effort=647 velocity=0.261799387799149
- joint left_joint3: limit lower=-3.14159265 upper=3.14159265 effort=484 velocity=1.309 -> lower=-3.14159265 upper=3.14159265 effort=484 velocity=0.261799387799149
- joint left_joint4: limit lower=-2.53072742 upper=2.53072742 effort=459 velocity=1.749 -> lower=-2.53072742 upper=2.53072742 effort=459 velocity=0.261799387799149
- joint left_joint5: limit lower=-3.14159265 upper=3.14159265 effort=217 velocity=2.618 -> lower=-3.14159265 upper=3.14159265 effort=217 velocity=0.523598775598299
- joint left_joint6: limit lower=-1.91986218 upper=1.91986218 effort=107 velocity=3.142 -> lower=-1.91986218 upper=1.91986218 effort=107 velocity=0.523598775598299
- joint left_joint7: limit lower=-3.14159265 upper=3.14159265 effort=36 velocity=3.142 -> lower=-3.14159265 upper=3.14159265 effort=36 velocity=0.523598775598299
- joint right_joint1: limit lower=-3.14159265 upper=3.14159265 effort=647 velocity=1.309 -> lower=-3.14159265 upper=3.14159265 effort=647 velocity=0.261799387799149
- joint right_joint2: limit lower=-1.8325957145940461 upper=1.8325957145940461 effort=647 velocity=1.309 -> lower=-1.8325957145940461 upper=1.8325957145940461 effort=647 velocity=0.261799387799149
- joint right_joint3: limit lower=-3.14159265 upper=3.14159265 effort=484 velocity=1.309 -> lower=-3.14159265 upper=3.14159265 effort=484 velocity=0.261799387799149
- joint right_joint4: limit lower=-2.53072742 upper=2.53072742 effort=459 velocity=1.749 -> lower=-2.53072742 upper=2.53072742 effort=459 velocity=0.261799387799149
- joint right_joint5: limit lower=-3.14159265 upper=3.14159265 effort=217 velocity=2.618 -> lower=-3.14159265 upper=3.14159265 effort=217 velocity=0.523598775598299
- joint right_joint6: limit lower=-1.91986218 upper=1.91986218 effort=107 velocity=3.142 -> lower=-1.91986218 upper=1.91986218 effort=107 velocity=0.523598775598299
- joint right_joint7: limit lower=-3.14159265 upper=3.14159265 effort=36 velocity=3.142 -> lower=-3.14159265 upper=3.14159265 effort=36 velocity=0.523598775598299

File: research/curobo_v3/generated/v3_analytic_071cb95/model/robot_meter_meshes.urdf (robot description, URDF)
Before this commit: robot alfa_robot_v3, 21 links, 20 joints
Joints:
- joint left_joint1: limit lower=-3.14159265 upper=3.14159265 effort=647 velocity=1.309 -> lower=-3.14159265 upper=3.14159265 effort=647 velocity=0.261799387799149
- joint left_joint2: limit lower=-1.8325957145940461 upper=1.8325957145940461 effort=647 velocity=1.309 -> lower=-1.8325957145940461 upper=1.8325957145940461 effort=647 velocity=0.261799387799149
- joint left_joint3: limit lower=-3.14159265 upper=3.14159265 effort=484 velocity=1.309 -> lower=-3.14159265 upper=3.14159265 effort=484 velocity=0.261799387799149
- joint left_joint4: limit lower=-2.53072742 upper=2.53072742 effort=459 velocity=1.749 -> lower=-2.53072742 upper=2.53072742 effort=459 velocity=0.261799387799149
- joint left_joint5: limit lower=-3.14159265 upper=3.14159265 effort=217 velocity=2.618 -> lower=-3.14159265 upper=3.14159265 effort=217 velocity=0.523598775598299
- joint left_joint6: limit lower=-1.91986218 upper=1.91986218 effort=107 velocity=3.142 -> lower=-1.91986218 upper=1.91986218 effort=107 velocity=0.523598775598299
- joint left_joint7: limit lower=-3.14159265 upper=3.14159265 effort=36 velocity=3.142 -> lower=-3.14159265 upper=3.14159265 effort=36 velocity=0.523598775598299
- joint right_joint1: limit lower=-3.14159265 upper=3.14159265 effort=647 velocity=1.309 -> lower=-3.14159265 upper=3.14159265 effort=647 velocity=0.261799387799149
- joint right_joint2: limit lower=-1.8325957145940461 upper=1.8325957145940461 effort=647 velocity=1.309 -> lower=-1.8325957145940461 upper=1.8325957145940461 effort=647 velocity=0.261799387799149
- joint right_joint3: limit lower=-3.14159265 upper=3.14159265 effort=484 velocity=1.309 -> lower=-3.14159265 upper=3.14159265 effort=484 velocity=0.261799387799149
- joint right_joint4: limit lower=-2.53072742 upper=2.53072742 effort=459 velocity=1.749 -> lower=-2.53072742 upper=2.53072742 effort=459 velocity=0.261799387799149
- joint right_joint5: limit lower=-3.14159265 upper=3.14159265 effort=217 velocity=2.618 -> lower=-3.14159265 upper=3.14159265 effort=217 velocity=0.523598775598299
- joint right_joint6: limit lower=-1.91986218 upper=1.91986218 effort=107 velocity=3.142 -> lower=-1.91986218 upper=1.91986218 effort=107 velocity=0.523598775598299
- joint right_joint7: limit lower=-3.14159265 upper=3.14159265 effort=36 velocity=3.142 -> lower=-3.14159265 upper=3.14159265 effort=36 velocity=0.523598775598299
