Commit message: [feat][motion] 同步当前零位191mm TCP与六段LM规划并兼容PR65 (#69)
* fix(curobo): 修正吸附目标面内翻转并保留顶吸旋转回归证据

* feat(curobo): 录制左臂接触前缀并提供工控机回放前端待接口对齐

* feat(curobo): 左臂录制回放接入FJT Action回执及取消

* docs(curobo): 记录左臂发送后掉使能的驱动与Action时间线

* feat(curobo): 压缩左臂发送轨迹并限制15度每秒60秒及增加实测可视化

* fix(curobo): 恢复控制台重启后的会话并重试过期控制器查询

* docs(curobo): 记录10Hz连续轨迹的离线试验及圆滑待定边界

* research(curobo): 保留原规划帧核验RT插值与局部定时问题

* feat(curobo): 可视化原帧七轴曲线和末段插值加速度峰值

* feat(curobo): 增加左臂临时平滑与全任务只读预览，记录GPU集成阻塞

* feat(curobo): 标记左Joint7与局部Z轴70毫米临时TCP

* feat(curobo): 增加固定升降70毫米测试杆解析IK候选与FK复核

* feat(curobo): 增加同点多朝向与五次插值，记录起点自碰撞门禁阻塞

* feat(curobo): 可视化测试杆诊断中的具体自碰撞球对

* fix(curobo): 复用底盘立方体替代逻辑，移除测试杆检查器重复球对检测

* feat(curobo): 接入测试杆同点多朝向打表、轨迹预览与手动FJT发送

* docs(curobo): 固化测试杆打表联调方案与接手恢复手册

* feat(curobo): 固定目标关节解析寻根并支持全零后独立到位预览

* docs(curobo): 记录本会话实机联调职责与既有执行边界

* chore(curobo): 为随机误差实验独立登记8170至8172端口

* chore(curobo): 随机误差Demo统一使用8171入口

* feat(curobo): 为8171接入当前模型随机误差规划与失败前缀回放

* feat(curobo): 同步电控左J5新零位并更新URDF IK与Viser版本门禁

* fix(curobo): 纠正转身后左右放箱目标并恢复双龙头车外观

* feat(curobo): 临时校准左J2反馈减1度与命令加1度并同步Viser

* fix(curobo): 按目标高度分段挖孔，补齐高箱下方碰撞实体

* fix(curobo): 避免回放重复应用底盘位姿导致转身显示抵消

* feat(curobo): 增加TCP标定快速到位模式与停稳实测姿态记录

* fix(curobo): 松开自动局部数值IK预览并修复快速轨迹播放和发送门禁

* feat(curobo): 预览默认五倍速且独立于实机轨迹时间

* research(curobo): 拟合十姿态同点触碰零位与TCP并区分J2已有补偿

* feat(curobo): 按授权启用十姿态零位拟合候选A并同步联调显示和执行

* docs(curobo): 归档用户实机验收通过的零位补偿联调结论

* fix(curobo): 整墙演示恢复顶吸前移停车位并贯通25箱13轮回放

* feat(curobo): 从入口逐面规划整箱300箱并支持完整连续回放

* feat(curobo): 按整轮双末端额外旋转选择25箱配对并提供回放

* feat(curobo): 按确认姿态重定义双臂零位并翻转J6供离线验收

* feat(curobo): 采用确认后的双臂零位J6正向及191毫米TCP并同步FKIK

* fix(curobo): 删除误加J4零位偏置与本地小角度拟合补偿

* feat(curobo): 接入六段LM前向预接触流程并适配当前零位与191毫米TCP

迁移8209算法及必要源码依赖；补齐16/64批量LM真实预热并共享长段求解器。旧2厘米升降网格跳过191毫米TCP下运输可行窗口，原范围内加密为5毫米，保留目标、限位、碰撞及包络验收。35项回归及三类任务四次GPU完整流程通过，8210页面实时计算通过；不涉及工控机，保留抽离途中空载验碰等研究边界。

Co-Authored-By: Codex <codex@openai.com>

* fix(curobo): 验证PR65集成与当前模型入口兼容及117任务合同

保留独立时间化入口和六段LM默认入口；当前模型及GPU完整任务回归通过，未更改实机或覆盖其他未提交工作。

Co-Authored-By: Codex <codex@openai.com>

---------

Co-authored-by: Codex <codex@openai.com>

File: research/curobo_v3/generated/zero_model_candidate_20261018/mobile/robot_rezero_candidate.urdf (robot description, URDF)
Before this commit: robot alfa_robot_v3, 24 links, 23 joints
Joints:
- joint left_joint6: axis -0 -0 -1 -> 0 0 1
- joint left_tool0_fixed: origin xyz=0 0 0.151 rpy=0 0 0 -> xyz=0 0 0.191 rpy=0 0 0
- joint right_joint6: axis -0 -0 -1 -> 0 0 1
- joint right_tool0_fixed: origin xyz=0 0 0.151 rpy=0 0 0 -> xyz=0 0 0.191 rpy=0 0 0

File: research/curobo_v3/generated/zero_model_candidate_20261018/robot_rezero_candidate.urdf (robot description, URDF)
Before this commit: robot alfa_robot_v3, 21 links, 20 joints
Joints:
- joint left_joint6: axis -0 -0 -1 -> 0 0 1
- joint left_tool0_fixed: origin xyz=0 0 0.151 rpy=0 0 0 -> xyz=0 0 0.191 rpy=0 0 0
- joint right_joint6: axis -0 -0 -1 -> 0 0 1
- joint right_tool0_fixed: origin xyz=0 0 0.151 rpy=0 0 0 -> xyz=0 0 0.191 rpy=0 0 0
